File: boatcontrol/boatcontrol.sch (KiCad schematic (older format))
At the start: 271 parts, among them J1 TBL008V-1000-02BE, J10 TBL008V-1000-08BE, J11 TBL008V-1000-02BE, J12 TBL008V-1000-08BE, J2 SS73100-047F, J3 SS73100-047F, J4 TBP01R2W-508-08BE, J5 TB007-508-16BE, J6 TBP01R2W-508-08BE, J7 RPi_GPIO, J8 TBL008V-1000-02BE (DC IN), J9 TBL008V-1000-02BE, K1 G5RL-K1A-E-DC12, K10 G5RL-K1A-E-DC12, K11 G5RL-K1A-E-DC12, K12 G5RL-K1A-E-DC12, K13 G5RL-K1A-E-DC12, K14 G5RL-K1A-E-DC12, K15 G5RL-K1A-E-DC12, K16 G5RL-K1A-E-DC12, K17 G5RL-K1A-E-DC12, K18 G5RL-K1A-E-DC12, K19 G5RL-K1A-E-DC12, K2 G5RL-K1A-E-DC12, K20 G5RL-K1A-E-DC12, K21 G5RL-K1A-E-DC12, K22 G5RL-K1A-E-DC12, K23 G5RL-K1A-E-DC12, K24 G5RL-K1A-E-DC12, K25 G5RL-K1A-E-DC12, K26 G5RL-K1A-E-DC12, K27 G5RL-K1A-E-DC12, K28 G5RL-K1A-E-DC12, K29 G5RL-K1A-E-DC12, K3 G5RL-K1A-E-DC12, K30 G5RL-K1A-E-DC12, K31 G5RL-K1A-E-DC12, K32 G5RL-K1A-E-DC12, K33 EW60-1A3-CL12D04, K34 EW60-1A3-CL12D04, K35 EW60-1A3-CL12D04, K36 EW60-1A3-CL12D04, K37 EW60-1A3-CL12D04, K38 EW60-1A3-CL12D04, K39 EW60-1A3-CL12D04, K4 G5RL-K1A-E-DC12, K40 EW60-1A3-CL12D04, K5 G5RL-K1A-E-DC12, K6 G5RL-K1A-E-DC12, K7 G5RL-K1A-E-DC12, K8 G5RL-K1A-E-DC12, K9 G5RL-K1A-E-DC12, Q1 SchurterCircuitBreaker 3a, Q10 SchurterCircuitBreaker 3a, Q11 SchurterCircuitBreaker 3a, Q12 SchurterCircuitBreaker 3a, Q13 SchurterCircuitBreaker 3a, Q14 SchurterCircuitBreaker 3a, Q15 SchurterCircuitBreaker 3a, Q16 SchurterCircuitBreaker 3a, Q17 SchurterCircuitBreaker 6a, Q18 SchurterCircuitBreaker 6a, Q19 SchurterCircuitBreaker 6a, Q2 SchurterCircuitBreaker 3a, Q20 SchurterCircuitBreaker 6a, Q21 SchurterCircuitBreaker 10a, Q22 SchurterCircuitBreaker 10a, Q23 SchurterCircuitBreaker 16a, Q24 SchurterCircuitBreaker 16a, Q25 SchurterCircuitBreaker 6a, Q26 SchurterCircuitBreaker 6a, Q27 SchurterCircuitBreaker 6a, Q28 SchurterCircuitBreaker 6a, Q29 SchurterCircuitBreaker 10a, Q3 SchurterCircuitBreaker 3a, Q30 SchurterCircuitBreaker 10a, Q31 SchurterCircuitBreaker 16a, Q32 SchurterCircuitBreaker 16a, Q33 SchurterCircuitBreaker 3a, Q4 SchurterCircuitBreaker 3a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

Commit message: Tracks
Connections:
- wire segments 2342 -> 2351

Commit message: Mid Restructure
Connections:
- wire segments 2351 -> 2098
Other:
- moved on the sheet: C1, C3, C5, C7, D41, D42, J11, J4, J5, J6, J8, J9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

Commit message: Refactoring done
Connections:
- wire segments 2098 -> 2393
Other:
- moved on the sheet: C1, C3, C5, C7, D41, D42, J1, J11, J2A, J3A, J4, J5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

Commit message: Change do DIP everywhere
Parts:
- U10, U13, U16, U19, U7: footprint Package_SO:SOIC-28W_7.5x17.9mm_P1.27mm -> Package_DIP:DIP-28_W7.62mm
Changed lines of the file:
@@
 F 0 "U10" V 28600 10950 50  0000 L CNN
 F 1 "MCP23017_SO" V 28700 10750 50  0000 L CNN
-F 2 "Package_SO:SOIC-28W_7.5x17.9mm_P1.27mm" H 28900 10000 50  0001 L CNN
+F 2 "Package_DIP:DIP-28_W7.62mm" H 28900 10000 50  0001 L CNN
 F 3 "http://ww1.microchip.com/downloads/en/DeviceDoc/20001952C.pdf" H 28900 9900 50  0001 L CNN
 	1    28700 11000
@@
 F 0 "U13" V 2000 5050 50  0000 L CNN
 F 1 "MCP23017_SO" V 1900 4850 50  0000 L CNN
-F 2 "Package_SO:SOIC-28W_7.5x17.9mm_P1.27mm" H 2150 4150 50  0001 L CNN
+F 2 "Package_DIP:DIP-28_W7.62mm" H 2150 4150 50  0001 L CNN
 F 3 "http://ww1.microchip.com/downloads/en/DeviceDoc/20001952C.pdf" H 2150 4050 50  0001 L CNN
 	1    1950 5150
@@
 F 0 "U16" V 28550 5250 50  0000 L CNN
 F 1 "MCP23017_SO" V 28650 5000 50  0000 L CNN
-F 2 "Package_SO:SOIC-28W_7.5x17.9mm_P1.27mm" H 28850 4250 50  0001 L CNN
+F 2 "Package_DIP:DIP-28_W7.62mm" H 28850 4250 50  0001 L CNN
 F 3 "http://ww1.microchip.com/downloads/en/DeviceDoc/20001952C.pdf" H 28850 4150 50  0001 L CNN
 	1    28650 5250
@@
 F 0 "U7" V 1850 10950 50  0000 L CNN
 F 1 "MCP23017_SO" V 1950 10750 50  0000 L CNN
-F 2 "Package_SO:SOIC-28W_7.5x17.9mm_P1.27mm" H 2150 9950 50  0001 L CNN
+F 2 "Package_DIP:DIP-28_W7.62mm" H 2150 9950 50  0001 L CNN
 F 3 "http://ww1.microchip.com/downloads/en/DeviceDoc/20001952C.pdf" H 2150 9850 50  0001 L CNN
 	1    1950 10950
@@
 F 0 "U19" V 1850 18300 50  0000 L CNN
 F 1 "MCP23017_SO" V 1950 18100 50  0000 L CNN
-F 2 "Package_SO:SOIC-28W_7.5x17.9mm_P1.27mm" H 2150 17300 50  0001 L CNN
+F 2 "Package_DIP:DIP-28_W7.62mm" H 2150 17300 50  0001 L CNN
 F 3 "http://ww1.microchip.com/downloads/en/DeviceDoc/20001952C.pdf" H 2150 17200 50  0001 L CNN
 	1    1950 18300

Commit message: Time to refactor the PCB
Parts:
- J1: Field4 31.3mm -> (none); Field5 Manufacturer recommendations -> (none); Field6 AC -> (none); Type (none) -> AC 230V Common
- J11: Field4 DC -> (none); Type (none) -> 12VDC Logic
- J8: value TBL008V-1000-02BE (DC IN) -> TBL008V-1000-02BE; Field4 31.3mm -> (none); Field5 Manufacturer recommendations -> (none); Type (none) -> DC12V Common Bank1
- J9: Field4 DC -> (none); Type (none) -> DC 12V Common Bank2
- U1, U10, U13, U16, U19, U4, U7: value MCP23017_SO -> MCP23017-E/SP
- renumbered U17 to U14, U14 to U17
Connections:
- wire segments 2393 -> 2245
Other:
- moved on the sheet: J11, J4, J5, J6, J8, J9, K17, K18, K19, K20, K21, K22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

Commit message: Power Routing done on a set
Parts:
- C4: value Illinois Capacitor -> Illinois Capacitor 227AVG050MGBJ
- J5: value TB007-508-16BE -> TBP01R2W-508-16BE
Connections:
- wire segments 2245 -> 2375
Other:
- moved on the sheet: U13, U16

Commit message: Let's sort out the switches
Connections:
- wire segments 2375 -> 2373
Other:
- moved on the sheet: J1, J9
Changed lines of the file:
@@
 L BoatControl:TBL008V-1000-02BE J9
 U 1 1 70FC1583
-P 25500 4500
-F 0 "J9" V 25450 4400 50  0000 R CNN
-F 1 "TBL008V-1000-02BE" V 25400 5550 50  0000 R CNN
-F 2 "CUI_TBL008V-1000-02BE" H 25500 4500 50  0001 L BNN
-F 3 "CUI" H 25500 4500 50  0001 L BNN
-F 4 "DC 12V Common Bank2" V 25200 5050 50  0000 C CNN "Type"
-	1    25500 4500
+P 25500 2050
+F 0 "J9" V 25450 1950 50  0000 R CNN
+F 1 "TBL008V-1000-02BE" V 25400 3100 50  0000 R CNN
+F 2 "CUI_TBL008V-1000-02BE" H 25500 2050 50  0001 L BNN
+F 3 "CUI" H 25500 2050 50  0001 L BNN
+F 4 "DC 12V Common Bank2" V 25200 2600 50  0000 C CNN "Type"
+	1    25500 2050
 	0    1    -1   0
 $EndComp
@@
 D32A
 Text Label 23350 4300 0    50   ~ 0
-K32B
+K31B
 Text Label 22500 4500 0    50   ~ 0
 D31B
@@
 	33400 4950 35500 4950
 Wire Wire Line
-	25600 4950 25600 4900
+	25600 4950 25600 2450
 Wire Wire Line
 	24950 4950 25600 4950
@@
 	-1   0    0    -1
 $EndComp
-Wire Wire Line
-	3900 4950 3900 6350
 $Comp
 L BoatControl:TBL008V-1000-02BE J1
 U 1 1 8ADFCE69
-P 4000 6750
-F 0 "J1" V 3846 6622 50  0000 R CNN
-F 1 "TBL008V-1000-02BE" V 4250 7200 50  0000 R CNN
-F 2 "CUI_TBL008V-1000-02BE" H 4000 6750 50  0001 L BNN
-F 3 "CUI" H 4000 6750 50  0001 L BNN
-F 4 "AC 230V Common" V 4350 6800 50  0000 C CNN "Type"
-	1    4000 6750
+P 4000 7150
+F 0 "J1" V 3846 7022 50  0000 R CNN
+F 1 "TBL008V-1000-02BE" V 4250 7600 50  0000 R CNN
+F 2 "CUI_TBL008V-1000-02BE" H 4000 7150 50  0001 L BNN
+F 3 "CUI" H 4000 7150 50  0001 L BNN
+F 4 "AC 230V Common" V 4350 7200 50  0000 C CNN "Type"
+	1    4000 7150
 	0    -1   1    0
 $EndComp
@@
 	13750 6500 13750 6350
 Wire Wire Line
-	13750 6350 4000 6350
-Wire Wire Line
 	1500 6350 1500 5500
 Wire Wire Line
 	1500 5500 1850 5500
-Connection ~ 3900 6350
-Wire Wire Line
-	3900 6350 1500 6350
-Connection ~ 4000 6350
-Wire Wire Line
-	4000 6350 3900 6350
 Wire Wire Line
 	13650 6500 13650 6400
@@
 Wire Wire Line
 	13550 2950 13550 2550
+Wire Wire Line
+	1500 6350 13750 6350
+Wire Wire Line
+	3900 4950 3900 6750
 Wire Bus Line
 	3450 17500 15400 17500

Commit message: Wired
Connections:
- wire segments 2373 -> 2376
Changed lines of the file:
@@
 Connection ~ 13450 3600
 Wire Wire Line
-	4150 5450 4150 5850
+	4150 5450 4150 5600
 Connection ~ 4150 5450
 Wire Wire Line
@@
 Connection ~ 12250 5450
 Wire Wire Line
-	3250 5850 4150 5850
-Wire Wire Line
 	15200 3600 15200 3050
 Connection ~ 15200 3600
@@
 	3050 3400 4000 3400
 Wire Wire Line
-	3200 3800 3200 5900
-Wire Wire Line
-	2650 4300 3100 4300
-Wire Wire Line
-	3100 4300 3100 6000
-Wire Wire Line
-	2650 4200 2900 4200
-Wire Wire Line
-	2900 4200 2900 3250
-Wire Wire Line
-	2950 3300 2950 4100
-Wire Wire Line
-	2950 4100 2650 4100
-Wire Wire Line
-	3150 4000 2650 4000
-Wire Wire Line
-	3150 4000 3150 5950
-Wire Wire Line
-	3200 3800 2650 3800
-Wire Wire Line
-	3250 3600 2650 3600
-Wire Wire Line
-	3250 3600 3250 5850
-Wire Wire Line
-	3000 3350 3000 3900
-Wire Wire Line
-	3000 3900 2650 3900
-Wire Wire Line
-	3050 3400 3050 3700
-Wire Wire Line
-	3050 3700 2650 3700
+	3000 3350 3000 3800
 Text Label 26950 5450 3    50   ~ 0
 D25B
@@
 Wire Wire Line
 	3900 4950 3900 6750
+Wire Wire Line
+	2900 3250 2900 4200
+Wire Wire Line
+	4150 5600 3250 5600
+Wire Wire Line
+	3100 4300 3100 6000
+Wire Wire Line
+	2650 4200 2900 4200
+Wire Wire Line
+	2650 4300 3100 4300
+Wire Wire Line
+	2650 4100 3150 4100
+Wire Wire Line
+	3150 4100 3150 5950
+Wire Wire Line
+	2950 4000 2950 3300
+Wire Wire Line
+	2950 4000 2650 4000
+Wire Wire Line
+	3200 3900 3200 5900
+Wire Wire Line
+	2650 3800 3000 3800
+Wire Wire Line
+	2650 3900 3200 3900
+Wire Wire Line
+	3250 3700 2650 3700
+Wire Wire Line
+	3250 3700 3250 5600
+Wire Wire Line
+	3050 3400 3050 3600
+Wire Wire Line
+	3050 3600 2650 3600
+Wire Wire Line
+	25000 5600 25300 5600
+Wire Wire Line
+	25300 5600 25300 3450
+Wire Wire Line
+	25300 3450 24050 3450
 Wire Bus Line
 	3450 17500 15400 17500
@@
 Wire Bus Line
 	3000 11350 25700 11350
+Connection ~ 25000 5600
+Connection ~ 24050 3450
 $EndSCHEMATC
