File: boatcontrol/boatcontrol.sch (KiCad schematic (older format))
At the start: 343 parts, among them J1 TBL008V-1000-02BE, J10 TBL008V-1000-08BE, J11 TBL008V-1000-02BE, J12 TBL008V-1000-08BE, J2 SS73100-047F, J3 SS73100-047F, J4 TBP01R2W-508-08BE, J5 TBP01R2W-508-16BE, J6 TBP01R2W-508-08BE, J7 RPi_GPIO, J8 TBL008V-1000-02BE, J9 TBL008V-1000-02BE, K1 G5RL-K1A-E-DC12, K10 G5RL-K1A-E-DC12, K11 G5RL-K1A-E-DC12, K12 G5RL-K1A-E-DC12, K13 G5RL-K1A-E-DC12, K14 G5RL-K1A-E-DC12, K15 G5RL-K1A-E-DC12, K16 G5RL-K1A-E-DC12, K17 G5RL-K1A-E-DC12, K18 G5RL-K1A-E-DC12, K19 G5RL-K1A-E-DC12, K2 G5RL-K1A-E-DC12, K20 G5RL-K1A-E-DC12, K21 G5RL-K1A-E-DC12, K22 G5RL-K1A-E-DC12, K23 G5RL-K1A-E-DC12, K24 G5RL-K1A-E-DC12, K25 G5RL-K1A-E-DC12, K26 G5RL-K1A-E-DC12, K27 G5RL-K1A-E-DC12, K28 G5RL-K1A-E-DC12, K29 G5RL-K1A-E-DC12, K3 G5RL-K1A-E-DC12, K30 G5RL-K1A-E-DC12, K31 G5RL-K1A-E-DC12, K32 G5RL-K1A-E-DC12, K33 EW60-1A3-CL12D04, K34 EW60-1A3-CL12D04, K35 EW60-1A3-CL12D04, K36 EW60-1A3-CL12D04, K37 EW60-1A3-CL12D04, K38 EW60-1A3-CL12D04, K39 EW60-1A3-CL12D04, K4 G5RL-K1A-E-DC12, K40 EW60-1A3-CL12D04, K5 G5RL-K1A-E-DC12, K6 G5RL-K1A-E-DC12, K7 G5RL-K1A-E-DC12, K8 G5RL-K1A-E-DC12, K9 G5RL-K1A-E-DC12, Q1 SchurterCircuitBreaker 3a, Q10 SchurterCircuitBreaker 3a, Q11 SchurterCircuitBreaker 3a, Q12 SchurterCircuitBreaker 3a, Q13 SchurterCircuitBreaker 3a, Q14 SchurterCircuitBreaker 3a, Q15 SchurterCircuitBreaker 3a, Q16 SchurterCircuitBreaker 3a, Q17 SchurterCircuitBreaker 6a, Q18 SchurterCircuitBreaker 6a, Q19 SchurterCircuitBreaker 6a, Q2 SchurterCircuitBreaker 3a, Q20 SchurterCircuitBreaker 6a, Q21 SchurterCircuitBreaker 10a, Q22 SchurterCircuitBreaker 10a, Q23 SchurterCircuitBreaker 16a, Q24 SchurterCircuitBreaker 16a, Q25 SchurterCircuitBreaker 6a, Q26 SchurterCircuitBreaker 6a, Q27 SchurterCircuitBreaker 6a, Q28 SchurterCircuitBreaker 6a, Q29 SchurterCircuitBreaker 10a, Q3 SchurterCircuitBreaker 3a, Q30 SchurterCircuitBreaker 10a, Q31 SchurterCircuitBreaker 16a, Q32 SchurterCircuitBreaker 16a, Q33 SchurterCircuitBreaker 3a, Q4 SchurterCircuitBreaker 3a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

Commit message: Routing RJ45
Connections:
- net at U7.28 (GPA7): now also U9.1 (I1)
Changed lines of the file:
@@
 Wire Wire Line
 	31950 16050 32250 16050
+Wire Wire Line
+	14500 8950 28750 8950
 Wire Bus Line
 	3300 17750 15250 17750

Commit message: Before Big Power
Parts:
- J7: symbol RPi_Hat-rescue:RPi_GPIO -> boatcontrol-rescue:RPi_GPIO-RPi_Hat-rescue
- renumbered SW34A2 to SW35A1, SW36B2 to SW37B1
Changed lines of the file:
@@
 	7250 19650 7350 19550
 $Comp
-L RPi_Hat-rescue:RPi_GPIO J7
+L boatcontrol-rescue:RPi_GPIO-RPi_Hat-rescue J7
 U 1 1 B9E969F9
 P 30000 6350
@@
 $EndComp
 $Comp
-L Switch:SW_Push_DPDT SW34A2
+L Switch:SW_Push_DPDT SW35A1
 U 1 1 FA3EDD46
 P 7450 19350
-F 0 "SW34A2" V 7300 19350 50  0000 C CNN
+F 0 "SW35A1" V 7300 19350 50  0000 C CNN
 F 1 " ESB30" V 7400 19400 50  0000 C CNN
 F 2 "BoatControl:SW_PUSH_ESB30_DPDT" H 7450 19550 50  0001 C CNN
@@
 $EndComp
 $Comp
-L Switch:SW_Push_DPDT SW36B2
+L Switch:SW_Push_DPDT SW37B1
 U 1 1 FD1E3E6B
 P 10650 18050
-F 0 "SW36B2" V 10500 18050 50  0000 C CNN
+F 0 "SW37B1" V 10500 18050 50  0000 C CNN
 F 1 " ESB30" V 10600 18050 50  0000 C CNN
 F 2 "BoatControl:SW_PUSH_ESB30_DPDT" H 10650 18250 50  0001 C CNN

Commit message: Split 60A to own daughter board.
Parts:
- removed J7: RPi_GPIO, BoatControl:Samtec_HLE-120-02-XXX-DV-BE-XX-XX, symbol boatcontrol-rescue:RPi_GPIO-RPi_Hat-rescue
- added J?: Raspberry_Pi_2_3, Connector_PinSocket_2.00mm:PinSocket_2x20_P2.00mm_Vertical, symbol Connector:Raspberry_Pi_2_3
- added J?: Conn_02x20_Odd_Even Header, Connector_PinSocket_2.00mm:PinSocket_2x20_P2.00mm_Vertical, symbol Connector_Generic:Conn_02x20_Odd_Even
- added J?: Conn_02x20_Odd_Even Socket, Connector_PinHeader_2.00mm:PinHeader_2x20_P2.00mm_Vertical, symbol Connector_Generic:Conn_02x20_Odd_Even
Connections:
- net D33A: no longer D33.1 (A1), RN2.9 (R8.2)
- net D33B: no longer D33.3 (A2), RN1.9 (R8.2), RN2.10 (R7.2)
- net D34A: no longer D34.1 (A1), RN2.11 (R6.2)
- net D34B: no longer D34.3 (A2), RN2.12 (R5.2)
- net D35A: no longer D35.1 (A1), RN2.13 (R4.2)
- net D35B: no longer D35.3 (A2), RN2.14 (R3.2)
- net D36A: no longer D36.1 (A1), RN2.15 (R2.2)
- net D36B: no longer D36.3 (A2), RN2.16 (R1.2)
- net D37A: no longer D37.1 (A1), RN1.16 (R1.2)
- net D37B: no longer D37.3 (A2), RN1.15 (R2.2)
- net D38A: no longer D38.1 (A1), RN1.14 (R3.2)
- net D38B: no longer D38.3 (A2), RN1.13 (R4.2)
- net D39A: no longer D39.1 (A1), RN1.12 (R5.2)
- net D39B: no longer D39.3 (A2), RN1.11 (R6.2)
- net D40A: no longer D40.1 (A1), RN1.10 (R7.2)
- net K33A: now also J?.1 (Pin_1); no longer RN2.8 (R8.1), SW33A1.2 (B), SW33A1.5 (B)
- net K33B: now also J?.2 (Pin_2); no longer RN1.8 (R8.1), RN2.7 (R7.1), SWSW33B1.2 (B), SWSW33B1.5 (B)
- net K34A: now also J?.3 (Pin_3); no longer RN2.6 (R6.1), SW34A1.2 (B), SW34A1.5 (B)
- net K34B: now also J?.4 (Pin_4); no longer RN2.5 (R5.1)
- net K35A: now also J?.5 (Pin_5); no longer RN2.4 (R4.1), SW35A1.2 (B), SW35A1.5 (B)
- net K35B: now also J?.6 (Pin_6); no longer RN2.3 (R3.1)
- net K36A: now also J?.7 (Pin_7); no longer RN2.2 (R2.1), SW36A1.2 (B), SW36A1.5 (B)
- net K36B: now also J?.8 (Pin_8); no longer RN2.1 (R1.1)
- net K37A: no longer RN1.1 (R1.1), SW37A1.2 (B), SW37A1.5 (B)
- net K37B: no longer RN1.2 (R2.1)
- net K38A: now also J?.9 (Pin_9); no longer RN1.3 (R3.1), SW38A1.2 (B), SW38A1.5 (B)
- net K38B: now also J?.10 (Pin_10); no longer RN1.4 (R4.1), SW38B1.2 (B), SW38B1.5 (B)
- net K39A: now also J?.11 (Pin_11); no longer RN1.5 (R5.1), SW39A1.2 (B), SW39A1.5 (B)
- net K39B: now also J?.12 (Pin_12); no longer RN1.6 (R6.1), SW39B1.2 (B), SW39B1.5 (B)
- net K40A: now also K40.A3, J?.13 (Pin_13); no longer RN1.7 (R7.1)
- net K40B: now also J?.14 (Pin_14)
- net at K33.1, K33.2, K33.3: now also J10.1_1 (01P), J10.1_2 (01P), J10.1_3 (01P); no longer J12.1_1 (01P), J12.1_2 (01P), J12.1_3 (01P)
- net at K33.4, K33.5, K33.6: now also J12.1_1 (01P), J12.1_2 (01P), J12.1_3 (01P); no longer J10.1_1 (01P), J10.1_2 (01P), J10.1_3 (01P)
- net at K33.A1, K34.A1, K35.A1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: now also J?.27 (Pin_27), J?.28 (Pin_28), J?.29 (Pin_29), J?.30 (Pin_30), J?.31 (Pin_31), J?.32 (Pin_32), J?.33 (Pin_33), J?.34 (Pin_34), J?.35 (Pin_35), J?.36 (Pin_36), J?.37 (Pin_37), J?.38 (Pin_38), J?.39 (Pin_39), J?.40 (Pin_40); no longer D33.2 (K), D34.2 (K), D35.2 (K), D36.2 (K), D37.2 (K), D38.2 (K), D39.2 (K), D40.2 (K)
- net at K34.1, K34.2, K34.3: now also J10.2_1 (02P), J10.2_2 (02P), J10.2_3 (02P); no longer J12.2_1 (02P), J12.2_2 (02P), J12.2_3 (02P)
- net at K34.4, K34.5, K34.6: now also J12.2_1 (02P), J12.2_2 (02P), J12.2_3 (02P); no longer J10.2_1 (02P), J10.2_2 (02P), J10.2_3 (02P)
- net at K35.1, K35.2, K35.3: now also J10.3_1 (03P), J10.3_2 (03P), J10.3_3 (03P); no longer J12.3_1 (03P), J12.3_2 (03P), J12.3_3 (03P)
- net at K35.4, K35.5, K35.6: now also J12.3_1 (03P), J12.3_2 (03P), J12.3_3 (03P); no longer J10.3_1 (03P), J10.3_2 (03P), J10.3_3 (03P)
- net at K36.1, K36.2, K36.3: now also J10.4_1 (04P), J10.4_2 (04P), J10.4_3 (04P); no longer J12.4_1 (04P), J12.4_2 (04P), J12.4_3 (04P)
- net at K36.4, K36.5, K36.6: now also J12.4_1 (04P), J12.4_2 (04P), J12.4_3 (04P); no longer J10.4_1 (04P), J10.4_2 (04P), J10.4_3 (04P)
- net at K37.1, K37.2, K37.3: now also J10.5_1 (05P), J10.5_2 (05P), J10.5_3 (05P); no longer J12.5_1 (05P), J12.5_2 (05P), J12.5_3 (05P)
- net at K37.4, K37.5, K37.6: now also J12.5_1 (05P), J12.5_2 (05P), J12.5_3 (05P); no longer J10.5_1 (05P), J10.5_2 (05P), J10.5_3 (05P)
- net at K38.1, K38.2, K38.3: now also J10.6_1 (06P), J10.6_2 (06P), J10.6_3 (06P); no longer J12.6_1 (06P), J12.6_2 (06P), J12.6_3 (06P)
- net at K38.4, K38.5, K38.6: now also J12.6_1 (06P), J12.6_2 (06P), J12.6_3 (06P); no longer J10.6_1 (06P), J10.6_2 (06P), J10.6_3 (06P)
- net at K39.1, K39.2, K39.3: now also J10.7_1 (07P), J10.7_2 (07P), J10.7_3 (07P); no longer J12.7_1 (07P), J12.7_2 (07P), J12.7_3 (07P)
- net at K39.4, K39.5, K39.6: now also J12.7_1 (07P), J12.7_2 (07P), J12.7_3 (07P); no longer J10.7_1 (07P), J10.7_2 (07P), J10.7_3 (07P)
- net at K40.1, K40.2, K40.3: now also J10.8_1 (08P), J10.8_2 (08P), J10.8_3 (08P); no longer J12.8_1 (08P), J12.8_2 (08P), J12.8_3 (08P)
- net at K40.4, K40.5, K40.6: now also J12.8_1 (08P), J12.8_2 (08P), J12.8_3 (08P); no longer J10.8_1 (08P), J10.8_2 (08P), J10.8_3 (08P)
- net at U19.21 (GPA0): no longer U21.11 (O8)
- net at U19.22 (GPA1): no longer U21.12 (O7)
- net at U19.23 (GPA2): no longer U21.13 (O6)
- net at U19.24 (GPA3): no longer U21.14 (O5)
- net at U19.5 (GPB4): no longer U20.15 (O4)
- net at U19.6 (GPB5): no longer U20.16 (O3)
- net at U19.7 (GPB6): no longer U20.17 (O2)
- net at U19.8 (GPB7): no longer U20.18 (O1)
- net at SW40B1.2 (B): no longer SW40B1.5 (B)
- net D40B: no longer names the net of D40.3 (A2)
- new net: D33.1 (A1), RN2.1 (R1.1)
- new net: D33.3 (A2), RN1.1 (R1.1)
- new net: D34.1 (A1), RN2.2 (R2.1)
- new net: D34.3 (A2), RN1.2 (R2.1)
- new net: D35.1 (A1), RN2.3 (R3.1)
- new net: D35.3 (A2), RN1.3 (R3.1)
- new net: D36.1 (A1), RN2.4 (R4.1)
- new net: D36.3 (A2), RN1.4 (R4.1)
- new net: D37.1 (A1), RN2.5 (R5.1)
- new net: D37.3 (A2), RN1.5 (R5.1)
- new net: D38.1 (A1), RN2.6 (R6.1)
- new net: D38.3 (A2), RN1.6 (R6.1)
- new net: D39.1 (A1), RN2.7 (R7.1)
- new net: D39.3 (A2), RN1.7 (R7.1)
- now unconnected: SW33A1.1 (A), SW33A1.3 (C), SW33A1.4 (A), SW33A1.6 (C), SW34A1.1 (A), SW34A1.3 (C), SW34A1.4 (A), SW34A1.6 (C), SW34B1.1 (A), SW34B1.3 (C), SW34B1.4 (A), SW34B1.6 (C), SW35A1.1 (A), SW35A1.3 (C), SW35A1.4 (A), SW35A1.6 (C), SW35B1.1 (A), SW35B1.3 (C), SW35B1.4 (A), SW35B1.6 (C), SW36A1.1 (A), SW36A1.3 (C), SW36A1.4 (A), SW36A1.6 (C), SW36B1.1 (A), SW36B1.3 (C), SW36B1.4 (A), SW36B1.6 (C), SW37A1.1 (A), SW37A1.3 (C), SW37A1.4 (A), SW37A1.6 (C), SW37B1.1 (A), SW37B1.3 (C), SW37B1.4 (A), SW37B1.6 (C), SW38A1.1 (A), SW38A1.3 (C), SW38A1.4 (A), SW38A1.6 (C), SW38B1.1 (A), SW38B1.3 (C), SW38B1.4 (A), SW38B1.6 (C), SW39A1.1 (A), SW39A1.3 (C), SW39A1.4 (A), SW39A1.6 (C), SW39B1.1 (A), SW39B1.3 (C), SW39B1.4 (A), SW39B1.6 (C), SW40A1.1 (A), SW40A1.2 (B), SW40A1.3 (C), SW40A1.4 (A), SW40A1.5 (B), SW40A1.6 (C), SW40B1.1 (A), SW40B1.3 (C), SW40B1.4 (A), SW40B1.6 (C), SWSW33B1.1 (A), SWSW33B1.3 (C), SWSW33B1.4 (A), SWSW33B1.6 (C), U20.1 (I1), U20.2 (I2), U20.3 (I3), U20.4 (I4), U20.5 (I5), U20.6 (I6), U20.7 (I7), U20.8 (I8), U21.1 (I1), U21.2 (I2), U21.3 (I3), U21.4 (I4), U21.5 (I5), U21.6 (I6), U21.7 (I7), U21.8 (I8), U21.9 (GND)
Other:
- moved on the sheet: D33, D34, D35, D36, D37, D38, D39, D40, J10, J12, K33, K34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

Commit message: Split high power
Connections:
- net at U19.1 (GPB0): now also U20.8 (I8); no longer U20.11 (O8)
- net at U19.2 (GPB1): now also U21.8 (I8); no longer U20.12 (O7)
- net at U19.21 (GPA0): now also U20.4 (I4)
- net at U19.22 (GPA1): now also U21.4 (I4)
- net at U19.23 (GPA2): now also U20.3 (I3)
- net at U19.24 (GPA3): now also U21.3 (I3)
- net at U19.25 (GPA4): now also U20.2 (I2); no longer U21.15 (O4)
- net at U19.26 (GPA5): now also U21.2 (I2); no longer U21.16 (O3)
- net at U19.27 (GPA6): now also U20.1 (I1); no longer U21.17 (O2)
- net at U19.28 (GPA7): now also U21.1 (I1); no longer U21.18 (O1)
- net at U19.3 (GPB2): now also U20.7 (I7); no longer U20.13 (O6)
- net at U19.4 (GPB3): now also U21.7 (I7); no longer U20.14 (O5)
- net at U19.5 (GPB4): now also U20.6 (I6)
- net at U19.6 (GPB5): now also U21.6 (I6)
- net at U19.7 (GPB6): now also U20.5 (I5)
- net at U19.8 (GPB7): now also U21.5 (I5)
- net at U20.15 (O4): now also J?.9 (Pin_9), RN2.12 (R5.2), SW37A1.2 (B), SW37A1.5 (B)
- net at U20.16 (O3): now also J?.11 (Pin_11), RN2.11 (R6.2), SW38A1.2 (B), SW38A1.5 (B)
- net at U20.17 (O2): now also J?.13 (Pin_13), RN2.10 (R7.2), SW39A1.2 (B), SW39A1.5 (B)
- net at U20.18 (O1): now also J?.15 (Pin_15), RN2.9 (R8.2), SW40A1.2 (B), SW40A1.5 (B)
- net at U21.11 (O8): now also J?.2 (Pin_2), RN1.16 (R1.2), SWSW33B1.2 (B), SWSW33B1.5 (B)
- net at U21.12 (O7): now also J?.4 (Pin_4), RN1.15 (R2.2), SW34B1.2 (B), SW34B1.5 (B)
- net at U21.13 (O6): now also RN1.14 (R3.2), SW35B1.2 (B)
- net at U21.14 (O5): now also J?.8 (Pin_8), RN1.13 (R4.2), SW36B1.2 (B), SW36B1.5 (B)
- net at D33.2 (K): now also D34.2 (K), D35.2 (K), D36.2 (K), D37.2 (K), D38.2 (K), D39.2 (K), D40.2 (K)
- net at D40.1 (A1): now also RN2.8 (R8.1)
- net at D40.3 (A2): now also RN1.8 (R8.1)
- net at RN2.13 (R4.2): now also J?.7 (Pin_7), SW36A1.2 (B), SW36A1.5 (B), U20.14 (O5)
- net at RN2.14 (R3.2): now also J?.5 (Pin_5), SW35A1.2 (B), SW35A1.5 (B), U20.13 (O6)
- net at RN2.15 (R2.2): now also J?.3 (Pin_3), SW34A1.2 (B), SW34A1.5 (B), U20.12 (O7)
- net at RN2.16 (R1.2): now also J?.1 (Pin_1), SW33A1.2 (B), SW33A1.5 (B), U20.11 (O8)
- net at RN1.10 (R7.2): now also J?.14 (Pin_14), SW39B1.2 (B), SW39B1.5 (B), U21.17 (O2)
- net at RN1.11 (R6.2): now also J?.12 (Pin_12), SW38B1.2 (B), SW38B1.5 (B), U21.16 (O3)
- net at RN1.12 (R5.2): now also J?.10 (Pin_10), SW37B1.2 (B), SW37B1.5 (B), U21.15 (O4)
- net at RN1.9 (R8.2): now also J?.16 (Pin_16), SW40B1.2 (B), SW40B1.5 (B), U21.18 (O1)
- net at J?.27 (Pin_27): now also J?.28 (Pin_28), J?.29 (Pin_29), J?.30 (Pin_30), J?.31 (Pin_31), J?.32 (Pin_32), J?.33 (Pin_33), J?.34 (Pin_34), J?.35 (Pin_35), J?.36 (Pin_36), J?.37 (Pin_37), J?.38 (Pin_38), J?.39 (Pin_39), J?.40 (Pin_40)
- net at J?.6 (Pin_6): now also SW35B1.5 (B)
- net at SWSW33B1.1 (A): now also SWSW33B1.3 (C), SWSW33B1.4 (A)
- net at SWSW33B1.6 (C): now also SW33A1.6 (C), SW34A1.6 (C), SW34B1.6 (C), SW35A1.6 (C), SW36A1.6 (C), SW37A1.6 (C), SW38A1.6 (C), SW39A1.6 (C)
- net at SW33A1.1 (A): now also SW33A1.3 (C), SW33A1.4 (A)
- net at SW34A1.1 (A): now also SW34A1.3 (C), SW34A1.4 (A)
- net at SW35A1.1 (A): now also SW35A1.3 (C), SW35A1.4 (A)
- net at SW36A1.1 (A): now also SW36A1.3 (C), SW36A1.4 (A)
- net at SW37A1.1 (A): now also SW37A1.3 (C), SW37A1.4 (A)
- net at SW38A1.1 (A): now also SW38A1.3 (C), SW38A1.4 (A)
- net at SW39A1.1 (A): now also SW39A1.3 (C), SW39A1.4 (A)
- net at SW40A1.1 (A): now also SW40A1.3 (C), SW40A1.4 (A)
- net at SW34B1.1 (A): now also SW34B1.3 (C), SW34B1.4 (A)
- net at SW35B1.1 (A): now also SW35B1.3 (C), SW35B1.4 (A)
- net at SW36B1.1 (A): now also SW36B1.3 (C), SW36B1.4 (A)
- net at SW36B1.6 (C): now also SW37B1.6 (C), SW38B1.6 (C), SW39B1.6 (C), SW40B1.6 (C)
- net at SW37B1.1 (A): now also SW37B1.3 (C), SW37B1.4 (A)
- net at SW38B1.1 (A): now also SW38B1.3 (C), SW38B1.4 (A)
- net at SW39B1.1 (A): now also SW39B1.3 (C), SW39B1.4 (A)
- net at SW40B1.1 (A): now also SW40B1.3 (C), SW40B1.4 (A)
Other:
- moved on the sheet: D33, D34, D35, D36, D37, D38, D39, D40, J5, J?, RN1, RN2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

Commit message: Lots of logical cleanup
Connections:
- net RPIBCM1_ID_SC: now also J?.28 (ID_SC/GPIO1)
- net RPIBCM20_MOSI: now also J?.38 (GPIO20/MOSI1)
- net RPi3.3V: now also J?.1 (3V3), J?.17 (3V3)
- net RPiBCM0_ID_SD: now also J?.27 (ID_SD/GPIO0)
- net RPiBCM10_MOSI: now also J?.19 (MOSI0/GPIO10)
- net RPiBCM11_SCLK: now also J?.23 (SCLK0/GPIO11)
- net RPiBCM12: now also J?.32 (PWM0/GPIO12)
- net RPiBCM13: now also J?.33 (PWM1/GPIO13)
- net RPiBCM14_TXD: now also J?.8 (GPIO14/TXD)
- net RPiBCM15_RXD: now also J?.10 (GPIO15/RXD)
- net RPiBCM16: now also J?.36 (GPIO16)
- net RPiBCM17: now also J?.11 (GPIO17)
- net RPiBCM19_MISO: now also J?.35 (GPIO19/MISO1)
- net RPiBCM21_SCLK: now also J?.40 (GPIO21/SCLK1)
- net RPiBCM22: now also J?.15 (GPIO22)
- net RPiBCM23: now also J?.16 (GPIO23)
- net RPiBCM24: now also J?.18 (GPIO24)
- net RPiBCM25: now also J?.22 (GPIO25)
- net RPiBCM27_PCM_D: now also J?.13 (GPIO27)
- net RPiBCM2_SDA: now also J?.3 (SDA/GPIO2)
- net RPiBCM3_SCL: now also J?.5 (SCL/GPIO3)
- net RPiBCM4_GPCLK0: now also J?.7 (GCLK0/GPIO4)
- net RPiBCM5: now also J?.29 (GCLK1/GPIO5)
- net RPiBCM6: now also J?.31 (GCLK2/GPIO6)
- net RPiBCM7_CE1: now also J?.26 (~CE1~/GPIO7)
- net RPiBCM8_CEO: now also J?.24 (~CE0~/GPIO8)
- net RPiBCM9_MISO: now also J?.21 (MISO0/GPIO9)
- net RPiGND: now also J?.14 (GND), J?.20 (GND), J?.25 (GND), J?.30 (GND), J?.34 (GND), J?.39 (GND), J?.6 (GND), J?.9 (GND)
- net at SW31A1.1 (A), SW31A1.3 (C), SW31A1.4 (A): no longer U18.11 (O8)
- net RPiBCM18: now reaches J?.12 (GPIO18/PWM0)
- net RPiBCM26: now reaches J?.37 (GPIO26)
- net at J2.A_2 (2): now also J2.A_4 (4), J2.A_6 (6), J2.A_8 (8), J2.B_2 (2), J2.B_4 (4), J2.B_6 (6), J2.B_8 (8), J2.C_2 (2), J2.C_4 (4), J2.C_6 (6), J2.C_8 (8), J2.D_2 (2), J2.D_4 (4), J2.D_6 (6), J2.D_8 (8), J2.E_2 (2), J2.E_4 (4), J2.E_6 (6), J2.E_8 (8), J2.F_2 (2), J2.F_4 (4), J2.F_6 (6), J2.F_8 (8), J2.G_2 (2), J2.G_4 (4), J2.G_6 (6), J2.G_8 (8), J2.H_2 (2), J2.H_4 (4), J2.H_6 (6), J2.H_8 (8)
- net at SW33A1.6 (C), SW34A1.6 (C), SW34B1.6 (C)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: now also SW35B1.6 (C), SW36B1.6 (C), SW37B1.6 (C), SW38B1.6 (C), SW39B1.6 (C), SW40A1.6 (C), SW40B1.6 (C)
Other:
- moved on the sheet: J2A, J?, RN10, RN3, RN4, RN5, RN6, RN7, RN8, RN9, U1, U2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

Commit message: Just need the controller wires now
Connections:
- net RPIBCM1_ID_SC: now also J2.K_6 (6)
- net RPIBCM20_MOSI: now also J2.J_4 (4)
- net RPi3.3V: now also J2.I_1 (1), J2.J_1 (1), J2.K_1 (1), J2.L_1 (1)
- net RPiBCM0_ID_SD: now also J2.K_5 (5)
- net RPiBCM10_MOSI: now also J2.I_4 (4)
- net RPiBCM11_SCLK: now also J2.I_5 (5)
- net RPiBCM12: now also J2.L_3 (3)
- net RPiBCM13: now also J2.L_4 (4)
- net RPiBCM14_TXD: now also J2.L_5 (5)
- net RPiBCM15_RXD: now also J2.L_6 (6)
- net RPiBCM16: now also J2.L_7 (7)
- net RPiBCM17: now also J2.L_8 (8)
- net RPiBCM19_MISO: now also J2.J_3 (3)
- net RPiBCM21_SCLK: now also J2.J_5 (5)
- net RPiBCM22: now also J2.K_7 (7)
- net RPiBCM23: now also J2.K_8 (8)
- net RPiBCM25: now also J2.J_8 (8)
- net RPiBCM26: now also J2.J_7 (7)
- net RPiBCM27_PCM_D: now also J2.J_6 (6)
- net RPiBCM2_SDA: now also J2.K_3 (3)
- net RPiBCM3_SCL: now also J2.K_4 (4)
- net RPiBCM4_GPCLK0: now also J2.I_6 (6)
- net RPiBCM5: now also J2.I_7 (7)
- net RPiBCM6: now also J2.I_8 (8)
- net RPiBCM9_MISO: now also J2.I_3 (3)
- net RPiGND: now also J2.I_2 (2), J2.J_2 (2), J2.K_2 (2), J2.L_2 (2)
- net SW33A1: now reaches J2.M_1 (1)
- net SW33A1: now also SW33A1.1 (A), SW33A1.3 (C), SW33A1.4 (A)
- net at J2.M_2 (2): now also J2.M_4 (4), J2.M_6 (6), J2.M_8 (8), J2.N_2 (2), J2.N_4 (4), J2.N_6 (6), J2.N_8 (8), J2.O_2 (2), J2.O_4 (4), J2.O_6 (6), J2.O_8 (8), J2.P_2 (2), J2.P_4 (4), J2.P_6 (6), J2.P_8 (8)
- net SW33B1: now reaches J2.M_3 (3)
- net SW33B1: now also SWSW33B1.1 (A), SWSW33B1.3 (C), SWSW33B1.4 (A)
- net SW34A1: now reaches J2.M_5 (5)
- net SW34A1: now also SW34A1.1 (A), SW34A1.3 (C), SW34A1.4 (A)
- net SW34B1: now reaches J2.M_7 (7)
- net SW34B1: now also SW34B1.1 (A), SW34B1.3 (C), SW34B1.4 (A)
- net SW35A1: now reaches J2.N_1 (1)
- net SW35A1: now also SW35A1.1 (A), SW35A1.3 (C), SW35A1.4 (A)
- net SW35B1: now reaches J2.N_3 (3)
- net SW35B1: now also SW35B1.1 (A), SW35B1.3 (C), SW35B1.4 (A)
- net SW36A1: now reaches J2.N_5 (5)
- net SW36A1: now also SW36A1.1 (A), SW36A1.3 (C), SW36A1.4 (A)
- net SW36B1: now reaches J2.N_7 (7)
- net SW36B1: now also SW36B1.1 (A), SW36B1.3 (C), SW36B1.4 (A)
- net SW37A1: now reaches J2.O_1 (1)
- net SW37A1: now also SW37A1.1 (A), SW37A1.3 (C), SW37A1.4 (A)
- net SW37B1: now reaches J2.O_3 (3)
- net SW37B1: now also SW37B1.1 (A), SW37B1.3 (C), SW37B1.4 (A)
- net SW38A1: now reaches J2.O_5 (5)
- net SW38A1: now also SW38A1.1 (A), SW38A1.3 (C), SW38A1.4 (A)
- net SW38B1: now reaches J2.O_7 (7)
- net SW38B1: now also SW38B1.1 (A), SW38B1.3 (C), SW38B1.4 (A)
- net SW39A1: now reaches J2.P_1 (1)
- net SW39A1: now also SW39A1.1 (A), SW39A1.3 (C), SW39A1.4 (A)
- net SW39B1: now reaches J2.P_3 (3)
- net SW39B1: now also SW39B1.1 (A), SW39B1.3 (C), SW39B1.4 (A)
- net SW40A1: now reaches J2.P_5 (5)
- net SW40A1: now also SW40A1.1 (A), SW40A1.3 (C), SW40A1.4 (A)
- net SW40B1: now reaches J2.P_7 (7)
- net SW40B1: now also SW40B1.1 (A), SW40B1.3 (C), SW40B1.4 (A)
- net RPiBCM18 renamed RPiBCM18_PWM0
Other:
- moved on the sheet: J?

Commit message: Everything Logically Wired in the Schematic
Parts:
- removed JP10, JP11, JP14, JP15, JP16, JP17, JP20, JP9: SolderJumper_2_Open, Jumper:SolderJumper-2_P1.3mm_Open_RoundedPad1.0x1.5mm, symbol Jumper:SolderJumper_2_Open
- removed JP12, JP13, JP18, JP19, JP21, JP4, JP5, JP6, JP7, JP8: SolderJumper_2_Bridged, Jumper:SolderJumper-2_P1.3mm_Bridged_RoundedPad1.0x1.5mm, symbol Jumper:SolderJumper_2_Bridged
- added JP? (x19): SolderJumper_2_Bridged, Jumper:SolderJumper-2_P1.3mm_Bridged_RoundedPad1.0x1.5mm, symbol Jumper:SolderJumper_2_Bridged
- added JP? (x20): SolderJumper_2_Open, Jumper:SolderJumper-2_P1.3mm_Open_RoundedPad1.0x1.5mm, symbol Jumper:SolderJumper_2_Open
Connections:
- net +5V: now also J?.2 (5V), J?.4 (5V), JP1.1 (A), JP2.1 (A), U1.9 (VDD), U10.10 (VSS), U13.9 (VDD), U16.9 (VDD), U19.9 (VDD), U4.9 (VDD), U7.9 (VDD), JP?.1 (A), JP?.1 (A), JP?.1 (A), JP?.1 (A), JP?.1 (A), JP?.1 (A), JP?.1 (A), JP?.1 (A), JP?.1 (A), JP?.1 (A), JP?.1 (A), JP?.1 (A), JP?.1 (A), JP?.1 (A), JP?.1 (A), JP?.1 (A), JP?.1 (A), JP?.1 (A), JP?.1 (A)
- net RPiGND: now also JP3.1 (A), U1.10 (VSS), U10.9 (VDD), U11.9 (GND), U13.10 (VSS), U14.9 (GND), U15.9 (GND), U16.10 (VSS), U17.9 (GND), U18.9 (GND), U19.10 (VSS), U2.9 (GND), U20.9 (GND), U21.9 (GND), U3.9 (GND), U4.10 (VSS), U5.9 (GND), U6.9 (GND), U7.10 (VSS), U8.9 (GND), JP?.1 (A), JP?.1 (A), JP?.1 (A), JP?.1 (A), JP?.1 (A), JP?.1 (A), JP?.1 (A), JP?.1 (A), JP?.1 (A), JP?.1 (A), JP?.1 (A), JP?.1 (A), JP?.1 (A), JP?.1 (A), JP?.1 (A), JP?.1 (A), JP?.1 (A), JP?.1 (A), JP?.1 (A), JP?.1 (A)
- net at C2.1, L1.2, U22.6 (FB): now also U11.10 (COM), U12.10 (COM), U14.10 (COM), U15.10 (COM), U17.10 (COM), U18.10 (COM), U2.10 (COM), U20.10 (COM), U21.10 (COM), U3.10 (COM), U5.10 (COM), U6.10 (COM), U8.10 (COM), U9.10 (COM)
- net at U13.15 (A0): now also JP?.2 (B), JP?.2 (B)
- net at U13.16 (A1): now also JP?.2 (B), JP?.2 (B)
- net at U13.17 (A2): now also JP?.2 (B), JP?.2 (B)
- net at U16.15 (A0): now also JP?.2 (B), JP?.2 (B)
- net at U16.16 (A1): now also JP?.2 (B), JP?.2 (B)
- net at U16.17 (A2): now also JP?.2 (B), JP?.2 (B)
- net at U1.15 (A0): now also JP?.2 (B), JP?.2 (B)
- net at U1.16 (A1): now also JP?.2 (B), JP?.2 (B)
- net at U1.17 (A2): now also JP?.2 (B), JP?.2 (B)
- net at U19.15 (A0): now also JP?.2 (B), JP?.2 (B)
- net at U19.16 (A1): now also JP?.2 (B), JP?.2 (B)
- net at U19.17 (A2): now also JP?.2 (B), JP?.2 (B)
- net at U10.15 (A0): now also JP3.2 (B), JP?.2 (B)
- net at U10.16 (A1): now also JP2.2 (B), JP?.2 (B)
- net at U10.17 (A2): now also JP1.2 (B), JP?.2 (B)
- net at U7.15 (A0): now also JP?.2 (B), JP?.2 (B)
- net at U7.16 (A1): now also JP?.2 (B), JP?.2 (B)
- net at U7.17 (A2): now also JP?.2 (B), JP?.2 (B)
- net at U4.15 (A0): now also JP?.2 (B), JP?.2 (B)
- net at U4.16 (A1): now also JP?.2 (B), JP?.2 (B)
- net at U4.17 (A2): now also JP?.2 (B), JP?.2 (B)
- no-connect marks 0 -> 3
Other:
- note added: "I2C Address 0x20"
- note added: "I2C Address 0x21"
- note added: "I2C Address 0x22"
- note added: "I2C Address 0x23"
- moved on the sheet: C1, C2, C3, C4, C5, C6, C7, C8, D41, D42, J11, JP1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

Commit message: Fix I2C Addresses
Parts:
- gave numbers to parts that had none: 42
Connections:
- net +5V: now also JP16.1 (A), JP18.1 (A), JP21.1 (A), JP24.1 (A), JP25.1 (A), JP28.1 (A), JP29.1 (A), JP3.1 (A), JP34.1 (A), JP42.1 (A), JP5.1 (A), JP6.1 (A), JP8.1 (A), U10.9 (VDD); no longer JP1.1 (A), JP12.1 (A), JP15.1 (A), JP17.1 (A), JP2.1 (A), JP22.1 (A), JP23.1 (A), JP26.1 (A), JP27.1 (A), JP30.1 (A), JP33.1 (A), JP4.1 (A), JP41.1 (A), U10.10 (VSS)
- net RPiGND: now also JP1.1 (A), JP12.1 (A), JP15.1 (A), JP17.1 (A), JP2.1 (A), JP22.1 (A), JP23.1 (A), JP26.1 (A), JP27.1 (A), JP30.1 (A), JP33.1 (A), JP4.1 (A), JP41.1 (A), U10.10 (VSS); no longer JP16.1 (A), JP18.1 (A), JP21.1 (A), JP24.1 (A), JP25.1 (A), JP28.1 (A), JP29.1 (A), JP3.1 (A), JP34.1 (A), JP42.1 (A), JP5.1 (A), JP6.1 (A), JP8.1 (A), U10.9 (VDD)
Other:
- note added: "I2C Address 0x24"
- note added: "I2C Address 0x25"
- note added: "I2C Address 0x26"
- moved on the sheet: JP15, JP16, JP17, JP18, JP21, JP22, JP23, JP24, JP25, JP26, JP27, JP28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
