File: boatcontrol/boatcontrol.kicad_pcb (KiCad board)
At the start: 2 copper layers, 271 parts, among them J1 TBL008V-1000-02BE, J10 TBL008V-1000-08BE, J11 TBL008V-1000-02BE, J12 TBL008V-1000-08BE, J2 SS73100-047F, J3 SS73100-047F, J4 TBP01R2W-508-08BE, J5 TB007-508-16BE, J6 TBP01R2W-508-08BE, J7 RPi_GPIO, J8 TBL008V-1000-02BE, J9 TBL008V-1000-02BE, K1 G5RL-K1A-E-DC12, K10 G5RL-K1A-E-DC12, K11 G5RL-K1A-E-DC12, K12 G5RL-K1A-E-DC12, K13 G5RL-K1A-E-DC12, K14 G5RL-K1A-E-DC12, K15 G5RL-K1A-E-DC12, K16 G5RL-K1A-E-DC12, K17 G5RL-K1A-E-DC12, K18 G5RL-K1A-E-DC12, K19 G5RL-K1A-E-DC12, K2 G5RL-K1A-E-DC12, K20 G5RL-K1A-E-DC12, K21 G5RL-K1A-E-DC12, K22 G5RL-K1A-E-DC12, K23 G5RL-K1A-E-DC12, K24 G5RL-K1A-E-DC12, K25 G5RL-K1A-E-DC12, K26 G5RL-K1A-E-DC12, K27 G5RL-K1A-E-DC12, K28 G5RL-K1A-E-DC12, K29 G5RL-K1A-E-DC12, K3 G5RL-K1A-E-DC12, K30 G5RL-K1A-E-DC12, K31 G5RL-K1A-E-DC12, K32 G5RL-K1A-E-DC12, K33 EW60-1A3-CL12D04, K34 EW60-1A3-CL12D04, K35 EW60-1A3-CL12D04, K36 EW60-1A3-CL12D04, K37 EW60-1A3-CL12D04, K38 EW60-1A3-CL12D04, K39 EW60-1A3-CL12D04, K4 G5RL-K1A-E-DC12, K40 EW60-1A3-CL12D04, K5 G5RL-K1A-E-DC12, K6 G5RL-K1A-E-DC12, K7 G5RL-K1A-E-DC12, K8 G5RL-K1A-E-DC12, K9 G5RL-K1A-E-DC12, Q1 SchurterCircuitBreaker 3a, Q10 SchurterCircuitBreaker 3a, Q11 SchurterCircuitBreaker 3a, Q12 SchurterCircuitBreaker 3a, Q13 SchurterCircuitBreaker 3a, Q14 SchurterCircuitBreaker 3a, Q15 SchurterCircuitBreaker 3a, Q16 SchurterCircuitBreaker 3a, Q17 SchurterCircuitBreaker 6a, Q18 SchurterCircuitBreaker 6a, Q19 SchurterCircuitBreaker 6a, Q2 SchurterCircuitBreaker 3a, Q20 SchurterCircuitBreaker 6a, Q21 SchurterCircuitBreaker 10a, Q22 SchurterCircuitBreaker 10a, Q23 SchurterCircuitBreaker 16a, Q24 SchurterCircuitBreaker 16a, Q25 SchurterCircuitBreaker 6a, Q26 SchurterCircuitBreaker 6a, Q27 SchurterCircuitBreaker 6a, Q28 SchurterCircuitBreaker 6a, Q29 SchurterCircuitBreaker 10a, Q3 SchurterCircuitBreaker 3a, Q30 SchurterCircuitBreaker 10a, Q31 SchurterCircuitBreaker 16a, Q32 SchurterCircuitBreaker 16a, Q33 SchurterCircuitBreaker 3a, Q4 SchurterCircuitBreaker 3a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

Commit message: Power Routing done on a set
Parts:
- C4: value Illinois Capacitor -> Illinois Capacitor 227AVG050MGBJ
- J5: value TB007-508-16BE -> TBP01R2W-508-16BE
- moved J3 192.1 mm to (431.5, 227.7)
- moved U15 124.7 mm to (249.6, 115.6), turned to 90 degrees
- moved J1 98.3 mm to (338.7, 90.9)
- moved U14 64.1 mm to (156.7, 115.6), turned to 90 degrees
- moved J9 17.0 mm to (45.0, 92.5)
- moved RN9 10.7 mm to (163.7, 123.3)
- moved U13 10.1 mm to (221.6, 115.7)
- moved RN5 7.92 mm to (256.2, 123.2)
Connections:
- D28 pad 1: /D12A -> /D28A
- J1 pad 2_1: Net-(J1-Pad2_1) -> Net-(J1-Pad1_1)
- J1 pad 2_2: Net-(J1-Pad2_1) -> Net-(J1-Pad1_1)
- J1 pad 2_3: Net-(J1-Pad2_1) -> Net-(J1-Pad1_1)
- J3 pad A_3: Net-(J3-PadA_3) -> Net-(J3-PadA_1)
- RN9 pad 14: (no net) -> /D28A
- U13 pad 1: (no net) -> Net-(U13-Pad1)
- U13 pad 2: (no net) -> Net-(J1-Pad1_1)
- U13 pad 21: (no net) -> Net-(U13-Pad21)
- U13 pad 22: (no net) -> Net-(U13-Pad22)
- U13 pad 23: (no net) -> Net-(U13-Pad23)
- U13 pad 24: (no net) -> Net-(U13-Pad24)
- U13 pad 25: (no net) -> Net-(U13-Pad25)
- U13 pad 26: (no net) -> Net-(U13-Pad26)
- U13 pad 27: (no net) -> Net-(U13-Pad27)
- U13 pad 28: (no net) -> Net-(U13-Pad28)
- U13 pad 3: (no net) -> Net-(U13-Pad3)
- U13 pad 4: (no net) -> Net-(U13-Pad4)
- U13 pad 5: (no net) -> Net-(U13-Pad5)
- U13 pad 6: (no net) -> Net-(U13-Pad6)
- U13 pad 7: (no net) -> Net-(U13-Pad7)
- U13 pad 8: (no net) -> Net-(U13-Pad8)
- U14 pad 1: (no net) -> Net-(U13-Pad28)
- U14 pad 11: Net-(SW32A1-Pad1) -> Net-(SW26A1-Pad1)
- U14 pad 12: Net-(SW32B1-Pad1) -> Net-(SW26B1-Pad1)
- U14 pad 13: Net-(SW30A1-Pad1) -> Net-(SW28A1-Pad1)
- U14 pad 14: Net-(SW30B1-Pad1) -> Net-(SW28B1-Pad1)
- U14 pad 15: Net-(SW28A1-Pad1) -> Net-(SW30A1-Pad1)
- U14 pad 16: Net-(SW28B1-Pad1) -> Net-(SW30B1-Pad1)
- U14 pad 17: Net-(SW26A1-Pad1) -> Net-(SW32A1-Pad1)
- U14 pad 18: Net-(SW26B1-Pad1) -> Net-(SW32B1-Pad1)
- U14 pad 2: (no net) -> Net-(U13-Pad27)
- U14 pad 3: (no net) -> Net-(U13-Pad26)
- U14 pad 4: (no net) -> Net-(U13-Pad25)
- U14 pad 5: (no net) -> Net-(U13-Pad24)
- U14 pad 6: (no net) -> Net-(U13-Pad23)
- U14 pad 7: (no net) -> Net-(U13-Pad22)
- U14 pad 8: (no net) -> Net-(U13-Pad21)
- U15 pad 1: (no net) -> Net-(U13-Pad1)
- U15 pad 11: Net-(SW24A1-Pad1) -> Net-(SW18A1-Pad1)
- U15 pad 12: Net-(SW24B1-Pad1) -> Net-(SW18B1-Pad1)
- U15 pad 13: Net-(SW22A1-Pad1) -> Net-(SW20A1-Pad1)
- U15 pad 14: Net-(SW22B1-Pad1) -> Net-(SW20B1-Pad1)
- U15 pad 15: Net-(SW20A1-Pad1) -> Net-(SW22A1-Pad1)
- U15 pad 16: Net-(SW20B1-Pad1) -> Net-(SW22B1-Pad1)
- U15 pad 17: Net-(SW18A1-Pad1) -> Net-(SW24A1-Pad1)
- U15 pad 18: Net-(SW18B1-Pad1) -> Net-(SW24B1-Pad1)
- U15 pad 2: (no net) -> Net-(J1-Pad1_1)
- U15 pad 3: (no net) -> Net-(U13-Pad3)
- U15 pad 4: (no net) -> Net-(U13-Pad4)
- U15 pad 5: (no net) -> Net-(U13-Pad5)
- U15 pad 6: (no net) -> Net-(U13-Pad6)
- U15 pad 7: (no net) -> Net-(U13-Pad7)
- U15 pad 8: (no net) -> Net-(U13-Pad8)
- U16 pad 1: (no net) -> Net-(U16-Pad1)
- U16 pad 2: (no net) -> Net-(U16-Pad2)
- U16 pad 21: (no net) -> Net-(U16-Pad21)
- U16 pad 22: (no net) -> Net-(U16-Pad22)
- U16 pad 23: (no net) -> Net-(U16-Pad23)
- U16 pad 24: (no net) -> Net-(U16-Pad24)
- U16 pad 25: (no net) -> Net-(U16-Pad25)
- U16 pad 26: (no net) -> Net-(U16-Pad26)
- U16 pad 27: (no net) -> Net-(U16-Pad27)
- U16 pad 28: (no net) -> Net-(U16-Pad28)
- U16 pad 3: (no net) -> Net-(U16-Pad3)
- U16 pad 4: (no net) -> Net-(U16-Pad4)
- U16 pad 5: (no net) -> Net-(U16-Pad5)
- U16 pad 6: (no net) -> Net-(U16-Pad6)
- U16 pad 7: (no net) -> Net-(U16-Pad7)
- U16 pad 8: (no net) -> Net-(U16-Pad8)
- U17 pad 1: (no net) -> Net-(U16-Pad28)
- U17 pad 2: (no net) -> Net-(U16-Pad27)
- U17 pad 3: (no net) -> Net-(U16-Pad26)
- U17 pad 4: (no net) -> Net-(U16-Pad25)
- U17 pad 5: (no net) -> Net-(U16-Pad24)
- U17 pad 6: (no net) -> Net-(U16-Pad23)
- U17 pad 7: (no net) -> Net-(U16-Pad22)
- U17 pad 8: (no net) -> Net-(U16-Pad21)
- U18 pad 1: (no net) -> Net-(U16-Pad8)
- U18 pad 2: (no net) -> Net-(U16-Pad7)
- U18 pad 3: (no net) -> Net-(U16-Pad6)
- U18 pad 4: (no net) -> Net-(U16-Pad5)
- U18 pad 5: (no net) -> Net-(U16-Pad4)
- U18 pad 6: (no net) -> Net-(U16-Pad3)
- U18 pad 7: (no net) -> Net-(U16-Pad2)
- U18 pad 8: (no net) -> Net-(U16-Pad1)
Routing:
- net (no net): track 785.3 -> 0.00 mm
- net Net-(K26-Pad3): track 0.00 -> 335.6 mm
- net Net-(K24-Pad3): track 0.00 -> 330.6 mm
- net Net-(J9-Pad1_1): track 0.00 -> 274.0 mm
- net Net-(K25-Pad3): track 0.00 -> 266.4 mm
- net Net-(J1-Pad1_1): track 0.00 -> 264.1 mm, vias 0 -> 1
- net Net-(K23-Pad3): track 0.00 -> 255.4 mm, vias 0 -> 1
- net Net-(K28-Pad3): track 0.00 -> 249.1 mm
- net Net-(K22-Pad3): track 0.00 -> 247.4 mm
- net Net-(K21-Pad3): track 0.00 -> 196.6 mm, vias 0 -> 1
- net Net-(K27-Pad3): track 0.00 -> 195.1 mm, vias 0 -> 1
- net Net-(K20-Pad3): track 0.00 -> 165.1 mm
- net Net-(K30-Pad3): track 0.00 -> 162.7 mm
- net Net-(K29-Pad3): track 0.00 -> 155.0 mm
- net Net-(K19-Pad3): track 0.00 -> 135.5 mm, vias 0 -> 1
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Other:
- net class Up to 16A 230V: via_dia 1 -> 8; via_drill 0.6 -> 6
- net class Up to 60A 12-230V AC\DC: via_dia 6 -> 9; via_drill 4 -> 7
- net class Up to16A 12V: via_dia 1 -> 8; via_drill 0.6 -> 6

Commit message: Let's sort out the switches
Parts:
- moved J3 72.5 mm to (474.8, 169.6)
Connections:
- J1 pad 2_1: Net-(J1-Pad1_1) -> Net-(J1-Pad2_1)
- J1 pad 2_2: Net-(J1-Pad1_1) -> Net-(J1-Pad2_1)
- J1 pad 2_3: Net-(J1-Pad1_1) -> Net-(J1-Pad2_1)
- K31 pad 8: /K32B -> /K31B
- RN10 pad 8: (no net) -> /K31B
- SW31B1 pad 2: /K32B -> /K31B
- SW31B1 pad 5: /K32B -> /K31B
- U13 pad 2: Net-(J1-Pad1_1) -> Net-(U13-Pad2)
- U15 pad 2: Net-(J1-Pad1_1) -> Net-(U13-Pad2)
Routing:
- net /K31B: track 0.00 -> 76.5 mm
- net Net-(SW17B1-Pad6): track 0.00 -> 47.9 mm
- net Net-(J9-Pad1_1): track 274.0 -> 316.0 mm
- net Net-(D17-Pad2): track 577.8 -> 608.6 mm
- net /K29A: track 68.1 -> 94.3 mm
- net Net-(J1-Pad1_1): track 264.1 -> 286.5 mm
- net /K32B: track 122.4 -> 104.0 mm
- net Net-(J9-Pad2_1): track 0.00 -> 5.00 mm
- net Net-(J1-Pad2_1): track 0.00 -> 5.00 mm
- net Net-(SW29A1-Pad1): track 38.0 -> 37.3 mm

Commit message: Wired
Parts:
- moved J3 71.9 mm to (441.7, 105.8)
- moved SW17B1 12.6 mm to (325.0, 62.9)
- moved SW19B1 12.0 mm to (293.9, 62.9)
- moved SW21B1 11.9 mm to (263.4, 62.9)
- moved SW21A1 11.1 mm to (251.8, 62.9)
- moved SW19A1 10.8 mm to (282.6, 62.9)
- moved SW17A1 10.7 mm to (313.2, 62.9)
- moved D23 5.09 mm to (208.9, 62.9), turned to 0 degrees
- moved SW23B1 1.30 mm to (232.4, 62.9)
- moved SW23A1 1.30 mm to (221.0, 62.9)
- moved D21 0.76 mm to (244.6, 62.9)
- moved D17 0.60 mm to (306.0, 62.9)
- moved D19 0.60 mm to (275.6, 62.9)
Connections:
- SW17B1 pad 6: Net-(SW17B1-Pad6) -> Net-(SW17A1-Pad6)
- SW18B1 pad 6: Net-(SW17B1-Pad6) -> Net-(SW17A1-Pad6)
- SW19B1 pad 6: Net-(SW17B1-Pad6) -> Net-(SW17A1-Pad6)
- SW20B1 pad 6: Net-(SW17B1-Pad6) -> Net-(SW17A1-Pad6)
- SW21B1 pad 6: Net-(SW17B1-Pad6) -> Net-(SW17A1-Pad6)
- SW22B1 pad 6: Net-(SW17B1-Pad6) -> Net-(SW17A1-Pad6)
- SW23B1 pad 6: Net-(SW17B1-Pad6) -> Net-(SW17A1-Pad6)
- SW24B1 pad 6: Net-(SW17B1-Pad6) -> Net-(SW17A1-Pad6)
- SW25B1 pad 6: Net-(SW17B1-Pad6) -> Net-(SW17A1-Pad6)
- SW26B1 pad 6: Net-(SW17B1-Pad6) -> Net-(SW17A1-Pad6)
- SW27B1 pad 6: Net-(SW17B1-Pad6) -> Net-(SW17A1-Pad6)
- SW28B1 pad 6: Net-(SW17B1-Pad6) -> Net-(SW17A1-Pad6)
- SW29B1 pad 6: Net-(SW17B1-Pad6) -> Net-(SW17A1-Pad6)
- SW30B1 pad 6: Net-(SW17B1-Pad6) -> Net-(SW17A1-Pad6)
- SW31B1 pad 6: Net-(SW17B1-Pad6) -> Net-(SW17A1-Pad6)
- SW32B1 pad 6: Net-(SW17B1-Pad6) -> Net-(SW17A1-Pad6)
- U17 pad 13: Net-(SW21B1-Pad1) -> Net-(SW21A1-Pad1)
- U17 pad 14: Net-(SW21A1-Pad1) -> Net-(SW21B1-Pad1)
- U17 pad 15: Net-(SW19B1-Pad1) -> Net-(SW19A1-Pad1)
- U17 pad 16: Net-(SW19A1-Pad1) -> Net-(SW19B1-Pad1)
- U17 pad 17: Net-(SW17B1-Pad1) -> Net-(SW17A1-Pad1)
- U17 pad 18: Net-(SW17A1-Pad1) -> Net-(SW17B1-Pad1)
Routing:
- net Net-(SW17A1-Pad6): track 257.8 -> 669.0 mm
- net Net-(SW17B1-Pad6): track 47.9 -> 0.00 mm
- net /K23B: track 92.9 -> 51.6 mm
- net /K18B: track 17.3 -> 45.6 mm
- net /K17B: track 54.0 -> 80.4 mm
- net Net-(D17-Pad2): track 608.6 -> 634.7 mm
- net /K21A: track 26.1 -> 52.2 mm
- net /K19B: track 33.4 -> 57.6 mm
- net /K21B: track 52.8 -> 71.2 mm
- net Net-(SW23A1-Pad1): track 18.2 -> 32.3 mm
- net Net-(J9-Pad1_1): track 316.0 -> 303.3 mm
- net Net-(SW25A1-Pad1): track 54.4 -> 67.0 mm, vias 1 -> 0
- net Net-(SW19B1-Pad1): track 53.7 -> 62.4 mm
- net Net-(SW21B1-Pad1): track 28.3 -> 37.0 mm
- net Net-(SW27A1-Pad1): track 32.7 -> 41.2 mm
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
Commit message: cleanup
Parts:
- moved J3 38.0 mm to (425.0, 71.7)
Connections:
- J2 pad A_3: /A3 -> (no net)
- J6 pad 4: Net-(J6-Pad4) -> (no net)
- J6 pad 5: Net-(J6-Pad4) -> (no net)
- U3 pad 13: /A3 -> (no net)

Commit message: Big Power in place
Parts:
- moved U4 172.6 mm to (-110.0, 94.2)
- moved J2 172.6 mm to (-48.4, 132.3)
- moved U1 172.6 mm to (-122.7, 129.2)
- moved U2 172.6 mm to (-82.1, 141.2)
- moved U3 172.6 mm to (-85.9, 162.2)
- moved U5 172.6 mm to (-81.5, 113.9)
- moved U6 172.6 mm to (-83.4, 75.8)
- moved U8 152.2 mm to (249.2, 197.8), turned to 90 degrees
- moved J6 112.1 mm to (21.5, 5.80), turned to 270 degrees
- moved U12 108.1 mm to (136.1, 136.5)
- moved J3 91.1 mm to (472.6, 149.4)
- moved U10 88.2 mm to (221.4, 128.9)
- moved RN8 73.2 mm to (163.3, 205.6)
- moved U7 73.1 mm to (221.4, 197.8)
- moved RN4 72.4 mm to (255.9, 205.2)
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Connections:
- D10 pad 3: /D10B -> (no net)
- D12 pad 1: /D12A -> (no net)
- J2 pad A_3: (no net) -> /A3
- J4 pad 1: (no net) -> Net-(J4-Pad1)
- J4 pad 2: (no net) -> Net-(J4-Pad2)
- J4 pad 3: (no net) -> Net-(J4-Pad3)
- J4 pad 4: (no net) -> Net-(J4-Pad4)
- J4 pad 5: (no net) -> Net-(J4-Pad5)
- J4 pad 6: (no net) -> Net-(J4-Pad6)
- J4 pad 7: (no net) -> Net-(J4-Pad7)
- J4 pad 8: (no net) -> Net-(J4-Pad8)
- J6 pad 1: (no net) -> Net-(J6-Pad1)
- J6 pad 2: (no net) -> Net-(J6-Pad2)
- J6 pad 3: (no net) -> Net-(J6-Pad3)
- J6 pad 4: (no net) -> Net-(J6-Pad4)
- J6 pad 5: (no net) -> Net-(J6-Pad5)
- J6 pad 6: (no net) -> Net-(J6-Pad6)
- J6 pad 7: (no net) -> Net-(J6-Pad7)
- J6 pad 8: (no net) -> Net-(J6-Pad8)
- K2 pad 1: /K2A -> /K18A
- K2 pad 8: /K2B -> /K18B
- Q10 pad P1: Net-(K10-Pad3) -> Net-(J5-Pad10)
- Q10 pad P2: Net-(J5-Pad10) -> Net-(K10-Pad3)
- Q11 pad P1: Net-(K11-Pad3) -> Net-(J5-Pad11)
- Q11 pad P2: Net-(J5-Pad11) -> Net-(K11-Pad3)
- Q12 pad P1: Net-(K12-Pad3) -> Net-(J5-Pad12)
- Q12 pad P2: Net-(J5-Pad12) -> Net-(K12-Pad3)
- Q13 pad P1: Net-(K13-Pad3) -> Net-(J5-Pad13)
- Q13 pad P2: Net-(J5-Pad13) -> Net-(K13-Pad3)
- Q14 pad P1: Net-(K14-Pad3) -> Net-(J5-Pad14)
- Q14 pad P2: Net-(J5-Pad14) -> Net-(K14-Pad3)
- Q15 pad P1: Net-(K15-Pad3) -> Net-(J5-Pad15)
- Q15 pad P2: Net-(J5-Pad15) -> Net-(K15-Pad3)
- Q16 pad P1: Net-(K16-Pad3) -> Net-(J5-Pad16)
- Q16 pad P2: Net-(J5-Pad16) -> Net-(K16-Pad3)
- Q17 pad P1: (no net) -> Net-(J4-Pad1)
- Q18 pad P1: (no net) -> Net-(J4-Pad2)
- Q19 pad P1: (no net) -> Net-(J4-Pad3)
- Q20 pad P1: (no net) -> Net-(J4-Pad4)
- Q21 pad P1: (no net) -> Net-(J4-Pad5)
- Q22 pad P1: (no net) -> Net-(J4-Pad6)
- Q23 pad P1: (no net) -> Net-(J4-Pad7)
- Q24 pad P1: (no net) -> Net-(J4-Pad8)
- Q25 pad P1: (no net) -> Net-(J6-Pad1)
- Q26 pad P1: (no net) -> Net-(J6-Pad2)
- Q27 pad P1: (no net) -> Net-(J6-Pad3)
- Q28 pad P1: (no net) -> Net-(J6-Pad4)
- Q29 pad P1: (no net) -> Net-(J6-Pad5)
- Q30 pad P1: (no net) -> Net-(J6-Pad6)
- Q31 pad P1: (no net) -> Net-(J6-Pad7)
- Q32 pad P1: (no net) -> Net-(J6-Pad8)
- Q9 pad P1: Net-(K9-Pad3) -> Net-(J5-Pad9)
- Q9 pad P2: Net-(J5-Pad9) -> Net-(K9-Pad3)
- RN3 pad 1: /K2A -> /K1A
- RN3 pad 10: /D8A -> /D7A
- RN3 pad 11: /D6B -> /D5B
- RN3 pad 12: /D6A -> /D5A
- RN3 pad 13: /D4B -> /D3B
- RN3 pad 14: /D4A -> /D3A
- RN3 pad 15: /D2B -> /D1B
- RN3 pad 16: /D2A -> /D1A
- RN3 pad 2: /K2B -> /K1B
- RN3 pad 3: /K4A -> /K3A
- RN3 pad 4: /K4B -> /K3B
- RN3 pad 5: /K6A -> /K5A
- RN3 pad 6: /K6B -> /K5B
- RN3 pad 7: /K8A -> /K7A
- RN3 pad 8: /K8B -> /K7B
- RN3 pad 9: /D8B -> /D7B
- RN4 pad 1: /K1A -> /K2A
- RN4 pad 10: /D7A -> /D8A
- RN4 pad 11: /D5B -> /D6B
- RN4 pad 12: /D5A -> /D6A
- RN4 pad 13: /D3B -> /D4B
- RN4 pad 14: /D3A -> /D4A
- RN4 pad 15: /D1B -> /D2B
- RN4 pad 16: /D1A -> /D2A
- RN4 pad 2: /K1B -> /K2B
- RN4 pad 3: /K3A -> /K4A
- RN4 pad 4: /K3B -> /K4B
- RN4 pad 5: /K5A -> /K6A
- RN4 pad 6: /K5B -> /K6B
- RN4 pad 7: /K7A -> /K8A
- RN4 pad 8: /K7B -> /K8B
- RN4 pad 9: /D7B -> /D8B
- RN7 pad 1: /K10A -> /K9A
- RN7 pad 10: /D16A -> /D15A
- RN7 pad 11: /D14B -> /D13B
- RN7 pad 12: /D14A -> /D13A
- RN7 pad 13: /D12B -> /D11B
- RN7 pad 14: /D12A -> /D11A
- RN7 pad 15: /D10B -> /D9B
- RN7 pad 16: /D10A -> /D9A
- RN7 pad 2: /K10B -> /K9B
- RN7 pad 3: /K12A -> /K11A
- RN7 pad 4: /K12B -> /K11B
- RN7 pad 5: /K14A -> /K13A
- RN7 pad 6: /K14B -> /K13B
- RN7 pad 7: /K16A -> /K15A
- RN7 pad 8: /K16B -> /K15B
- RN7 pad 9: /D16B -> /D15B
- RN8 pad 1: /K9A -> /K10A
- RN8 pad 10: /D15A -> /D18A
- RN8 pad 11: /D13B -> /D16B
- RN8 pad 12: /D13A -> /D16A
- RN8 pad 13: /D11B -> /D14B
- RN8 pad 14: /D11A -> /D14A
- RN8 pad 15: /D9B -> /D12B
- RN8 pad 16: /D9A -> /D10A
- RN8 pad 2: /K9B -> /K10B
- RN8 pad 3: /K11A -> /K12A
- RN8 pad 4: /K11B -> /K12B
- RN8 pad 5: /K13A -> /K14A
- RN8 pad 6: /K13B -> /K14B
- RN8 pad 7: /K15A -> /K16A
- RN8 pad 8: /K15B -> /K16B
- RN8 pad 9: /D15B -> /D18B
- SW10A1 pad 2: /K10B -> /K10A
- SW10A1 pad 5: /K10B -> /K10A
- SW10A1 pad 6: Net-(J5-Pad9) -> Net-(SW10A1-Pad6)
- SW10B1 pad 2: /K10A -> /K10B
- SW10B1 pad 5: /K10A -> /K10B
- SW10B1 pad 6: (no net) -> Net-(SW10A1-Pad6)
- SW11A1 pad 2: /K11B -> /K11A
- SW11A1 pad 5: /K11B -> /K11A
- SW11A1 pad 6: Net-(J5-Pad9) -> Net-(SW10A1-Pad6)
- SW11B1 pad 2: /K11A -> /K11B
- SW11B1 pad 5: /K11A -> /K11B
- SW11B1 pad 6: (no net) -> Net-(SW10A1-Pad6)
- SW12A1 pad 2: /K12B -> /K12A
- SW12A1 pad 5: /K12B -> /K12A
- SW12A1 pad 6: Net-(J5-Pad9) -> Net-(SW10A1-Pad6)
- SW12B1 pad 2: /K12A -> /K12B
- SW12B1 pad 5: /K12A -> /K12B
- SW12B1 pad 6: (no net) -> Net-(SW10A1-Pad6)
- SW13A1 pad 2: /K13B -> /K13A
- SW13A1 pad 5: /K13B -> /K13A
- SW13A1 pad 6: Net-(J5-Pad9) -> Net-(SW10A1-Pad6)
- SW13B1 pad 2: /K13A -> /K13B
- SW13B1 pad 5: /K13A -> /K13B
- SW13B1 pad 6: (no net) -> Net-(SW10A1-Pad6)
- SW14A1 pad 2: /K14B -> /K14A
- SW14A1 pad 5: /K14B -> /K14A
- SW14A1 pad 6: Net-(J5-Pad9) -> Net-(SW10A1-Pad6)
- SW14B1 pad 2: /K14A -> /K14B
- SW14B1 pad 5: /K14A -> /K14B
- SW14B1 pad 6: (no net) -> Net-(SW10A1-Pad6)
- SW15A1 pad 2: /K15B -> /K15A
- SW15A1 pad 5: /K15B -> /K15A
- SW15A1 pad 6: Net-(J5-Pad9) -> Net-(SW10A1-Pad6)
- SW15B1 pad 2: /K15A -> /K15B
- SW15B1 pad 5: /K15A -> /K15B
- SW15B1 pad 6: (no net) -> Net-(SW10A1-Pad6)
- SW16A1 pad 2: /K16B -> /K16A
- SW16A1 pad 5: /K16B -> /K16A
- SW16A1 pad 6: Net-(J5-Pad9) -> Net-(SW10A1-Pad6)
- SW16B1 pad 2: /K16A -> /K16B
- SW16B1 pad 5: /K16A -> /K16B
- SW16B1 pad 6: (no net) -> Net-(SW10A1-Pad6)
- SW1A1 pad 2: /K1B -> /K1A
- SW1A1 pad 5: /K1B -> /K1A
- SW1A1 pad 6: Net-(J5-Pad9) -> Net-(SW10A1-Pad6)
- SW1B1 pad 2: /K1A -> /K1B
- SW1B1 pad 5: /K1A -> /K1B
- SW1B1 pad 6: (no net) -> Net-(SW10A1-Pad6)
- SW2A1 pad 2: /K2B -> /K18A
- SW2A1 pad 5: /K2B -> /K18A
- SW2A1 pad 6: Net-(J5-Pad9) -> Net-(SW10A1-Pad6)
- SW2B1 pad 2: /K2A -> /K18B
- SW2B1 pad 5: /K2A -> /K18B
- SW2B1 pad 6: (no net) -> Net-(SW10A1-Pad6)
- SW3A1 pad 2: /K3B -> /K3A
- SW3A1 pad 5: /K3B -> /K3A
- SW3A1 pad 6: Net-(J5-Pad9) -> Net-(SW10A1-Pad6)
- SW3B1 pad 2: /K3A -> /K3B
- SW3B1 pad 5: /K3A -> /K3B
- SW3B1 pad 6: (no net) -> Net-(SW10A1-Pad6)
- SW4A1 pad 2: /K4B -> /K4A
- SW4A1 pad 5: /K4B -> /K4A
- SW4A1 pad 6: Net-(J5-Pad9) -> Net-(SW10A1-Pad6)
- SW4B1 pad 2: /K4A -> /K4B
- SW4B1 pad 5: /K4A -> /K4B
- SW4B1 pad 6: (no net) -> Net-(SW10A1-Pad6)
- SW5A1 pad 2: /K5B -> /K5A
- SW5A1 pad 5: /K5B -> /K5A
- SW5A1 pad 6: Net-(J5-Pad9) -> Net-(SW10A1-Pad6)
- SW5B1 pad 2: /K5A -> /K5B
- SW5B1 pad 5: /K5A -> /K5B
- SW5B1 pad 6: (no net) -> Net-(SW10A1-Pad6)
- SW6A1 pad 2: /K6B -> /K6A
- SW6A1 pad 5: /K6B -> /K6A
- SW6A1 pad 6: Net-(J5-Pad9) -> Net-(SW10A1-Pad6)
- SW6B1 pad 2: /K6A -> /K6B
- SW6B1 pad 5: /K6A -> /K6B
- SW6B1 pad 6: (no net) -> Net-(SW10A1-Pad6)
- SW7A1 pad 2: /K7B -> /K7A
- SW7A1 pad 5: /K7B -> /K7A
- SW7A1 pad 6: Net-(J5-Pad9) -> Net-(SW10A1-Pad6)
- SW7B1 pad 2: /K7A -> /K7B
- SW7B1 pad 5: /K7A -> /K7B
- SW7B1 pad 6: (no net) -> Net-(SW10A1-Pad6)
- SW8A1 pad 2: /K8B -> /K8A
- SW8A1 pad 5: /K8B -> /K8A
- SW8A1 pad 6: Net-(J5-Pad9) -> Net-(SW10A1-Pad6)
- SW8B1 pad 2: /K8A -> /K8B
- SW8B1 pad 5: /K8A -> /K8B
- SW8B1 pad 6: (no net) -> Net-(SW10A1-Pad6)
- SW9A1 pad 2: /K9B -> /K9A
- SW9A1 pad 5: /K9B -> /K9A
- SW9A1 pad 6: Net-(J5-Pad9) -> Net-(SW10A1-Pad6)
- SW9B1 pad 2: /K9A -> /K9B
- SW9B1 pad 5: /K9A -> /K9B
- SW9B1 pad 6: (no net) -> Net-(SW10A1-Pad6)
- U11 pad 1: Net-(U11-Pad1) -> Net-(U10-Pad28)
- U11 pad 11: Net-(SW15B1-Pad1) -> Net-(SW7A1-Pad1)
- U11 pad 12: Net-(SW13B1-Pad1) -> Net-(SW7B1-Pad1)
- U11 pad 13: Net-(SW11B1-Pad1) -> Net-(SW5A1-Pad1)
- U11 pad 14: Net-(SW9B1-Pad1) -> Net-(SW5B1-Pad1)
- U11 pad 15: Net-(SW7B1-Pad1) -> Net-(SW3A1-Pad1)
- U11 pad 16: Net-(SW5B1-Pad1) -> Net-(SW3B1-Pad1)
- U11 pad 17: Net-(SW3B1-Pad1) -> Net-(SW1A1-Pad1)
- U11 pad 2: Net-(U11-Pad2) -> Net-(U10-Pad27)
- U11 pad 3: Net-(U11-Pad3) -> Net-(U10-Pad26)
- U11 pad 4: Net-(U11-Pad4) -> Net-(U10-Pad25)
- U11 pad 5: Net-(U11-Pad5) -> Net-(U10-Pad24)
- U11 pad 6: Net-(U11-Pad6) -> Net-(U10-Pad23)
- U11 pad 7: Net-(U11-Pad7) -> Net-(U10-Pad22)
- U11 pad 8: Net-(U11-Pad8) -> Net-(U10-Pad21)
- U12 pad 1: Net-(U10-Pad28) -> Net-(U10-Pad8)
- U12 pad 11: Net-(SW16B1-Pad1) -> Net-(SW15A1-Pad1)
- U12 pad 12: Net-(SW14B1-Pad1) -> Net-(SW15B1-Pad1)
- U12 pad 13: Net-(SW12B1-Pad1) -> Net-(SW13A1-Pad1)
- U12 pad 14: Net-(SW10B1-Pad1) -> Net-(SW13B1-Pad1)
- U12 pad 15: Net-(SW8B1-Pad1) -> Net-(SW11A1-Pad1)
- U12 pad 16: Net-(SW6B1-Pad1) -> Net-(SW11B1-Pad1)
- U12 pad 17: Net-(SW4B1-Pad1) -> Net-(SW9A1-Pad1)
- U12 pad 18: Net-(SW2B1-Pad1) -> Net-(SW9B1-Pad1)
- U12 pad 2: Net-(U10-Pad27) -> Net-(U10-Pad7)
- U12 pad 3: Net-(U10-Pad26) -> Net-(U10-Pad6)
- U12 pad 4: Net-(U10-Pad25) -> Net-(U10-Pad5)
- U12 pad 5: Net-(U10-Pad24) -> Net-(U10-Pad4)
- U12 pad 6: Net-(U10-Pad23) -> Net-(U10-Pad3)
- U12 pad 7: Net-(U10-Pad22) -> Net-(U10-Pad2)
- U12 pad 8: Net-(U10-Pad21) -> Net-(U10-Pad1)
- U3 pad 13: (no net) -> /A3
- U7 pad 1: Net-(U11-Pad8) -> Net-(U7-Pad1)
- U7 pad 2: Net-(U11-Pad7) -> Net-(U7-Pad2)
- U7 pad 28: Net-(U7-Pad28) -> (no net)
- U7 pad 3: Net-(U11-Pad6) -> Net-(U7-Pad3)
- U7 pad 4: Net-(U11-Pad5) -> Net-(U7-Pad4)
- U7 pad 5: Net-(U11-Pad4) -> Net-(U7-Pad5)
- U7 pad 6: Net-(U11-Pad3) -> Net-(U7-Pad6)
- U7 pad 7: Net-(U11-Pad2) -> Net-(U7-Pad7)
- U7 pad 8: Net-(U11-Pad1) -> Net-(U7-Pad8)
- U8 pad 1: Net-(U7-Pad21) -> Net-(U7-Pad1)
- U8 pad 11: Net-(SW15A1-Pad1) -> Net-(SW2A1-Pad1)
- U8 pad 12: Net-(SW13A1-Pad1) -> Net-(SW2B1-Pad1)
- U8 pad 13: Net-(SW11A1-Pad1) -> Net-(SW4A1-Pad1)
- U8 pad 14: Net-(SW9A1-Pad1) -> Net-(SW4B1-Pad1)
- U8 pad 15: Net-(SW7A1-Pad1) -> Net-(SW6A1-Pad1)
- U8 pad 16: Net-(SW5A1-Pad1) -> Net-(SW6B1-Pad1)
- U8 pad 17: Net-(SW3A1-Pad1) -> Net-(SW8A1-Pad1)
- U8 pad 18: Net-(SW1A1-Pad1) -> Net-(SW8B1-Pad1)
- U8 pad 2: Net-(U7-Pad22) -> Net-(U7-Pad2)
- U8 pad 3: Net-(U7-Pad23) -> Net-(U7-Pad3)
- U8 pad 4: Net-(U7-Pad24) -> Net-(U7-Pad4)
- U8 pad 5: Net-(U7-Pad25) -> Net-(U7-Pad5)
- U8 pad 6: Net-(U7-Pad26) -> Net-(U7-Pad6)
- U8 pad 7: Net-(U7-Pad27) -> Net-(U7-Pad7)
- U8 pad 8: Net-(U7-Pad28) -> Net-(U7-Pad8)
- U9 pad 1: Net-(U10-Pad1) -> (no net)
- U9 pad 11: Net-(SW16A1-Pad1) -> Net-(SW10A1-Pad1)
- U9 pad 12: Net-(SW14A1-Pad1) -> Net-(SW10B1-Pad1)
- U9 pad 14: Net-(SW10A1-Pad1) -> Net-(SW12B1-Pad1)
- U9 pad 15: Net-(SW8A1-Pad1) -> Net-(SW14A1-Pad1)
- U9 pad 16: Net-(SW6A1-Pad1) -> Net-(SW14B1-Pad1)
- U9 pad 17: Net-(SW4A1-Pad1) -> Net-(SW16A1-Pad1)
- U9 pad 18: Net-(SW2A1-Pad1) -> Net-(SW16B1-Pad1)
- U9 pad 2: Net-(U10-Pad2) -> Net-(U7-Pad27)
- U9 pad 3: Net-(U10-Pad3) -> Net-(U7-Pad26)
- U9 pad 4: Net-(U10-Pad4) -> Net-(U7-Pad25)
- U9 pad 5: Net-(U10-Pad5) -> Net-(U7-Pad24)
- U9 pad 6: Net-(U10-Pad6) -> Net-(U7-Pad23)
- U9 pad 7: Net-(U10-Pad7) -> Net-(U7-Pad22)
- U9 pad 8: Net-(U10-Pad8) -> Net-(U7-Pad21)
Routing:
- net Net-(J8-Pad1_1): track 7.50 -> 548.8 mm
- net Net-(C2-Pad1): track 537.2 -> 0.00 mm
- net Net-(K12-Pad3): track 0.00 -> 395.7 mm
- net Net-(K6-Pad3): track 0.00 -> 359.2 mm
- net Net-(K10-Pad3): track 0.00 -> 351.4 mm
- net Net-(K9-Pad3): track 0.00 -> 309.2 mm
- net Net-(K8-Pad3): track 0.00 -> 298.7 mm
- net Net-(SW10A1-Pad6): track 0.00 -> 281.6 mm
- net Net-(K7-Pad3): track 0.00 -> 242.3 mm
- net Net-(K13-Pad3): track 0.00 -> 236.5 mm
- net Net-(K4-Pad3): track 0.00 -> 229.6 mm
- net Net-(K11-Pad3): track 0.00 -> 214.8 mm
- net Net-(K3-Pad3): track 0.00 -> 189.0 mm, vias 0 -> 1
- net Net-(J6-Pad1): track 0.00 -> 182.8 mm
- net Net-(K14-Pad3): track 0.00 -> 177.9 mm
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
Commit message: Wired and tidy
Parts:
- moved J2 549.1 mm to (490.5, 27.0)
- moved U1 549.1 mm to (416.2, 23.9)
- moved U2 549.1 mm to (456.8, 35.9)
- moved U3 549.1 mm to (453.0, 56.9)
- moved U4 549.1 mm to (428.9, -11.1)
- moved U5 549.1 mm to (457.4, 8.62)
- moved U6 549.1 mm to (455.5, -29.5)
- moved J3 454.1 mm to (20.8, 103.7), turned to 270 degrees
- moved RN8 0.22 mm to (163.4, 205.4)
- moved U9 0.10 mm to (156.3, 197.7)
Connections:
- D10 pad 3: (no net) -> /D10B
- D12 pad 1: (no net) -> /D12A
- K2 pad 1: /K18A -> /K2A
- K2 pad 8: /K18B -> /K2B
- RN8 pad 10: /D18A -> /D16A
- RN8 pad 11: /D16B -> /D14B
- RN8 pad 12: /D16A -> /D14A
- RN8 pad 13: /D14B -> /D12B
- RN8 pad 14: /D14A -> /D12A
- RN8 pad 15: /D12B -> /D10B
- RN8 pad 9: /D18B -> /D16B
- SW2A1 pad 2: /K18A -> /K2A
- SW2A1 pad 5: /K18A -> /K2A
- SW2B1 pad 2: /K18B -> /K2B
- SW2B1 pad 5: /K18B -> /K2B
Routing:
- net /K16B: track 17.3 -> 149.7 mm
- net /D16B: track 0.00 -> 101.4 mm
- net /K16A: track 17.3 -> 106.8 mm
- net Net-(SW4A1-Pad1): track 7.00 -> 95.2 mm
- net /D4A: track 0.00 -> 86.7 mm
- net Net-(U7-Pad27): track 0.00 -> 83.6 mm
- net Net-(D1-Pad2): track 566.8 -> 649.3 mm
- net Net-(U7-Pad26): track 0.00 -> 78.1 mm
- net Net-(SW2B1-Pad1): track 21.7 -> 97.9 mm
- net Net-(U7-Pad25): track 0.00 -> 72.7 mm
- net Net-(SW10A1-Pad6): track 281.6 -> 350.6 mm
- net /K14A: track 17.3 -> 85.5 mm
- net /D16A: track 0.00 -> 67.7 mm
- net Net-(U7-Pad24): track 0.00 -> 67.2 mm
- net Net-(U7-Pad23): track 0.00 -> 61.8 mm
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
Commit message: Rewired and Cleanup
Parts:
- moved J3 346.1 mm to (361.0, 167.2), turned to 90 degrees
- moved J1 14.3 mm to (352.9, 89.6), turned to 90 degrees
- moved D3 5.25 mm to (269.4, 145.6), turned to 0 degrees
- moved D5 5.18 mm to (239.0, 145.6), turned to 0 degrees
- moved D1 5.14 mm to (300.0, 145.6), turned to 0 degrees
- moved D23 5.10 mm to (214.0, 62.8), turned to 180 degrees
- moved D7 5.10 mm to (208.6, 145.5), turned to 0 degrees
Routing:
- net Net-(SW10A1-Pad6): track 350.6 -> 703.1 mm
- net /K13A: track 90.7 -> 261.1 mm
- net /K13B: track 70.6 -> 184.7 mm
- net /K19B: track 57.6 -> 155.3 mm
- net /D4B: track 25.9 -> 108.2 mm
- net /K3B: track 57.2 -> 139.1 mm
- net Net-(SW1B1-Pad1): track 87.4 -> 13.8 mm
- net Net-(SW2A1-Pad1): track 58.4 -> 127.5 mm
- net /K19A: track 39.5 -> 106.5 mm
- net Net-(SW1A1-Pad1): track 78.5 -> 13.9 mm
- net /D13A: track 63.6 -> 127.9 mm
- net /K15A: track 98.6 -> 155.8 mm
- net /K3A: track 38.1 -> 92.5 mm
- net /D11A: track 38.3 -> 86.6 mm
- net Net-(SW3B1-Pad1): track 61.9 -> 13.8 mm
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