File: boatcontrol/boatcontrol.kicad_pcb (KiCad board)
At the start: 2 copper layers, 271 parts, among them J1 TBL008V-1000-02BE, J10 TBL008V-1000-08BE, J11 TBL008V-1000-02BE, J12 TBL008V-1000-08BE, J2 SS73100-047F, J3 SS73100-047F, J4 TBP01R2W-508-08BE, J5 TBP01R2W-508-16BE, J6 TBP01R2W-508-08BE, J7 RPi_GPIO, J8 TBL008V-1000-02BE, J9 TBL008V-1000-02BE, K1 G5RL-K1A-E-DC12, K10 G5RL-K1A-E-DC12, K11 G5RL-K1A-E-DC12, K12 G5RL-K1A-E-DC12, K13 G5RL-K1A-E-DC12, K14 G5RL-K1A-E-DC12, K15 G5RL-K1A-E-DC12, K16 G5RL-K1A-E-DC12, K17 G5RL-K1A-E-DC12, K18 G5RL-K1A-E-DC12, K19 G5RL-K1A-E-DC12, K2 G5RL-K1A-E-DC12, K20 G5RL-K1A-E-DC12, K21 G5RL-K1A-E-DC12, K22 G5RL-K1A-E-DC12, K23 G5RL-K1A-E-DC12, K24 G5RL-K1A-E-DC12, K25 G5RL-K1A-E-DC12, K26 G5RL-K1A-E-DC12, K27 G5RL-K1A-E-DC12, K28 G5RL-K1A-E-DC12, K29 G5RL-K1A-E-DC12, K3 G5RL-K1A-E-DC12, K30 G5RL-K1A-E-DC12, K31 G5RL-K1A-E-DC12, K32 G5RL-K1A-E-DC12, K33 EW60-1A3-CL12D04, K34 EW60-1A3-CL12D04, K35 EW60-1A3-CL12D04, K36 EW60-1A3-CL12D04, K37 EW60-1A3-CL12D04, K38 EW60-1A3-CL12D04, K39 EW60-1A3-CL12D04, K4 G5RL-K1A-E-DC12, K40 EW60-1A3-CL12D04, K5 G5RL-K1A-E-DC12, K6 G5RL-K1A-E-DC12, K7 G5RL-K1A-E-DC12, K8 G5RL-K1A-E-DC12, K9 G5RL-K1A-E-DC12, Q1 SchurterCircuitBreaker 3a, Q10 SchurterCircuitBreaker 3a, Q11 SchurterCircuitBreaker 3a, Q12 SchurterCircuitBreaker 3a, Q13 SchurterCircuitBreaker 3a, Q14 SchurterCircuitBreaker 3a, Q15 SchurterCircuitBreaker 3a, Q16 SchurterCircuitBreaker 3a, Q17 SchurterCircuitBreaker 6a, Q18 SchurterCircuitBreaker 6a, Q19 SchurterCircuitBreaker 6a, Q2 SchurterCircuitBreaker 3a, Q20 SchurterCircuitBreaker 6a, Q21 SchurterCircuitBreaker 10a, Q22 SchurterCircuitBreaker 10a, Q23 SchurterCircuitBreaker 16a, Q24 SchurterCircuitBreaker 16a, Q25 SchurterCircuitBreaker 6a, Q26 SchurterCircuitBreaker 6a, Q27 SchurterCircuitBreaker 6a, Q28 SchurterCircuitBreaker 6a, Q29 SchurterCircuitBreaker 10a, Q3 SchurterCircuitBreaker 3a, Q30 SchurterCircuitBreaker 10a, Q31 SchurterCircuitBreaker 16a, Q32 SchurterCircuitBreaker 16a, Q33 SchurterCircuitBreaker 3a, Q4 SchurterCircuitBreaker 3a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

Commit message: Cleaner, faster stronger
Parts:
- added C10: 107CKS016M 100UF, Capacitor_THT:CP_Radial_D5.0mm_P2.00mm, F.Cu at (464.5, 42.3)
- added C11: 107CKS016M 100UF, Capacitor_THT:CP_Radial_D5.0mm_P2.00mm, F.Cu at (485.8, 15.3)
- added C12: 107CKS016M 100UF, Capacitor_THT:CP_Radial_D5.0mm_P2.00mm, F.Cu at (438.0, 35.8)
- added C13: 107CKS016M 100UF, Capacitor_THT:CP_Radial_D5.0mm_P2.00mm, F.Cu at (431.3, 42.3)
- added C14: 107CKS016M 100UF, Capacitor_THT:CP_Radial_D5.0mm_P2.00mm, F.Cu at (444.6, 35.8)
- added C15: 107CKS016M 100UF, Capacitor_THT:CP_Radial_D5.0mm_P2.00mm, F.Cu at (438.0, 42.3)
- added C16: 107CKS016M 100UF, Capacitor_THT:CP_Radial_D5.0mm_P2.00mm, F.Cu at (451.2, 35.8)
- added C17: 107CKS016M 100UF, Capacitor_THT:CP_Radial_D5.0mm_P2.00mm, F.Cu at (431.3, 35.8)
- added C18: 107CKS016M 100UF, Capacitor_THT:CP_Radial_D5.0mm_P2.00mm, F.Cu at (444.6, 42.3)
- added C19: 107CKS016M 100UF, Capacitor_THT:CP_Radial_D5.0mm_P2.00mm, F.Cu at (451.2, 42.3)
- added C20: 107CKS016M 100UF, Capacitor_THT:CP_Radial_D5.0mm_P2.00mm, F.Cu at (457.9, 35.8)
- added C21: 107CKS016M 100UF, Capacitor_THT:CP_Radial_D5.0mm_P2.00mm, F.Cu at (472.5, 21.9)
- added C22: 107CKS016M 100UF, Capacitor_THT:CP_Radial_D5.0mm_P2.00mm, F.Cu at (479.1, 15.3)
- added C23: 107CKS016M 100UF, Capacitor_THT:CP_Radial_D5.0mm_P2.00mm, F.Cu at (457.9, 42.3)
- added C24: 107CKS016M 100UF, Capacitor_THT:CP_Radial_D5.0mm_P2.00mm, F.Cu at (464.5, 35.8)
- added C25: 107CKS016M 100UF, Capacitor_THT:CP_Radial_D5.0mm_P2.00mm, F.Cu at (472.5, 28.4)
- added C26: 107CKS016M 100UF, Capacitor_THT:CP_Radial_D5.0mm_P2.00mm, F.Cu at (479.1, 21.9)
- added C27: 107CKS016M 100UF, Capacitor_THT:CP_Radial_D5.0mm_P2.00mm, F.Cu at (477.8, 35.0)
- added C28: 107CKS016M 100UF, Capacitor_THT:CP_Radial_D5.0mm_P2.00mm, F.Cu at (491.0, 41.5)
- added C29: 107CKS016M 100UF, Capacitor_THT:CP_Radial_D5.0mm_P2.00mm, F.Cu at (491.0, 35.0)
- added C30: 107CKS016M 100UF, Capacitor_THT:CP_Radial_D5.0mm_P2.00mm, F.Cu at (484.4, 41.5)
- added C31: 107CKS016M 100UF, Capacitor_THT:CP_Radial_D5.0mm_P2.00mm, F.Cu at (492.4, 28.4)
- added C32: 107CKS016M 100UF, Capacitor_THT:CP_Radial_D5.0mm_P2.00mm, F.Cu at (477.8, 41.5)
- added C33: 107CKS016M 100UF, Capacitor_THT:CP_Radial_D5.0mm_P2.00mm, F.Cu at (484.4, 35.0)
- added C34: 107CKS016M 100UF, Capacitor_THT:CP_Radial_D5.0mm_P2.00mm, F.Cu at (492.4, 21.9)
- added C35: 107CKS016M 100UF, Capacitor_THT:CP_Radial_D5.0mm_P2.00mm, F.Cu at (485.8, 28.4)
- added C36: 107CKS016M 100UF, Capacitor_THT:CP_Radial_D5.0mm_P2.00mm, F.Cu at (471.1, 35.8)
- added C37: 107CKS016M 100UF, Capacitor_THT:CP_Radial_D5.0mm_P2.00mm, F.Cu at (471.1, 42.3)
- added C38: 107CKS016M 100UF, Capacitor_THT:CP_Radial_D5.0mm_P2.00mm, F.Cu at (492.4, 15.3)
- added C39: 107CKS016M 100UF, Capacitor_THT:CP_Radial_D5.0mm_P2.00mm, F.Cu at (485.8, 21.9)
- added C40: 107CKS016M 100UF, Capacitor_THT:CP_Radial_D5.0mm_P2.00mm, F.Cu at (479.1, 28.4)
- added C9: 107CKS016M 100UF, Capacitor_THT:CP_Radial_D5.0mm_P2.00mm, F.Cu at (472.5, 15.3)
- added RN11: 4120R-1-103LF, BoatControl:DIP254P762X432-16P, F.Cu at (468.8, 31.1)
- added RN12: 4120R-1-103LF, BoatControl:DIP254P762X432-16P, F.Cu at (458.5, 31.1)
- added RN13: 4120R-1-103LF, BoatControl:DIP254P762X432-16P, F.Cu at (448.2, 31.1)
- added RN14: 4120R-1-103LF, BoatControl:DIP254P762X432-16P, F.Cu at (437.9, 31.1)
- moved J2 473.7 mm to (24.8, 114.2), turned to 270 degrees
- moved U6 451.2 mm to (45.5, 158.7), turned to 180 degrees
- moved U5 430.0 mm to (45.4, 131.7), turned to 180 degrees
- moved U2 417.0 mm to (45.2, 102.6), turned to 180 degrees
- moved U3 408.1 mm to (45.3, 74.7), turned to 180 degrees
- moved U4 400.0 mm to (65.2, 155.4), turned to 270 degrees
- moved K40 372.0 mm to (388.9, 159.8), turned to 90 degrees
- moved K39 360.2 mm to (400.3, 121.1), turned to 270 degrees
- moved U1 358.7 mm to (65.4, 99.0)
- moved K38 335.2 mm to (407.3, 159.8), turned to 90 degrees
- moved K37 324.6 mm to (418.7, 121.1), turned to 270 degrees
- moved K36 298.4 mm to (425.7, 159.8), turned to 90 degrees
- moved K35 289.4 mm to (437.1, 121.1), turned to 270 degrees
- moved J12 270.6 mm to (459.4, 95.1), turned to 180 degrees
- moved C5 265.4 mm to (538.7, 37.9), turned to 180 degrees
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Connections:
- C1 pad 2: +12V -> GND
- C2 pad 2: +12V -> GND
- C4 pad 2: +12V -> GND
- C5 pad 2: +12V -> GND
- C6 pad 2: +12V -> GND
- C8 pad 2: +12V -> GND
- D41 pad 2: +12V -> GND
- D42 pad 2: +12V -> GND
- J11 pad 1_1: Net-(J11-Pad1_1) -> GND
- J11 pad 1_2: Net-(J11-Pad1_1) -> GND
- J11 pad 1_3: Net-(J11-Pad1_1) -> GND
- J11 pad 2_1: Net-(J11-Pad2_1) -> +12V
- J11 pad 2_2: Net-(J11-Pad2_1) -> +12V
- J11 pad 2_3: Net-(J11-Pad2_1) -> +12V
- J2 pad A_3: /A3 -> (no net)
- J3 pad A_3: Net-(J3-PadA_1) -> Net-(J3-PadA_3)
- J3 pad I_2: /K17A -> Net-(C9-Pad2)
- J3 pad I_4: /K17B -> Net-(C10-Pad2)
- J3 pad I_6: /K18A -> Net-(C11-Pad2)
- J3 pad I_8: /K18B -> Net-(C12-Pad2)
- J3 pad J_2: /K19A -> Net-(C13-Pad2)
- J3 pad J_4: /K19B -> Net-(C14-Pad2)
- J3 pad J_6: /K20A -> Net-(C15-Pad2)
- J3 pad J_8: /K20B -> Net-(C16-Pad2)
- J3 pad K_2: /K21A -> Net-(C17-Pad2)
- J3 pad K_4: /K21B -> Net-(C18-Pad2)
- J3 pad K_6: /K22A -> Net-(C19-Pad2)
- J3 pad K_8: /K22B -> Net-(C20-Pad2)
- J3 pad L_2: /K23A -> Net-(C21-Pad2)
- J3 pad L_4: /K23B -> Net-(C22-Pad2)
- J3 pad L_6: /K24A -> Net-(C23-Pad2)
- J3 pad L_8: /K24B -> Net-(C24-Pad2)
- J3 pad M_2: /K25A -> Net-(C25-Pad2)
- J3 pad M_4: /K25B -> Net-(C26-Pad2)
- J3 pad M_6: /K26A -> Net-(C27-Pad2)
- J3 pad M_8: /K26B -> Net-(C28-Pad2)
- J3 pad N_2: /K27A -> Net-(C29-Pad2)
- J3 pad N_4: /K27B -> Net-(C30-Pad2)
- J3 pad N_6: /K28A -> Net-(C31-Pad2)
- J3 pad N_8: /K28B -> Net-(C32-Pad2)
- J3 pad O_2: /K29A -> Net-(C33-Pad2)
- J3 pad O_4: /K29B -> Net-(C34-Pad2)
- J3 pad O_6: /K30A -> Net-(C35-Pad2)
- J3 pad O_8: /K30B -> Net-(C36-Pad2)
- J3 pad P_2: /K31A -> Net-(C37-Pad2)
- J3 pad P_4: /K21B -> Net-(C38-Pad2)
- J3 pad P_6: /K32A -> Net-(C39-Pad2)
- J3 pad P_8: /K32B -> Net-(C40-Pad2)
- U22 pad 4: +12V -> GND
- U23 pad 4: +12V -> GND
- U3 pad 13: /A3 -> (no net)
Routing:
- net Net-(J8-Pad1_1): track 549.1 -> 917.8 mm
- net Net-(J1-Pad1_1): track 301.3 -> 509.1 mm, vias 1 -> 0
- net Net-(J9-Pad1_1): track 305.7 -> 501.8 mm
- net Net-(K29-Pad3): track 155.0 -> 127.6 mm
- net /K1B: track 100.0 -> 74.2 mm
- net /D5B: track 50.7 -> 74.3 mm
- net /K13B: track 184.7 -> 174.5 mm
- net /K1A: track 115.9 -> 106.3 mm
- net /K15B: track 147.2 -> 139.3 mm
- net /K13A: track 261.1 -> 253.4 mm
- net Net-(J5-Pad10): track 43.1 -> 38.0 mm
- net Net-(J9-Pad2_1): track 5.00 -> 0.00 mm
- net Net-(J1-Pad2_1): track 5.00 -> 0.00 mm
- net Net-(D1-Pad2): track 650.1 -> 645.1 mm
- net Net-(K14-Pad3): track 177.9 -> 173.4 mm
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Other:
- net class Up to 32A 12V DC added: clearance 0.2, trace_width 4, via_dia 9, via_drill 7
- net class Up to16A 12V removed
- net class Up to16A 12V DC added: clearance 0.2, trace_width 2.5, via_dia 8, via_drill 6
