File: boatcontrol/boatcontrol.kicad_pcb (KiCad board)
At the start: 2 copper layers, 789.3 x 680.1 mm, 567 parts, among them IC1301 CD74HCT221E, IC1401 CD74HCT221E, IC1501 CD74HCT221E, IC1601 CD74HCT221E, IC2201 CD74HCT221E, IC2301 CD74HCT221E, IC2401 CD74HCT221E, IC2501 CD74HCT221E, IC3101 CD74HCT221E, IC3201 CD74HCT221E, IC3301 CD74HCT221E, IC3401 CD74HCT221E, IC401 CD74HCT221E, IC501 CD74HCT221E, IC5301 CD74HCT221E, IC5401 CD74HCT221E, IC5501 CD74HCT221E, IC5601 CD74HCT221E, IC601 CD74HCT221E, IC6201 CD74HCT221E, IC6301 CD74HCT221E, IC6401 CD74HCT221E, IC6501 CD74HCT221E, IC701 CD74HCT221E, IC7101 CD74HCT221E, IC7201 CD74HCT221E, IC7301 CD74HCT221E, IC7401 CD74HCT221E, IC8001 CD74HCT221E, IC8101 CD74HCT221E, IC8201 CD74HCT221E, IC8301 CD74HCT221E, J101 Conn_01x01_Male, J102 Conn_01x01_Male, J103 Conn_01x01_Male, J105 Conn_01x02_Male, J106 Conn_01x01_Male, J107 SS73100-047F, J108 SS73100-047F, J111 TBL008V-1000-02BE, J201 Conn_01x01_Male, J202 Conn_01x01_Male, J203 TBP01R2W-508-16BE, J204 Conn_01x01_Male, J205 Conn_01x01_Male, J206 TBL008V-1000-02BE, J3 40HAT, J3901 Conn_01x01_Male, J3902 Conn_01x01_Male, J3903 Conn_02x20_Odd_Even Socket, J5101 Conn_01x01_Male, J5102 TBP01R2W-508-08BE, J5103 Conn_01x01_Male, J5104 TBL008V-1000-02BE, J5105 TBP01R2W-508-08BE, J5106 Conn_01x01_Male, J5107 Conn_01x01_Male, J5108 TBL008V-1000-02BE, J8801 Conn_01x01_Male, J8802 Conn_01x01_Male, J8803 Conn_02x20_Odd_Even Socket, K1001 G5RL-K1A-E-DC12, K1101 G5RL-K1A-E-DC12, K1701 G5RL-K1A-E-DC12, K1801 G5RL-K1A-E-DC12, K1901 G5RL-K1A-E-DC12, K2001 G5RL-K1A-E-DC12, K2601 G5RL-K1A-E-DC12, K2701 G5RL-K1A-E-DC12, K2801 G5RL-K1A-E-DC12, K2901 G5RL-K1A-E-DC12, K3501 G5RL-K1A-E-DC12, K3601 G5RL-K1A-E-DC12, K3701 G5RL-K1A-E-DC12, K3801 G5RL-K1A-E-DC12, K5701 G5RL-K1A-E-DC12, K5801 G5RL-K1A-E-DC12, K5901 G5RL-K1A-E-DC12, K6001 G5RL-K1A-E-DC12, K6601 G5RL-K1A-E-DC12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

Commit message: vibrator cleanup and layout
Parts:
- moved RN7901 23.1 mm to (124.5, 157.5), turned to 0 degrees
- moved RN6103 23.0 mm to (73.5, 172.5), turned to 0 degrees
- moved RN7004 23.0 mm to (249.5, 187.5), turned to 0 degrees
- moved RN5201 23.0 mm to (301.0, 157.5), turned to 0 degrees
- moved RN5203 23.0 mm to (301.0, 172.5), turned to 0 degrees
- moved RN5204 23.0 mm to (301.0, 187.5), turned to 0 degrees
- moved RN6101 23.0 mm to (73.5, 157.5), turned to 0 degrees
- moved RN6104 23.0 mm to (73.5, 187.5), turned to 0 degrees
- moved RN7904 23.0 mm to (124.5, 187.5), turned to 0 degrees
- moved RN7001 23.0 mm to (249.5, 157.5), turned to 0 degrees
- moved RN7003 23.0 mm to (249.5, 172.5), turned to 0 degrees
- moved RN7903 23.0 mm to (124.5, 172.5), turned to 0 degrees
- moved C1209 14.0 mm to (174.0, 224.0)
- moved C1210 14.0 mm to (180.0, 224.0)
- moved RN1202 14.0 mm to (152.0, 225.0)
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Routing:
- net +12P: track 753.2 -> 0.00 mm
- net /12V DC Common Bank/12V DC Block 1/3AC3/ON_LED: track 12.8 -> 0.00 mm
- net /12V DC Common Bank/12V DC Block 2/MultiVibrator3A3/R2: track 9.86 -> 12.1 mm
- net /Mixed 12V DC / 230V AC Common Bank/12V DC 6A Block/MultiVibrator6A4/R2: track 9.86 -> 12.1 mm
- net /Mixed 12V DC / 230V AC Common Bank/230V AC 6A Block/MultiVibrator6A1/R2: track 9.86 -> 12.1 mm
- net /Mixed 12V DC / 230V AC Common Bank/12V DC 10/16A Block/MultiVibrator10A1/R2: track 9.86 -> 12.1 mm
- net /Mixed 12V DC / 230V AC Common Bank/12V DC 6A Block/MultiVibrator6A2/R2: track 9.86 -> 12.1 mm
- net /Mixed 12V DC / 230V AC Common Bank/12V DC 6A Block/MultiVibrator6A1/R2: track 9.86 -> 12.1 mm
- net /Mixed 12V DC / 230V AC Common Bank/12V DC 10/16A Block/MultiVibrator16A2/R2: track 9.86 -> 12.1 mm
- net /Mixed 12V DC / 230V AC Common Bank/12V DC 10/16A Block/MultiVibrator16A1/R2: track 9.86 -> 12.1 mm
- net /12V DC Common Bank/12V DC Block 4/MultiVibrator3A4/R2: track 9.86 -> 12.1 mm
- net /Mixed 12V DC / 230V AC Common Bank/230V AC 6A Block/MultiVibrator6A4/R2: track 9.86 -> 12.1 mm
- net /Mixed 12V DC / 230V AC Common Bank/230V AC 6A Block/MultiVibrator6A3/R2: track 9.86 -> 12.1 mm
- net /Mixed 12V DC / 230V AC Common Bank/230V AC 6A Block/MultiVibrator6A2/R2: track 9.86 -> 12.1 mm
- net /Mixed 12V DC / 230V AC Common Bank/230V AC 10/16A Block/MultiVibrator16A1/R2: track 9.86 -> 12.1 mm
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
Commit message: More cleanup
Parts:
- D5701, D5801, D5901, D6001, D8401, D8501, D8601, D8701: value 20mA R/G -> 20mA R/G CA
- D6601, D6901, D7501, D7801: value WP115VGYW -> 20mA R/G CA
- moved C5209 85.2 mm to (358.0, 122.0)
- moved C5210 85.2 mm to (352.0, 122.0)
- moved RN5202 85.2 mm to (323.0, 115.5)
- moved U5201 85.2 mm to (327.0, 123.5)
- moved RN6102 5.41 mm to (92.5, 115.5)
- moved C6109 4.00 mm to (126.5, 117.0)
- moved C6110 4.00 mm to (120.5, 117.0)
- moved U6101 4.00 mm to (95.5, 123.0)
- moved C7009 2.00 mm to (300.0, 122.0)
- moved C7010 2.00 mm to (294.0, 117.0)
- moved RN7002 2.00 mm to (265.0, 115.5)
- moved U7001 2.00 mm to (269.0, 123.0)
- moved C7909 1.50 mm to (193.0, 117.0)
- moved C7910 1.50 mm to (187.0, 117.0)
- moved RN7902 1.50 mm to (155.5, 115.5)
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
Commit message: Fix resistor network values
Parts:
- moved U202 9.50 mm to (375.5, 189.0)
- moved U5101 9.50 mm to (111.5, 189.0)
- moved U5102 9.50 mm to (287.5, 189.0)
- moved U201 9.00 mm to (199.5, 189.0)
- moved C3001 0.50 mm to (387.0, 183.0)
- moved C3002 0.50 mm to (412.5, 177.0)
- moved C3003 0.50 mm to (387.0, 153.0)
- moved C3004 0.50 mm to (412.5, 147.0)
- moved C3005 0.50 mm to (387.0, 168.0)
- moved C3006 0.50 mm to (412.5, 162.0)
- moved C3007 0.50 mm to (387.0, 198.0)
- moved C3008 0.50 mm to (412.5, 192.0)
- moved C3101 0.50 mm to (381.5, 178.0)
- moved C3201 0.50 mm to (381.5, 148.0)
- moved C3301 0.50 mm to (381.5, 163.0)
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
Commit message: Multi
Parts:
- RN5201, RN5204, RN7901, RN7904: value 100K Ohm -> 100KΩ
- RN5203, RN7903: value 10M Ohm -> 10MΩ
