File: boatcontrol/boatcontrol.kicad_pcb (KiCad board)
At the start: 2 copper layers, 789.3 x 680.1 mm, 567 parts, among them IC1301 CD74HCT221E, IC1401 CD74HCT221E, IC1501 CD74HCT221E, IC1601 CD74HCT221E, IC2201 CD74HCT221E, IC2301 CD74HCT221E, IC2401 CD74HCT221E, IC2501 CD74HCT221E, IC3101 CD74HCT221E, IC3201 CD74HCT221E, IC3301 CD74HCT221E, IC3401 CD74HCT221E, IC401 CD74HCT221E, IC501 CD74HCT221E, IC5301 CD74HCT221E, IC5401 CD74HCT221E, IC5501 CD74HCT221E, IC5601 CD74HCT221E, IC601 CD74HCT221E, IC6201 CD74HCT221E, IC6301 CD74HCT221E, IC6401 CD74HCT221E, IC6501 CD74HCT221E, IC701 CD74HCT221E, IC7101 CD74HCT221E, IC7201 CD74HCT221E, IC7301 CD74HCT221E, IC7401 CD74HCT221E, IC8001 CD74HCT221E, IC8101 CD74HCT221E, IC8201 CD74HCT221E, IC8301 CD74HCT221E, J101 Conn_01x01_Male, J102 Conn_01x01_Male, J103 Conn_01x01_Male, J105 Conn_01x02_Male, J106 Conn_01x01_Male, J107 SS73100-047F, J108 SS73100-047F, J111 TBL008V-1000-02BE, J201 Conn_01x01_Male, J202 Conn_01x01_Male, J203 TBP01R2W-508-16BE, J204 Conn_01x01_Male, J205 Conn_01x01_Male, J206 TBL008V-1000-02BE, J3 40HAT, J3901 Conn_01x01_Male, J3902 Conn_01x01_Male, J3903 Conn_02x20_Odd_Even Socket, J5101 Conn_01x01_Male, J5102 TBP01R2W-508-08BE, J5103 Conn_01x01_Male, J5104 TBL008V-1000-02BE, J5105 TBP01R2W-508-08BE, J5106 Conn_01x01_Male, J5107 Conn_01x01_Male, J5108 TBL008V-1000-02BE, J8801 Conn_01x01_Male, J8802 Conn_01x01_Male, J8803 Conn_02x20_Odd_Even Socket, K1001 G5RL-K1A-E-DC12, K1101 G5RL-K1A-E-DC12, K1701 G5RL-K1A-E-DC12, K1801 G5RL-K1A-E-DC12, K1901 G5RL-K1A-E-DC12, K2001 G5RL-K1A-E-DC12, K2601 G5RL-K1A-E-DC12, K2701 G5RL-K1A-E-DC12, K2801 G5RL-K1A-E-DC12, K2901 G5RL-K1A-E-DC12, K3501 G5RL-K1A-E-DC12, K3601 G5RL-K1A-E-DC12, K3701 G5RL-K1A-E-DC12, K3801 G5RL-K1A-E-DC12, K5701 G5RL-K1A-E-DC12, K5801 G5RL-K1A-E-DC12, K5901 G5RL-K1A-E-DC12, K6001 G5RL-K1A-E-DC12, K6601 G5RL-K1A-E-DC12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

Commit message: Left Sorted
Changed lines of the file:
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@@
     (add_net "/Add-On Relay Board 1/I2C_A2")
     (add_net "/Add-On Relay Board 1/INT_A")
-    (add_net "/Add-On Relay Board 1/INT_B")
     (add_net "/Add-On Relay Board 1/MixedBlock1/MixedControl1/DIG_OFF")
     (add_net "/Add-On Relay Board 1/MixedBlock1/MixedControl1/DIG_ON")
@@
     (add_net "/Add-On Relay Board 2/I2C_A2")
     (add_net "/Add-On Relay Board 2/INT_A")
-    (add_net "/Add-On Relay Board 2/INT_B")
     (add_net "/Add-On Relay Board 2/MixedBlock1/MixedControl1/DIG_OFF")
     (add_net "/Add-On Relay Board 2/MixedBlock1/MixedControl1/DIG_ON")
@@
     (add_net "Net-(JP5108-Pad2)")
     (add_net "Net-(Q104-Pad1)")
-    (add_net "Net-(Q104-Pad14)")
     (add_net "Net-(Q104-Pad5)")
     (add_net "Net-(U101-Pad1)")
@@
     (add_net "Net-(U101-Pad7)")
     (add_net "Net-(U101-Pad8)")
-    (add_net "Net-(U102-Pad11)")
-    (add_net "Net-(U102-Pad14)")
     (add_net "Net-(U102-Pad21)")
     (add_net "Net-(U102-Pad22)")
@@
     (add_net "Net-(U102-Pad27)")
     (add_net "Net-(U102-Pad28)")
-    (add_net "Net-(U104-Pad1)")
-    (add_net "Net-(U104-Pad2)")
-    (add_net "Net-(U104-Pad3)")
-    (add_net "Net-(U107-Pad5)")
-    (add_net "Net-(U108-Pad5)")
-    (add_net "Net-(U201-Pad11)")
-    (add_net "Net-(U201-Pad14)")
-    (add_net "Net-(U202-Pad11)")
-    (add_net "Net-(U202-Pad14)")
-    (add_net "Net-(U202-Pad2)")
-    (add_net "Net-(U3901-Pad11)")
-    (add_net "Net-(U3901-Pad14)")
-    (add_net "Net-(U3901-Pad20)")
-    (add_net "Net-(U5101-Pad11)")
-    (add_net "Net-(U5101-Pad14)")
-    (add_net "Net-(U5102-Pad11)")
-    (add_net "Net-(U5102-Pad14)")
-    (add_net "Net-(U8801-Pad11)")
-    (add_net "Net-(U8801-Pad14)")
-    (add_net "Net-(U8801-Pad20)")
     (add_net SCK)
     (add_net SDA)
@@
     (descr "N (R-PDIP-T)")
     (tags "Integrated Circuit")
-    (fp_text reference IC6501 (at 0 -11.43 90) (layer F.SilkS)
+    (fp_text reference IC6501 (at -4.5 13.000001 180) (layer F.SilkS)
       (effects (font (size 1 1) (thickness 0.2)))
     )
@@
     (descr "N (R-PDIP-T)")
     (tags "Integrated Circuit")
-    (fp_text reference IC6401 (at 0 -11.43 90) (layer F.SilkS)
+    (fp_text reference IC6401 (at -4.5 13 180) (layer F.SilkS)
       (effects (font (size 1 1) (thickness 0.2)))
     )
@@
     (descr "N (R-PDIP-T)")
     (tags "Integrated Circuit")
-    (fp_text reference IC6301 (at 0 -11.43 90) (layer F.SilkS)
+    (fp_text reference IC6301 (at -4.5 13 180) (layer F.SilkS)
       (effects (font (size 1 1) (thickness 0.2)))
     )
@@
     (descr "C, Disc series, Radial, pin pitch=5.00mm, , diameter*width=7.5*5.0mm^2, Capacitor, http://www.vishay.com/docs/28535/vy2series.pdf")
     (tags "C Disc series Radial pin pitch 5.00mm  diameter 7.5mm width 5.0mm Capacitor")
-    (fp_text reference C6501 (at 9 -3.75 90) (layer F.SilkS)
+    (fp_text reference C6501 (at -4 2.5 90) (layer F.SilkS)
       (effects (font (size 1 1) (thickness 0.15)))
     )
-    (fp_text value 0.1μF (at 2.5 3.75 180) (layer F.Fab)
+    (fp_text value 0.1μF (at -4 1 270) (layer F.Fab)
       (effects (font (size 1 1) (thickness 0.15)))
     )
@@
     (fp_line (start 6.5 2.75) (end 6.5 -2.75) (layer F.CrtYd) (width 0.05))
     (fp_line (start 6.5 -2.75) (end -1.5 -2.75) (layer F.CrtYd) (width 0.05))
-    (fp_text user %R (at 9 0 90) (layer F.Fab)
+    (fp_text user %R (at -4 2.5 90) (layer F.Fab)
       (effects (font (size 1 1) (thickness 0.15)))
     )
@@
     (descr "C, Disc series, Radial, pin pitch=5.00mm, , diameter*width=7.5*5.0mm^2, Capacitor, http://www.vishay.com/docs/28535/vy2series.pdf")
     (tags "C Disc series Radial pin pitch 5.00mm  diameter 7.5mm width 5.0mm Capacitor")
-    (fp_text reference C6401 (at 9 -3.75 90) (layer F.SilkS)
+    (fp_text reference C6401 (at -4 2.5 90) (layer F.SilkS)
       (effects (font (size 1 1) (thickness 0.15)))
     )
-    (fp_text value 0.1μF (at 2.5 3.75 180) (layer F.Fab)
+    (fp_text value 0.1μF (at -4 1 270) (layer F.Fab)
       (effects (font (size 1 1) (thickness 0.15)))
     )
@@
     (fp_line (start 6.5 2.75) (end 6.5 -2.75) (layer F.CrtYd) (width 0.05))
     (fp_line (start 6.5 -2.75) (end -1.5 -2.75) (layer F.CrtYd) (width 0.05))
-    (fp_text user %R (at 9 0 90) (layer F.Fab)
+    (fp_text user %R (at -4 2.5 90) (layer F.Fab)
       (effects (font (size 1 1) (thickness 0.15)))
     )
@@
     (descr "C, Disc series, Radial, pin pitch=5.00mm, , diameter*width=7.5*5.0mm^2, Capacitor, http://www.vishay.com/docs/28535/vy2series.pdf")
     (tags "C Disc series Radial pin pitch 5.00mm  diameter 7.5mm width 5.0mm Capacitor")
-    (fp_text reference C6301 (at 9 -3.75 90) (layer F.SilkS)
+    (fp_text reference C6301 (at -3.999999 2.5 90) (layer F.SilkS)
       (effects (font (size 1 1) (thickness 0.15)))
     )
-    (fp_text value 0.1μF (at 2.5 3.75 180) (layer F.Fab)
+    (fp_text value 0.1μF (at -3.999999 1 270) (layer F.Fab)
       (effects (font (size 1 1) (thickness 0.15)))
     )
@@
     (fp_line (start 6.5 2.75) (end 6.5 -2.75) (layer F.CrtYd) (width 0.05))
     (fp_line (start 6.5 -2.75) (end -1.5 -2.75) (layer F.CrtYd) (width 0.05))
-    (fp_text user %R (at 9 0 90) (layer F.Fab)
+    (fp_text user %R (at -3.999999 2.5 90) (layer F.Fab)
       (effects (font (size 1 1) (thickness 0.15)))
     )
@@
     (descr "C, Disc series, Radial, pin pitch=5.00mm, , diameter*width=7.5*5.0mm^2, Capacitor, http://www.vishay.com/docs/28535/vy2series.pdf")
     (tags "C Disc series Radial pin pitch 5.00mm  diameter 7.5mm width 5.0mm Capacitor")
-    (fp_text reference C6201 (at -4 1.9 90) (layer F.SilkS)
+    (fp_text reference C6201 (at -4 2.5 90) (layer F.SilkS)
       (effects (font (size 1 1) (thickness 0.15)))
     )
-    (fp_text value 0.1μF (at -3.8 -0.1 90) (layer F.Fab)
+    (fp_text value 0.1μF (at -3.8 1 90) (layer F.Fab)
       (effects (font (size 1 1) (thickness 0.15)))
     )
@@
     (fp_line (start 6.5 2.75) (end 6.5 -2.75) (layer F.CrtYd) (width 0.05))
     (fp_line (start 6.5 -2.75) (end -1.5 -2.75) (layer F.CrtYd) (width 0.05))
-    (fp_text user %R (at 2.6 1.9 90) (layer F.Fab)
+    (fp_text user %R (at -4 2.5 90) (layer F.Fab)
       (effects (font (size 1 1) (thickness 0.15)))
     )
@@
     (descr "C, Disc series, Radial, pin pitch=5.00mm, , diameter*width=7.5*5.0mm^2, Capacitor, http://www.vishay.com/docs/28535/vy2series.pdf")
     (tags "C Disc series Radial pin pitch 5.00mm  diameter 7.5mm width 5.0mm Capacitor")
-    (fp_text reference C6107 (at -4 -3.75 90) (layer F.SilkS)
+    (fp_text reference C6107 (at 9 -2.5 90) (layer F.SilkS)
       (effects (font (size 1 1) (thickness 0.15)))
     )
-    (fp_text value 1µF (at 2.5 3.75 180) (layer F.Fab)
+    (fp_text value 1µF (at 8.5 -1 270) (layer F.Fab)
       (effects (font (size 1 1) (thickness 0.15)))
     )
@@
     (fp_line (start 6.5 2.75) (end 6.5 -2.75) (layer F.CrtYd) (width 0.05))
     (fp_line (start 6.5 -2.75) (end -1.5 -2.75) (layer F.CrtYd) (width 0.05))
-    (fp_text user %R (at -4 0 90) (layer F.Fab)
+    (fp_text user %R (at 9 -2.5 90) (layer F.Fab)
       (effects (font (size 1 1) (thickness 0.15)))
     )
@@
     (descr "C, Disc series, Radial, pin pitch=5.00mm, , diameter*width=7.5*5.0mm^2, Capacitor, http://www.vishay.com/docs/28535/vy2series.pdf")
     (tags "C Disc series Radial pin pitch 5.00mm  diameter 7.5mm width 5.0mm Capacitor")
-    (fp_text reference C6105 (at -4 -3.75 90) (layer F.SilkS)
+    (fp_text reference C6105 (at 9 -2.5 90) (layer F.SilkS)
       (effects (font (size 1 1) (thickness 0.15)))
     )
-    (fp_text value 1µF (at 2.5 3.75 180) (layer F.Fab)
+    (fp_text value 1µF (at 8.5 -1 270) (layer F.Fab)
       (effects (font (size 1 1) (thickness 0.15)))
     )
@@
     (fp_line (start 6.5 2.75) (end 6.5 -2.75) (layer F.CrtYd) (width 0.05))
     (fp_line (start 6.5 -2.75) (end -1.5 -2.75) (layer F.CrtYd) (width 0.05))
-    (fp_text user %R (at -4 0 90) (layer F.Fab)
+    (fp_text user %R (at 9 -2.5 90) (layer F.Fab)
       (effects (font (size 1 1) (thickness 0.15)))
     )
@@
     (descr "C, Disc series, Radial, pin pitch=5.00mm, , diameter*width=7.5*5.0mm^2, Capacitor, http://www.vishay.com/docs/28535/vy2series.pdf")
     (tags "C Disc series Radial pin pitch 5.00mm  diameter 7.5mm width 5.0mm Capacitor")
-    (fp_text reference C6103 (at -4 -3.75 90) (layer F.SilkS)
+    (fp_text reference C6103 (at 8.999999 -2.5 90) (layer F.SilkS)
       (effects (font (size 1 1) (thickness 0.15)))
     )
-    (fp_text value 1µF (at 2.5 3.75 180) (layer F.Fab)
+    (fp_text value 1µF (at 8.499999 -1 270) (layer F.Fab)
       (effects (font (size 1 1) (thickness 0.15)))
     )
@@
     (fp_line (start 6.5 2.75) (end 6.5 -2.75) (layer F.CrtYd) (width 0.05))
     (fp_line (start 6.5 -2.75) (end -1.5 -2.75) (layer F.CrtYd) (width 0.05))
-    (fp_text user %R (at -4 0 90) (layer F.Fab)
+    (fp_text user %R (at 8.999999 -2.5 90) (layer F.Fab)
       (effects (font (size 1 1) (thickness 0.15)))
     )
@@
     (descr "C, Disc series, Radial, pin pitch=5.00mm, , diameter*width=7.5*5.0mm^2, Capacitor, http://www.vishay.com/docs/28535/vy2series.pdf")
     (tags "C Disc series Radial pin pitch 5.00mm  diameter 7.5mm width 5.0mm Capacitor")
-    (fp_text reference C6101 (at 8.8 -1.8 90) (layer F.SilkS)
+    (fp_text reference C6101 (at 9 -2.5 90) (layer F.SilkS)
       (effects (font (size 1 1) (thickness 0.15)))
     )
-    (fp_text value 1µF (at 8 0 270) (layer F.Fab)
+    (fp_text value 1µF (at 8 -1 270) (layer F.Fab)
       (effects (font (size 1 1) (thickness 0.15)))
     )
@@
     (fp_line (start 6.5 2.75) (end 6.5 -2.75) (layer F.CrtYd) (width 0.05))
     (fp_line (start 6.5 -2.75) (end -1.5 -2.75) (layer F.CrtYd) (width 0.05))
-    (fp_text user %R (at 2.6 -1.8 90) (layer F.Fab)
+    (fp_text user %R (at 9 -2.5 90) (layer F.Fab)
       (effects (font (size 1 1) (thickness 0.15)))
     )

Commit message: Fix cap
Parts:
- moved C7003 26.7 mm to (248.0, 168.0), turned to 90 degrees
- moved C7004 26.7 mm to (274.0, 162.0), turned to 270 degrees
- moved IC1601 0.50 mm to (224.5, 195.0)
- moved IC1401 0.50 mm to (224.5, 165.0)
- moved IC2201 0.50 mm to (349.5, 150.0)
- moved IC2301 0.50 mm to (349.5, 165.0)
- moved IC2401 0.50 mm to (349.5, 180.0)
- moved IC2501 0.50 mm to (349.5, 195.0)
- moved IC3101 0.50 mm to (400.0, 180.0)
- moved IC3201 0.50 mm to (400.0, 150.0)
- moved IC3301 0.50 mm to (400.0, 165.0)
- moved IC3401 0.50 mm to (400.0, 195.0)
- turned IC7201 to 90 degrees
Routing:
- net /Mixed 12V DC / 230V AC Common Bank/12V DC 10/16A Block/MultiVibrator10A2/R2: track 9.86 -> 12.1 mm

Commit message: Text cleanup
Parts:
- moved C1203 0.50 mm to (211.0, 168.0)
- moved C1207 0.50 mm to (211.0, 198.0)
- moved C1401 0.50 mm to (205.5, 163.0)
- moved C1601 0.50 mm to (205.5, 193.0)
- moved C2101 0.50 mm to (336.0, 153.0)
- moved C2103 0.50 mm to (336.0, 168.0)
- moved C2105 0.50 mm to (336.0, 183.0)
- moved C2107 0.50 mm to (336.0, 198.0)
- moved C2201 0.50 mm to (330.5, 148.0)
- moved C2301 0.50 mm to (330.5, 163.0)
- moved C2401 0.50 mm to (330.5, 178.0)
- moved C2501 0.50 mm to (330.5, 193.0)
- moved C3002 0.50 mm to (413.0, 177.0)
- moved C3004 0.50 mm to (413.0, 147.0)
- moved C3006 0.50 mm to (413.0, 162.0)
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Routing:
- net /12V DC Common Bank/12V DC Block 4/MultiVibrator3A1/RC2: track 7.47 -> 7.97 mm
- net /12V DC Common Bank/12V DC Block 4/MultiVibrator3A1/R2: track 12.1 -> 12.6 mm
- net /12V DC Common Bank/12V DC Block 4/MultiVibrator3A4/RC2: track 7.47 -> 7.97 mm
- net /12V DC Common Bank/12V DC Block 4/MultiVibrator3A4/R2: track 12.1 -> 12.6 mm
- net /12V DC Common Bank/12V DC Block 4/MultiVibrator3A3/RC2: track 7.47 -> 7.97 mm
- net /12V DC Common Bank/12V DC Block 4/MultiVibrator3A3/R2: track 12.1 -> 12.6 mm
- net /12V DC Common Bank/12V DC Block 4/MultiVibrator3A2/RC2: track 7.47 -> 7.97 mm
- net /12V DC Common Bank/12V DC Block 4/MultiVibrator3A2/R2: track 12.1 -> 12.6 mm
- net /12V DC Common Bank/12V DC Block 3/MultiVibrator3A4/RC2: track 7.47 -> 7.97 mm
- net /12V DC Common Bank/12V DC Block 3/MultiVibrator3A4/R2: track 12.1 -> 12.6 mm
- net /12V DC Common Bank/12V DC Block 3/MultiVibrator3A3/RC2: track 7.47 -> 7.97 mm
- net /12V DC Common Bank/12V DC Block 3/MultiVibrator3A3/R2: track 12.1 -> 12.6 mm
- net /12V DC Common Bank/12V DC Block 3/MultiVibrator3A2/RC2: track 7.47 -> 7.97 mm
- net /12V DC Common Bank/12V DC Block 3/MultiVibrator3A2/R2: track 12.1 -> 12.6 mm
- net /12V DC Common Bank/12V DC Block 3/MultiVibrator3A1/RC2: track 7.47 -> 7.97 mm
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
Commit message: Rewiring resistors done
Routing:
- net +5V: track 414.3 -> 756.4 mm
- net (no net): track 0.00 -> 70.1 mm

Commit message: SecondBlock
Connections:
- RN5201 pad 3: 12V_DC_C17_OFF -> /Mixed 12V DC / 230V AC Common Bank/12V DC 6A Block/DIG_ON_C1
- RN5201 pad 4: /Mixed 12V DC / 230V AC Common Bank/12V DC 6A Block/DIG_ON_C1 -> /Mixed 12V DC / 230V AC Common Bank/12V DC 6A Block/DIG_OFF_C1
- RN5201 pad 5: /Mixed 12V DC / 230V AC Common Bank/12V DC 6A Block/DIG_OFF_C1 -> 12V_DC_C17_OFF
- RN5201 pad 7: 12V_DC_C18_OFF -> /Mixed 12V DC / 230V AC Common Bank/12V DC 6A Block/DIG_ON_C2
- RN5201 pad 8: /Mixed 12V DC / 230V AC Common Bank/12V DC 6A Block/DIG_ON_C2 -> /Mixed 12V DC / 230V AC Common Bank/12V DC 6A Block/DIG_OFF_C2
- RN5201 pad 9: /Mixed 12V DC / 230V AC Common Bank/12V DC 6A Block/DIG_OFF_C2 -> 12V_DC_C18_OFF
- RN5203 pad 2: /Mixed 12V DC / 230V AC Common Bank/12V DC 6A Block/MultiVibrator6A1/R1 -> /Mixed 12V DC / 230V AC Common Bank/12V DC 6A Block/MultiVibrator6A2/R1
- RN5203 pad 4: /Mixed 12V DC / 230V AC Common Bank/12V DC 6A Block/MultiVibrator6A2/R1 -> /Mixed 12V DC / 230V AC Common Bank/12V DC 6A Block/MultiVibrator6A1/R1
- RN5203 pad 6: /Mixed 12V DC / 230V AC Common Bank/12V DC 6A Block/MultiVibrator6A3/R1 -> /Mixed 12V DC / 230V AC Common Bank/12V DC 6A Block/MultiVibrator6A3/R2
- RN5203 pad 7: /Mixed 12V DC / 230V AC Common Bank/12V DC 6A Block/MultiVibrator6A3/R2 -> /Mixed 12V DC / 230V AC Common Bank/12V DC 6A Block/MultiVibrator6A3/R1
- RN5204 pad 3: 12V_DC_C19_OFF -> /Mixed 12V DC / 230V AC Common Bank/12V DC 6A Block/DIG_ON_C3
- RN5204 pad 4: /Mixed 12V DC / 230V AC Common Bank/12V DC 6A Block/DIG_ON_C3 -> /Mixed 12V DC / 230V AC Common Bank/12V DC 6A Block/DIG_OFF_C3
- RN5204 pad 5: /Mixed 12V DC / 230V AC Common Bank/12V DC 6A Block/DIG_OFF_C3 -> 12V_DC_C19_OFF
- RN5204 pad 7: 12V_DC_C20_OFF -> /Mixed 12V DC / 230V AC Common Bank/12V DC 6A Block/DIG_ON_C4
- RN5204 pad 8: /Mixed 12V DC / 230V AC Common Bank/12V DC 6A Block/DIG_ON_C4 -> /Mixed 12V DC / 230V AC Common Bank/12V DC 6A Block/DIG_OFF_C4
- RN5204 pad 9: /Mixed 12V DC / 230V AC Common Bank/12V DC 6A Block/DIG_OFF_C4 -> 12V_DC_C20_OFF
- RN6101 pad 3: 230V_AC_C5_OFF -> /Mixed 12V DC / 230V AC Common Bank/230V AC 10/16A Block/DIG_ON_C1
- RN6101 pad 4: /Mixed 12V DC / 230V AC Common Bank/230V AC 10/16A Block/DIG_ON_C1 -> /Mixed 12V DC / 230V AC Common Bank/230V AC 10/16A Block/DIG_OFF_C1
- RN6101 pad 5: /Mixed 12V DC / 230V AC Common Bank/230V AC 10/16A Block/DIG_OFF_C1 -> 230V_AC_C5_OFF
- RN6101 pad 7: 230V_AC_C6_OFF -> /Mixed 12V DC / 230V AC Common Bank/230V AC 10/16A Block/DIG_ON_C2
- RN6101 pad 8: /Mixed 12V DC / 230V AC Common Bank/230V AC 10/16A Block/DIG_ON_C2 -> /Mixed 12V DC / 230V AC Common Bank/230V AC 10/16A Block/DIG_OFF_C2
- RN6101 pad 9: /Mixed 12V DC / 230V AC Common Bank/230V AC 10/16A Block/DIG_OFF_C2 -> 230V_AC_C6_OFF
- RN6103 pad 2: /Mixed 12V DC / 230V AC Common Bank/230V AC 10/16A Block/MultiVibrator10A1/R1 -> /Mixed 12V DC / 230V AC Common Bank/230V AC 10/16A Block/MultiVibrator10A2/R1
- RN6103 pad 4: /Mixed 12V DC / 230V AC Common Bank/230V AC 10/16A Block/MultiVibrator10A2/R1 -> /Mixed 12V DC / 230V AC Common Bank/230V AC 10/16A Block/MultiVibrator10A1/R1
- RN6103 pad 6: /Mixed 12V DC / 230V AC Common Bank/230V AC 10/16A Block/MultiVibrator16A1/R1 -> /Mixed 12V DC / 230V AC Common Bank/230V AC 10/16A Block/MultiVibrator16A1/R2
- RN6103 pad 7: /Mixed 12V DC / 230V AC Common Bank/230V AC 10/16A Block/MultiVibrator16A1/R2 -> /Mixed 12V DC / 230V AC Common Bank/230V AC 10/16A Block/MultiVibrator16A1/R1
- RN6104 pad 3: 230V_AC_C7_OFF -> /Mixed 12V DC / 230V AC Common Bank/230V AC 10/16A Block/DIG_ON_C3
- RN6104 pad 4: /Mixed 12V DC / 230V AC Common Bank/230V AC 10/16A Block/DIG_ON_C3 -> /Mixed 12V DC / 230V AC Common Bank/230V AC 10/16A Block/DIG_OFF_C3
- RN6104 pad 5: /Mixed 12V DC / 230V AC Common Bank/230V AC 10/16A Block/DIG_OFF_C3 -> 230V_AC_C7_OFF
- RN6104 pad 7: 230V_AC_C8_OFF -> /Mixed 12V DC / 230V AC Common Bank/230V AC 10/16A Block/DIG_ON_C4
- RN6104 pad 8: /Mixed 12V DC / 230V AC Common Bank/230V AC 10/16A Block/DIG_ON_C4 -> /Mixed 12V DC / 230V AC Common Bank/230V AC 10/16A Block/DIG_OFF_C4
- RN6104 pad 9: /Mixed 12V DC / 230V AC Common Bank/230V AC 10/16A Block/DIG_OFF_C4 -> 230V_AC_C8_OFF
- RN7001 pad 3: 12V_DC_C21_OFF -> /Mixed 12V DC / 230V AC Common Bank/12V DC 10/16A Block/DIG_ON_C1
- RN7001 pad 4: /Mixed 12V DC / 230V AC Common Bank/12V DC 10/16A Block/DIG_ON_C1 -> /Mixed 12V DC / 230V AC Common Bank/12V DC 10/16A Block/DIG_OFF_C1
- RN7001 pad 5: /Mixed 12V DC / 230V AC Common Bank/12V DC 10/16A Block/DIG_OFF_C1 -> 12V_DC_C21_OFF
- RN7001 pad 7: 12V_DC_C22_OFF -> /Mixed 12V DC / 230V AC Common Bank/12V DC 10/16A Block/DIG_ON_C2
- RN7001 pad 8: /Mixed 12V DC / 230V AC Common Bank/12V DC 10/16A Block/DIG_ON_C2 -> /Mixed 12V DC / 230V AC Common Bank/12V DC 10/16A Block/DIG_OFF_C2
- RN7001 pad 9: /Mixed 12V DC / 230V AC Common Bank/12V DC 10/16A Block/DIG_OFF_C2 -> 12V_DC_C22_OFF
- RN7003 pad 2: /Mixed 12V DC / 230V AC Common Bank/12V DC 10/16A Block/MultiVibrator10A1/R1 -> /Mixed 12V DC / 230V AC Common Bank/12V DC 10/16A Block/MultiVibrator10A2/R1
- RN7003 pad 4: /Mixed 12V DC / 230V AC Common Bank/12V DC 10/16A Block/MultiVibrator10A2/R1 -> /Mixed 12V DC / 230V AC Common Bank/12V DC 10/16A Block/MultiVibrator10A1/R1
- RN7003 pad 6: /Mixed 12V DC / 230V AC Common Bank/12V DC 10/16A Block/MultiVibrator16A1/R1 -> /Mixed 12V DC / 230V AC Common Bank/12V DC 10/16A Block/MultiVibrator16A1/R2
- RN7003 pad 7: /Mixed 12V DC / 230V AC Common Bank/12V DC 10/16A Block/MultiVibrator16A1/R2 -> /Mixed 12V DC / 230V AC Common Bank/12V DC 10/16A Block/MultiVibrator16A1/R1
- RN7004 pad 3: 12V_DC_C23_OFF -> /Mixed 12V DC / 230V AC Common Bank/12V DC 10/16A Block/DIG_ON_C3
- RN7004 pad 4: /Mixed 12V DC / 230V AC Common Bank/12V DC 10/16A Block/DIG_ON_C3 -> /Mixed 12V DC / 230V AC Common Bank/12V DC 10/16A Block/DIG_OFF_C3
- RN7004 pad 5: /Mixed 12V DC / 230V AC Common Bank/12V DC 10/16A Block/DIG_OFF_C3 -> 12V_DC_C23_OFF
- RN7004 pad 7: 12V_DC_C24_OFF -> /Mixed 12V DC / 230V AC Common Bank/12V DC 10/16A Block/DIG_ON_C4
- RN7004 pad 8: /Mixed 12V DC / 230V AC Common Bank/12V DC 10/16A Block/DIG_ON_C4 -> /Mixed 12V DC / 230V AC Common Bank/12V DC 10/16A Block/DIG_OFF_C4
- RN7004 pad 9: /Mixed 12V DC / 230V AC Common Bank/12V DC 10/16A Block/DIG_OFF_C4 -> 12V_DC_C24_OFF
- RN7901 pad 3: 230V_AC_C1_OFF -> /Mixed 12V DC / 230V AC Common Bank/230V AC 6A Block/DIG_ON_C1
- RN7901 pad 4: /Mixed 12V DC / 230V AC Common Bank/230V AC 6A Block/DIG_ON_C1 -> /Mixed 12V DC / 230V AC Common Bank/230V AC 6A Block/DIG_OFF_C1
- RN7901 pad 5: /Mixed 12V DC / 230V AC Common Bank/230V AC 6A Block/DIG_OFF_C1 -> 230V_AC_C1_OFF
- RN7901 pad 7: 230V_AC_C2_OFF -> /Mixed 12V DC / 230V AC Common Bank/230V AC 6A Block/DIG_ON_C2
- RN7901 pad 8: /Mixed 12V DC / 230V AC Common Bank/230V AC 6A Block/DIG_ON_C2 -> /Mixed 12V DC / 230V AC Common Bank/230V AC 6A Block/DIG_OFF_C2
- RN7901 pad 9: /Mixed 12V DC / 230V AC Common Bank/230V AC 6A Block/DIG_OFF_C2 -> 230V_AC_C2_OFF
- RN7903 pad 2: /Mixed 12V DC / 230V AC Common Bank/230V AC 6A Block/MultiVibrator6A1/R1 -> /Mixed 12V DC / 230V AC Common Bank/230V AC 6A Block/MultiVibrator6A2/R1
- RN7903 pad 4: /Mixed 12V DC / 230V AC Common Bank/230V AC 6A Block/MultiVibrator6A2/R1 -> /Mixed 12V DC / 230V AC Common Bank/230V AC 6A Block/MultiVibrator6A1/R1
- RN7903 pad 6: /Mixed 12V DC / 230V AC Common Bank/230V AC 6A Block/MultiVibrator6A3/R1 -> /Mixed 12V DC / 230V AC Common Bank/230V AC 6A Block/MultiVibrator6A3/R2
- RN7903 pad 7: /Mixed 12V DC / 230V AC Common Bank/230V AC 6A Block/MultiVibrator6A3/R2 -> /Mixed 12V DC / 230V AC Common Bank/230V AC 6A Block/MultiVibrator6A3/R1
- RN7904 pad 3: 230V_AC_C3_OFF -> /Mixed 12V DC / 230V AC Common Bank/230V AC 6A Block/DIG_ON_C3
- RN7904 pad 4: /Mixed 12V DC / 230V AC Common Bank/230V AC 6A Block/DIG_ON_C3 -> /Mixed 12V DC / 230V AC Common Bank/230V AC 6A Block/DIG_OFF_C3
- RN7904 pad 5: /Mixed 12V DC / 230V AC Common Bank/230V AC 6A Block/DIG_OFF_C3 -> 230V_AC_C3_OFF
- RN7904 pad 7: 230V_AC_C4_OFF -> /Mixed 12V DC / 230V AC Common Bank/230V AC 6A Block/DIG_ON_C4
- RN7904 pad 8: /Mixed 12V DC / 230V AC Common Bank/230V AC 6A Block/DIG_ON_C4 -> /Mixed 12V DC / 230V AC Common Bank/230V AC 6A Block/DIG_OFF_C4
- RN7904 pad 9: /Mixed 12V DC / 230V AC Common Bank/230V AC 6A Block/DIG_OFF_C4 -> 230V_AC_C4_OFF
Routing:
- net /Mixed 12V DC / 230V AC Common Bank/230V AC 6A Block/MultiVibrator6A1/R1: track 12.1 -> 54.5 mm
- net /Mixed 12V DC / 230V AC Common Bank/230V AC 6A Block/MultiVibrator6A1/R2: track 12.1 -> 36.0 mm
- net /Mixed 12V DC / 230V AC Common Bank/230V AC 6A Block/MultiVibrator6A4/R1: track 12.1 -> 36.0 mm
- net /Mixed 12V DC / 230V AC Common Bank/230V AC 6A Block/MultiVibrator6A4/R2: track 12.1 -> 35.5 mm
- net /Mixed 12V DC / 230V AC Common Bank/230V AC 6A Block/DIG_OFF_C3: track 0.00 -> 16.0 mm
- net /Mixed 12V DC / 230V AC Common Bank/230V AC 6A Block/DIG_OFF_C1: track 0.00 -> 16.0 mm
- net 230V_AC_C3_OFF: track 0.00 -> 16.0 mm
- net 230V_AC_C1_OFF: track 0.00 -> 16.0 mm
- net /Mixed 12V DC / 230V AC Common Bank/230V AC 6A Block/DIG_ON_C2: track 0.00 -> 15.8 mm
- net 230V_AC_C2_ON: track 0.00 -> 15.8 mm
- net 230V_AC_C4_ON: track 0.00 -> 15.8 mm
- net /Mixed 12V DC / 230V AC Common Bank/230V AC 6A Block/DIG_ON_C4: track 0.00 -> 15.8 mm
- net /Mixed 12V DC / 230V AC Common Bank/230V AC 6A Block/MultiVibrator6A3/R2: track 12.1 -> 27.3 mm
- net /Mixed 12V DC / 230V AC Common Bank/230V AC 6A Block/MultiVibrator6A2/R1: track 12.1 -> 18.3 mm
- net 230V_AC_C4_OFF: track 0.00 -> 3.56 mm
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