File: boatcontrol/MinexBlock.sch (KiCad schematic (older format))
At the start: 2 parts

Commit message: Add mixed blocks
Parts:
- removed RN?: 4116R-1-471, BoatControl:DIP254P762X432-16P, symbol Device:R_Pack08
- removed U?: ULN2803A, Package_DIP:DIP-18_W7.62mm, symbol Transistor_Array:ULN2803A
- added RN?: 4116R-1-471, BoatControl:DIP254P762X432-16P, symbol Device:R_Pack08
- added U?: ULN2803A, Package_DIP:DIP-18_W7.62mm, symbol Transistor_Array:ULN2803A
Connections:
- net +12P: now also U?.10 (COM)
- net GND: now also U?.9 (GND)
- net LOGIC_OFF_C1: now also RN?.2 (R2.1), U?.2 (I2)
- net LOGIC_OFF_C2: now also RN?.4 (R4.1), U?.4 (I4)
- net LOGIC_OFF_C3: now also RN?.6 (R6.1), U?.6 (I6)
- net LOGIC_OFF_C4: now also RN?.8 (R8.1), U?.8 (I8)
- net LOGIC_ON_C1: now also RN?.1 (R1.1), U?.1 (I1)
- net LOGIC_ON_C2: now also RN?.3 (R3.1), U?.3 (I3)
- net LOGIC_ON_C3: now also RN?.5 (R5.1), U?.5 (I5)
- net LOGIC_ON_C4: now also RN?.7 (R7.1), U?.7 (I7)
- new net 6AC1/OFF_C?: U?.17 (O2)
- new net 6AC1/OFF_LED_C?: RN?.15 (R2.2)
- new net 6AC1/ON_C?: U?.18 (O1)
- new net 6AC1/ON_LED_C?: RN?.16 (R1.2)
- new net 6AC2/OFF_C?: U?.15 (O4)
- new net 6AC2/OFF_LED_C?: RN?.13 (R4.2)
- new net 6AC2/ON_C?: U?.16 (O3)
- new net 6AC2/ON_LED_C?: RN?.14 (R3.2)
- new net 6AC3/OFF_C?: U?.13 (O6)
- new net 6AC3/OFF_LED_C?: RN?.11 (R6.2)
- new net 6AC3/ON_C?: U?.14 (O5)
- new net 6AC3/ON_LED_C?: RN?.12 (R5.2)
- new net 6AC4/OFF_C?: U?.11 (O8)
- new net 6AC4/OFF_LED_C?: RN?.9 (R8.2)
- new net 6AC4/ON_C?: U?.12 (O7)
- new net 6AC4/ON_LED_C?: RN?.10 (R7.2)
Changed lines of the file:
@@
 $Descr A4 11693 8268
 encoding utf-8
-Sheet 29 64
+Sheet 63 80
 Title ""
 Date ""
@@
 $Comp
 L Transistor_Array:ULN2803A U?
-U 1 1 81A9CC94
+U 1 1 D2F31428
 P 4000 3300
-AR Path="/81A9CC94" Ref="U?"  Part="1"
-AR Path="/8148B1BC/81A9CC94" Ref="U?"  Part="1"
-AR Path="/81CB63BE/81A9CC94" Ref="U?"  Part="1"
-AR Path="/822CFB36/81A9CC94" Ref="U?"  Part="1"
-AR Path="/828E1EFD/81A9CC94" Ref="U?"  Part="1"
-AR Path="/828E1F0F/81A9CC94" Ref="U?"  Part="1"
-AR Path="/D16552B4/D1AAA1B8/81A9CC94" Ref="U?"  Part="1"
-AR Path="/D16552B4/D1AAA1CA/81A9CC94" Ref="U?"  Part="1"
-AR Path="/D16552B4/D1AAA1DC/81A9CC94" Ref="U?"  Part="1"
-AR Path="/D16552B4/D1AAA1EE/81A9CC94" Ref="U?"  Part="1"
-AR Path="/D1BB8DB4/D1AAA1B8/81A9CC94" Ref="U?"  Part="1"
-AR Path="/D1BB8DB4/D2B4FEF5/81A9CC94" Ref="U?"  Part="1"
-AR Path="/D1BB8DB4/D2B4FEF7/81A9CC94" Ref="U?"  Part="1"
-AR Path="/E0EE2714/E1383403/E142CBAC/81A9CC94" Ref="U?"  Part="1"
-AR Path="/E0EE2714/E1383403/E142CD42/81A9CC94" Ref="U?"  Part="1"
+AR Path="/D2F31428" Ref="U?"  Part="1"
+AR Path="/8148B1BC/D2F31428" Ref="U?"  Part="1"
+AR Path="/81CB63BE/D2F31428" Ref="U?"  Part="1"
+AR Path="/822CFB36/D2F31428" Ref="U?"  Part="1"
+AR Path="/828E1EFD/D2F31428" Ref="U?"  Part="1"
+AR Path="/828E1F0F/D2F31428" Ref="U?"  Part="1"
+AR Path="/D16552B4/D1AAA1B8/D2F31428" Ref="U?"  Part="1"
+AR Path="/D16552B4/D1AAA1CA/D2F31428" Ref="U?"  Part="1"
+AR Path="/D16552B4/D1AAA1DC/D2F31428" Ref="U?"  Part="1"
+AR Path="/D16552B4/D1AAA1EE/D2F31428" Ref="U?"  Part="1"
+AR Path="/D1BB8DB4/D1AAA1B8/D2F31428" Ref="U?"  Part="1"
+AR Path="/D1BB8DB4/D2B4FEF6/D2F31428" Ref="U?"  Part="1"
+AR Path="/E0EE2714/E1383403/E142CB9A/D2F31428" Ref="U?"  Part="1"
+AR Path="/E0EE2714/E1383403/E142CD30/D2F31428" Ref="U?"  Part="1"
 F 0 "U?" H 3950 3100 50  0000 L CNN
 F 1 "ULN2803A" H 3800 3800 50  0000 L CNN
@@
 $Sheet
 S 5300 2650 1000 700
-U 81A9CCA4
-F0 "10AC2" 50
-F1 "10AmpCircuit.sch" 50
+U D2F31429
+F0 "6AC2" 50
+F1 "6AmpCircuit.sch" 50
 F2 "ON_C?" B L 5300 2750 50
 F3 "OFF_C?" B L 5300 2900 50
@@
 $EndSheet
 $Sheet
+S 5300 3550 1000 700
+U D2F3142A
+F0 "6AC3" 50
+F1 "6AmpCircuit.sch" 50
+F2 "ON_C?" B L 5300 3650 50
+F3 "OFF_C?" B L 5300 3800 50
+F4 "ON_LED_C?" I R 6300 3650 50
+F5 "OFF_LED_C?" I R 6300 3800 50
+F6 "OUT_C?" O R 6300 4150 50
+F7 "IN_C?" I L 5300 4150 50
+$EndSheet
+$Sheet
 S 5300 4450 1000 700
-U 81A9CCB4
-F0 "16AC2" 50
-F1 "16AmpCircuit.sch" 50
+U D2B5CDA6
+F0 "6AC4" 50
+F1 "6AmpCircuit.sch" 50
 F2 "ON_C?" B L 5300 4550 50
 F3 "OFF_C?" B L 5300 4700 50
@@
 $Comp
 L power:GND #PWR?
-U 1 1 81AA51E9
+U 1 1 D2B5CDA7
 P 4000 4250
-AR Path="/8148B1BC/81AA51E9" Ref="#PWR?"  Part="1"
-AR Path="/81CB63BE/81AA51E9" Ref="#PWR?"  Part="1"
-AR Path="/822CFB36/81AA51E9" Ref="#PWR?"  Part="1"
-AR Path="/828E1EFD/81AA51E9" Ref="#PWR?"  Part="1"
-AR Path="/828E1F0F/81AA51E9" Ref="#PWR?"  Part="1"
-AR Path="/D16552B4/D1AAA1B8/81AA51E9" Ref="#PWR?"  Part="1"
-AR Path="/D16552B4/D1AAA1CA/81AA51E9" Ref="#PWR?"  Part="1"
-AR Path="/D16552B4/D1AAA1DC/81AA51E9" Ref="#PWR?"  Part="1"
-AR Path="/D16552B4/D1AAA1EE/81AA51E9" Ref="#PWR?"  Part="1"
-AR Path="/D1BB8DB4/D1AAA1B8/81AA51E9" Ref="#PWR?"  Part="1"
-AR Path="/D1BB8DB4/D2B4FEF5/81AA51E9" Ref="#PWR?"  Part="1"
-AR Path="/D1BB8DB4/D2B4FEF7/81AA51E9" Ref="#PWR?"  Part="1"
-AR Path="/E0EE2714/E1383403/E142CBAC/81AA51E9" Ref="#PWR?"  Part="1"
-AR Path="/E0EE2714/E1383403/E142CD42/81AA51E9" Ref="#PWR?"  Part="1"
+AR Path="/8148B1BC/D2B5CDA7" Ref="#PWR?"  Part="1"
+AR Path="/81CB63BE/D2B5CDA7" Ref="#PWR?"  Part="1"
+AR Path="/822CFB36/D2B5CDA7" Ref="#PWR?"  Part="1"
+AR Path="/828E1EFD/D2B5CDA7" Ref="#PWR?"  Part="1"
+AR Path="/828E1F0F/D2B5CDA7" Ref="#PWR?"  Part="1"
+AR Path="/D16552B4/D1AAA1B8/D2B5CDA7" Ref="#PWR?"  Part="1"
+AR Path="/D16552B4/D1AAA1CA/D2B5CDA7" Ref="#PWR?"  Part="1"
+AR Path="/D16552B4/D1AAA1DC/D2B5CDA7" Ref="#PWR?"  Part="1"
+AR Path="/D16552B4/D1AAA1EE/D2B5CDA7" Ref="#PWR?"  Part="1"
+AR Path="/D1BB8DB4/D1AAA1B8/D2B5CDA7" Ref="#PWR?"  Part="1"
+AR Path="/D1BB8DB4/D2B4FEF6/D2B5CDA7" Ref="#PWR?"  Part="1"
+AR Path="/E0EE2714/E1383403/E142CB9A/D2B5CDA7" Ref="#PWR?"  Part="1"
+AR Path="/E0EE2714/E1383403/E142CD30/D2B5CDA7" Ref="#PWR?"  Part="1"
 F 0 "#PWR?" H 4000 4000 50  0001 C CNN
 F 1 "GND" H 4005 4077 50  0000 C CNN
@@
 $Comp
 L power:+12P #PWR?
-U 1 1 81B610D3
+U 1 1 D2B5CDA8
 P 4000 2500
-AR Path="/8148B1BC/81B610D3" Ref="#PWR?"  Part="1"
-AR Path="/81CB63BE/81B610D3" Ref="#PWR?"  Part="1"
-AR Path="/822CFB36/81B610D3" Ref="#PWR?"  Part="1"
-AR Path="/828E1EFD/81B610D3" Ref="#PWR?"  Part="1"
-AR Path="/828E1F0F/81B610D3" Ref="#PWR?"  Part="1"
-AR Path="/D16552B4/D1AAA1B8/81B610D3" Ref="#PWR?"  Part="1"
-AR Path="/D16552B4/D1AAA1CA/81B610D3" Ref="#PWR?"  Part="1"
-AR Path="/D16552B4/D1AAA1DC/81B610D3" Ref="#PWR?"  Part="1"
-AR Path="/D16552B4/D1AAA1EE/81B610D3" Ref="#PWR?"  Part="1"
-AR Path="/D1BB8DB4/D1AAA1B8/81B610D3" Ref="#PWR?"  Part="1"
-AR Path="/D1BB8DB4/D2B4FEF5/81B610D3" Ref="#PWR?"  Part="1"
-AR Path="/D1BB8DB4/D2B4FEF7/81B610D3" Ref="#PWR?"  Part="1"
-AR Path="/E0EE2714/E1383403/E142CBAC/81B610D3" Ref="#PWR?"  Part="1"
-AR Path="/E0EE2714/E1383403/E142CD42/81B610D3" Ref="#PWR?"  Part="1"
+AR Path="/8148B1BC/D2B5CDA8" Ref="#PWR?"  Part="1"
+AR Path="/81CB63BE/D2B5CDA8" Ref="#PWR?"  Part="1"
+AR Path="/822CFB36/D2B5CDA8" Ref="#PWR?"  Part="1"
+AR Path="/828E1EFD/D2B5CDA8" Ref="#PWR?"  Part="1"
+AR Path="/828E1F0F/D2B5CDA8" Ref="#PWR?"  Part="1"
+AR Path="/D16552B4/D1AAA1B8/D2B5CDA8" Ref="#PWR?"  Part="1"
+AR Path="/D16552B4/D1AAA1CA/D2B5CDA8" Ref="#PWR?"  Part="1"
+AR Path="/D16552B4/D1AAA1DC/D2B5CDA8" Ref="#PWR?"  Part="1"
+AR Path="/D16552B4/D1AAA1EE/D2B5CDA8" Ref="#PWR?"  Part="1"
+AR Path="/D1BB8DB4/D1AAA1B8/D2B5CDA8" Ref="#PWR?"  Part="1"
+AR Path="/D1BB8DB4/D2B4FEF6/D2B5CDA8" Ref="#PWR?"  Part="1"
+AR Path="/E0EE2714/E1383403/E142CB9A/D2B5CDA8" Ref="#PWR?"  Part="1"
+AR Path="/E0EE2714/E1383403/E142CD30/D2B5CDA8" Ref="#PWR?"  Part="1"
 F 0 "#PWR?" H 4000 2350 50  0001 C CNN
 F 1 "+12P" H 4015 2673 50  0000 C CNN
@@
 $Comp
 L Device:R_Pack08 RN?
-U 1 1 D2F31427
+U 1 1 D2B5CDA1
 P 7400 3500
-AR Path="/D2F31427" Ref="RN?"  Part="1"
-AR Path="/8148B1BC/D2F31427" Ref="RN?"  Part="1"
-AR Path="/81CB63BE/D2F31427" Ref="RN?"  Part="1"
-AR Path="/822CFB36/D2F31427" Ref="RN?"  Part="1"
-AR Path="/828E1EFD/D2F31427" Ref="RN?"  Part="1"
-AR Path="/828E1F0F/D2F31427" Ref="RN?"  Part="1"
-AR Path="/D16552B4/D1AAA1B8/D2F31427" Ref="RN?"  Part="1"
-AR Path="/D16552B4/D1AAA1CA/D2F31427" Ref="RN?"  Part="1"
-AR Path="/D16552B4/D1AAA1DC/D2F31427" Ref="RN?"  Part="1"
-AR Path="/D16552B4/D1AAA1EE/D2F31427" Ref="RN?"  Part="1"
-AR Path="/D1BB8DB4/D1AAA1B8/D2F31427" Ref="RN?"  Part="1"
-AR Path="/D1BB8DB4/D2B4FEF5/D2F31427" Ref="RN?"  Part="1"
-AR Path="/D1BB8DB4/D2B4FEF7/D2F31427" Ref="RN?"  Part="1"
-AR Path="/E0EE2714/E1383403/E142CBAC/D2F31427" Ref="RN?"  Part="1"
-AR Path="/E0EE2714/E1383403/E142CD42/D2F31427" Ref="RN?"  Part="1"
+AR Path="/D2B5CDA1" Ref="RN?"  Part="1"
+AR Path="/8148B1BC/D2B5CDA1" Ref="RN?"  Part="1"
+AR Path="/81CB63BE/D2B5CDA1" Ref="RN?"  Part="1"
+AR Path="/822CFB36/D2B5CDA1" Ref="RN?"  Part="1"
+AR Path="/828E1EFD/D2B5CDA1" Ref="RN?"  Part="1"
+AR Path="/828E1F0F/D2B5CDA1" Ref="RN?"  Part="1"
+AR Path="/D16552B4/D1AAA1B8/D2B5CDA1" Ref="RN?"  Part="1"
+AR Path="/D16552B4/D1AAA1CA/D2B5CDA1" Ref="RN?"  Part="1"
+AR Path="/D16552B4/D1AAA1DC/D2B5CDA1" Ref="RN?"  Part="1"
+AR Path="/D16552B4/D1AAA1EE/D2B5CDA1" Ref="RN?"  Part="1"
+AR Path="/D1BB8DB4/D1AAA1B8/D2B5CDA1" Ref="RN?"  Part="1"
+AR Path="/D1BB8DB4/D2B4FEF6/D2B5CDA1" Ref="RN?"  Part="1"
+AR Path="/E0EE2714/E1383403/E142CB9A/D2B5CDA1" Ref="RN?"  Part="1"
+AR Path="/E0EE2714/E1383403/E142CD30/D2B5CDA1" Ref="RN?"  Part="1"
 F 0 "RN?" V 7800 3425 50  0000 L CNN
 F 1 "4116R-1-471" H 7100 3050 50  0000 L CNN
@@
 $Sheet
 S 5300 1750 1000 700
-U 81A9CC9C
-F0 "10AC1" 50
-F1 "10AmpCircuit.sch" 50
+U D2F4DB5C
+F0 "6AC1" 50
+F1 "6AmpCircuit.sch" 50
 F2 "ON_C?" B L 5300 1850 50
 F3 "OFF_C?" B L 5300 2000 50
@@
 $EndSheet
 $Sheet
-S 5300 3550 1000 700
-U 81A9CCAC
-F0 "16AC1" 50
-F1 "16AmpCircuit.sch" 50
-F2 "ON_C?" B L 5300 3650 50
-F3 "OFF_C?" B L 5300 3800 50
-F4 "ON_LED_C?" I R 6300 3650 50
-F5 "OFF_LED_C?" I R 6300 3800 50
-F6 "OUT_C?" O R 6300 4150 50
-F7 "IN_C?" I L 5300 4150 50
+S 9250 1750 1100 600
+U E14BA326
+F0 "sheetE14BA31B" 50
+F1 "CircuitControl.sch" 50
+F2 "ON_LED_C?" I L 9250 2150 50
+F3 "OFF_LED_C?" I L 9250 2250 50
+F4 "ON_C?" B L 9250 1850 50
+F5 "OFF_C?" B L 9250 1950 50
+F6 "OFF_SIGNAL?" O R 10350 2000 50
+F7 "ON_SIGNAL?" O R 10350 1900 50
+$EndSheet
+$Sheet
+S 9250 2550 1100 600
+U E14BA32E
+F0 "sheetE14BA31C" 50
+F1 "CircuitControl.sch" 50
+F2 "ON_LED_C?" I L 9250 2950 50
+F3 "OFF_LED_C?" I L 9250 3050 50
+F4 "ON_C?" B L 9250 2650 50
+F5 "OFF_C?" B L 9250 2750 50
+F6 "OFF_SIGNAL?" O R 10350 2800 50
+F7 "ON_SIGNAL?" O R 10350 2700 50
+$EndSheet
+$Sheet
+S 9250 3350 1100 600
+U E14BA336
+F0 "sheetE14BA31D" 50
+F1 "CircuitControl.sch" 50
+F2 "ON_LED_C?" I L 9250 3750 50
+F3 "OFF_LED_C?" I L 9250 3850 50
+F4 "ON_C?" B L 9250 3450 50
+F5 "OFF_C?" B L 9250 3550 50
+F6 "OFF_SIGNAL?" O R 10350 3600 50
+F7 "ON_SIGNAL?" O R 10350 3500 50
+$EndSheet
+$Sheet
+S 9250 4150 1100 600
+U E14BA33E
+F0 "sheetE14BA31E" 50
+F1 "CircuitControl.sch" 50
+F2 "ON_LED_C?" I L 9250 4550 50
+F3 "OFF_LED_C?" I L 9250 4650 50
+F4 "ON_C?" B L 9250 4250 50
+F5 "OFF_C?" B L 9250 4350 50
+F6 "OFF_SIGNAL?" O R 10350 4400 50
+F7 "ON_SIGNAL?" O R 10350 4300 50
 $EndSheet
 $EndSCHEMATC
