File: boatcontrol/MixedBlock.sch (KiCad schematic (older format))
At the start: 2 parts, among them U22 ULN2803A

Commit message: Start re-routing PCB
Parts:
- renumbered RN17 to RN9, U22 to U16
Changed lines of the file:
@@
 AR Path="/E0EE2714/E1383403/E142CD30/D2F31428" Ref="U?"  Part="1"
 AR Path="/E0EE2714/E1383403/E15855D9/D2F31428" Ref="U?"  Part="1"
-AR Path="/E171B33C/E142CD30/D2F31428" Ref="U22"  Part="1"
-AR Path="/E171B33C/E15855D9/D2F31428" Ref="U23"  Part="1"
-F 0 "U22" H 3950 3100 50  0000 L CNN
+AR Path="/E171B33C/E142CD30/D2F31428" Ref="U16"  Part="1"
+AR Path="/E171B33C/E15855D9/D2F31428" Ref="U17"  Part="1"
+F 0 "U17" H 3950 3100 50  0000 L CNN
 F 1 "ULN2803A" H 3800 3800 50  0000 L CNN
 F 2 "Package_DIP:DIP-18_W7.62mm" H 4050 2650 50  0001 L CNN
@@
 AR Path="/E0EE2714/E1383403/E142CD30/5F29B0EF" Ref="#PWR?"  Part="1"
 AR Path="/E0EE2714/E1383403/E15855D9/5F29B0EF" Ref="#PWR?"  Part="1"
-AR Path="/E171B33C/E142CD30/5F29B0EF" Ref="#PWR0134"  Part="1"
-AR Path="/E171B33C/E15855D9/5F29B0EF" Ref="#PWR0140"  Part="1"
-F 0 "#PWR0140" H 4000 4000 50  0001 C CNN
+AR Path="/E171B33C/E142CD30/5F29B0EF" Ref="#PWR084"  Part="1"
+AR Path="/E171B33C/E15855D9/5F29B0EF" Ref="#PWR094"  Part="1"
+F 0 "#PWR094" H 4000 4000 50  0001 C CNN
 F 1 "GND" H 4005 4077 50  0000 C CNN
 F 2 "" H 4000 4250 50  0001 C CNN
@@
 AR Path="/E0EE2714/E1383403/E142CD30/D2B5CDA8" Ref="#PWR?"  Part="1"
 AR Path="/E0EE2714/E1383403/E15855D9/D2B5CDA8" Ref="#PWR?"  Part="1"
-AR Path="/E171B33C/E142CD30/D2B5CDA8" Ref="#PWR0133"  Part="1"
-AR Path="/E171B33C/E15855D9/D2B5CDA8" Ref="#PWR0139"  Part="1"
-F 0 "#PWR0139" H 4000 2350 50  0001 C CNN
+AR Path="/E171B33C/E142CD30/D2B5CDA8" Ref="#PWR083"  Part="1"
+AR Path="/E171B33C/E15855D9/D2B5CDA8" Ref="#PWR093"  Part="1"
+F 0 "#PWR093" H 4000 2350 50  0001 C CNN
 F 1 "+12P" H 4015 2673 50  0000 C CNN
 F 2 "" H 4000 2500 50  0001 C CNN
@@
 AR Path="/E0EE2714/E1383403/E142CD30/D2B5CDA1" Ref="RN?"  Part="1"
 AR Path="/E0EE2714/E1383403/E15855D9/D2B5CDA1" Ref="RN?"  Part="1"
-AR Path="/E171B33C/E142CD30/D2B5CDA1" Ref="RN17"  Part="1"
-AR Path="/E171B33C/E15855D9/D2B5CDA1" Ref="RN18"  Part="1"
-F 0 "RN17" V 7800 3425 50  0000 L CNN
+AR Path="/E171B33C/E142CD30/D2B5CDA1" Ref="RN9"  Part="1"
+AR Path="/E171B33C/E15855D9/D2B5CDA1" Ref="RN10"  Part="1"
+F 0 "RN10" V 7800 3425 50  0000 L CNN
 F 1 "4116R-1-471" H 7100 3050 50  0000 L CNN
 F 2 "BoatControl:DIP254P762X432-16P" V 7875 3500 50  0001 C CNN
