File: boatcontrol/MixedControl.sch (KiCad schematic (older format))
At the start: 8 parts

Commit message: Refactor Mixed Control
Parts:
- removed J?: TBP01R2W-508-08BE, CUI_TBP01R2W-508-08BE, symbol BoatControl:TBP01R2W-508-08BE
- added H? (x4): MountingHole, MountingHole:MountingHole_3mm, symbol Mechanical:MountingHole
- added J?: Conn_02x20_Odd_Even Socket, Connector_PinHeader_2.54mm:PinHeader_2x20_P2.54mm_Vertical, symbol Connector_Generic:Conn_02x20_Odd_Even
Connections:
- wire segments 95 -> 138

Commit message: Refactored
Connections:
- net MixedBlock1/LOGIC_OFF_C1 renamed IND_C1_OFF
- net MixedBlock1/LOGIC_OFF_C2 renamed IND_C2_OFF
- net MixedBlock1/LOGIC_OFF_C3 renamed IND_C3_OFF
- net MixedBlock1/LOGIC_OFF_C4 renamed IND_C4_OFF
- net MixedBlock1/LOGIC_ON_C1 renamed IND_C1_ON
- net MixedBlock1/LOGIC_ON_C2 renamed IND_C2_ON
- net MixedBlock1/LOGIC_ON_C3 renamed IND_C3_ON
- net MixedBlock1/LOGIC_ON_C4 renamed IND_C4_ON
- net MixedBlock2/LOGIC_OFF_C1 renamed IND_C5_OFF
- net MixedBlock2/LOGIC_OFF_C2 renamed IND_C6_OFF
- net MixedBlock2/LOGIC_OFF_C3 renamed IND_C7_OFF
- net MixedBlock2/LOGIC_OFF_C4 renamed IND_C8_OFF
- net MixedBlock2/LOGIC_ON_C1 renamed IND_C5_ON
- net MixedBlock2/LOGIC_ON_C2 renamed IND_C6_ON
- net MixedBlock2/LOGIC_ON_C3 renamed IND_C7_ON
- net MixedBlock2/LOGIC_ON_C4 renamed IND_C8_ON
Other:
- moved on the sheet: J?, JP?, U?

Commit message: Fix bugs
Parts:
- gave numbers to parts that had none: 12
Connections:
- net GND: now also J31.18 (Pin_18)
- net at U21.18 (~RESET~): now also JP27.1
Changed lines of the file:
@@
 $Descr A4 11693 8268
 encoding utf-8
-Sheet 45 55
+Sheet 24 55
 Title ""
 Date ""
@@
 AR Path="/D1BB8DB4/E142CB7C" Ref="U?"  Part="1"
 AR Path="/E0EE2714/E1383403/E142CB7C" Ref="U?"  Part="1"
-AR Path="/E171B33C/E142CB7C" Ref="U?"  Part="1"
-F 0 "U?" V 4000 3750 50  0000 L CNN
+AR Path="/E171B33C/E142CB7C" Ref="U21"  Part="1"
+F 0 "U21" V 4000 3750 50  0000 L CNN
 F 1 "MCP23017-E/SP" V 3900 3550 50  0000 L CNN
 F 2 "Package_DIP:DIP-28_W7.62mm" H 4150 2850 50  0001 L CNN
@@
 AR Path="/D1BB8DB4/E142CC74" Ref="JP?"  Part="1"
 AR Path="/E0EE2714/E1383403/E142CC74" Ref="JP?"  Part="1"
-AR Path="/E171B33C/E142CC74" Ref="JP?"  Part="1"
-F 0 "JP?" H 3000 4000 50  0000 C CNN
+AR Path="/E171B33C/E142CC74" Ref="JP27"  Part="1"
+F 0 "JP27" H 3000 4000 50  0000 C CNN
 F 1 "Jumper_NO_Small" H 3050 3850 50  0001 C CNN
 F 2 "Connector_PinHeader_2.54mm:PinHeader_1x01_P2.54mm_Vertical" H 3000 3950 50  0001 C CNN
@@
 AR Path="/D1BB8DB4/E142CC7A" Ref="J?"  Part="1"
 AR Path="/E0EE2714/E1383403/E142CC7A" Ref="J?"  Part="1"
-AR Path="/E171B33C/E142CC7A" Ref="J?"  Part="1"
-F 0 "J?" H 2872 3682 50  0000 R CNN
+AR Path="/E171B33C/E142CC7A" Ref="J30"  Part="1"
+F 0 "J30" H 2872 3682 50  0000 R CNN
 F 1 "Conn_01x01_Male" H 2872 3773 50  0001 R CNN
 F 2 "Connector_PinHeader_2.54mm:PinHeader_1x01_P2.54mm_Vertical" H 2900 3750 50  0001 C CNN
@@
 AR Path="/D1BB8DB4/E142CC81" Ref="JP?"  Part="1"
 AR Path="/E0EE2714/E1383403/E142CC81" Ref="JP?"  Part="1"
-AR Path="/E171B33C/E142CC81" Ref="JP?"  Part="1"
-F 0 "JP?" H 2950 4400 50  0000 C CNN
+AR Path="/E171B33C/E142CC81" Ref="JP26"  Part="1"
+F 0 "JP26" H 2950 4400 50  0000 C CNN
 F 1 "SolderJumper_3_Open" V 2800 4750 50  0001 C CNN
 F 2 "Jumper:SolderJumper-3_P1.3mm_Open_RoundedPad1.0x1.5mm_NumberLabels" H 2950 4300 50  0001 C CNN
@@
 AR Path="/D1BB8DB4/E142CC87" Ref="JP?"  Part="1"
 AR Path="/E0EE2714/E1383403/E142CC87" Ref="JP?"  Part="1"
-AR Path="/E171B33C/E142CC87" Ref="JP?"  Part="1"
-F 0 "JP?" H 2400 4500 50  0000 C CNN
+AR Path="/E171B33C/E142CC87" Ref="JP25"  Part="1"
+F 0 "JP25" H 2400 4500 50  0000 C CNN
 F 1 "SolderJumper_3_Open" V 2250 4850 50  0001 C CNN
 F 2 "Jumper:SolderJumper-3_P1.3mm_Open_RoundedPad1.0x1.5mm_NumberLabels" H 2400 4400 50  0001 C CNN
@@
 AR Path="/D1BB8DB4/E142CC8D" Ref="JP?"  Part="1"
 AR Path="/E0EE2714/E1383403/E142CC8D" Ref="JP?"  Part="1"
-AR Path="/E171B33C/E142CC8D" Ref="JP?"  Part="1"
-F 0 "JP?" H 1900 4600 50  0000 C CNN
+AR Path="/E171B33C/E142CC8D" Ref="JP24"  Part="1"
+F 0 "JP24" H 1900 4600 50  0000 C CNN
 F 1 "SolderJumper_3_Open" V 1750 4950 50  0001 C CNN
 F 2 "Jumper:SolderJumper-3_P1.3mm_Open_RoundedPad1.0x1.5mm_NumberLabels" H 1900 4500 50  0001 C CNN
@@
 AR Path="/D1BB8DB4/E142CC93" Ref="J?"  Part="1"
 AR Path="/E0EE2714/E1383403/E142CC93" Ref="J?"  Part="1"
-AR Path="/E171B33C/E142CC93" Ref="J?"  Part="1"
-F 0 "J?" H 2872 3582 50  0000 R CNN
+AR Path="/E171B33C/E142CC93" Ref="J29"  Part="1"
+F 0 "J29" H 2872 3582 50  0000 R CNN
 F 1 "Conn_01x01_Male" H 2872 3673 50  0001 R CNN
 F 2 "Connector_PinHeader_2.54mm:PinHeader_1x01_P2.54mm_Vertical" H 2900 3650 50  0001 C CNN
@@
 AR Path="/D1BB8DB4/E142CCB8" Ref="#PWR?"  Part="1"
 AR Path="/E0EE2714/E1383403/E142CCB8" Ref="#PWR?"  Part="1"
-AR Path="/E171B33C/E142CCB8" Ref="#PWR?"  Part="1"
-F 0 "#PWR?" H 3950 4700 50  0001 C CNN
+AR Path="/E171B33C/E142CCB8" Ref="#PWR0131"  Part="1"
+F 0 "#PWR0131" H 3950 4700 50  0001 C CNN
 F 1 "GND" H 4100 4900 50  0000 C CNN
 F 2 "" H 3950 4950 50  0001 C CNN
@@
 AR Path="/D1BB8DB4/E142CCC5" Ref="#PWR?"  Part="1"
 AR Path="/E0EE2714/E1383403/E142CCC5" Ref="#PWR?"  Part="1"
-AR Path="/E171B33C/E142CCC5" Ref="#PWR?"  Part="1"
-F 0 "#PWR?" H 3950 2600 50  0001 C CNN
+AR Path="/E171B33C/E142CCC5" Ref="#PWR0130"  Part="1"
+F 0 "#PWR0130" H 3950 2600 50  0001 C CNN
 F 1 "+5V" H 4100 2800 50  0000 C CNN
 F 2 "" H 3950 2750 50  0001 C CNN
@@
 	1    0    0    -1
 $EndComp
-Text HLabel 3250 3050 0    50   Output ~ 0
-SDA
-Text HLabel 3250 3150 0    50   Output ~ 0
-SCK
 Connection ~ 3950 4950
 $Sheet
@@
 AR Path="/E0EE2714/E15696A6" Ref="H?"  Part="1"
 AR Path="/E0EE2714/E1383403/E15696A6" Ref="H?"  Part="1"
-AR Path="/E171B33C/E15696A6" Ref="H?"  Part="1"
-F 0 "H?" H 9700 3800 50  0000 L CNN
+AR Path="/E171B33C/E15696A6" Ref="H29"  Part="1"
+F 0 "H29" H 9700 3800 50  0000 L CNN
 F 1 "MountingHole" V 9750 3750 50  0001 L CNN
 F 2 "MountingHole:MountingHole_3mm" H 9750 3650 50  0001 C CNN
@@
 AR Path="/E0EE2714/E15696A0" Ref="H?"  Part="1"
 AR Path="/E0EE2714/E1383403/E15696A0" Ref="H?"  Part="1"
-AR Path="/E171B33C/E15696A0" Ref="H?"  Part="1"
-F 0 "H?" H 9700 3850 50  0000 L CNN
+AR Path="/E171B33C/E15696A0" Ref="H30"  Part="1"
+F 0 "H30" H 9700 3850 50  0000 L CNN
 F 1 "MountingHole" H 9850 3955 50  0001 L CNN
 F 2 "MountingHole:MountingHole_3mm" H 9750 4000 50  0001 C CNN
@@
 AR Path="/E0EE2714/E156969A" Ref="J?"  Part="1"
 AR Path="/E0EE2714/E1383403/E156969A" Ref="J?"  Part="1"
-AR Path="/E171B33C/E156969A" Ref="J?"  Part="1"
-F 0 "J?" V 8600 4900 50  0000 R CNN
+AR Path="/E171B33C/E156969A" Ref="J31"  Part="1"
+F 0 "J31" V 8600 4900 50  0000 R CNN
 F 1 "Conn_02x20_Odd_Even Socket" V 8600 4200 50  0000 R CNN
 F 2 "Connector_PinHeader_2.54mm:PinHeader_2x20_P2.54mm_Vertical" H 8550 3800 50  0001 C CNN
@@
 AR Path="/E0EE2714/E15696AC" Ref="H?"  Part="1"
 AR Path="/E0EE2714/E1383403/E15696AC" Ref="H?"  Part="1"
-AR Path="/E171B33C/E15696AC" Ref="H?"  Part="1"
-F 0 "H?" V 7600 3600 50  0000 L CNN
+AR Path="/E171B33C/E15696AC" Ref="H27"  Part="1"
+F 0 "H27" V 7600 3600 50  0000 L CNN
 F 1 "MountingHole" H 7550 3605 50  0001 L CNN
 F 2 "MountingHole:MountingHole_3mm" H 7450 3650 50  0001 C CNN
@@
 AR Path="/E0EE2714/E15696B2" Ref="H?"  Part="1"
 AR Path="/E0EE2714/E1383403/E15696B2" Ref="H?"  Part="1"
-AR Path="/E171B33C/E15696B2" Ref="H?"  Part="1"
-F 0 "H?" V 7300 3950 50  0000 L CNN
+AR Path="/E171B33C/E15696B2" Ref="H28"  Part="1"
+F 0 "H28" V 7300 3950 50  0000 L CNN
 F 1 "MountingHole" H 7550 3955 50  0001 L CNN
 F 2 "MountingHole:MountingHole_3mm" H 7450 4000 50  0001 C CNN
@@
 P 9650 3850
 AR Path="/E0EE2714/E1383403/E16C27B4" Ref="#PWR?"  Part="1"
-AR Path="/E171B33C/E16C27B4" Ref="#PWR?"  Part="1"
-F 0 "#PWR?" H 9650 3600 50  0001 C CNN
+AR Path="/E171B33C/E16C27B4" Ref="#PWR0132"  Part="1"
+F 0 "#PWR0132" H 9650 3600 50  0001 C CNN
 F 1 "GND" V 9650 3750 50  0000 R CNN
 F 2 "" H 9650 3850 50  0001 C CNN
@@
 Text GLabel 4850 5300 2    50   Input ~ 0
 IND_C8_OFF
+Text GLabel 3250 3050 0    50   Input ~ 0
+SDA
+Text GLabel 3250 3150 0    50   Input ~ 0
+SCK
+Wire Wire Line
+	8550 4100 8450 4100
+Connection ~ 8550 4100
+Wire Wire Line
+	3250 3950 3100 3950
 $EndSCHEMATC

Commit message: Error Free
Parts:
- JP27: footprint Connector_PinHeader_2.54mm:PinHeader_1x01_P2.54mm_Vertical -> Connector_PinHeader_2.54mm:PinHeader_1x02_P2.54mm_Vertical
Changed lines of the file:
@@
 AR Path="/E0EE2714/E1383403/E142CC74" Ref="JP?"  Part="1"
 AR Path="/E171B33C/E142CC74" Ref="JP27"  Part="1"
-F 0 "JP27" H 3000 4000 50  0000 C CNN
+F 0 "JP27" H 3000 4050 50  0000 C CNN
 F 1 "Jumper_NO_Small" H 3050 3850 50  0001 C CNN
-F 2 "Connector_PinHeader_2.54mm:PinHeader_1x01_P2.54mm_Vertical" H 3000 3950 50  0001 C CNN
+F 2 "Connector_PinHeader_2.54mm:PinHeader_1x02_P2.54mm_Vertical" H 3000 3950 50  0001 C CNN
 F 3 "~" H 3000 3950 50  0001 C CNN
 	1    3000 3950
@@
 AR Path="/E0EE2714/E1383403/E142CC7A" Ref="J?"  Part="1"
 AR Path="/E171B33C/E142CC7A" Ref="J30"  Part="1"
-F 0 "J30" H 2872 3682 50  0000 R CNN
+F 0 "J30" H 2950 3800 50  0000 R CNN
 F 1 "Conn_01x01_Male" H 2872 3773 50  0001 R CNN
 F 2 "Connector_PinHeader_2.54mm:PinHeader_1x01_P2.54mm_Vertical" H 2900 3750 50  0001 C CNN
@@
 AR Path="/E0EE2714/E1383403/E142CC93" Ref="J?"  Part="1"
 AR Path="/E171B33C/E142CC93" Ref="J29"  Part="1"
-F 0 "J29" H 2872 3582 50  0000 R CNN
+F 0 "J29" H 2950 3700 50  0000 R CNN
 F 1 "Conn_01x01_Male" H 2872 3673 50  0001 R CNN
 F 2 "Connector_PinHeader_2.54mm:PinHeader_1x01_P2.54mm_Vertical" H 2900 3650 50  0001 C CNN
@@
 Wire Wire Line
 	3250 3950 3100 3950
+Connection ~ 3050 4100
 $EndSCHEMATC

Commit message: Start re-routing PCB
Parts:
- renumbered J29 to J21, J30 to J22, J31 to J23, JP24 to JP16, JP25 to JP17, JP26 to JP18, JP27 to JP19, U21 to U15
Changed lines of the file:
@@
 AR Path="/D1BB8DB4/E142CB7C" Ref="U?"  Part="1"
 AR Path="/E0EE2714/E1383403/E142CB7C" Ref="U?"  Part="1"
-AR Path="/E171B33C/E142CB7C" Ref="U21"  Part="1"
-F 0 "U21" V 4000 3750 50  0000 L CNN
+AR Path="/E171B33C/E142CB7C" Ref="U15"  Part="1"
+F 0 "U15" V 4000 3750 50  0000 L CNN
 F 1 "MCP23017-E/SP" V 3900 3550 50  0000 L CNN
 F 2 "Package_DIP:DIP-28_W7.62mm" H 4150 2850 50  0001 L CNN
@@
 AR Path="/D1BB8DB4/E142CC74" Ref="JP?"  Part="1"
 AR Path="/E0EE2714/E1383403/E142CC74" Ref="JP?"  Part="1"
-AR Path="/E171B33C/E142CC74" Ref="JP27"  Part="1"
-F 0 "JP27" H 3000 4050 50  0000 C CNN
+AR Path="/E171B33C/E142CC74" Ref="JP19"  Part="1"
+F 0 "JP19" H 3000 4050 50  0000 C CNN
 F 1 "Jumper_NO_Small" H 3050 3850 50  0001 C CNN
 F 2 "Connector_PinHeader_2.54mm:PinHeader_1x02_P2.54mm_Vertical" H 3000 3950 50  0001 C CNN
@@
 AR Path="/D1BB8DB4/E142CC7A" Ref="J?"  Part="1"
 AR Path="/E0EE2714/E1383403/E142CC7A" Ref="J?"  Part="1"
-AR Path="/E171B33C/E142CC7A" Ref="J30"  Part="1"
-F 0 "J30" H 2950 3800 50  0000 R CNN
+AR Path="/E171B33C/E142CC7A" Ref="J22"  Part="1"
+F 0 "J22" H 2950 3800 50  0000 R CNN
 F 1 "Conn_01x01_Male" H 2872 3773 50  0001 R CNN
 F 2 "Connector_PinHeader_2.54mm:PinHeader_1x01_P2.54mm_Vertical" H 2900 3750 50  0001 C CNN
@@
 AR Path="/D1BB8DB4/E142CC81" Ref="JP?"  Part="1"
 AR Path="/E0EE2714/E1383403/E142CC81" Ref="JP?"  Part="1"
-AR Path="/E171B33C/E142CC81" Ref="JP26"  Part="1"
-F 0 "JP26" H 2950 4400 50  0000 C CNN
+AR Path="/E171B33C/E142CC81" Ref="JP18"  Part="1"
+F 0 "JP18" H 2950 4400 50  0000 C CNN
 F 1 "SolderJumper_3_Open" V 2800 4750 50  0001 C CNN
 F 2 "Jumper:SolderJumper-3_P1.3mm_Open_RoundedPad1.0x1.5mm_NumberLabels" H 2950 4300 50  0001 C CNN
@@
 AR Path="/D1BB8DB4/E142CC87" Ref="JP?"  Part="1"
 AR Path="/E0EE2714/E1383403/E142CC87" Ref="JP?"  Part="1"
-AR Path="/E171B33C/E142CC87" Ref="JP25"  Part="1"
-F 0 "JP25" H 2400 4500 50  0000 C CNN
+AR Path="/E171B33C/E142CC87" Ref="JP17"  Part="1"
+F 0 "JP17" H 2400 4500 50  0000 C CNN
 F 1 "SolderJumper_3_Open" V 2250 4850 50  0001 C CNN
 F 2 "Jumper:SolderJumper-3_P1.3mm_Open_RoundedPad1.0x1.5mm_NumberLabels" H 2400 4400 50  0001 C CNN
@@
 AR Path="/D1BB8DB4/E142CC8D" Ref="JP?"  Part="1"
 AR Path="/E0EE2714/E1383403/E142CC8D" Ref="JP?"  Part="1"
-AR Path="/E171B33C/E142CC8D" Ref="JP24"  Part="1"
-F 0 "JP24" H 1900 4600 50  0000 C CNN
+AR Path="/E171B33C/E142CC8D" Ref="JP16"  Part="1"
+F 0 "JP16" H 1900 4600 50  0000 C CNN
 F 1 "SolderJumper_3_Open" V 1750 4950 50  0001 C CNN
 F 2 "Jumper:SolderJumper-3_P1.3mm_Open_RoundedPad1.0x1.5mm_NumberLabels" H 1900 4500 50  0001 C CNN
@@
 AR Path="/D1BB8DB4/E142CC93" Ref="J?"  Part="1"
 AR Path="/E0EE2714/E1383403/E142CC93" Ref="J?"  Part="1"
-AR Path="/E171B33C/E142CC93" Ref="J29"  Part="1"
-F 0 "J29" H 2950 3700 50  0000 R CNN
+AR Path="/E171B33C/E142CC93" Ref="J21"  Part="1"
+F 0 "J21" H 2950 3700 50  0000 R CNN
 F 1 "Conn_01x01_Male" H 2872 3673 50  0001 R CNN
 F 2 "Connector_PinHeader_2.54mm:PinHeader_1x01_P2.54mm_Vertical" H 2900 3650 50  0001 C CNN
@@
 AR Path="/D1BB8DB4/E142CCB8" Ref="#PWR?"  Part="1"
 AR Path="/E0EE2714/E1383403/E142CCB8" Ref="#PWR?"  Part="1"
-AR Path="/E171B33C/E142CCB8" Ref="#PWR0131"  Part="1"
-F 0 "#PWR0131" H 3950 4700 50  0001 C CNN
+AR Path="/E171B33C/E142CCB8" Ref="#PWR081"  Part="1"
+F 0 "#PWR081" H 3950 4700 50  0001 C CNN
 F 1 "GND" H 4100 4900 50  0000 C CNN
 F 2 "" H 3950 4950 50  0001 C CNN
@@
 AR Path="/D1BB8DB4/E142CCC5" Ref="#PWR?"  Part="1"
 AR Path="/E0EE2714/E1383403/E142CCC5" Ref="#PWR?"  Part="1"
-AR Path="/E171B33C/E142CCC5" Ref="#PWR0130"  Part="1"
-F 0 "#PWR0130" H 3950 2600 50  0001 C CNN
+AR Path="/E171B33C/E142CCC5" Ref="#PWR080"  Part="1"
+F 0 "#PWR080" H 3950 2600 50  0001 C CNN
 F 1 "+5V" H 4100 2800 50  0000 C CNN
 F 2 "" H 3950 2750 50  0001 C CNN
@@
 AR Path="/E0EE2714/E156969A" Ref="J?"  Part="1"
 AR Path="/E0EE2714/E1383403/E156969A" Ref="J?"  Part="1"
-AR Path="/E171B33C/E156969A" Ref="J31"  Part="1"
-F 0 "J31" V 8600 4900 50  0000 R CNN
+AR Path="/E171B33C/E156969A" Ref="J23"  Part="1"
+F 0 "J23" V 8600 4900 50  0000 R CNN
 F 1 "Conn_02x20_Odd_Even Socket" V 8600 4200 50  0000 R CNN
 F 2 "Connector_PinHeader_2.54mm:PinHeader_2x20_P2.54mm_Vertical" H 8550 3800 50  0001 C CNN
@@
 P 9650 3850
 AR Path="/E0EE2714/E1383403/E16C27B4" Ref="#PWR?"  Part="1"
-AR Path="/E171B33C/E16C27B4" Ref="#PWR0132"  Part="1"
-F 0 "#PWR0132" H 9650 3600 50  0001 C CNN
+AR Path="/E171B33C/E16C27B4" Ref="#PWR082"  Part="1"
+F 0 "#PWR082" H 9650 3600 50  0001 C CNN
 F 1 "GND" V 9650 3750 50  0000 R CNN
 F 2 "" H 9650 3850 50  0001 C CNN
