File: boatcontrol/RelayBoard.sch (KiCad schematic (older format))
At the start: 15 parts, among them J18 Conn_02x20_Odd_Even Header, J19 TBL008V-1000-08BE, J20 TBL008V-1000-08BE, K17 EW60-1A3-CL12D04, K18 EW60-1A3-CL12D04, K19 EW60-1A3-CL12D04, K20 EW60-1A3-CL12D04, K21 EW60-1A3-CL12D04, K22 EW60-1A3-CL12D04, K23 EW60-1A3-CL12D04, K24 EW60-1A3-CL12D04

Commit message: Before starting the PCB fresh
Parts:
- renumbered H23 to H2301, H24 to H2302, H25 to H2303, H26 to H2304, J18 to J2301, J19 to J2302, J20 to J2303, K17 to K2301, K18 to K2302, K19 to K2303, K20 to K2304, K21 to K2305, K22 to K2306, K23 to K2307, K24 to K2308
Changed lines of the file:
@@
 AR Path="/E1098DA6" Ref="#PWR?"  Part="1"
 AR Path="/E0EE2714/E107FCD3/E1098DA6" Ref="#PWR?"  Part="1"
-AR Path="/E171B338/E1098DA6" Ref="#PWR072"  Part="1"
-F 0 "#PWR072" H 3200 3800 50  0001 C CNN
+AR Path="/E171B338/E1098DA6" Ref="#PWR02301"  Part="1"
+F 0 "#PWR02301" H 3200 3800 50  0001 C CNN
 F 1 "GND" H 3400 4050 50  0000 R CNN
 F 2 "" H 3200 4050 50  0001 C CNN
@@
 AR Path="/E1098DAC" Ref="#PWR?"  Part="1"
 AR Path="/E0EE2714/E107FCD3/E1098DAC" Ref="#PWR?"  Part="1"
-AR Path="/E171B338/E1098DAC" Ref="#PWR073"  Part="1"
-F 0 "#PWR073" H 4250 3800 50  0001 C CNN
+AR Path="/E171B338/E1098DAC" Ref="#PWR02302"  Part="1"
+F 0 "#PWR02302" H 4250 3800 50  0001 C CNN
 F 1 "GND" H 4450 4050 50  0000 R CNN
 F 2 "" H 4250 4050 50  0001 C CNN
@@
 AR Path="/E1098DB2" Ref="#PWR?"  Part="1"
 AR Path="/E0EE2714/E107FCD3/E1098DB2" Ref="#PWR?"  Part="1"
-AR Path="/E171B338/E1098DB2" Ref="#PWR074"  Part="1"
-F 0 "#PWR074" H 5300 3800 50  0001 C CNN
+AR Path="/E171B338/E1098DB2" Ref="#PWR02303"  Part="1"
+F 0 "#PWR02303" H 5300 3800 50  0001 C CNN
 F 1 "GND" H 5500 4050 50  0000 R CNN
 F 2 "" H 5300 4050 50  0001 C CNN
@@
 AR Path="/E1098DB8" Ref="#PWR?"  Part="1"
 AR Path="/E0EE2714/E107FCD3/E1098DB8" Ref="#PWR?"  Part="1"
-AR Path="/E171B338/E1098DB8" Ref="#PWR075"  Part="1"
-F 0 "#PWR075" H 6350 3800 50  0001 C CNN
+AR Path="/E171B338/E1098DB8" Ref="#PWR02304"  Part="1"
+F 0 "#PWR02304" H 6350 3800 50  0001 C CNN
 F 1 "GND" H 6550 4050 50  0000 R CNN
 F 2 "" H 6350 4050 50  0001 C CNN
@@
 AR Path="/E1098DC4" Ref="#PWR?"  Part="1"
 AR Path="/E0EE2714/E107FCD3/E1098DC4" Ref="#PWR?"  Part="1"
-AR Path="/E171B338/E1098DC4" Ref="#PWR077"  Part="1"
-F 0 "#PWR077" H 8450 3800 50  0001 C CNN
+AR Path="/E171B338/E1098DC4" Ref="#PWR02306"  Part="1"
+F 0 "#PWR02306" H 8450 3800 50  0001 C CNN
 F 1 "GND" H 8650 4050 50  0000 R CNN
 F 2 "" H 8450 4050 50  0001 C CNN
@@
 AR Path="/E1098DCA" Ref="#PWR?"  Part="1"
 AR Path="/E0EE2714/E107FCD3/E1098DCA" Ref="#PWR?"  Part="1"
-AR Path="/E171B338/E1098DCA" Ref="#PWR078"  Part="1"
-F 0 "#PWR078" H 9500 3800 50  0001 C CNN
+AR Path="/E171B338/E1098DCA" Ref="#PWR02307"  Part="1"
+F 0 "#PWR02307" H 9500 3800 50  0001 C CNN
 F 1 "GND" H 9700 4050 50  0000 R CNN
 F 2 "" H 9500 4050 50  0001 C CNN
@@
 AR Path="/E1098DD0" Ref="#PWR?"  Part="1"
 AR Path="/E0EE2714/E107FCD3/E1098DD0" Ref="#PWR?"  Part="1"
-AR Path="/E171B338/E1098DD0" Ref="#PWR079"  Part="1"
-F 0 "#PWR079" H 10550 3800 50  0001 C CNN
+AR Path="/E171B338/E1098DD0" Ref="#PWR02308"  Part="1"
+F 0 "#PWR02308" H 10550 3800 50  0001 C CNN
 F 1 "GND" H 10750 4050 50  0000 R CNN
 F 2 "" H 10550 4050 50  0001 C CNN
@@
 AR Path="/E1098DD9" Ref="J?"  Part="1"
 AR Path="/E0EE2714/E107FCD3/E1098DD9" Ref="J?"  Part="1"
-AR Path="/E171B338/E1098DD9" Ref="J20"  Part="1"
-F 0 "J20" V 7146 4922 50  0000 R CNN
+AR Path="/E171B338/E1098DD9" Ref="J2303"  Part="1"
+F 0 "J2303" V 7146 4922 50  0000 R CNN
 F 1 "TBL008V-1000-08BE" V 7400 5800 50  0000 R CNN
 F 2 "CUI_TBL008V-1000-08BE" H 7300 5350 50  0001 L BNN
@@
 AR Path="/E1098DE2" Ref="J?"  Part="1"
 AR Path="/E0EE2714/E107FCD3/E1098DE2" Ref="J?"  Part="1"
-AR Path="/E171B338/E1098DE2" Ref="J19"  Part="1"
-F 0 "J19" V 7146 2372 50  0000 R CNN
+AR Path="/E171B338/E1098DE2" Ref="J2302"  Part="1"
+F 0 "J2302" V 7146 2372 50  0000 R CNN
 F 1 "TBL008V-1000-08BE" V 7400 3250 50  0000 R CNN
 F 2 "CUI_TBL008V-1000-08BE" H 7300 2800 50  0001 L BNN
@@
 AR Path="/E1098DE8" Ref="K?"  Part="1"
 AR Path="/E0EE2714/E107FCD3/E1098DE8" Ref="K?"  Part="1"
-AR Path="/E171B338/E1098DE8" Ref="K18"  Part="1"
-F 0 "K18" V 4800 3850 50  0000 L CNN
+AR Path="/E171B338/E1098DE8" Ref="K2302"  Part="1"
+F 0 "K2302" V 4800 3850 50  0000 L CNN
 F 1 "EW60-1A3-CL12D04" V 4550 3600 50  0000 L CNN
 F 2 "BoatControl:TE_2071366-2" H 4750 4400 50  0001 L BNN
@@
 AR Path="/E1098DEE" Ref="K?"  Part="1"
 AR Path="/E0EE2714/E107FCD3/E1098DEE" Ref="K?"  Part="1"
-AR Path="/E171B338/E1098DEE" Ref="K19"  Part="1"
-F 0 "K19" V 5850 3850 50  0000 L CNN
+AR Path="/E171B338/E1098DEE" Ref="K2303"  Part="1"
+F 0 "K2303" V 5850 3850 50  0000 L CNN
 F 1 "EW60-1A3-CL12D04" V 5600 3600 50  0000 L CNN
 F 2 "BoatControl:TE_2071366-2" H 5800 4400 50  0001 L BNN
@@
 AR Path="/E1098DF4" Ref="K?"  Part="1"
 AR Path="/E0EE2714/E107FCD3/E1098DF4" Ref="K?"  Part="1"
-AR Path="/E171B338/E1098DF4" Ref="K20"  Part="1"
-F 0 "K20" V 6900 3850 50  0000 L CNN
+AR Path="/E171B338/E1098DF4" Ref="K2304"  Part="1"
+F 0 "K2304" V 6900 3850 50  0000 L CNN
 F 1 "EW60-1A3-CL12D04" V 6650 3600 50  0000 L CNN
 F 2 "BoatControl:TE_2071366-2" H 6850 4400 50  0001 L BNN
@@
 AR Path="/E1098DFA" Ref="K?"  Part="1"
 AR Path="/E0EE2714/E107FCD3/E1098DFA" Ref="K?"  Part="1"
-AR Path="/E171B338/E1098DFA" Ref="K21"  Part="1"
-F 0 "K21" V 7950 3850 50  0000 L CNN
+AR Path="/E171B338/E1098DFA" Ref="K2305"  Part="1"
+F 0 "K2305" V 7950 3850 50  0000 L CNN
 F 1 "EW60-1A3-CL12D04" V 7700 3600 50  0000 L CNN
 F 2 "BoatControl:TE_2071366-2" H 7900 4400 50  0001 L BNN
@@
 AR Path="/E1098E00" Ref="K?"  Part="1"
 AR Path="/E0EE2714/E107FCD3/E1098E00" Ref="K?"  Part="1"
-AR Path="/E171B338/E1098E00" Ref="K22"  Part="1"
-F 0 "K22" V 9000 3850 50  0000 L CNN
+AR Path="/E171B338/E1098E00" Ref="K2306"  Part="1"
+F 0 "K2306" V 9000 3850 50  0000 L CNN
 F 1 "EW60-1A3-CL12D04" V 8750 3600 50  0000 L CNN
 F 2 "BoatControl:TE_2071366-2" H 8950 4400 50  0001 L BNN
@@
 AR Path="/E1098E06" Ref="K?"  Part="1"
 AR Path="/E0EE2714/E107FCD3/E1098E06" Ref="K?"  Part="1"
-AR Path="/E171B338/E1098E06" Ref="K23"  Part="1"
-F 0 "K23" V 10050 3850 50  0000 L CNN
+AR Path="/E171B338/E1098E06" Ref="K2307"  Part="1"
+F 0 "K2307" V 10050 3850 50  0000 L CNN
 F 1 "EW60-1A3-CL12D04" V 9800 3600 50  0000 L CNN
 F 2 "BoatControl:TE_2071366-2" H 10000 4400 50  0001 L BNN
@@
 AR Path="/E1098E0C" Ref="K?"  Part="1"
 AR Path="/E0EE2714/E107FCD3/E1098E0C" Ref="K?"  Part="1"
-AR Path="/E171B338/E1098E0C" Ref="K24"  Part="1"
-F 0 "K24" V 11100 3850 50  0000 L CNN
+AR Path="/E171B338/E1098E0C" Ref="K2308"  Part="1"
+F 0 "K2308" V 11100 3850 50  0000 L CNN
 F 1 "EW60-1A3-CL12D04" V 10850 3550 50  0000 L CNN
 F 2 "BoatControl:TE_2071366-2" H 11050 4400 50  0001 L BNN
@@
 AR Path="/E1098E6E" Ref="J?"  Part="1"
 AR Path="/E0EE2714/E107FCD3/E1098E6E" Ref="J?"  Part="1"
-AR Path="/E171B338/E1098E6E" Ref="J18"  Part="1"
-F 0 "J18" V 1346 2913 50  0000 R CNN
+AR Path="/E171B338/E1098E6E" Ref="J2301"  Part="1"
+F 0 "J2301" V 1346 2913 50  0000 R CNN
 F 1 "Conn_02x20_Odd_Even Header" V 1300 4450 50  0000 R CNN
 F 2 "Connector_PinSocket_2.54mm:PinSocket_2x20_P2.54mm_Vertical" H 1250 4000 50  0001 C CNN
@@
 AR Path="/E1098E74" Ref="H?"  Part="1"
 AR Path="/E0EE2714/E107FCD3/E1098E74" Ref="H?"  Part="1"
-AR Path="/E171B338/E1098E74" Ref="H23"  Part="1"
-F 0 "H23" H 150 3946 50  0000 L CNN
+AR Path="/E171B338/E1098E74" Ref="H2301"  Part="1"
+F 0 "H2301" H 150 3946 50  0000 L CNN
 F 1 "MountingHole" H 150 3855 50  0000 L CNN
 F 2 "MountingHole:MountingHole_3mm" H 50  3900 50  0001 C CNN
@@
 AR Path="/E1098E7A" Ref="H?"  Part="1"
 AR Path="/E0EE2714/E107FCD3/E1098E7A" Ref="H?"  Part="1"
-AR Path="/E171B338/E1098E7A" Ref="H24"  Part="1"
-F 0 "H24" H 150 4296 50  0000 L CNN
+AR Path="/E171B338/E1098E7A" Ref="H2302"  Part="1"
+F 0 "H2302" H 150 4296 50  0000 L CNN
 F 1 "MountingHole" H 150 4205 50  0000 L CNN
 F 2 "MountingHole:MountingHole_3mm" H 50  4250 50  0001 C CNN
@@
 AR Path="/E1098E80" Ref="H?"  Part="1"
 AR Path="/E0EE2714/E107FCD3/E1098E80" Ref="H?"  Part="1"
-AR Path="/E171B338/E1098E80" Ref="H26"  Part="1"
-F 0 "H26" H 2450 4296 50  0000 L CNN
+AR Path="/E171B338/E1098E80" Ref="H2304"  Part="1"
+F 0 "H2304" H 2450 4296 50  0000 L CNN
 F 1 "MountingHole" H 2450 4205 50  0000 L CNN
 F 2 "MountingHole:MountingHole_3mm" H 2350 4250 50  0001 C CNN
@@
 AR Path="/E1098E86" Ref="H?"  Part="1"
 AR Path="/E0EE2714/E107FCD3/E1098E86" Ref="H?"  Part="1"
-AR Path="/E171B338/E1098E86" Ref="H25"  Part="1"
-F 0 "H25" H 2450 3946 50  0000 L CNN
+AR Path="/E171B338/E1098E86" Ref="H2303"  Part="1"
+F 0 "H2303" H 2450 3946 50  0000 L CNN
 F 1 "MountingHole" H 2450 3855 50  0000 L CNN
 F 2 "MountingHole:MountingHole_3mm" H 2350 3900 50  0001 C CNN
@@
 AR Path="/E1098E92" Ref="K?"  Part="1"
 AR Path="/E0EE2714/E107FCD3/E1098E92" Ref="K?"  Part="1"
-AR Path="/E171B338/E1098E92" Ref="K17"  Part="1"
-F 0 "K17" V 3750 3850 50  0000 L CNN
+AR Path="/E171B338/E1098E92" Ref="K2301"  Part="1"
+F 0 "K2301" V 3750 3850 50  0000 L CNN
 F 1 "EW60-1A3-CL12D04" V 3500 3600 50  0000 L CNN
 F 2 "BoatControl:TE_2071366-2" H 3700 4400 50  0001 L BNN
@@
 AR Path="/5F4F4DC8" Ref="#PWR?"  Part="1"
 AR Path="/E0EE2714/E107FCD3/5F4F4DC8" Ref="#PWR?"  Part="1"
-AR Path="/E171B338/5F4F4DC8" Ref="#PWR076"  Part="1"
-F 0 "#PWR076" H 7400 3800 50  0001 C CNN
+AR Path="/E171B338/5F4F4DC8" Ref="#PWR02305"  Part="1"
+F 0 "#PWR02305" H 7400 3800 50  0001 C CNN
 F 1 "GND" H 7600 4050 50  0000 R CNN
 F 2 "" H 7400 4050 50  0001 C CNN

Commit message: Structured
Changed lines of the file:
@@
 $Descr A4 11693 8268
 encoding utf-8
-Sheet 23 55
+Sheet 34 55
 Title "Boat Control Hat"
 Date "2020-07-09"
@@
 AR Path="/E0EE2714/E107FCD3/E1098DA6" Ref="#PWR?"  Part="1"
 AR Path="/E171B338/E1098DA6" Ref="#PWR02301"  Part="1"
-F 0 "#PWR02301" H 3200 3800 50  0001 C CNN
+AR Path="/E171B33C/5F80BAC6/E1098DA6" Ref="#PWR?"  Part="1"
+F 0 "#PWR?" H 3200 3800 50  0001 C CNN
 F 1 "GND" H 3400 4050 50  0000 R CNN
 F 2 "" H 3200 4050 50  0001 C CNN
@@
 AR Path="/E0EE2714/E107FCD3/E1098DAC" Ref="#PWR?"  Part="1"
 AR Path="/E171B338/E1098DAC" Ref="#PWR02302"  Part="1"
-F 0 "#PWR02302" H 4250 3800 50  0001 C CNN
+AR Path="/E171B33C/5F80BAC6/E1098DAC" Ref="#PWR?"  Part="1"
+F 0 "#PWR?" H 4250 3800 50  0001 C CNN
 F 1 "GND" H 4450 4050 50  0000 R CNN
 F 2 "" H 4250 4050 50  0001 C CNN
@@
 AR Path="/E0EE2714/E107FCD3/E1098DB2" Ref="#PWR?"  Part="1"
 AR Path="/E171B338/E1098DB2" Ref="#PWR02303"  Part="1"
-F 0 "#PWR02303" H 5300 3800 50  0001 C CNN
+AR Path="/E171B33C/5F80BAC6/E1098DB2" Ref="#PWR?"  Part="1"
+F 0 "#PWR?" H 5300 3800 50  0001 C CNN
 F 1 "GND" H 5500 4050 50  0000 R CNN
 F 2 "" H 5300 4050 50  0001 C CNN
@@
 AR Path="/E0EE2714/E107FCD3/E1098DB8" Ref="#PWR?"  Part="1"
 AR Path="/E171B338/E1098DB8" Ref="#PWR02304"  Part="1"
-F 0 "#PWR02304" H 6350 3800 50  0001 C CNN
+AR Path="/E171B33C/5F80BAC6/E1098DB8" Ref="#PWR?"  Part="1"
+F 0 "#PWR?" H 6350 3800 50  0001 C CNN
 F 1 "GND" H 6550 4050 50  0000 R CNN
 F 2 "" H 6350 4050 50  0001 C CNN
@@
 AR Path="/E0EE2714/E107FCD3/E1098DC4" Ref="#PWR?"  Part="1"
 AR Path="/E171B338/E1098DC4" Ref="#PWR02306"  Part="1"
-F 0 "#PWR02306" H 8450 3800 50  0001 C CNN
+AR Path="/E171B33C/5F80BAC6/E1098DC4" Ref="#PWR?"  Part="1"
+F 0 "#PWR?" H 8450 3800 50  0001 C CNN
 F 1 "GND" H 8650 4050 50  0000 R CNN
 F 2 "" H 8450 4050 50  0001 C CNN
@@
 AR Path="/E0EE2714/E107FCD3/E1098DCA" Ref="#PWR?"  Part="1"
 AR Path="/E171B338/E1098DCA" Ref="#PWR02307"  Part="1"
-F 0 "#PWR02307" H 9500 3800 50  0001 C CNN
+AR Path="/E171B33C/5F80BAC6/E1098DCA" Ref="#PWR?"  Part="1"
+F 0 "#PWR?" H 9500 3800 50  0001 C CNN
 F 1 "GND" H 9700 4050 50  0000 R CNN
 F 2 "" H 9500 4050 50  0001 C CNN
@@
 AR Path="/E0EE2714/E107FCD3/E1098DD0" Ref="#PWR?"  Part="1"
 AR Path="/E171B338/E1098DD0" Ref="#PWR02308"  Part="1"
-F 0 "#PWR02308" H 10550 3800 50  0001 C CNN
+AR Path="/E171B33C/5F80BAC6/E1098DD0" Ref="#PWR?"  Part="1"
+F 0 "#PWR?" H 10550 3800 50  0001 C CNN
 F 1 "GND" H 10750 4050 50  0000 R CNN
 F 2 "" H 10550 4050 50  0001 C CNN
@@
 AR Path="/E0EE2714/E107FCD3/E1098DD9" Ref="J?"  Part="1"
 AR Path="/E171B338/E1098DD9" Ref="J2303"  Part="1"
-F 0 "J2303" V 7146 4922 50  0000 R CNN
+AR Path="/E171B33C/5F80BAC6/E1098DD9" Ref="J?"  Part="1"
+F 0 "J?" V 7146 4922 50  0000 R CNN
 F 1 "TBL008V-1000-08BE" V 7400 5800 50  0000 R CNN
 F 2 "CUI_TBL008V-1000-08BE" H 7300 5350 50  0001 L BNN
@@
 AR Path="/E0EE2714/E107FCD3/E1098DE2" Ref="J?"  Part="1"
 AR Path="/E171B338/E1098DE2" Ref="J2302"  Part="1"
-F 0 "J2302" V 7146 2372 50  0000 R CNN
+AR Path="/E171B33C/5F80BAC6/E1098DE2" Ref="J?"  Part="1"
+F 0 "J?" V 7146 2372 50  0000 R CNN
 F 1 "TBL008V-1000-08BE" V 7400 3250 50  0000 R CNN
 F 2 "CUI_TBL008V-1000-08BE" H 7300 2800 50  0001 L BNN
@@
 AR Path="/E0EE2714/E107FCD3/E1098DE8" Ref="K?"  Part="1"
 AR Path="/E171B338/E1098DE8" Ref="K2302"  Part="1"
-F 0 "K2302" V 4800 3850 50  0000 L CNN
+AR Path="/E171B33C/5F80BAC6/E1098DE8" Ref="K?"  Part="1"
+F 0 "K?" V 4800 3850 50  0000 L CNN
 F 1 "EW60-1A3-CL12D04" V 4550 3600 50  0000 L CNN
 F 2 "BoatControl:TE_2071366-2" H 4750 4400 50  0001 L BNN
@@
 AR Path="/E0EE2714/E107FCD3/E1098DEE" Ref="K?"  Part="1"
 AR Path="/E171B338/E1098DEE" Ref="K2303"  Part="1"
-F 0 "K2303" V 5850 3850 50  0000 L CNN
+AR Path="/E171B33C/5F80BAC6/E1098DEE" Ref="K?"  Part="1"
+F 0 "K?" V 5850 3850 50  0000 L CNN
 F 1 "EW60-1A3-CL12D04" V 5600 3600 50  0000 L CNN
 F 2 "BoatControl:TE_2071366-2" H 5800 4400 50  0001 L BNN
@@
 AR Path="/E0EE2714/E107FCD3/E1098DF4" Ref="K?"  Part="1"
 AR Path="/E171B338/E1098DF4" Ref="K2304"  Part="1"
-F 0 "K2304" V 6900 3850 50  0000 L CNN
+AR Path="/E171B33C/5F80BAC6/E1098DF4" Ref="K?"  Part="1"
+F 0 "K?" V 6900 3850 50  0000 L CNN
 F 1 "EW60-1A3-CL12D04" V 6650 3600 50  0000 L CNN
 F 2 "BoatControl:TE_2071366-2" H 6850 4400 50  0001 L BNN
@@
 AR Path="/E0EE2714/E107FCD3/E1098DFA" Ref="K?"  Part="1"
 AR Path="/E171B338/E1098DFA" Ref="K2305"  Part="1"
-F 0 "K2305" V 7950 3850 50  0000 L CNN
+AR Path="/E171B33C/5F80BAC6/E1098DFA" Ref="K?"  Part="1"
+F 0 "K?" V 7950 3850 50  0000 L CNN
 F 1 "EW60-1A3-CL12D04" V 7700 3600 50  0000 L CNN
 F 2 "BoatControl:TE_2071366-2" H 7900 4400 50  0001 L BNN
@@
 AR Path="/E0EE2714/E107FCD3/E1098E00" Ref="K?"  Part="1"
 AR Path="/E171B338/E1098E00" Ref="K2306"  Part="1"
-F 0 "K2306" V 9000 3850 50  0000 L CNN
+AR Path="/E171B33C/5F80BAC6/E1098E00" Ref="K?"  Part="1"
+F 0 "K?" V 9000 3850 50  0000 L CNN
 F 1 "EW60-1A3-CL12D04" V 8750 3600 50  0000 L CNN
 F 2 "BoatControl:TE_2071366-2" H 8950 4400 50  0001 L BNN
@@
 AR Path="/E0EE2714/E107FCD3/E1098E06" Ref="K?"  Part="1"
 AR Path="/E171B338/E1098E06" Ref="K2307"  Part="1"
-F 0 "K2307" V 10050 3850 50  0000 L CNN
+AR Path="/E171B33C/5F80BAC6/E1098E06" Ref="K?"  Part="1"
+F 0 "K?" V 10050 3850 50  0000 L CNN
 F 1 "EW60-1A3-CL12D04" V 9800 3600 50  0000 L CNN
 F 2 "BoatControl:TE_2071366-2" H 10000 4400 50  0001 L BNN
@@
 AR Path="/E0EE2714/E107FCD3/E1098E0C" Ref="K?"  Part="1"
 AR Path="/E171B338/E1098E0C" Ref="K2308"  Part="1"
-F 0 "K2308" V 11100 3850 50  0000 L CNN
+AR Path="/E171B33C/5F80BAC6/E1098E0C" Ref="K?"  Part="1"
+F 0 "K?" V 11100 3850 50  0000 L CNN
 F 1 "EW60-1A3-CL12D04" V 10850 3550 50  0000 L CNN
 F 2 "BoatControl:TE_2071366-2" H 11050 4400 50  0001 L BNN
@@
 AR Path="/E0EE2714/E107FCD3/E1098E6E" Ref="J?"  Part="1"
 AR Path="/E171B338/E1098E6E" Ref="J2301"  Part="1"
-F 0 "J2301" V 1346 2913 50  0000 R CNN
+AR Path="/E171B33C/5F80BAC6/E1098E6E" Ref="J?"  Part="1"
+F 0 "J?" V 1346 2913 50  0000 R CNN
 F 1 "Conn_02x20_Odd_Even Header" V 1300 4450 50  0000 R CNN
 F 2 "Connector_PinSocket_2.54mm:PinSocket_2x20_P2.54mm_Vertical" H 1250 4000 50  0001 C CNN
@@
 AR Path="/E0EE2714/E107FCD3/E1098E74" Ref="H?"  Part="1"
 AR Path="/E171B338/E1098E74" Ref="H2301"  Part="1"
-F 0 "H2301" H 150 3946 50  0000 L CNN
+AR Path="/E171B33C/5F80BAC6/E1098E74" Ref="H?"  Part="1"
+F 0 "H?" H 150 3946 50  0000 L CNN
 F 1 "MountingHole" H 150 3855 50  0000 L CNN
 F 2 "MountingHole:MountingHole_3mm" H 50  3900 50  0001 C CNN
@@
 AR Path="/E0EE2714/E107FCD3/E1098E7A" Ref="H?"  Part="1"
 AR Path="/E171B338/E1098E7A" Ref="H2302"  Part="1"
-F 0 "H2302" H 150 4296 50  0000 L CNN
+AR Path="/E171B33C/5F80BAC6/E1098E7A" Ref="H?"  Part="1"
+F 0 "H?" H 150 4296 50  0000 L CNN
 F 1 "MountingHole" H 150 4205 50  0000 L CNN
 F 2 "MountingHole:MountingHole_3mm" H 50  4250 50  0001 C CNN
@@
 AR Path="/E0EE2714/E107FCD3/E1098E80" Ref="H?"  Part="1"
 AR Path="/E171B338/E1098E80" Ref="H2304"  Part="1"
-F 0 "H2304" H 2450 4296 50  0000 L CNN
+AR Path="/E171B33C/5F80BAC6/E1098E80" Ref="H?"  Part="1"
+F 0 "H?" H 2450 4296 50  0000 L CNN
 F 1 "MountingHole" H 2450 4205 50  0000 L CNN
 F 2 "MountingHole:MountingHole_3mm" H 2350 4250 50  0001 C CNN
@@
 AR Path="/E0EE2714/E107FCD3/E1098E86" Ref="H?"  Part="1"
 AR Path="/E171B338/E1098E86" Ref="H2303"  Part="1"
-F 0 "H2303" H 2450 3946 50  0000 L CNN
+AR Path="/E171B33C/5F80BAC6/E1098E86" Ref="H?"  Part="1"
+F 0 "H?" H 2450 3946 50  0000 L CNN
 F 1 "MountingHole" H 2450 3855 50  0000 L CNN
 F 2 "MountingHole:MountingHole_3mm" H 2350 3900 50  0001 C CNN
@@
 AR Path="/E0EE2714/E107FCD3/E1098E92" Ref="K?"  Part="1"
 AR Path="/E171B338/E1098E92" Ref="K2301"  Part="1"
-F 0 "K2301" V 3750 3850 50  0000 L CNN
+AR Path="/E171B33C/5F80BAC6/E1098E92" Ref="K?"  Part="1"
+F 0 "K?" V 3750 3850 50  0000 L CNN
 F 1 "EW60-1A3-CL12D04" V 3500 3600 50  0000 L CNN
 F 2 "BoatControl:TE_2071366-2" H 3700 4400 50  0001 L BNN
@@
 AR Path="/E0EE2714/E107FCD3/5F4F4DC8" Ref="#PWR?"  Part="1"
 AR Path="/E171B338/5F4F4DC8" Ref="#PWR02305"  Part="1"
-F 0 "#PWR02305" H 7400 3800 50  0001 C CNN
+AR Path="/E171B33C/5F80BAC6/5F4F4DC8" Ref="#PWR?"  Part="1"
+F 0 "#PWR?" H 7400 3800 50  0001 C CNN
 F 1 "GND" H 7600 4050 50  0000 R CNN
 F 2 "" H 7400 4050 50  0001 C CNN
