File: boatcontrol/RelayBoard.sch (KiCad schematic (older format))
At the start: 15 parts, among them J5001 TBL008V-1000-08BE, J5002 Conn_02x20_Odd_Even Header, J5003 TBL008V-1000-08BE, K5001 EW60-1A3-CL12D04, K5002 EW60-1A3-CL12D04, K5003 EW60-1A3-CL12D04, K5004 EW60-1A3-CL12D04, K5005 EW60-1A3-CL12D04, K5006 EW60-1A3-CL12D04, K5007 EW60-1A3-CL12D04, K5008 EW60-1A3-CL12D04

Commit message: Defina add-on boards
Changed lines of the file:
@@
 AR Path="/E171B338/E1098DA6" Ref="#PWR?"  Part="1"
 AR Path="/E171B33C/5F80BAC6/E1098DA6" Ref="#PWR05001"  Part="1"
-F 0 "#PWR05001" H 3200 3800 50  0001 C CNN
+AR Path="/601318CC/5F80BAC6/E1098DA6" Ref="#PWR?"  Part="1"
+F 0 "#PWR?" H 3200 3800 50  0001 C CNN
 F 1 "GND" H 3400 4050 50  0000 R CNN
 F 2 "" H 3200 4050 50  0001 C CNN
@@
 AR Path="/E171B338/E1098DAC" Ref="#PWR?"  Part="1"
 AR Path="/E171B33C/5F80BAC6/E1098DAC" Ref="#PWR05002"  Part="1"
-F 0 "#PWR05002" H 4250 3800 50  0001 C CNN
+AR Path="/601318CC/5F80BAC6/E1098DAC" Ref="#PWR?"  Part="1"
+F 0 "#PWR?" H 4250 3800 50  0001 C CNN
 F 1 "GND" H 4450 4050 50  0000 R CNN
 F 2 "" H 4250 4050 50  0001 C CNN
@@
 AR Path="/E171B338/E1098DB2" Ref="#PWR?"  Part="1"
 AR Path="/E171B33C/5F80BAC6/E1098DB2" Ref="#PWR05003"  Part="1"
-F 0 "#PWR05003" H 5300 3800 50  0001 C CNN
+AR Path="/601318CC/5F80BAC6/E1098DB2" Ref="#PWR?"  Part="1"
+F 0 "#PWR?" H 5300 3800 50  0001 C CNN
 F 1 "GND" H 5500 4050 50  0000 R CNN
 F 2 "" H 5300 4050 50  0001 C CNN
@@
 AR Path="/E171B338/E1098DB8" Ref="#PWR?"  Part="1"
 AR Path="/E171B33C/5F80BAC6/E1098DB8" Ref="#PWR05004"  Part="1"
-F 0 "#PWR05004" H 6350 3800 50  0001 C CNN
+AR Path="/601318CC/5F80BAC6/E1098DB8" Ref="#PWR?"  Part="1"
+F 0 "#PWR?" H 6350 3800 50  0001 C CNN
 F 1 "GND" H 6550 4050 50  0000 R CNN
 F 2 "" H 6350 4050 50  0001 C CNN
@@
 AR Path="/E171B338/E1098DC4" Ref="#PWR?"  Part="1"
 AR Path="/E171B33C/5F80BAC6/E1098DC4" Ref="#PWR05006"  Part="1"
-F 0 "#PWR05006" H 8450 3800 50  0001 C CNN
+AR Path="/601318CC/5F80BAC6/E1098DC4" Ref="#PWR?"  Part="1"
+F 0 "#PWR?" H 8450 3800 50  0001 C CNN
 F 1 "GND" H 8650 4050 50  0000 R CNN
 F 2 "" H 8450 4050 50  0001 C CNN
@@
 AR Path="/E171B338/E1098DCA" Ref="#PWR?"  Part="1"
 AR Path="/E171B33C/5F80BAC6/E1098DCA" Ref="#PWR05007"  Part="1"
-F 0 "#PWR05007" H 9500 3800 50  0001 C CNN
+AR Path="/601318CC/5F80BAC6/E1098DCA" Ref="#PWR?"  Part="1"
+F 0 "#PWR?" H 9500 3800 50  0001 C CNN
 F 1 "GND" H 9700 4050 50  0000 R CNN
 F 2 "" H 9500 4050 50  0001 C CNN
@@
 AR Path="/E171B338/E1098DD0" Ref="#PWR?"  Part="1"
 AR Path="/E171B33C/5F80BAC6/E1098DD0" Ref="#PWR05008"  Part="1"
-F 0 "#PWR05008" H 10550 3800 50  0001 C CNN
+AR Path="/601318CC/5F80BAC6/E1098DD0" Ref="#PWR?"  Part="1"
+F 0 "#PWR?" H 10550 3800 50  0001 C CNN
 F 1 "GND" H 10750 4050 50  0000 R CNN
 F 2 "" H 10550 4050 50  0001 C CNN
@@
 AR Path="/E171B338/E1098DD9" Ref="J?"  Part="1"
 AR Path="/E171B33C/5F80BAC6/E1098DD9" Ref="J5003"  Part="1"
-F 0 "J5003" V 7146 4922 50  0000 R CNN
+AR Path="/601318CC/5F80BAC6/E1098DD9" Ref="J?"  Part="1"
+F 0 "J?" V 7146 4922 50  0000 R CNN
 F 1 "TBL008V-1000-08BE" V 7400 5800 50  0000 R CNN
 F 2 "CUI_TBL008V-1000-08BE" H 7300 5350 50  0001 L BNN
@@
 AR Path="/E171B338/E1098DE2" Ref="J?"  Part="1"
 AR Path="/E171B33C/5F80BAC6/E1098DE2" Ref="J5001"  Part="1"
-F 0 "J5001" V 7146 2372 50  0000 R CNN
+AR Path="/601318CC/5F80BAC6/E1098DE2" Ref="J?"  Part="1"
+F 0 "J?" V 7146 2372 50  0000 R CNN
 F 1 "TBL008V-1000-08BE" V 7400 3250 50  0000 R CNN
 F 2 "CUI_TBL008V-1000-08BE" H 7300 2800 50  0001 L BNN
@@
 AR Path="/E171B338/E1098DE8" Ref="K?"  Part="1"
 AR Path="/E171B33C/5F80BAC6/E1098DE8" Ref="K5001"  Part="1"
-F 0 "K5001" V 4800 3850 50  0000 L CNN
+AR Path="/601318CC/5F80BAC6/E1098DE8" Ref="K?"  Part="1"
+F 0 "K?" V 4800 3850 50  0000 L CNN
 F 1 "EW60-1A3-CL12D04" V 4550 3600 50  0000 L CNN
 F 2 "BoatControl:TE_2071366-2" H 4750 4400 50  0001 L BNN
@@
 AR Path="/E171B338/E1098DF4" Ref="K?"  Part="1"
 AR Path="/E171B33C/5F80BAC6/E1098DF4" Ref="K5002"  Part="1"
-F 0 "K5002" V 6900 3850 50  0000 L CNN
+AR Path="/601318CC/5F80BAC6/E1098DF4" Ref="K?"  Part="1"
+F 0 "K?" V 6900 3850 50  0000 L CNN
 F 1 "EW60-1A3-CL12D04" V 6650 3600 50  0000 L CNN
 F 2 "BoatControl:TE_2071366-2" H 6850 4400 50  0001 L BNN
@@
 AR Path="/E171B338/E1098E00" Ref="K?"  Part="1"
 AR Path="/E171B33C/5F80BAC6/E1098E00" Ref="K5003"  Part="1"
-F 0 "K5003" V 9000 3850 50  0000 L CNN
+AR Path="/601318CC/5F80BAC6/E1098E00" Ref="K?"  Part="1"
+F 0 "K?" V 9000 3850 50  0000 L CNN
 F 1 "EW60-1A3-CL12D04" V 8750 3600 50  0000 L CNN
 F 2 "BoatControl:TE_2071366-2" H 8950 4400 50  0001 L BNN
@@
 AR Path="/E171B338/E1098E0C" Ref="K?"  Part="1"
 AR Path="/E171B33C/5F80BAC6/E1098E0C" Ref="K5004"  Part="1"
-F 0 "K5004" V 11100 3850 50  0000 L CNN
+AR Path="/601318CC/5F80BAC6/E1098E0C" Ref="K?"  Part="1"
+F 0 "K?" V 11100 3850 50  0000 L CNN
 F 1 "EW60-1A3-CL12D04" V 10850 3550 50  0000 L CNN
 F 2 "BoatControl:TE_2071366-2" H 11050 4400 50  0001 L BNN
@@
 AR Path="/E171B338/5F4F4DC8" Ref="#PWR?"  Part="1"
 AR Path="/E171B33C/5F80BAC6/5F4F4DC8" Ref="#PWR05005"  Part="1"
-F 0 "#PWR05005" H 7400 3800 50  0001 C CNN
+AR Path="/601318CC/5F80BAC6/5F4F4DC8" Ref="#PWR?"  Part="1"
+F 0 "#PWR?" H 7400 3800 50  0001 C CNN
 F 1 "GND" H 7600 4050 50  0000 R CNN
 F 2 "" H 7400 4050 50  0001 C CNN
@@
 AR Path="/E171B338/E1098E86" Ref="H?"  Part="1"
 AR Path="/E171B33C/5F80BAC6/E1098E86" Ref="H5002"  Part="1"
-F 0 "H5002" H 2450 3946 50  0000 L CNN
+AR Path="/601318CC/5F80BAC6/E1098E86" Ref="H?"  Part="1"
+F 0 "H?" H 2450 3946 50  0000 L CNN
 F 1 "MountingHole" H 2450 3855 50  0000 L CNN
 F 2 "MountingHole:MountingHole_3mm" H 2350 3900 50  0001 C CNN
@@
 AR Path="/E171B338/E1098E80" Ref="H?"  Part="1"
 AR Path="/E171B33C/5F80BAC6/E1098E80" Ref="H5004"  Part="1"
-F 0 "H5004" H 2450 4296 50  0000 L CNN
+AR Path="/601318CC/5F80BAC6/E1098E80" Ref="H?"  Part="1"
+F 0 "H?" H 2450 4296 50  0000 L CNN
 F 1 "MountingHole" H 2450 4205 50  0000 L CNN
 F 2 "MountingHole:MountingHole_3mm" H 2350 4250 50  0001 C CNN
@@
 AR Path="/E171B338/E1098E7A" Ref="H?"  Part="1"
 AR Path="/E171B33C/5F80BAC6/E1098E7A" Ref="H5003"  Part="1"
-F 0 "H5003" H 150 4296 50  0000 L CNN
+AR Path="/601318CC/5F80BAC6/E1098E7A" Ref="H?"  Part="1"
+F 0 "H?" H 150 4296 50  0000 L CNN
 F 1 "MountingHole" H 150 4205 50  0000 L CNN
 F 2 "MountingHole:MountingHole_3mm" H 50  4250 50  0001 C CNN
@@
 AR Path="/E171B338/E1098E74" Ref="H?"  Part="1"
 AR Path="/E171B33C/5F80BAC6/E1098E74" Ref="H5001"  Part="1"
-F 0 "H5001" H 150 3946 50  0000 L CNN
+AR Path="/601318CC/5F80BAC6/E1098E74" Ref="H?"  Part="1"
+F 0 "H?" H 150 3946 50  0000 L CNN
 F 1 "MountingHole" H 150 3855 50  0000 L CNN
 F 2 "MountingHole:MountingHole_3mm" H 50  3900 50  0001 C CNN
@@
 AR Path="/E171B338/E1098E06" Ref="K?"  Part="1"
 AR Path="/E171B33C/5F80BAC6/E1098E06" Ref="K5008"  Part="1"
-F 0 "K5008" V 10050 3950 50  0000 L CNN
+AR Path="/601318CC/5F80BAC6/E1098E06" Ref="K?"  Part="1"
+F 0 "K?" V 10050 3950 50  0000 L CNN
 F 1 "EW60-1A3-CL12D04" V 9800 3700 50  0000 L CNN
 F 2 "BoatControl:TE_2071366-2" H 10000 4500 50  0001 L BNN
@@
 AR Path="/E171B338/E1098DFA" Ref="K?"  Part="1"
 AR Path="/E171B33C/5F80BAC6/E1098DFA" Ref="K5007"  Part="1"
-F 0 "K5007" V 7950 3950 50  0000 L CNN
+AR Path="/601318CC/5F80BAC6/E1098DFA" Ref="K?"  Part="1"
+F 0 "K?" V 7950 3950 50  0000 L CNN
 F 1 "EW60-1A3-CL12D04" V 7700 3700 50  0000 L CNN
 F 2 "BoatControl:TE_2071366-2" H 7900 4500 50  0001 L BNN
@@
 AR Path="/E171B338/E1098DEE" Ref="K?"  Part="1"
 AR Path="/E171B33C/5F80BAC6/E1098DEE" Ref="K5006"  Part="1"
-F 0 "K5006" V 5850 3950 50  0000 L CNN
+AR Path="/601318CC/5F80BAC6/E1098DEE" Ref="K?"  Part="1"
+F 0 "K?" V 5850 3950 50  0000 L CNN
 F 1 "EW60-1A3-CL12D04" V 5600 3700 50  0000 L CNN
 F 2 "BoatControl:TE_2071366-2" H 5800 4500 50  0001 L BNN
@@
 AR Path="/E171B338/E1098E92" Ref="K?"  Part="1"
 AR Path="/E171B33C/5F80BAC6/E1098E92" Ref="K5005"  Part="1"
-F 0 "K5005" V 3750 3950 50  0000 L CNN
+AR Path="/601318CC/5F80BAC6/E1098E92" Ref="K?"  Part="1"
+F 0 "K?" V 3750 3950 50  0000 L CNN
 F 1 "EW60-1A3-CL12D04" V 3500 3700 50  0000 L CNN
 F 2 "BoatControl:TE_2071366-2" H 3700 4500 50  0001 L BNN
@@
 AR Path="/E171B338/E1098E6E" Ref="J?"  Part="1"
 AR Path="/E171B33C/5F80BAC6/E1098E6E" Ref="J5002"  Part="1"
-F 0 "J5002" V 1346 2913 50  0000 R CNN
+AR Path="/601318CC/5F80BAC6/E1098E6E" Ref="J?"  Part="1"
+F 0 "J?" V 1346 2913 50  0000 R CNN
 F 1 "Conn_02x20_Odd_Even Header" V 1300 4450 50  0000 R CNN
 F 2 "Connector_PinSocket_2.54mm:PinSocket_2x20_P2.54mm_Vertical" H 1250 4000 50  0001 C CNN
@@
 U 1 1 60E5FB29
 P 250 4300
-F 0 "#PWR05009" H 250 4050 50  0001 C CNN
+AR Path="/E171B33C/5F80BAC6/60E5FB29" Ref="#PWR05009"  Part="1"
+AR Path="/601318CC/5F80BAC6/60E5FB29" Ref="#PWR?"  Part="1"
+F 0 "#PWR?" H 250 4050 50  0001 C CNN
 F 1 "GND" H 255 4127 50  0000 C CNN
 F 2 "" H 250 4300 50  0001 C CNN
