File: boatcontrol/3AmpBlock.sch (KiCad schematic (older format))
At the start: 13 parts, among them U3001 ULN2803A

Commit message: Cleanup
Connections:
- net labels added: AN_OFF_C2, AN_OFF_C3, AN_OFF_C4, AN_ON_C2, AN_ON_C3, AN_ON_C4, DIG_OFF_C2, DIG_OFF_C3, DIG_OFF_C4, DIG_ON_C2, DIG_ON_C3, DIG_ON_C4
Changed lines of the file:
@@
 $Descr A4 11693 8268
 encoding utf-8
-Sheet 30 87
+Sheet 21 87
 Title "Boat Control Hat"
 Date "2020-07-09"
@@
 AR Path="/D16552B4/5FA17F52/D2F3142C" Ref="#PWR01202"  Part="1"
 AR Path="/D16552B4/5FA17F6C/D2F3142C" Ref="#PWR02102"  Part="1"
-F 0 "#PWR03002" H 5800 3000 50  0001 C CNN
+F 0 "#PWR02102" H 5800 3000 50  0001 C CNN
 F 1 "GND" H 5805 3077 50  0000 C CNN
 F 2 "" H 5800 3250 50  0001 C CNN
@@
 AR Path="/D16552B4/5FA17F52/81A9CC8E" Ref="RN1202"  Part="1"
 AR Path="/D16552B4/5FA17F6C/81A9CC8E" Ref="RN2102"  Part="1"
-F 0 "RN3002" V 5650 825 50  0000 L CNN
+F 0 "RN2102" V 5650 825 50  0000 L CNN
 F 1 "4116R-1-471" H 4200 900 50  0000 L CNN
 F 2 "BoatControl:DIP254P762X432-16P" V 5725 900 50  0001 C CNN
@@
 AR Path="/D16552B4/5FA17F6C/5FF784D2" Ref="RN2104"  Part="1"
 AR Path="/D16552B4/5FA17F86/5FF784D2" Ref="RN3004"  Part="1"
-F 0 "RN3004" V 6450 7000 50  0000 C CNN
+F 0 "RN2104" V 6450 7000 50  0000 C CNN
 F 1 "4116R-1-103LF" V 6350 7000 50  0000 C CNN
 F 2 "DIP787W49P254L2197H469Q16N" H 7300 7400 50  0001 L CNN
@@
 AR Path="/D16552B4/5FA17F6C/5FD52518" Ref="RN2101"  Part="1"
 AR Path="/D16552B4/5FA17F86/5FD52518" Ref="RN3001"  Part="1"
-F 0 "RN3001" V 4650 7000 50  0000 C CNN
+F 0 "RN2101" V 4650 7000 50  0000 C CNN
 F 1 "4116R-1-103LF" V 4550 7000 50  0001 C CNN
 F 2 "DIP787W49P254L2197H469Q16N" H 5500 7400 50  0001 L CNN
@@
 AR Path="/D16552B4/5FA17F6C/5FF7A29F" Ref="#PWR02103"  Part="1"
 AR Path="/D16552B4/5FA17F86/5FF7A29F" Ref="#PWR03003"  Part="1"
-F 0 "#PWR03003" H 6550 7150 50  0001 C CNN
+F 0 "#PWR02103" H 6550 7150 50  0001 C CNN
 F 1 "+5V" H 6565 7473 50  0000 C CNN
 F 2 "" H 6550 7300 50  0001 C CNN
@@
 $EndSheet
 Text HLabel 5650 4650 0    50   Output ~ 0
-AN_ON_C1
+AN_ON_C3
 Text HLabel 5650 4750 0    50   Output ~ 0
-AN_OFF_C1
+AN_OFF_C3
 Text HLabel 5650 4850 0    50   Output ~ 0
-DIG_ON_C1
+DIG_ON_C3
 Text HLabel 5650 4950 0    50   Output ~ 0
-DIG_OFF_C1
+DIG_OFF_C3
 Text HLabel 7100 4650 0    50   Output ~ 0
-AN_ON_C1
+AN_ON_C4
 Text HLabel 7100 4750 0    50   Output ~ 0
-AN_OFF_C1
+AN_OFF_C4
 Text HLabel 7100 4850 0    50   Output ~ 0
-DIG_ON_C1
+DIG_ON_C4
 Text HLabel 7100 4950 0    50   Output ~ 0
-DIG_OFF_C1
+DIG_OFF_C4
 Text Notes 6500 950  2    50   ~ 0
 Resistors for diodes
@@
 AR Path="/D16552B4/5FA17F52/D2B5CDA2" Ref="U1201"  Part="1"
 AR Path="/D16552B4/5FA17F6C/D2B5CDA2" Ref="U2101"  Part="1"
-F 0 "U3001" H 5050 3050 50  0000 L CNN
+F 0 "U2101" H 5050 3050 50  0000 L CNN
 F 1 "ULN2803A" H 4900 3750 50  0000 L CNN
 F 2 "Package_DIP:DIP-18_W7.62mm" H 5150 2600 50  0001 L CNN
@@
 $EndSheet
 Text HLabel 4200 4950 0    50   Output ~ 0
-DIG_OFF_C1
+DIG_OFF_C2
 Text HLabel 4200 4850 0    50   Output ~ 0
-DIG_ON_C1
+DIG_ON_C2
 Text HLabel 4200 4750 0    50   Output ~ 0
-AN_OFF_C1
+AN_OFF_C2
 Text HLabel 4200 4650 0    50   Output ~ 0
-AN_ON_C1
+AN_ON_C2
 Text HLabel 2750 4950 0    50   Output ~ 0
 DIG_OFF_C1
@@
 AR Path="/D16552B4/5FA17F52/5F542D5F" Ref="RN1203"  Part="1"
 AR Path="/D16552B4/5FA17F6C/5F542D5F" Ref="RN2103"  Part="1"
-F 0 "RN3003" H 5200 6800 50  0000 L CNN
+F 0 "RN2103" H 5200 6800 50  0000 L CNN
 F 1 "4120R-1-103LF" H 5000 6700 50  0000 L CNN
 F 2 "BoatControl:DIP254P762X432-16P" V 5825 7100 50  0001 C CNN
@@
 AR Path="/D16552B4/5FA17F52/D2F3142D" Ref="#PWR01201"  Part="1"
 AR Path="/D16552B4/5FA17F6C/D2F3142D" Ref="#PWR02101"  Part="1"
-F 0 "#PWR03001" H 4800 2700 50  0001 C CNN
+F 0 "#PWR02101" H 4800 2700 50  0001 C CNN
 F 1 "+12P" H 4650 2950 50  0000 C CNN
 F 2 "" H 4800 2850 50  0001 C CNN
@@
 AR Path="/D16552B4/5FA17F52/5FDBB725" Ref="C1208"  Part="1"
 AR Path="/D16552B4/5FA17F6C/5FDBB725" Ref="C2108"  Part="1"
-F 0 "C3008" V 5700 6550 50  0000 L CNN
+F 0 "C2108" V 5700 6550 50  0000 L CNN
 F 1 "107CKS016M 100UF" H 4500 6700 50  0001 L CNN
 F 2 "Capacitor_THT:CP_Radial_D5.0mm_P2.00mm" H 5650 6700 50  0001 C CNN
@@
 AR Path="/D16552B4/5FA17F52/5FDBB72C" Ref="C1207"  Part="1"
 AR Path="/D16552B4/5FA17F6C/5FDBB72C" Ref="C2107"  Part="1"
-F 0 "C3007" V 5600 6450 50  0000 L CNN
+F 0 "C2107" V 5600 6450 50  0000 L CNN
 F 1 "107CKS016M 100UF" H 4450 6600 50  0001 L CNN
 F 2 "Capacitor_THT:CP_Radial_D5.0mm_P2.00mm" H 5550 6600 50  0001 C CNN
@@
 AR Path="/D16552B4/5FA17F52/5FDB4626" Ref="C1206"  Part="1"
 AR Path="/D16552B4/5FA17F6C/5FDB4626" Ref="C2106"  Part="1"
-F 0 "C3006" V 5500 6300 50  0000 L CNN
+F 0 "C2106" V 5500 6300 50  0000 L CNN
 F 1 "107CKS016M 100UF" H 4300 6450 50  0001 L CNN
 F 2 "Capacitor_THT:CP_Radial_D5.0mm_P2.00mm" H 5450 6450 50  0001 C CNN
@@
 AR Path="/D16552B4/5FA17F52/5FDB462D" Ref="C1205"  Part="1"
 AR Path="/D16552B4/5FA17F6C/5FDB462D" Ref="C2105"  Part="1"
-F 0 "C3005" V 5400 6200 50  0000 L CNN
+F 0 "C2105" V 5400 6200 50  0000 L CNN
 F 1 "107CKS016M 100UF" H 4250 6350 50  0001 L CNN
 F 2 "Capacitor_THT:CP_Radial_D5.0mm_P2.00mm" H 5350 6350 50  0001 C CNN
@@
 AR Path="/D16552B4/5FA17F52/5FD94312" Ref="C1204"  Part="1"
 AR Path="/D16552B4/5FA17F6C/5FD94312" Ref="C2104"  Part="1"
-F 0 "C3004" V 5300 6550 50  0000 L CNN
+F 0 "C2104" V 5300 6550 50  0000 L CNN
 F 1 "107CKS016M 100UF" H 4100 6700 50  0001 L CNN
 F 2 "Capacitor_THT:CP_Radial_D5.0mm_P2.00mm" H 5250 6700 50  0001 C CNN
@@
 AR Path="/D16552B4/5FA17F52/5FD94319" Ref="C1203"  Part="1"
 AR Path="/D16552B4/5FA17F6C/5FD94319" Ref="C2103"  Part="1"
-F 0 "C3003" V 5200 6450 50  0000 L CNN
+F 0 "C2103" V 5200 6450 50  0000 L CNN
 F 1 "107CKS016M 100UF" H 4050 6600 50  0001 L CNN
 F 2 "Capacitor_THT:CP_Radial_D5.0mm_P2.00mm" H 5150 6600 50  0001 C CNN
@@
 AR Path="/D16552B4/5FA17F52/5F542D59" Ref="C1201"  Part="1"
 AR Path="/D16552B4/5FA17F6C/5F542D59" Ref="C2101"  Part="1"
-F 0 "C3001" V 5000 6100 50  0000 L CNN
+F 0 "C2101" V 5000 6100 50  0000 L CNN
 F 1 "107CKS016M 100UF" H 4100 6250 50  0001 L CNN
 F 2 "Capacitor_THT:CP_Radial_D5.0mm_P2.00mm" H 4950 6350 50  0001 C CNN
@@
 AR Path="/D16552B4/5FA17F52/5F59CDBA" Ref="C1202"  Part="1"
 AR Path="/D16552B4/5FA17F6C/5F59CDBA" Ref="C2102"  Part="1"
-F 0 "C3002" V 5100 6200 50  0000 L CNN
+F 0 "C2102" V 5100 6200 50  0000 L CNN
 F 1 "107CKS016M 100UF" H 3900 6450 50  0001 L CNN
 F 2 "Capacitor_THT:CP_Radial_D5.0mm_P2.00mm" H 5050 6450 50  0001 C CNN
