File: boatcontrol/3AmpBlock.sch (KiCad schematic (older format))
At the start: 13 parts, among them U3001 ULN2803A

Commit message: bugfixing
Connections:
- wire segments 288 -> 284
Changed lines of the file:
@@
 AR Path="/D16552B4/5FA17F52/D2F3142C" Ref="#PWR01202"  Part="1"
 AR Path="/D16552B4/5FA17F6C/D2F3142C" Ref="#PWR02102"  Part="1"
-F 0 "#PWR0302" H 5800 3000 50  0001 C CNN
+F 0 "#PWR03002" H 5800 3000 50  0001 C CNN
 F 1 "GND" H 5805 3077 50  0000 C CNN
 F 2 "" H 5800 3250 50  0001 C CNN
@@
 AR Path="/D16552B4/5FA17F6C/5FF7A29F" Ref="#PWR02103"  Part="1"
 AR Path="/D16552B4/5FA17F86/5FF7A29F" Ref="#PWR03003"  Part="1"
-F 0 "#PWR0303" H 6550 7150 50  0001 C CNN
+F 0 "#PWR03003" H 6550 7150 50  0001 C CNN
 F 1 "+5V" H 6565 7473 50  0000 C CNN
 F 2 "" H 6550 7300 50  0001 C CNN
@@
 AR Path="/D16552B4/5FA17F52/D2F3142D" Ref="#PWR01201"  Part="1"
 AR Path="/D16552B4/5FA17F6C/D2F3142D" Ref="#PWR02101"  Part="1"
-F 0 "#PWR0301" H 4800 2700 50  0001 C CNN
+F 0 "#PWR03001" H 4800 2700 50  0001 C CNN
 F 1 "+12P" H 4650 2950 50  0000 C CNN
 F 2 "" H 4800 2850 50  0001 C CNN
@@
 $EndComp
 Wire Wire Line
-	5400 3650 5400 3850
-Wire Wire Line
 	5950 1500 5950 2450
 Wire Wire Line
-	5300 3650 5300 3800
-Wire Wire Line
-	5300 3800 5850 3800
-Wire Wire Line
 	5250 500  5250 700
-Connection ~ 5300 3800
-Wire Wire Line
-	5300 3800 5300 4500
-Wire Wire Line
-	5400 3850 5900 3850
 Wire Wire Line
 	5350 550  5350 700
-Connection ~ 5400 3850
-Wire Wire Line
-	5400 3850 5400 4400
 Wire Wire Line
 	5450 600  5450 700
@@
 	5550 650  7650 650
 Connection ~ 7650 1650
+Wire Wire Line
+	5400 3650 5400 4400
+Wire Wire Line
+	5300 3650 5300 4500
 $EndSCHEMATC

Commit message: possible
Changed lines of the file:
@@
 $Descr A4 11693 8268
 encoding utf-8
-Sheet 3 87
+Sheet 30 87
 Title "Boat Control Hat"
 Date "2020-07-09"
@@
 AR Path="/D16552B4/5FA17F52/81A9CC8E" Ref="RN1202"  Part="1"
 AR Path="/D16552B4/5FA17F6C/81A9CC8E" Ref="RN2102"  Part="1"
-F 0 "RN302" H 4500 900 50  0000 L CNN
+F 0 "RN3002" H 4500 900 50  0000 L CNN
 F 1 "4116R-1-471" H 5650 900 50  0000 L CNN
 F 2 "BoatControl:DIP254P762X432-16P" V 5725 900 50  0001 C CNN
@@
 AR Path="/D16552B4/5FA17F6C/5FF784D2" Ref="RN2104"  Part="1"
 AR Path="/D16552B4/5FA17F86/5FF784D2" Ref="RN3004"  Part="1"
-F 0 "RN304" V 6450 7000 50  0000 C CNN
+F 0 "RN3004" V 6450 7000 50  0000 C CNN
 F 1 "4116R-1-103LF" V 6350 7000 50  0000 C CNN
 F 2 "DIP787W49P254L2197H469Q16N" H 7300 7400 50  0001 L CNN
@@
 AR Path="/D16552B4/5FA17F6C/5FD52518" Ref="RN2101"  Part="1"
 AR Path="/D16552B4/5FA17F86/5FD52518" Ref="RN3001"  Part="1"
-F 0 "RN301" V 4650 7000 50  0000 C CNN
+F 0 "RN3001" V 4650 7000 50  0000 C CNN
 F 1 "4116R-1-103LF" V 4550 7000 50  0001 C CNN
 F 2 "DIP787W49P254L2197H469Q16N" H 5500 7400 50  0001 L CNN
@@
 AR Path="/D16552B4/5FA17F52/D2B5CDA2" Ref="U1201"  Part="1"
 AR Path="/D16552B4/5FA17F6C/D2B5CDA2" Ref="U2101"  Part="1"
-F 0 "U301" H 5050 3050 50  0000 L CNN
+F 0 "U3001" H 5050 3050 50  0000 L CNN
 F 1 "ULN2803A" H 4900 3750 50  0000 L CNN
 F 2 "Package_DIP:DIP-18_W7.62mm" H 5150 2600 50  0001 L CNN
@@
 AR Path="/D16552B4/5FA17F52/5F542D5F" Ref="RN1203"  Part="1"
 AR Path="/D16552B4/5FA17F6C/5F542D5F" Ref="RN2103"  Part="1"
-F 0 "RN303" H 5200 6800 50  0000 L CNN
+F 0 "RN3003" H 5200 6800 50  0000 L CNN
 F 1 "4120R-1-103LF" H 5000 6700 50  0000 L CNN
 F 2 "BoatControl:DIP254P762X432-16P" V 5825 7100 50  0001 C CNN
@@
 AR Path="/D16552B4/5FA17F52/5FDBB725" Ref="C1208"  Part="1"
 AR Path="/D16552B4/5FA17F6C/5FDBB725" Ref="C2108"  Part="1"
-F 0 "C308" V 5700 6550 50  0000 L CNN
+F 0 "C3008" V 5700 6550 50  0000 L CNN
 F 1 "107CKS016M 100UF" H 4500 6700 50  0001 L CNN
 F 2 "Capacitor_THT:CP_Radial_D5.0mm_P2.00mm" H 5650 6700 50  0001 C CNN
@@
 AR Path="/D16552B4/5FA17F52/5FDBB72C" Ref="C1207"  Part="1"
 AR Path="/D16552B4/5FA17F6C/5FDBB72C" Ref="C2107"  Part="1"
-F 0 "C307" V 5600 6450 50  0000 L CNN
+F 0 "C3007" V 5600 6450 50  0000 L CNN
 F 1 "107CKS016M 100UF" H 4450 6600 50  0001 L CNN
 F 2 "Capacitor_THT:CP_Radial_D5.0mm_P2.00mm" H 5550 6600 50  0001 C CNN
@@
 AR Path="/D16552B4/5FA17F52/5FDB4626" Ref="C1206"  Part="1"
 AR Path="/D16552B4/5FA17F6C/5FDB4626" Ref="C2106"  Part="1"
-F 0 "C306" V 5500 6300 50  0000 L CNN
+F 0 "C3006" V 5500 6300 50  0000 L CNN
 F 1 "107CKS016M 100UF" H 4300 6450 50  0001 L CNN
 F 2 "Capacitor_THT:CP_Radial_D5.0mm_P2.00mm" H 5450 6450 50  0001 C CNN
@@
 AR Path="/D16552B4/5FA17F52/5FDB462D" Ref="C1205"  Part="1"
 AR Path="/D16552B4/5FA17F6C/5FDB462D" Ref="C2105"  Part="1"
-F 0 "C305" V 5400 6200 50  0000 L CNN
+F 0 "C3005" V 5400 6200 50  0000 L CNN
 F 1 "107CKS016M 100UF" H 4250 6350 50  0001 L CNN
 F 2 "Capacitor_THT:CP_Radial_D5.0mm_P2.00mm" H 5350 6350 50  0001 C CNN
@@
 AR Path="/D16552B4/5FA17F52/5FD94312" Ref="C1204"  Part="1"
 AR Path="/D16552B4/5FA17F6C/5FD94312" Ref="C2104"  Part="1"
-F 0 "C304" V 5300 6550 50  0000 L CNN
+F 0 "C3004" V 5300 6550 50  0000 L CNN
 F 1 "107CKS016M 100UF" H 4100 6700 50  0001 L CNN
 F 2 "Capacitor_THT:CP_Radial_D5.0mm_P2.00mm" H 5250 6700 50  0001 C CNN
@@
 AR Path="/D16552B4/5FA17F52/5FD94319" Ref="C1203"  Part="1"
 AR Path="/D16552B4/5FA17F6C/5FD94319" Ref="C2103"  Part="1"
-F 0 "C303" V 5200 6450 50  0000 L CNN
+F 0 "C3003" V 5200 6450 50  0000 L CNN
 F 1 "107CKS016M 100UF" H 4050 6600 50  0001 L CNN
 F 2 "Capacitor_THT:CP_Radial_D5.0mm_P2.00mm" H 5150 6600 50  0001 C CNN
@@
 AR Path="/D16552B4/5FA17F52/5F542D59" Ref="C1201"  Part="1"
 AR Path="/D16552B4/5FA17F6C/5F542D59" Ref="C2101"  Part="1"
-F 0 "C301" V 5000 6100 50  0000 L CNN
+F 0 "C3001" V 5000 6100 50  0000 L CNN
 F 1 "107CKS016M 100UF" H 4100 6250 50  0001 L CNN
 F 2 "Capacitor_THT:CP_Radial_D5.0mm_P2.00mm" H 4950 6350 50  0001 C CNN
@@
 AR Path="/D16552B4/5FA17F52/5F59CDBA" Ref="C1202"  Part="1"
 AR Path="/D16552B4/5FA17F6C/5F59CDBA" Ref="C2102"  Part="1"
-F 0 "C302" V 5100 6200 50  0000 L CNN
+F 0 "C3002" V 5100 6200 50  0000 L CNN
 F 1 "107CKS016M 100UF" H 3900 6450 50  0001 L CNN
 F 2 "Capacitor_THT:CP_Radial_D5.0mm_P2.00mm" H 5050 6450 50  0001 C CNN

Commit message: Cleanup, re-ordering
Changed lines of the file:
@@
 $Descr A4 11693 8268
 encoding utf-8
-Sheet 30 87
+Sheet 3 87
 Title "Boat Control Hat"
 Date "2020-07-09"
@@
 AR Path="/D16552B4/5FA17F52/D2F3142C" Ref="#PWR01202"  Part="1"
 AR Path="/D16552B4/5FA17F6C/D2F3142C" Ref="#PWR02102"  Part="1"
-F 0 "#PWR03002" H 5800 3000 50  0001 C CNN
+F 0 "#PWR0302" H 5800 3000 50  0001 C CNN
 F 1 "GND" H 5805 3077 50  0000 C CNN
 F 2 "" H 5800 3250 50  0001 C CNN
@@
 AR Path="/D16552B4/5FA17F52/81A9CC8E" Ref="RN1202"  Part="1"
 AR Path="/D16552B4/5FA17F6C/81A9CC8E" Ref="RN2102"  Part="1"
-F 0 "RN3002" H 4500 900 50  0000 L CNN
+F 0 "RN302" H 4500 900 50  0000 L CNN
 F 1 "4116R-1-471" H 5650 900 50  0000 L CNN
 F 2 "BoatControl:DIP254P762X432-16P" V 5725 900 50  0001 C CNN
@@
 AR Path="/D16552B4/5FA17F6C/5FF784D2" Ref="RN2104"  Part="1"
 AR Path="/D16552B4/5FA17F86/5FF784D2" Ref="RN3004"  Part="1"
-F 0 "RN3004" V 6450 7000 50  0000 C CNN
+F 0 "RN304" V 6450 7000 50  0000 C CNN
 F 1 "4116R-1-103LF" V 6350 7000 50  0000 C CNN
 F 2 "DIP787W49P254L2197H469Q16N" H 7300 7400 50  0001 L CNN
@@
 AR Path="/D16552B4/5FA17F6C/5FD52518" Ref="RN2101"  Part="1"
 AR Path="/D16552B4/5FA17F86/5FD52518" Ref="RN3001"  Part="1"
-F 0 "RN3001" V 4650 7000 50  0000 C CNN
+F 0 "RN301" V 4650 7000 50  0000 C CNN
 F 1 "4116R-1-103LF" V 4550 7000 50  0001 C CNN
 F 2 "DIP787W49P254L2197H469Q16N" H 5500 7400 50  0001 L CNN
@@
 AR Path="/D16552B4/5FA17F6C/5FF7A29F" Ref="#PWR02103"  Part="1"
 AR Path="/D16552B4/5FA17F86/5FF7A29F" Ref="#PWR03003"  Part="1"
-F 0 "#PWR03003" H 6550 7150 50  0001 C CNN
+F 0 "#PWR0303" H 6550 7150 50  0001 C CNN
 F 1 "+5V" H 6565 7473 50  0000 C CNN
 F 2 "" H 6550 7300 50  0001 C CNN
@@
 AR Path="/D16552B4/5FA17F52/D2B5CDA2" Ref="U1201"  Part="1"
 AR Path="/D16552B4/5FA17F6C/D2B5CDA2" Ref="U2101"  Part="1"
-F 0 "U3001" H 5050 3050 50  0000 L CNN
+F 0 "U301" H 5050 3050 50  0000 L CNN
 F 1 "ULN2803A" H 4900 3750 50  0000 L CNN
 F 2 "Package_DIP:DIP-18_W7.62mm" H 5150 2600 50  0001 L CNN
@@
 AR Path="/D16552B4/5FA17F52/5F542D5F" Ref="RN1203"  Part="1"
 AR Path="/D16552B4/5FA17F6C/5F542D5F" Ref="RN2103"  Part="1"
-F 0 "RN3003" H 5200 6800 50  0000 L CNN
+F 0 "RN303" H 5200 6800 50  0000 L CNN
 F 1 "4120R-1-103LF" H 5000 6700 50  0000 L CNN
 F 2 "BoatControl:DIP254P762X432-16P" V 5825 7100 50  0001 C CNN
@@
 AR Path="/D16552B4/5FA17F52/D2F3142D" Ref="#PWR01201"  Part="1"
 AR Path="/D16552B4/5FA17F6C/D2F3142D" Ref="#PWR02101"  Part="1"
-F 0 "#PWR03001" H 4800 2700 50  0001 C CNN
+F 0 "#PWR0301" H 4800 2700 50  0001 C CNN
 F 1 "+12P" H 4650 2950 50  0000 C CNN
 F 2 "" H 4800 2850 50  0001 C CNN
@@
 AR Path="/D16552B4/5FA17F52/5FDBB725" Ref="C1208"  Part="1"
 AR Path="/D16552B4/5FA17F6C/5FDBB725" Ref="C2108"  Part="1"
-F 0 "C3008" V 5700 6550 50  0000 L CNN
+F 0 "C308" V 5700 6550 50  0000 L CNN
 F 1 "107CKS016M 100UF" H 4500 6700 50  0001 L CNN
 F 2 "Capacitor_THT:CP_Radial_D5.0mm_P2.00mm" H 5650 6700 50  0001 C CNN
@@
 AR Path="/D16552B4/5FA17F52/5FDBB72C" Ref="C1207"  Part="1"
 AR Path="/D16552B4/5FA17F6C/5FDBB72C" Ref="C2107"  Part="1"
-F 0 "C3007" V 5600 6450 50  0000 L CNN
+F 0 "C307" V 5600 6450 50  0000 L CNN
 F 1 "107CKS016M 100UF" H 4450 6600 50  0001 L CNN
 F 2 "Capacitor_THT:CP_Radial_D5.0mm_P2.00mm" H 5550 6600 50  0001 C CNN
@@
 AR Path="/D16552B4/5FA17F52/5FDB4626" Ref="C1206"  Part="1"
 AR Path="/D16552B4/5FA17F6C/5FDB4626" Ref="C2106"  Part="1"
-F 0 "C3006" V 5500 6300 50  0000 L CNN
+F 0 "C306" V 5500 6300 50  0000 L CNN
 F 1 "107CKS016M 100UF" H 4300 6450 50  0001 L CNN
 F 2 "Capacitor_THT:CP_Radial_D5.0mm_P2.00mm" H 5450 6450 50  0001 C CNN
@@
 AR Path="/D16552B4/5FA17F52/5FDB462D" Ref="C1205"  Part="1"
 AR Path="/D16552B4/5FA17F6C/5FDB462D" Ref="C2105"  Part="1"
-F 0 "C3005" V 5400 6200 50  0000 L CNN
+F 0 "C305" V 5400 6200 50  0000 L CNN
 F 1 "107CKS016M 100UF" H 4250 6350 50  0001 L CNN
 F 2 "Capacitor_THT:CP_Radial_D5.0mm_P2.00mm" H 5350 6350 50  0001 C CNN
@@
 AR Path="/D16552B4/5FA17F52/5FD94312" Ref="C1204"  Part="1"
 AR Path="/D16552B4/5FA17F6C/5FD94312" Ref="C2104"  Part="1"
-F 0 "C3004" V 5300 6550 50  0000 L CNN
+F 0 "C304" V 5300 6550 50  0000 L CNN
 F 1 "107CKS016M 100UF" H 4100 6700 50  0001 L CNN
 F 2 "Capacitor_THT:CP_Radial_D5.0mm_P2.00mm" H 5250 6700 50  0001 C CNN
@@
 AR Path="/D16552B4/5FA17F52/5FD94319" Ref="C1203"  Part="1"
 AR Path="/D16552B4/5FA17F6C/5FD94319" Ref="C2103"  Part="1"
-F 0 "C3003" V 5200 6450 50  0000 L CNN
+F 0 "C303" V 5200 6450 50  0000 L CNN
 F 1 "107CKS016M 100UF" H 4050 6600 50  0001 L CNN
 F 2 "Capacitor_THT:CP_Radial_D5.0mm_P2.00mm" H 5150 6600 50  0001 C CNN
@@
 AR Path="/D16552B4/5FA17F52/5F542D59" Ref="C1201"  Part="1"
 AR Path="/D16552B4/5FA17F6C/5F542D59" Ref="C2101"  Part="1"
-F 0 "C3001" V 5000 6100 50  0000 L CNN
+F 0 "C301" V 5000 6100 50  0000 L CNN
 F 1 "107CKS016M 100UF" H 4100 6250 50  0001 L CNN
 F 2 "Capacitor_THT:CP_Radial_D5.0mm_P2.00mm" H 4950 6350 50  0001 C CNN
@@
 AR Path="/D16552B4/5FA17F52/5F59CDBA" Ref="C1202"  Part="1"
 AR Path="/D16552B4/5FA17F6C/5F59CDBA" Ref="C2102"  Part="1"
-F 0 "C3002" V 5100 6200 50  0000 L CNN
+F 0 "C302" V 5100 6200 50  0000 L CNN
 F 1 "107CKS016M 100UF" H 3900 6450 50  0001 L CNN
 F 2 "Capacitor_THT:CP_Radial_D5.0mm_P2.00mm" H 5050 6450 50  0001 C CNN

Commit message: Rotate multivibrators
Connections:
- wire segments 284 -> 253
Other:
- note added: "Amplify 5V logic signals to 12V\nto operate relay coils, includes filtering"
- note added: "Resistors for multivibrator pull-up\nand timer circuits for relay pulses.\n\nThese can be swapped for higher/lower\nvalues as needed for longer pulses or\nmore noise resistance."
- note removed: "Amplify 5V logic signals to 12V to operate relay coils, includes filtering"
- note removed: "Resistors for multivibrator pull-up and timer circuits for relay pulses.\nThese can be swapped for higher/lower values as needed for longer pulses or more noise resistance."
- moved on the sheet: C301, C302, C303, C304, C305, C306, C307, C308, RN302, RN303, U301

Commit message: Nice
Parts:
- RN3002: value 4116R-1-471 -> 470 Ohm; Field4 (none) -> 4116R-1-471
Connections:
- wire segments 253 -> 230
Other:
- note added: "Amplify 5V logic signals to 12V\nto operate relay coils,\nincludes filtering"
- note added: "Resistors for LEDs"
- note removed: "Amplify 5V logic signals to 12V\nto operate relay coils, includes filtering"
- note removed: "Resistors for diodes"
- moved on the sheet: RN302

Commit message: Fix up 10/16A
Connections:
- wire segments 230 -> 226
Changed lines of the file:
@@
 	0    1    1    0
 $EndComp
-Wire Wire Line
-	7600 7200 7600 7100
-Wire Wire Line
-	8150 7200 7600 7200
-Wire Wire Line
-	7750 7150 7750 7100
-Wire Wire Line
-	8100 7150 7750 7150
 Text HLabel 4250 1900 0    50   Output ~ 0
 AN_OFF_C1
@@
 Text Notes 6450 2450 2    50   ~ 0
 Amplify 5V logic signals to 12V\nto operate relay coils,\nincludes filtering
-Text HLabel 7250 7100 3    50   Output ~ 0
+Text HLabel 9050 5250 2    50   Output ~ 0
 OUT_C4
 $Comp
@@
 Text HLabel 9050 3450 2    50   Output ~ 0
 OUT_C2
-Text HLabel 9050 5250 2    50   Output ~ 0
+Text HLabel 9050 4350 2    50   Output ~ 0
 OUT_C3
 Text Notes 7400 2800 2    50   ~ 0

Commit message: Cleaner flow
Parts:
- RN3002: value 470 Ohm -> 4116R-1-471; Field4 4116R-1-471 -> (none)
- RN304: value 4116R-1-103LF -> 10K Ohm; Field12 (none) -> 4116R-1-103LF
Changed lines of the file:
@@
 	1950 3450 1950 3350
-$Comp
-L BoatControl:4116R-1-103LF RN304
-U 1 1 5FF784D2
-P 1950 4950
-AR Path="/D16552B4/5FA17F38/5FF784D2" Ref="RN304"  Part="1"
-AR Path="/D16552B4/5FA17F52/5FF784D2" Ref="RN1204"  Part="1"
-AR Path="/D16552B4/5FA17F6C/5FF784D2" Ref="RN2104"  Part="1"
-AR Path="/D16552B4/5FA17F86/5FF784D2" Ref="RN3004"  Part="1"
-F 0 "RN304" V 1850 4650 50  0000 C CNN
-F 1 "4116R-1-103LF" V 1750 4650 50  0000 C CNN
-F 2 "DIP787W49P254L2197H469Q16N" H 2700 5050 50  0001 L CNN
-F 3 "http://www.bourns.com/pdfs/4100R.pdf" H 2700 4950 50  0001 L CNN
-F 4 "Bourns Isolated Resistor Array 10k +/-2% 8 Resistors, 2.25W Total, DIP package 4100R Through Hole" H 2700 4850 50  0001 L CNN "Description"
-F 5 "4.69" H 2700 4750 50  0001 L CNN "Height"
-F 6 "Bourns" H 2700 4650 50  0001 L CNN "Manufacturer_Name"
-F 7 "4116R-1-103LF" H 2700 4550 50  0001 L CNN "Manufacturer_Part_Number"
-F 8 "4116R-1-103LF" H 2700 4450 50  0001 L CNN "Arrow Part Number"
-F 9 "https://www.arrow.com/en/products/4116r-1-103lf/bourns" H 2700 4350 50  0001 L CNN "Arrow Price/Stock"
-F 10 "652-4116R-1LF-10K" H 2700 4250 50  0001 L CNN "Mouser Part Number"
-F 11 "https://www.mouser.co.uk/ProductDetail/Bourns/4116R-1-103LF?qs=jew24QT47erdvJ3qcVRaMA%3D%3D" H 2700 4150 50  0001 L CNN "Mouser Price/Stock"
-	1    1950 4950
-	1    0    0    1
-$EndComp
-$Comp
-L BoatControl:4116R-1-103LF RN301
-U 1 1 5FD52518
-P 1950 3150
-AR Path="/D16552B4/5FA17F38/5FD52518" Ref="RN301"  Part="1"
-AR Path="/D16552B4/5FA17F52/5FD52518" Ref="RN1201"  Part="1"
-AR Path="/D16552B4/5FA17F6C/5FD52518" Ref="RN2101"  Part="1"
-AR Path="/D16552B4/5FA17F86/5FD52518" Ref="RN3001"  Part="1"
-F 0 "RN301" V 1850 2850 50  0000 C CNN
-F 1 "4116R-1-103LF" V 1750 2850 50  0000 C CNN
-F 2 "DIP787W49P254L2197H469Q16N" H 2700 3250 50  0001 L CNN
-F 3 "http://www.bourns.com/pdfs/4100R.pdf" H 2700 3150 50  0001 L CNN
-F 4 "Bourns Isolated Resistor Array 10k +/-2% 8 Resistors, 2.25W Total, DIP package 4100R Through Hole" H 2700 3050 50  0001 L CNN "Description"
-F 5 "4.69" H 2700 2950 50  0001 L CNN "Height"
-F 6 "Bourns" H 2700 2850 50  0001 L CNN "Manufacturer_Name"
-F 7 "4116R-1-103LF" H 2700 2750 50  0001 L CNN "Manufacturer_Part_Number"
-F 8 "4116R-1-103LF" H 2700 2650 50  0001 L CNN "Arrow Part Number"
-F 9 "https://www.arrow.com/en/products/4116r-1-103lf/bourns" H 2700 2550 50  0001 L CNN "Arrow Price/Stock"
-F 10 "652-4116R-1LF-10K" H 2700 2450 50  0001 L CNN "Mouser Part Number"
-F 11 "https://www.mouser.co.uk/ProductDetail/Bourns/4116R-1-103LF?qs=jew24QT47erdvJ3qcVRaMA%3D%3D" H 2700 2350 50  0001 L CNN "Mouser Price/Stock"
-	1    1950 3150
-	1    0    0    1
-$EndComp
 $Comp
 L power:+5V #PWR0303
@@
 AR Path="/D16552B4/5FA17F6C/5F542D5F" Ref="RN2103"  Part="1"
 F 0 "RN303" H 2000 3450 50  0000 L CNN
-F 1 "4120R-1-103LF" H 1800 3350 50  0000 L CNN
+F 1 "4120R-1-103LF" H 1800 3350 50  0001 L CNN
 F 2 "BoatControl:DIP254P762X432-16P" V 2625 3750 50  0001 C CNN
 F 3 "~" H 2150 3750 50  0001 C CNN
@@
 AR Path="/D16552B4/5FA17F52/81A9CC8E" Ref="RN1202"  Part="1"
 AR Path="/D16552B4/5FA17F6C/81A9CC8E" Ref="RN2102"  Part="1"
-F 0 "RN302" V 6600 3600 50  0000 L CNN
-F 1 "470 Ohm" V 6700 3550 50  0000 L CNN
+F 0 "RN302" V 6650 3600 50  0000 L CNN
+F 1 "4116R-1-471" V 6700 3550 50  0001 L CNN
 F 2 "BoatControl:DIP254P762X432-16P" V 7675 3700 50  0001 C CNN
 F 3 "https://www.bourns.com/docs/Product-Datasheets/4100R.pdf" H 7200 3700 50  0001 C CNN
-F 4 "4116R-1-471" V 7200 3700 50  0001 C CNN "Field4"
+F 4 "" V 7200 3700 50  0001 C CNN "Field4"
 	1    7200 3700
 	0    1    1    0
@@
 Wire Wire Line
 	6550 4000 7000 4000
+$Comp
+L BoatControl:4116R-1-103LF RN301
+U 1 1 5FD52518
+P 1950 3150
+AR Path="/D16552B4/5FA17F38/5FD52518" Ref="RN301"  Part="1"
+AR Path="/D16552B4/5FA17F52/5FD52518" Ref="RN1201"  Part="1"
+AR Path="/D16552B4/5FA17F6C/5FD52518" Ref="RN2101"  Part="1"
+AR Path="/D16552B4/5FA17F86/5FD52518" Ref="RN3001"  Part="1"
+F 0 "RN301" V 1850 2850 50  0000 C CNN
+F 1 "4116R-1-103LF" V 1750 2850 50  0001 C CNN
+F 2 "DIP787W49P254L2197H469Q16N" H 2700 3250 50  0001 L CNN
+F 3 "http://www.bourns.com/pdfs/4100R.pdf" H 2700 3150 50  0001 L CNN
+F 4 "Bourns Isolated Resistor Array 10k +/-2% 8 Resistors, 2.25W Total, DIP package 4100R Through Hole" H 2700 3050 50  0001 L CNN "Description"
+F 5 "4.69" H 2700 2950 50  0001 L CNN "Height"
+F 6 "Bourns" H 2700 2850 50  0001 L CNN "Manufacturer_Name"
+F 7 "4116R-1-103LF" H 2700 2750 50  0001 L CNN "Manufacturer_Part_Number"
+F 8 "4116R-1-103LF" H 2700 2650 50  0001 L CNN "Arrow Part Number"
+F 9 "https://www.arrow.com/en/products/4116r-1-103lf/bourns" H 2700 2550 50  0001 L CNN "Arrow Price/Stock"
+F 10 "652-4116R-1LF-10K" H 2700 2450 50  0001 L CNN "Mouser Part Number"
+F 11 "https://www.mouser.co.uk/ProductDetail/Bourns/4116R-1-103LF?qs=jew24QT47erdvJ3qcVRaMA%3D%3D" H 2700 2350 50  0001 L CNN "Mouser Price/Stock"
+	1    1950 3150
+	1    0    0    1
+$EndComp
+$Comp
+L BoatControl:4116R-1-103LF RN304
+U 1 1 5FF784D2
+P 1950 4950
+AR Path="/D16552B4/5FA17F38/5FF784D2" Ref="RN304"  Part="1"
+AR Path="/D16552B4/5FA17F52/5FF784D2" Ref="RN1204"  Part="1"
+AR Path="/D16552B4/5FA17F6C/5FF784D2" Ref="RN2104"  Part="1"
+AR Path="/D16552B4/5FA17F86/5FF784D2" Ref="RN3004"  Part="1"
+F 0 "RN304" V 1850 4650 50  0000 C CNN
+F 1 "10K Ohm" V 1750 4650 50  0001 C CNN
+F 2 "DIP787W49P254L2197H469Q16N" H 2700 5050 50  0001 L CNN
+F 3 "http://www.bourns.com/pdfs/4100R.pdf" H 2700 4950 50  0001 L CNN
+F 4 "Bourns Isolated Resistor Array 10k +/-2% 8 Resistors, 2.25W Total, DIP package 4100R Through Hole" H 2700 4850 50  0001 L CNN "Description"
+F 5 "4.69" H 2700 4750 50  0001 L CNN "Height"
+F 6 "Bourns" H 2700 4650 50  0001 L CNN "Manufacturer_Name"
+F 7 "4116R-1-103LF" H 2700 4550 50  0001 L CNN "Manufacturer_Part_Number"
+F 8 "4116R-1-103LF" H 2700 4450 50  0001 L CNN "Arrow Part Number"
+F 9 "https://www.arrow.com/en/products/4116r-1-103lf/bourns" H 2700 4350 50  0001 L CNN "Arrow Price/Stock"
+F 10 "652-4116R-1LF-10K" H 2700 4250 50  0001 L CNN "Mouser Part Number"
+F 11 "https://www.mouser.co.uk/ProductDetail/Bourns/4116R-1-103LF?qs=jew24QT47erdvJ3qcVRaMA%3D%3D" H 2700 4150 50  0001 L CNN "Mouser Price/Stock"
+F 12 "4116R-1-103LF" V 1950 4950 50  0001 C CNN "Field12"
+	1    1950 4950
+	1    0    0    1
+$EndComp
 $EndSCHEMATC
