File: boatcontrol/3AmpBlock.sch (KiCad schematic (older format))
At the start: 13 parts, among them U3001 ULN2803A

Commit message: Add filter caps
Changed lines of the file:
@@
 $Descr A4 11693 8268
 encoding utf-8
-Sheet 3 87
+Sheet 30 87
 Title "Boat Control Hat"
 Date "2020-07-09"
@@
 AR Path="/D16552B4/5FA17F52/5F59CDBA" Ref="C1202"  Part="1"
 AR Path="/D16552B4/5FA17F6C/5F59CDBA" Ref="C2102"  Part="1"
-F 0 "C302" V 4100 2550 50  0000 L CNN
+F 0 "C3002" V 4100 2550 50  0000 L CNN
 F 1 "107CKS016M 100UF" H 3000 2500 50  0001 L CNN
 F 2 "Capacitor_THT:CP_Radial_D5.0mm_P2.00mm" H 4150 2500 50  0001 C CNN
@@
 AR Path="/D16552B4/5FA17F52/5F542D59" Ref="C1201"  Part="1"
 AR Path="/D16552B4/5FA17F6C/5F542D59" Ref="C2101"  Part="1"
-F 0 "C301" V 4100 2350 50  0000 L CNN
+F 0 "C3001" V 4100 2350 50  0000 L CNN
 F 1 "107CKS016M 100UF" H 3300 2200 50  0001 L CNN
 F 2 "Capacitor_THT:CP_Radial_D5.0mm_P2.00mm" H 4150 2300 50  0001 C CNN
@@
 AR Path="/D16552B4/5FA17F52/5FD94319" Ref="C1203"  Part="1"
 AR Path="/D16552B4/5FA17F6C/5FD94319" Ref="C2103"  Part="1"
-F 0 "C303" V 4100 3350 50  0000 L CNN
+F 0 "C3003" V 4100 3350 50  0000 L CNN
 F 1 "107CKS016M 100UF" H 3050 3300 50  0001 L CNN
 F 2 "Capacitor_THT:CP_Radial_D5.0mm_P2.00mm" H 4150 3300 50  0001 C CNN
@@
 AR Path="/D16552B4/5FA17F52/5FD94312" Ref="C1204"  Part="1"
 AR Path="/D16552B4/5FA17F6C/5FD94312" Ref="C2104"  Part="1"
-F 0 "C304" V 4100 3550 50  0000 L CNN
+F 0 "C3004" V 4100 3550 50  0000 L CNN
 F 1 "107CKS016M 100UF" H 3000 3500 50  0001 L CNN
 F 2 "Capacitor_THT:CP_Radial_D5.0mm_P2.00mm" H 4150 3500 50  0001 C CNN
@@
 AR Path="/D16552B4/5FA17F52/5FDB462D" Ref="C1205"  Part="1"
 AR Path="/D16552B4/5FA17F6C/5FDB462D" Ref="C2105"  Part="1"
-F 0 "C305" V 4100 4350 50  0000 L CNN
+F 0 "C3005" V 4100 4350 50  0000 L CNN
 F 1 "107CKS016M 100UF" H 3050 4300 50  0001 L CNN
 F 2 "Capacitor_THT:CP_Radial_D5.0mm_P2.00mm" H 4150 4300 50  0001 C CNN
@@
 AR Path="/D16552B4/5FA17F52/5FDB4626" Ref="C1206"  Part="1"
 AR Path="/D16552B4/5FA17F6C/5FDB4626" Ref="C2106"  Part="1"
-F 0 "C306" V 4100 4550 50  0000 L CNN
+F 0 "C3006" V 4100 4550 50  0000 L CNN
 F 1 "107CKS016M 100UF" H 3000 4500 50  0001 L CNN
 F 2 "Capacitor_THT:CP_Radial_D5.0mm_P2.00mm" H 4150 4500 50  0001 C CNN
@@
 AR Path="/D16552B4/5FA17F52/5FDBB72C" Ref="C1207"  Part="1"
 AR Path="/D16552B4/5FA17F6C/5FDBB72C" Ref="C2107"  Part="1"
-F 0 "C307" V 4100 5350 50  0000 L CNN
+F 0 "C3007" V 4100 5350 50  0000 L CNN
 F 1 "107CKS016M 100UF" H 3050 5300 50  0001 L CNN
 F 2 "Capacitor_THT:CP_Radial_D5.0mm_P2.00mm" H 4150 5300 50  0001 C CNN
@@
 AR Path="/D16552B4/5FA17F52/5FDBB725" Ref="C1208"  Part="1"
 AR Path="/D16552B4/5FA17F6C/5FDBB725" Ref="C2108"  Part="1"
-F 0 "C308" V 4100 5550 50  0000 L CNN
+F 0 "C3008" V 4100 5550 50  0000 L CNN
 F 1 "107CKS016M 100UF" H 3000 5500 50  0001 L CNN
 F 2 "Capacitor_THT:CP_Radial_D5.0mm_P2.00mm" H 4150 5500 50  0001 C CNN
@@
 AR Path="/D16552B4/5FA17F52/D2F3142D" Ref="#PWR01201"  Part="1"
 AR Path="/D16552B4/5FA17F6C/D2F3142D" Ref="#PWR02101"  Part="1"
-F 0 "#PWR0301" H 6400 3050 50  0001 C CNN
+F 0 "#PWR03001" H 6400 3050 50  0001 C CNN
 F 1 "+12P" H 6250 3300 50  0000 C CNN
 F 2 "" H 6400 3200 50  0001 C CNN
@@
 AR Path="/D16552B4/5FA17F52/D2B5CDA2" Ref="U1201"  Part="1"
 AR Path="/D16552B4/5FA17F6C/D2B5CDA2" Ref="U2101"  Part="1"
-F 0 "U301" H 5950 3300 50  0000 L CNN
+F 0 "U3001" H 5950 3300 50  0000 L CNN
 F 1 "ULN2803A" H 5800 4000 50  0000 L CNN
 F 2 "Package_DIP:DIP-18_W7.62mm" H 6050 2850 50  0001 L CNN
@@
 AR Path="/D16552B4/5FA17F52/D2F3142C" Ref="#PWR01202"  Part="1"
 AR Path="/D16552B4/5FA17F6C/D2F3142C" Ref="#PWR02102"  Part="1"
-F 0 "#PWR0302" H 6000 3950 50  0001 C CNN
+F 0 "#PWR03002" H 6000 3950 50  0001 C CNN
 F 1 "GND" H 6005 4027 50  0000 C CNN
 F 2 "" H 6000 4200 50  0001 C CNN
@@
 AR Path="/D16552B4/5FA17F6C/5FF7A29F" Ref="#PWR02103"  Part="1"
 AR Path="/D16552B4/5FA17F86/5FF7A29F" Ref="#PWR03003"  Part="1"
-F 0 "#PWR0303" H 1950 4800 50  0001 C CNN
+F 0 "#PWR03003" H 1950 4800 50  0001 C CNN
 F 1 "+5V" H 1965 5123 50  0000 C CNN
 F 2 "" H 1950 4950 50  0001 C CNN
@@
 AR Path="/D16552B4/5FA17F52/5F542D5F" Ref="RN1203"  Part="1"
 AR Path="/D16552B4/5FA17F6C/5F542D5F" Ref="RN2103"  Part="1"
-F 0 "RN303" H 2000 3450 50  0000 L CNN
+F 0 "RN3003" H 2000 3450 50  0000 L CNN
 F 1 "4120R-1-103LF" H 1800 3350 50  0001 L CNN
 F 2 "BoatControl:DIP254P762X432-16P" V 2625 3750 50  0001 C CNN
@@
 AR Path="/D16552B4/5FA17F52/81A9CC8E" Ref="RN1202"  Part="1"
 AR Path="/D16552B4/5FA17F6C/81A9CC8E" Ref="RN2102"  Part="1"
-F 0 "RN302" V 6650 3600 50  0000 L CNN
+F 0 "RN3002" V 6650 3600 50  0000 L CNN
 F 1 "4116R-1-471" V 6700 3550 50  0001 L CNN
 F 2 "BoatControl:DIP254P762X432-16P" V 7675 3700 50  0001 C CNN
@@
 AR Path="/D16552B4/5FA17F6C/5FD52518" Ref="RN2101"  Part="1"
 AR Path="/D16552B4/5FA17F86/5FD52518" Ref="RN3001"  Part="1"
-F 0 "RN301" V 1850 2850 50  0000 C CNN
+F 0 "RN3001" V 1850 2850 50  0000 C CNN
 F 1 "4116R-1-103LF" V 1750 2850 50  0001 C CNN
 F 2 "DIP787W49P254L2197H469Q16N" H 2700 3250 50  0001 L CNN
@@
 AR Path="/D16552B4/5FA17F6C/5FF784D2" Ref="RN2104"  Part="1"
 AR Path="/D16552B4/5FA17F86/5FF784D2" Ref="RN3004"  Part="1"
-F 0 "RN304" V 1850 4650 50  0000 C CNN
+F 0 "RN3004" V 1850 4650 50  0000 C CNN
 F 1 "10K Ohm" V 1750 4650 50  0001 C CNN
 F 2 "DIP787W49P254L2197H469Q16N" H 2700 5050 50  0001 L CNN
