File: boatcontrol/10_16AmpBlock.sch (KiCad schematic (older format))
At the start: 13 parts, among them U6101 ULN2803A

Commit message: Move In
Parts:
- C7001, C7002, C7003, C7004, C7005, C7006, C7007, C7008: value 1uF -> 1µF
- RN6101, RN6104: value 100K Ohm -> 100KΩ
- RN6102: value 680Ohm -> 680Ω
- RN7003: value 10M Ohm -> 10MΩ
Connections:
- net 10AC1/OFF: now also U6101.11 (O8); no longer U6101.17 (O2)
- net 10AC1/OFF_LED: now also RN6102.8 (R8.1); no longer RN6102.2 (R2.1)
- net 10AC1/ON: now also U6101.12 (O7); no longer U6101.18 (O1)
- net 10AC1/ON_LED: now also RN6102.7 (R7.1); no longer RN6102.1 (R1.1)
- net 10AC2/OFF: now also U6101.13 (O6); no longer U6101.15 (O4)
- net 10AC2/OFF_LED: now also RN6102.6 (R6.1); no longer RN6102.4 (R4.1)
- net 10AC2/ON: now also U6101.14 (O5); no longer U6101.16 (O3)
- net 10AC2/ON_LED: now also RN6102.5 (R5.1); no longer RN6102.3 (R3.1)
- net 16AC1/OFF: now also U6101.15 (O4); no longer U6101.13 (O6)
- net 16AC1/OFF_LED: now also RN6102.4 (R4.1); no longer RN6102.6 (R6.1)
- net 16AC1/ON: now also U6101.16 (O3); no longer U6101.14 (O5)
- net 16AC1/ON_LED: now also RN6102.3 (R3.1); no longer RN6102.5 (R5.1)
- net 16AC2/OFF: now also U6101.17 (O2); no longer U6101.11 (O8)
- net 16AC2/OFF_LED: now also RN6102.2 (R2.1); no longer RN6102.8 (R8.1)
- net 16AC2/ON: now also U6101.18 (O1); no longer U6101.12 (O7)
- net 16AC2/ON_LED: now also RN6102.1 (R1.1); no longer RN6102.7 (R7.1)
- removed net OFF_COIL: RN6102.11 (R6.2), RN6102.13 (R4.2), RN6102.15 (R2.2), RN6102.9 (R8.2)
- removed net ON_COIL: RN6102.10 (R7.2), RN6102.12 (R5.2), RN6102.14 (R3.2), RN6102.16 (R1.2)
- new net 10AC1/OFF_COIL: RN6102.9 (R8.2)
- new net 10AC1/ON_COIL: RN6102.10 (R7.2)
- new net 10AC2/OFF_COIL: RN6102.11 (R6.2)
- new net 10AC2/ON_COIL: RN6102.12 (R5.2)
- new net 16AC1/OFF_COIL: RN6102.13 (R4.2)
- new net 16AC1/ON_COIL: RN6102.14 (R3.2)
- new net 16AC2/OFF_COIL: RN6102.15 (R2.2)
- new net 16AC2/ON_COIL: RN6102.16 (R1.2)
Changed lines of the file:
@@
 Wire Wire Line
 	6900 3500 7050 3500
-$Sheet
-S 8550 4850 1000 700
-U 604748F7
-F0 "16AC2" 50
-F1 "16AmpCircuit.sch" 50
-F2 "ON" B L 8550 4900 50
-F3 "OFF" B L 8550 5000 50
-F4 "ON_LED" I R 9550 5200 50
-F5 "OFF_LED" I R 9550 5300 50
-F6 "OUT" O R 9550 5500 50
-F7 "IN" I L 8550 5450 50
-$EndSheet
-$Sheet
-S 8550 3050 1000 700
-U 60474907
-F0 "10AC2" 50
-F1 "10AmpCircuit.sch" 50
-F2 "ON" B L 8550 3100 50
-F3 "OFF" B L 8550 3200 50
-F4 "ON_LED" I R 9550 3450 50
-F5 "OFF_LED" I R 9550 3550 50
-F6 "OUT" O R 9550 3700 50
-F7 "IN" I L 8550 3650 50
-$EndSheet
 Text HLabel 8550 2750 0    50   Input ~ 0
 IN_C1
@@
 AR Path="/D1BB8DB4/5F75E923/60474926" Ref="RN7002"  Part="1"
 F 0 "RN6102" V 10200 4350 50  0000 L CNN
-F 1 "680Ohm" V 9800 3750 50  0001 L CNN
+F 1 "680Ω" V 9800 3750 50  0001 L CNN
 F 2 "BoatControl:DIP254P762X432-16P" V 10775 3900 50  0001 C CNN
 F 3 "https://www.bourns.com/docs/Product-Datasheets/4100R.pdf" H 10300 3900 50  0001 C CNN
@@
 AR Path="/D1BB8DB4/5F76AF55/62B5C7B5" Ref="C6101"  Part="1"
 F 0 "C6101" V 4600 2550 50  0000 L CNN
-F 1 "1uF" H 3800 2400 50  0001 L CNN
+F 1 "1µF" H 3800 2400 50  0001 L CNN
 F 2 "Capacitor_THT:C_Disc_D7.5mm_W5.0mm_P5.00mm" H 4650 2500 50  0001 C CNN
 F 3 "https://www.digikey.com/en/products/detail/kemet/C330C105K5R5TA7301/3726162" H 4650 2500 50  0001 C CNN
@@
 AR Path="/D1BB8DB4/5F76AF55/62B76848" Ref="C6102"  Part="1"
 F 0 "C6102" V 4600 2750 50  0000 L CNN
-F 1 "1uF" H 3800 2600 50  0001 L CNN
+F 1 "1µF" H 3800 2600 50  0001 L CNN
 F 2 "Capacitor_THT:C_Disc_D7.5mm_W5.0mm_P5.00mm" H 4650 2700 50  0001 C CNN
 F 3 "https://www.digikey.com/en/products/detail/kemet/C330C105K5R5TA7301/3726162" H 4650 2700 50  0001 C CNN
@@
 AR Path="/D1BB8DB4/5F76AF55/62B86A50" Ref="C6103"  Part="1"
 F 0 "C6103" V 4600 3550 50  0000 L CNN
-F 1 "1uF" H 3800 3400 50  0001 L CNN
+F 1 "1µF" H 3800 3400 50  0001 L CNN
 F 2 "Capacitor_THT:C_Disc_D7.5mm_W5.0mm_P5.00mm" H 4650 3500 50  0001 C CNN
 F 3 "https://www.digikey.com/en/products/detail/kemet/C330C105K5R5TA7301/3726162" H 4650 3500 50  0001 C CNN
@@
 AR Path="/D1BB8DB4/5F76AF55/62B939DB" Ref="C6104"  Part="1"
 F 0 "C6104" V 4600 3750 50  0000 L CNN
-F 1 "1uF" H 3800 3600 50  0001 L CNN
+F 1 "1µF" H 3800 3600 50  0001 L CNN
 F 2 "Capacitor_THT:C_Disc_D7.5mm_W5.0mm_P5.00mm" H 4650 3700 50  0001 C CNN
 F 3 "https://www.digikey.com/en/products/detail/kemet/C330C105K5R5TA7301/3726162" H 4650 3700 50  0001 C CNN
@@
 AR Path="/D1BB8DB4/5F76AF55/62BA14CE" Ref="C6105"  Part="1"
 F 0 "C6105" V 4600 4550 50  0000 L CNN
-F 1 "1uF" H 3800 4400 50  0001 L CNN
+F 1 "1µF" H 3800 4400 50  0001 L CNN
 F 2 "Capacitor_THT:C_Disc_D7.5mm_W5.0mm_P5.00mm" H 4650 4500 50  0001 C CNN
 F 3 "https://www.digikey.com/en/products/detail/kemet/C330C105K5R5TA7301/3726162" H 4650 4500 50  0001 C CNN
@@
 AR Path="/D1BB8DB4/5F76AF55/62BAE342" Ref="C6106"  Part="1"
 F 0 "C6106" V 4600 4750 50  0000 L CNN
-F 1 "1uF" H 3800 4600 50  0001 L CNN
+F 1 "1µF" H 3800 4600 50  0001 L CNN
 F 2 "Capacitor_THT:C_Disc_D7.5mm_W5.0mm_P5.00mm" H 4650 4700 50  0001 C CNN
 F 3 "https://www.digikey.com/en/products/detail/kemet/C330C105K5R5TA7301/3726162" H 4650 4700 50  0001 C CNN
@@
 AR Path="/D1BB8DB4/5F76AF55/62BBBC28" Ref="C6107"  Part="1"
 F 0 "C6107" V 4600 5550 50  0000 L CNN
-F 1 "1uF" H 3800 5400 50  0001 L CNN
+F 1 "1µF" H 3800 5400 50  0001 L CNN
 F 2 "Capacitor_THT:C_Disc_D7.5mm_W5.0mm_P5.00mm" H 4650 5500 50  0001 C CNN
 F 3 "https://www.digikey.com/en/products/detail/kemet/C330C105K5R5TA7301/3726162" H 4650 5500 50  0001 C CNN
@@
 AR Path="/D1BB8DB4/5F76AF55/62BC8A92" Ref="C6108"  Part="1"
 F 0 "C6108" V 4600 5750 50  0000 L CNN
-F 1 "1uF" H 3800 5600 50  0001 L CNN
+F 1 "1µF" H 3800 5600 50  0001 L CNN
 F 2 "Capacitor_THT:C_Disc_D7.5mm_W5.0mm_P5.00mm" H 4650 5700 50  0001 C CNN
 F 3 "https://www.digikey.com/en/products/detail/kemet/C330C105K5R5TA7301/3726162" H 4650 5700 50  0001 C CNN
@@
 AR Path="/D1BB8DB4/5F76AF55/62CB5764" Ref="RN6103"  Part="1"
 F 0 "RN6103" V 2150 3900 50  0000 L CNN
-F 1 "10M Ohm" H 2300 3550 50  0001 L CNN
+F 1 "10MΩ" H 2300 3550 50  0001 L CNN
 F 2 "Resistor_THT:R_Array_SIP9" V 3125 3950 50  0001 C CNN
 F 3 "https://www.bourns.com/docs/Product-Datasheets/4600x.pdf" H 2650 3950 50  0001 C CNN
@@
 AR Path="/D1BB8DB4/5F75E923/630078FE" Ref="RN7001"  Part="1"
 F 0 "RN6101" V 2150 3050 50  0000 C CNN
-F 1 "100K Ohm" V 2450 2750 50  0001 C CNN
+F 1 "100KΩ" V 2450 2750 50  0001 C CNN
 F 2 "Resistor_THT:R_Array_SIP9" H 3400 3150 50  0001 L CNN
 F 3 "http://www.bourns.com/pdfs/4100R.pdf" H 3400 3050 50  0001 L CNN
@@
 AR Path="/D1BB8DB4/5F75E923/63015012" Ref="RN7004"  Part="1"
 F 0 "RN6104" V 2150 4850 50  0000 C CNN
-F 1 "100K Ohm" V 2450 4550 50  0001 C CNN
+F 1 "100KΩ" V 2450 4550 50  0001 C CNN
 F 2 "Resistor_THT:R_Array_SIP9" H 3400 4950 50  0001 L CNN
 F 3 "http://www.bourns.com/pdfs/4100R.pdf" H 3400 4850 50  0001 L CNN
@@
 	9800 4150 9550 4150
 Wire Wire Line
-	9550 5300 10050 5300
-Wire Wire Line
 	10650 4400 9800 4400
 Wire Wire Line
@@
 	10000 4100 10100 4100
 Wire Wire Line
-	10000 5200 10000 4100
-Wire Wire Line
-	9550 5200 10000 5200
-Wire Wire Line
 	10050 4200 10100 4200
 Wire Wire Line
-	10050 5300 10050 4200
-Wire Wire Line
 	10700 3150 9550 3150
 Wire Wire Line
@@
 Wire Wire Line
 	9550 2350 10550 2350
-Text HLabel 9550 2250 0    50   Input ~ 0
-OFF_COIL
-Text HLabel 9550 2350 0    50   Input ~ 0
-ON_COIL
-Text HLabel 9550 3150 0    50   Input ~ 0
-OFF_COIL
-Text HLabel 9550 3250 0    50   Input ~ 0
-ON_COIL
-Text HLabel 9550 4050 0    50   Input ~ 0
-OFF_COIL
-Text HLabel 9550 4150 0    50   Input ~ 0
-ON_COIL
-Text HLabel 9550 4950 0    50   Input ~ 0
-OFF_COIL
-Text HLabel 9550 5050 0    50   Input ~ 0
-ON_COIL
 $Sheet
-S 8550 3950 1000 700
+S 8550 4850 1000 700
+U 60474911
+F0 "10AC1" 50
+F1 "10AmpCircuit.sch" 50
+F2 "ON" B L 8550 4900 50
+F3 "OFF" B L 8550 5000 50
+F4 "ON_LED" I R 9550 5250 50
+F5 "OFF_LED" I R 9550 5350 50
+F6 "OUT" O R 9550 5500 50
+F7 "IN" I L 8550 5450 50
+F8 "ON_COIL" I R 9550 5050 50
+F9 "OFF_COIL" I R 9550 4950 50
+$EndSheet
+Wire Wire Line
+	10050 2550 9550 2550
+Wire Wire Line
+	10050 2550 10050 3500
+Wire Wire Line
+	9550 2650 10000 2650
+Wire Wire Line
+	10000 2650 10000 3600
+Wire Wire Line
+	10050 5350 9550 5350
+Wire Wire Line
+	10050 4200 10050 5350
+Wire Wire Line
+	10000 5250 9550 5250
+Wire Wire Line
+	10000 4100 10000 5250
+$Sheet
+S 8550 3050 1000 700
 U 604748FF
 F0 "16AC1" 50
 F1 "16AmpCircuit.sch" 50
+F2 "ON" B L 8550 3100 50
+F3 "OFF" B L 8550 3200 50
+F4 "ON_LED" I R 9550 3450 50
+F5 "OFF_LED" I R 9550 3550 50
+F6 "OUT" O R 9550 3700 50
+F7 "IN" I L 8550 3650 50
+F8 "ON_COIL" I R 9550 3250 50
+F9 "OFF_COIL" I R 9550 3150 50
+$EndSheet
+$Sheet
+S 8550 2150 1000 700
+U 604748F7
+F0 "16AC2" 50
+F1 "16AmpCircuit.sch" 50
+F2 "ON" B L 8550 2200 50
+F3 "OFF" B L 8550 2300 50
+F4 "ON_LED" I R 9550 2550 50
+F5 "OFF_LED" I R 9550 2650 50
+F6 "OUT" O R 9550 2800 50
+F7 "IN" I L 8550 2750 50
+F8 "ON_COIL" I R 9550 2350 50
+F9 "OFF_COIL" I R 9550 2250 50
+$EndSheet
+$Sheet
+S 8550 3950 1000 700
+U 60474907
+F0 "10AC2" 50
+F1 "10AmpCircuit.sch" 50
 F2 "ON" B L 8550 4000 50
 F3 "OFF" B L 8550 4100 50
@@
 F6 "OUT" O R 9550 4600 50
 F7 "IN" I L 8550 4550 50
+F8 "ON_COIL" I R 9550 4150 50
+F9 "OFF_COIL" I R 9550 4050 50
 $EndSheet
-$Sheet
-S 8550 2150 1000 700
-U 60474911
-F0 "10AC1" 50
-F1 "10AmpCircuit.sch" 50
-F2 "ON" B L 8550 2200 50
-F3 "OFF" B L 8550 2300 50
-F4 "ON_LED" I R 9550 2550 50
-F5 "OFF_LED" I R 9550 2650 50
-F6 "OUT" O R 9550 2800 50
-F7 "IN" I L 8550 2750 50
-$EndSheet
-Wire Wire Line
-	10050 2550 9550 2550
-Wire Wire Line
-	10050 2550 10050 3500
-Wire Wire Line
-	9550 2650 10000 2650
-Wire Wire Line
-	10000 2650 10000 3600
 $EndSCHEMATC

Commit message: Figure out wiring cluster
Changed lines of the file:
@@
 $Descr A4 11693 8268
 encoding utf-8
-Sheet 61 87
+Sheet 70 87
 Title "Boat Control Hat"
 Date "2020-07-09"
@@
 AR Path="/D1BB8DB4/5F76AF55/604747A2" Ref="#PWR06101"  Part="1"
 AR Path="/D1BB8DB4/5F75E923/604747A2" Ref="#PWR07001"  Part="1"
-F 0 "#PWR06101" H 6900 3250 50  0001 C CNN
+F 0 "#PWR07001" H 6900 3250 50  0001 C CNN
 F 1 "+12P" H 6750 3500 50  0000 C CNN
 F 2 "" H 6900 3400 50  0001 C CNN
@@
 AR Path="/D1BB8DB4/5F76AF55/604747AF" Ref="U6101"  Part="1"
 AR Path="/D1BB8DB4/5F75E923/604747AF" Ref="U7001"  Part="1"
-F 0 "U6101" H 6450 3500 50  0000 L CNN
+F 0 "U7001" H 6450 3500 50  0000 L CNN
 F 1 "ULN2803A" H 6300 4200 50  0000 L CNN
 F 2 "Package_DIP:DIP-18_W7.62mm" H 6550 3050 50  0001 L CNN
@@
 Text Notes 6950 2650 2    50   ~ 0
 Amplify 5V logic signals to 12V\nto operate relay coils,\nincludes filtering
-Text HLabel 9550 5500 2    50   Output ~ 0
+Text HLabel 9550 2800 2    50   Output ~ 0
 OUT_C4
 $Comp
@@
 AR Path="/D1BB8DB4/5F76AF55/604747C1" Ref="#PWR06102"  Part="1"
 AR Path="/D1BB8DB4/5F75E923/604747C1" Ref="#PWR07002"  Part="1"
-F 0 "#PWR06102" H 6500 4150 50  0001 C CNN
+F 0 "#PWR07002" H 6500 4150 50  0001 C CNN
 F 1 "GND" H 6505 4227 50  0000 C CNN
 F 2 "" H 6500 4400 50  0001 C CNN
@@
 AR Path="/D1BB8DB4/5F76AF55/6047484A" Ref="#PWR06103"  Part="1"
 AR Path="/D1BB8DB4/5F75E923/6047484A" Ref="#PWR07003"  Part="1"
-F 0 "#PWR06103" H 2450 5000 50  0001 C CNN
+F 0 "#PWR07003" H 2450 5000 50  0001 C CNN
 F 1 "+5V" H 2465 5323 50  0000 C CNN
 F 2 "" H 2450 5150 50  0001 C CNN
@@
 Wire Wire Line
 	6900 3500 7050 3500
-Text HLabel 8550 2750 0    50   Input ~ 0
+Text HLabel 8550 2800 0    50   Input ~ 0
 IN_C1
-Text HLabel 9550 2800 2    50   Output ~ 0
+Text HLabel 9550 5500 2    50   Output ~ 0
 OUT_C1
-Text HLabel 8550 4550 0    50   Input ~ 0
+Text HLabel 8550 4600 0    50   Input ~ 0
 IN_C3
-Text HLabel 8550 5450 0    50   Input ~ 0
+Text HLabel 8550 5500 0    50   Input ~ 0
 IN_C4
+Text HLabel 9550 4600 2    50   Output ~ 0
+OUT_C2
 Text HLabel 9550 3700 2    50   Output ~ 0
-OUT_C2
-Text HLabel 9550 4600 2    50   Output ~ 0
 OUT_C3
-Text HLabel 8550 3650 0    50   Input ~ 0
+Text HLabel 8550 3700 0    50   Input ~ 0
 IN_C2
 Wire Wire Line
@@
 AR Path="/D1BB8DB4/5F76AF55/60474926" Ref="RN6102"  Part="1"
 AR Path="/D1BB8DB4/5F75E923/60474926" Ref="RN7002"  Part="1"
-F 0 "RN6102" V 10200 4350 50  0000 L CNN
+F 0 "RN7002" V 10200 4350 50  0000 L CNN
 F 1 "680Ω" V 9800 3750 50  0001 L CNN
 F 2 "BoatControl:DIP254P762X432-16P" V 10775 3900 50  0001 C CNN
@@
 AR Path="/D1BB8DB4/5F75E923/62B5C7B5" Ref="C7001"  Part="1"
 AR Path="/D1BB8DB4/5F76AF55/62B5C7B5" Ref="C6101"  Part="1"
-F 0 "C6101" V 4600 2550 50  0000 L CNN
+F 0 "C7001" V 4600 2550 50  0000 L CNN
 F 1 "1µF" H 3800 2400 50  0001 L CNN
 F 2 "Capacitor_THT:C_Disc_D7.5mm_W5.0mm_P5.00mm" H 4650 2500 50  0001 C CNN
@@
 AR Path="/D1BB8DB4/5F75E923/62B76848" Ref="C7002"  Part="1"
 AR Path="/D1BB8DB4/5F76AF55/62B76848" Ref="C6102"  Part="1"
-F 0 "C6102" V 4600 2750 50  0000 L CNN
+F 0 "C7002" V 4600 2750 50  0000 L CNN
 F 1 "1µF" H 3800 2600 50  0001 L CNN
 F 2 "Capacitor_THT:C_Disc_D7.5mm_W5.0mm_P5.00mm" H 4650 2700 50  0001 C CNN
@@
 AR Path="/D1BB8DB4/5F75E923/62B86A50" Ref="C7003"  Part="1"
 AR Path="/D1BB8DB4/5F76AF55/62B86A50" Ref="C6103"  Part="1"
-F 0 "C6103" V 4600 3550 50  0000 L CNN
+F 0 "C7003" V 4600 3550 50  0000 L CNN
 F 1 "1µF" H 3800 3400 50  0001 L CNN
 F 2 "Capacitor_THT:C_Disc_D7.5mm_W5.0mm_P5.00mm" H 4650 3500 50  0001 C CNN
@@
 AR Path="/D1BB8DB4/5F75E923/62B939DB" Ref="C7004"  Part="1"
 AR Path="/D1BB8DB4/5F76AF55/62B939DB" Ref="C6104"  Part="1"
-F 0 "C6104" V 4600 3750 50  0000 L CNN
+F 0 "C7004" V 4600 3750 50  0000 L CNN
 F 1 "1µF" H 3800 3600 50  0001 L CNN
 F 2 "Capacitor_THT:C_Disc_D7.5mm_W5.0mm_P5.00mm" H 4650 3700 50  0001 C CNN
@@
 AR Path="/D1BB8DB4/5F75E923/62BA14CE" Ref="C7005"  Part="1"
 AR Path="/D1BB8DB4/5F76AF55/62BA14CE" Ref="C6105"  Part="1"
-F 0 "C6105" V 4600 4550 50  0000 L CNN
+F 0 "C7005" V 4600 4550 50  0000 L CNN
 F 1 "1µF" H 3800 4400 50  0001 L CNN
 F 2 "Capacitor_THT:C_Disc_D7.5mm_W5.0mm_P5.00mm" H 4650 4500 50  0001 C CNN
@@
 AR Path="/D1BB8DB4/5F75E923/62BAE342" Ref="C7006"  Part="1"
 AR Path="/D1BB8DB4/5F76AF55/62BAE342" Ref="C6106"  Part="1"
-F 0 "C6106" V 4600 4750 50  0000 L CNN
+F 0 "C7006" V 4600 4750 50  0000 L CNN
 F 1 "1µF" H 3800 4600 50  0001 L CNN
 F 2 "Capacitor_THT:C_Disc_D7.5mm_W5.0mm_P5.00mm" H 4650 4700 50  0001 C CNN
@@
 AR Path="/D1BB8DB4/5F75E923/62BBBC28" Ref="C7007"  Part="1"
 AR Path="/D1BB8DB4/5F76AF55/62BBBC28" Ref="C6107"  Part="1"
-F 0 "C6107" V 4600 5550 50  0000 L CNN
+F 0 "C7007" V 4600 5550 50  0000 L CNN
 F 1 "1µF" H 3800 5400 50  0001 L CNN
 F 2 "Capacitor_THT:C_Disc_D7.5mm_W5.0mm_P5.00mm" H 4650 5500 50  0001 C CNN
@@
 AR Path="/D1BB8DB4/5F75E923/62BC8A92" Ref="C7008"  Part="1"
 AR Path="/D1BB8DB4/5F76AF55/62BC8A92" Ref="C6108"  Part="1"
-F 0 "C6108" V 4600 5750 50  0000 L CNN
+F 0 "C7008" V 4600 5750 50  0000 L CNN
 F 1 "1µF" H 3800 5600 50  0001 L CNN
 F 2 "Capacitor_THT:C_Disc_D7.5mm_W5.0mm_P5.00mm" H 4650 5700 50  0001 C CNN
@@
 AR Path="/D1BB8DB4/5F75E923/62CB5764" Ref="RN7003"  Part="1"
 AR Path="/D1BB8DB4/5F76AF55/62CB5764" Ref="RN6103"  Part="1"
-F 0 "RN6103" V 2150 3900 50  0000 L CNN
+F 0 "RN7003" V 2150 3900 50  0000 L CNN
 F 1 "10MΩ" H 2300 3550 50  0001 L CNN
 F 2 "Resistor_THT:R_Array_SIP9" V 3125 3950 50  0001 C CNN
@@
 AR Path="/D1BB8DB4/5F76AF55/630078FE" Ref="RN6101"  Part="1"
 AR Path="/D1BB8DB4/5F75E923/630078FE" Ref="RN7001"  Part="1"
-F 0 "RN6101" V 2150 3050 50  0000 C CNN
+F 0 "RN7001" V 2150 3050 50  0000 C CNN
 F 1 "100KΩ" V 2450 2750 50  0001 C CNN
 F 2 "Resistor_THT:R_Array_SIP9" H 3400 3150 50  0001 L CNN
@@
 AR Path="/D1BB8DB4/5F76AF55/63015012" Ref="RN6104"  Part="1"
 AR Path="/D1BB8DB4/5F75E923/63015012" Ref="RN7004"  Part="1"
-F 0 "RN6104" V 2150 4850 50  0000 C CNN
+F 0 "RN7004" V 2150 4850 50  0000 C CNN
 F 1 "100KΩ" V 2450 4550 50  0001 C CNN
 F 2 "Resistor_THT:R_Array_SIP9" H 3400 4950 50  0001 L CNN
@@
 F5 "OFF_LED" I R 9550 5350 50
 F6 "OUT" O R 9550 5500 50
-F7 "IN" I L 8550 5450 50
+F7 "IN" I L 8550 5500 50
 F8 "ON_COIL" I R 9550 5050 50
 F9 "OFF_COIL" I R 9550 4950 50
@@
 F5 "OFF_LED" I R 9550 3550 50
 F6 "OUT" O R 9550 3700 50
-F7 "IN" I L 8550 3650 50
+F7 "IN" I L 8550 3700 50
 F8 "ON_COIL" I R 9550 3250 50
 F9 "OFF_COIL" I R 9550 3150 50
@@
 F5 "OFF_LED" I R 9550 2650 50
 F6 "OUT" O R 9550 2800 50
-F7 "IN" I L 8550 2750 50
+F7 "IN" I L 8550 2800 50
 F8 "ON_COIL" I R 9550 2350 50
 F9 "OFF_COIL" I R 9550 2250 50
@@
 F5 "OFF_LED" I R 9550 4450 50
 F6 "OUT" O R 9550 4600 50
-F7 "IN" I L 8550 4550 50
+F7 "IN" I L 8550 4600 50
 F8 "ON_COIL" I R 9550 4150 50
 F9 "OFF_COIL" I R 9550 4050 50
