File: boatcontrol/6AmpBlock.sch (KiCad schematic (older format))
At the start: 15 parts, among them U7901 ULN2803A

Commit message: mwire
Connections:
- net 6AC1/OFF_COIL: now also RN7902.10 (R7.2); no longer RN7902.9 (R8.2)
- net 6AC1/ON_COIL: now also RN7902.9 (R8.2); no longer RN7902.10 (R7.2)
- net 6AC2/OFF_COIL: now also RN7902.12 (R5.2); no longer RN7902.11 (R6.2)
- net 6AC2/ON_COIL: now also RN7902.11 (R6.2); no longer RN7902.12 (R5.2)
- net 6AC3/OFF_COIL: now also RN7902.14 (R3.2); no longer RN7902.13 (R4.2)
- net 6AC3/ON_COIL: now also RN7902.13 (R4.2); no longer RN7902.14 (R3.2)
- net 6AC4/OFF_COIL: now also RN7902.16 (R1.2); no longer RN7902.15 (R2.2)
- net 6AC4/ON_COIL: now also RN7902.15 (R2.2); no longer RN7902.16 (R1.2)
Changed lines of the file:
@@
 $Descr A4 11693 8268
 encoding utf-8
-Sheet 51 97
+Sheet 67 97
 Title "Boat Control Hat"
 Date "2020-07-09"
@@
 F6 "OUT" O R 9350 3850 50
 F7 "IN" I L 8350 3850 50
-F8 "ON_COIL" I R 9350 3400 50
-F9 "OFF_COIL" I R 9350 3300 50
+F8 "ON_COIL" I R 9350 3300 50
+F9 "OFF_COIL" I R 9350 3400 50
 $EndSheet
 Text HLabel 8350 5650 0    50   Input ~ 0
@@
 F6 "OUT" O R 9350 5650 50
 F7 "IN" I L 8350 5650 50
-F8 "ON_COIL" I R 9350 5200 50
-F9 "OFF_COIL" I R 9350 5100 50
+F8 "ON_COIL" I R 9350 5100 50
+F9 "OFF_COIL" I R 9350 5200 50
 $EndSheet
 $Comp
@@
 F6 "OUT" O R 9350 2950 50
 F7 "IN" I L 8350 2950 50
-F8 "ON_COIL" I R 9350 2500 50
-F9 "OFF_COIL" I R 9350 2400 50
+F8 "ON_COIL" I R 9350 2400 50
+F9 "OFF_COIL" I R 9350 2500 50
 $EndSheet
 $Sheet
@@
 F6 "OUT" O R 9350 4750 50
 F7 "IN" I L 8350 4750 50
-F8 "ON_COIL" I R 9350 4300 50
-F9 "OFF_COIL" I R 9350 4200 50
+F8 "ON_COIL" I R 9350 4200 50
+F9 "OFF_COIL" I R 9350 4300 50
 $EndSheet
 $Comp
