File: boatcontrol/6AmpBlock.sch (KiCad schematic (older format))
At the start: 15 parts, among them U7901 ULN2803A

Commit message: Re-label
Changed lines of the file:
@@
 AR Path="/D1BB8DB4/5F317CB5/60365AE4" Ref="#PWR07901"  Part="1"
 AR Path="/D1BB8DB4/5F746103/60365AE4" Ref="#PWR05201"  Part="1"
-F 0 "#PWR07901" H 6700 3400 50  0001 C CNN
+F 0 "#PWR05201" H 6700 3400 50  0001 C CNN
 F 1 "+12P" H 6550 3650 50  0000 C CNN
 F 2 "" H 6700 3550 50  0001 C CNN
@@
 AR Path="/D1BB8DB4/5F317CB5/60365AF1" Ref="U7901"  Part="1"
 AR Path="/D1BB8DB4/5F746103/60365AF1" Ref="U5201"  Part="1"
-F 0 "U7901" H 6250 3650 50  0000 L CNN
+F 0 "U5201" H 6250 3650 50  0000 L CNN
 F 1 "ULN2803A" H 6100 4350 50  0000 L CNN
 F 2 "Package_DIP:DIP-18_W7.62mm" H 6350 3200 50  0001 L CNN
@@
 AR Path="/D1BB8DB4/5F317CB5/60365B03" Ref="#PWR07902"  Part="1"
 AR Path="/D1BB8DB4/5F746103/60365B03" Ref="#PWR05202"  Part="1"
-F 0 "#PWR07902" H 6300 4300 50  0001 C CNN
+F 0 "#PWR05202" H 6300 4300 50  0001 C CNN
 F 1 "GND" H 6305 4377 50  0000 C CNN
 F 2 "" H 6300 4550 50  0001 C CNN
@@
 AR Path="/D1BB8DB4/5F317CB5/60365B8C" Ref="#PWR07903"  Part="1"
 AR Path="/D1BB8DB4/5F746103/60365B8C" Ref="#PWR05203"  Part="1"
-F 0 "#PWR07903" H 2250 5150 50  0001 C CNN
+F 0 "#PWR05203" H 2250 5150 50  0001 C CNN
 F 1 "+5V" H 2265 5473 50  0000 C CNN
 F 2 "" H 2250 5300 50  0001 C CNN
@@
 AR Path="/D1BB8DB4/5F317CB5/60365C68" Ref="RN7902"  Part="1"
 AR Path="/D1BB8DB4/5F746103/60365C68" Ref="RN5202"  Part="1"
-F 0 "RN7902" V 10000 4550 50  0000 L CNN
+F 0 "RN5202" V 10000 4550 50  0000 L CNN
 F 1 "680Ω" V 9600 3900 50  0001 L CNN
 F 2 "BoatControl:DIP254P762X432-16P" V 10575 4050 50  0001 C CNN
@@
 AR Path="/D1BB8DB4/5F746103/62AB509B" Ref="C5201"  Part="1"
 AR Path="/D1BB8DB4/5F317CB5/62AB509B" Ref="C7901"  Part="1"
-F 0 "C7901" V 4400 2700 50  0000 L CNN
+F 0 "C5201" V 4400 2700 50  0000 L CNN
 F 1 "1µF" H 3600 2550 50  0001 L CNN
 F 2 "Capacitor_THT:C_Disc_D7.5mm_W5.0mm_P5.00mm" H 4450 2650 50  0001 C CNN
@@
 AR Path="/D1BB8DB4/5F746103/62AC1E93" Ref="C5202"  Part="1"
 AR Path="/D1BB8DB4/5F317CB5/62AC1E93" Ref="C7902"  Part="1"
-F 0 "C7902" V 4400 2900 50  0000 L CNN
+F 0 "C5202" V 4400 2900 50  0000 L CNN
 F 1 "1µF" H 3600 2750 50  0001 L CNN
 F 2 "Capacitor_THT:C_Disc_D7.5mm_W5.0mm_P5.00mm" H 4450 2850 50  0001 C CNN
@@
 AR Path="/D1BB8DB4/5F746103/62ADD9A6" Ref="C5208"  Part="1"
 AR Path="/D1BB8DB4/5F317CB5/62ADD9A6" Ref="C7908"  Part="1"
-F 0 "C7908" V 4400 5900 50  0000 L CNN
+F 0 "C5208" V 4400 5900 50  0000 L CNN
 F 1 "1µF" H 3600 5750 50  0001 L CNN
 F 2 "Capacitor_THT:C_Disc_D7.5mm_W5.0mm_P5.00mm" H 4450 5850 50  0001 C CNN
@@
 AR Path="/D1BB8DB4/5F746103/62AEACF8" Ref="C5207"  Part="1"
 AR Path="/D1BB8DB4/5F317CB5/62AEACF8" Ref="C7907"  Part="1"
-F 0 "C7907" V 4400 5700 50  0000 L CNN
+F 0 "C5207" V 4400 5700 50  0000 L CNN
 F 1 "1µF" H 3600 5550 50  0001 L CNN
 F 2 "Capacitor_THT:C_Disc_D7.5mm_W5.0mm_P5.00mm" H 4450 5650 50  0001 C CNN
@@
 AR Path="/D1BB8DB4/5F746103/62AF81A3" Ref="C5206"  Part="1"
 AR Path="/D1BB8DB4/5F317CB5/62AF81A3" Ref="C7906"  Part="1"
-F 0 "C7906" V 4400 4900 50  0000 L CNN
+F 0 "C5206" V 4400 4900 50  0000 L CNN
 F 1 "1µF" H 3600 4750 50  0001 L CNN
 F 2 "Capacitor_THT:C_Disc_D7.5mm_W5.0mm_P5.00mm" H 4450 4850 50  0001 C CNN
@@
 AR Path="/D1BB8DB4/5F746103/62B05762" Ref="C5205"  Part="1"
 AR Path="/D1BB8DB4/5F317CB5/62B05762" Ref="C7905"  Part="1"
-F 0 "C7905" V 4400 4700 50  0000 L CNN
+F 0 "C5205" V 4400 4700 50  0000 L CNN
 F 1 "1µF" H 3600 4550 50  0001 L CNN
 F 2 "Capacitor_THT:C_Disc_D7.5mm_W5.0mm_P5.00mm" H 4450 4650 50  0001 C CNN
@@
 AR Path="/D1BB8DB4/5F746103/62B3C5BA" Ref="C5203"  Part="1"
 AR Path="/D1BB8DB4/5F317CB5/62B3C5BA" Ref="C7903"  Part="1"
-F 0 "C7903" V 4400 3700 50  0000 L CNN
+F 0 "C5203" V 4400 3700 50  0000 L CNN
 F 1 "1µF" H 3600 3550 50  0001 L CNN
 F 2 "Capacitor_THT:C_Disc_D7.5mm_W5.0mm_P5.00mm" H 4450 3650 50  0001 C CNN
@@
 AR Path="/D1BB8DB4/5F746103/62B4996D" Ref="C5204"  Part="1"
 AR Path="/D1BB8DB4/5F317CB5/62B4996D" Ref="C7904"  Part="1"
-F 0 "C7904" V 4400 3900 50  0000 L CNN
+F 0 "C5204" V 4400 3900 50  0000 L CNN
 F 1 "1µF" H 3600 3750 50  0001 L CNN
 F 2 "Capacitor_THT:C_Disc_D7.5mm_W5.0mm_P5.00mm" H 4450 3850 50  0001 C CNN
@@
 AR Path="/D1BB8DB4/5F317CB5/62C7A7CE" Ref="RN7903"  Part="1"
 AR Path="/D1BB8DB4/5F746103/62C7A7CE" Ref="RN5203"  Part="1"
-F 0 "RN7903" V 1950 4050 50  0000 L CNN
+F 0 "RN5203" V 1950 4050 50  0000 L CNN
 F 1 "10MΩ" H 2100 3700 50  0001 L CNN
 F 2 "Resistor_THT:R_Array_SIP9" V 2925 4100 50  0001 C CNN
@@
 AR Path="/D1BB8DB4/5F317CB5/62F1D24C" Ref="RN7904"  Part="1"
 AR Path="/D1BB8DB4/5F746103/62F1D24C" Ref="RN5204"  Part="1"
-F 0 "RN7904" V 1950 5000 50  0000 C CNN
+F 0 "RN5204" V 1950 5000 50  0000 C CNN
 F 1 "100KΩ" V 2250 4700 50  0001 C CNN
 F 2 "Resistor_THT:R_Array_SIP9" H 3200 5100 50  0001 L CNN
@@
 AR Path="/D1BB8DB4/5F317CB5/62F2A731" Ref="RN7901"  Part="1"
 AR Path="/D1BB8DB4/5F746103/62F2A731" Ref="RN5201"  Part="1"
-F 0 "RN7901" V 1950 3200 50  0000 C CNN
+F 0 "RN5201" V 1950 3200 50  0000 C CNN
 F 1 "100KΩ" V 2250 2900 50  0001 C CNN
 F 2 "Resistor_THT:R_Array_SIP9" H 3200 3300 50  0001 L CNN
@@
 AR Path="/D1BB8DB4/5F317CB5/624D8B2F" Ref="C7909"  Part="1"
 AR Path="/D1BB8DB4/5F746103/624D8B2F" Ref="C5209"  Part="1"
-F 0 "C7909" H 6100 2950 50  0000 L CNN
+F 0 "C5209" H 6100 2950 50  0000 L CNN
 F 1 "10uF" H 6291 3105 50  0001 L CNN
 F 2 "Capacitor_THT:C_Disc_D7.5mm_W5.0mm_P5.00mm" H 6200 3150 50  0001 C CNN
@@
 AR Path="/D1BB8DB4/5F317CB5/624D8B37" Ref="C7910"  Part="1"
 AR Path="/D1BB8DB4/5F746103/624D8B37" Ref="C5210"  Part="1"
-F 0 "C7910" H 6350 2950 50  0000 L CNN
+F 0 "C5210" H 6350 2950 50  0000 L CNN
 F 1 "0.1uF" H 6541 3105 50  0001 L CNN
 F 2 "Capacitor_THT:C_Disc_D7.5mm_W5.0mm_P5.00mm" H 6450 3150 50  0001 C CNN
@@
 AR Path="/D1BB8DB4/5F317CB5/624D8B3E" Ref="#PWR0204"  Part="1"
 AR Path="/D1BB8DB4/5F746103/624D8B3E" Ref="#PWR0198"  Part="1"
-F 0 "#PWR0204" H 6450 2800 50  0001 C CNN
+F 0 "#PWR0198" H 6450 2800 50  0001 C CNN
 F 1 "GND" V 6455 2922 50  0000 R CNN
 F 2 "" H 6450 3050 50  0001 C CNN

Commit message: shuffle
Changed lines of the file:
@@
 $Descr A4 11693 8268
 encoding utf-8
-Sheet 40 97
+Sheet 67 97
 Title "Boat Control Hat"
 Date "2020-07-09"
@@
 AR Path="/D1BB8DB4/5F317CB5/60365AE4" Ref="#PWR07901"  Part="1"
 AR Path="/D1BB8DB4/5F746103/60365AE4" Ref="#PWR05201"  Part="1"
-F 0 "#PWR05201" H 6700 3400 50  0001 C CNN
+F 0 "#PWR07901" H 6700 3400 50  0001 C CNN
 F 1 "+12P" H 6550 3650 50  0000 C CNN
 F 2 "" H 6700 3550 50  0001 C CNN
@@
 AR Path="/D1BB8DB4/5F317CB5/60365AF1" Ref="U7901"  Part="1"
 AR Path="/D1BB8DB4/5F746103/60365AF1" Ref="U5201"  Part="1"
-F 0 "U5201" H 6250 3650 50  0000 L CNN
+F 0 "U7901" H 6250 3650 50  0000 L CNN
 F 1 "ULN2803A" H 6100 4350 50  0000 L CNN
 F 2 "Package_DIP:DIP-18_W7.62mm" H 6350 3200 50  0001 L CNN
@@
 AR Path="/D1BB8DB4/5F317CB5/60365B03" Ref="#PWR07902"  Part="1"
 AR Path="/D1BB8DB4/5F746103/60365B03" Ref="#PWR05202"  Part="1"
-F 0 "#PWR05202" H 6300 4300 50  0001 C CNN
+F 0 "#PWR07902" H 6300 4300 50  0001 C CNN
 F 1 "GND" H 6305 4377 50  0000 C CNN
 F 2 "" H 6300 4550 50  0001 C CNN
@@
 AR Path="/D1BB8DB4/5F317CB5/60365B8C" Ref="#PWR07903"  Part="1"
 AR Path="/D1BB8DB4/5F746103/60365B8C" Ref="#PWR05203"  Part="1"
-F 0 "#PWR05203" H 2250 5150 50  0001 C CNN
+F 0 "#PWR07903" H 2250 5150 50  0001 C CNN
 F 1 "+5V" H 2265 5473 50  0000 C CNN
 F 2 "" H 2250 5300 50  0001 C CNN
@@
 AR Path="/D1BB8DB4/5F317CB5/60365C68" Ref="RN7902"  Part="1"
 AR Path="/D1BB8DB4/5F746103/60365C68" Ref="RN5202"  Part="1"
-F 0 "RN5202" V 10000 4550 50  0000 L CNN
+F 0 "RN7902" V 10000 4550 50  0000 L CNN
 F 1 "680Ω" V 9600 3900 50  0001 L CNN
 F 2 "BoatControl:DIP254P762X432-16P" V 10575 4050 50  0001 C CNN
@@
 AR Path="/D1BB8DB4/5F746103/62AB509B" Ref="C5201"  Part="1"
 AR Path="/D1BB8DB4/5F317CB5/62AB509B" Ref="C7901"  Part="1"
-F 0 "C5201" V 4400 2700 50  0000 L CNN
+F 0 "C7901" V 4400 2700 50  0000 L CNN
 F 1 "1µF" H 3600 2550 50  0001 L CNN
 F 2 "Capacitor_THT:C_Disc_D7.5mm_W5.0mm_P5.00mm" H 4450 2650 50  0001 C CNN
@@
 AR Path="/D1BB8DB4/5F746103/62AC1E93" Ref="C5202"  Part="1"
 AR Path="/D1BB8DB4/5F317CB5/62AC1E93" Ref="C7902"  Part="1"
-F 0 "C5202" V 4400 2900 50  0000 L CNN
+F 0 "C7902" V 4400 2900 50  0000 L CNN
 F 1 "1µF" H 3600 2750 50  0001 L CNN
 F 2 "Capacitor_THT:C_Disc_D7.5mm_W5.0mm_P5.00mm" H 4450 2850 50  0001 C CNN
@@
 AR Path="/D1BB8DB4/5F746103/62ADD9A6" Ref="C5208"  Part="1"
 AR Path="/D1BB8DB4/5F317CB5/62ADD9A6" Ref="C7908"  Part="1"
-F 0 "C5208" V 4400 5900 50  0000 L CNN
+F 0 "C7908" V 4400 5900 50  0000 L CNN
 F 1 "1µF" H 3600 5750 50  0001 L CNN
 F 2 "Capacitor_THT:C_Disc_D7.5mm_W5.0mm_P5.00mm" H 4450 5850 50  0001 C CNN
@@
 AR Path="/D1BB8DB4/5F746103/62AEACF8" Ref="C5207"  Part="1"
 AR Path="/D1BB8DB4/5F317CB5/62AEACF8" Ref="C7907"  Part="1"
-F 0 "C5207" V 4400 5700 50  0000 L CNN
+F 0 "C7907" V 4400 5700 50  0000 L CNN
 F 1 "1µF" H 3600 5550 50  0001 L CNN
 F 2 "Capacitor_THT:C_Disc_D7.5mm_W5.0mm_P5.00mm" H 4450 5650 50  0001 C CNN
@@
 AR Path="/D1BB8DB4/5F746103/62AF81A3" Ref="C5206"  Part="1"
 AR Path="/D1BB8DB4/5F317CB5/62AF81A3" Ref="C7906"  Part="1"
-F 0 "C5206" V 4400 4900 50  0000 L CNN
+F 0 "C7906" V 4400 4900 50  0000 L CNN
 F 1 "1µF" H 3600 4750 50  0001 L CNN
 F 2 "Capacitor_THT:C_Disc_D7.5mm_W5.0mm_P5.00mm" H 4450 4850 50  0001 C CNN
@@
 AR Path="/D1BB8DB4/5F746103/62B05762" Ref="C5205"  Part="1"
 AR Path="/D1BB8DB4/5F317CB5/62B05762" Ref="C7905"  Part="1"
-F 0 "C5205" V 4400 4700 50  0000 L CNN
+F 0 "C7905" V 4400 4700 50  0000 L CNN
 F 1 "1µF" H 3600 4550 50  0001 L CNN
 F 2 "Capacitor_THT:C_Disc_D7.5mm_W5.0mm_P5.00mm" H 4450 4650 50  0001 C CNN
@@
 AR Path="/D1BB8DB4/5F746103/62B3C5BA" Ref="C5203"  Part="1"
 AR Path="/D1BB8DB4/5F317CB5/62B3C5BA" Ref="C7903"  Part="1"
-F 0 "C5203" V 4400 3700 50  0000 L CNN
+F 0 "C7903" V 4400 3700 50  0000 L CNN
 F 1 "1µF" H 3600 3550 50  0001 L CNN
 F 2 "Capacitor_THT:C_Disc_D7.5mm_W5.0mm_P5.00mm" H 4450 3650 50  0001 C CNN
@@
 AR Path="/D1BB8DB4/5F746103/62B4996D" Ref="C5204"  Part="1"
 AR Path="/D1BB8DB4/5F317CB5/62B4996D" Ref="C7904"  Part="1"
-F 0 "C5204" V 4400 3900 50  0000 L CNN
+F 0 "C7904" V 4400 3900 50  0000 L CNN
 F 1 "1µF" H 3600 3750 50  0001 L CNN
 F 2 "Capacitor_THT:C_Disc_D7.5mm_W5.0mm_P5.00mm" H 4450 3850 50  0001 C CNN
@@
 AR Path="/D1BB8DB4/5F317CB5/62C7A7CE" Ref="RN7903"  Part="1"
 AR Path="/D1BB8DB4/5F746103/62C7A7CE" Ref="RN5203"  Part="1"
-F 0 "RN5203" V 1950 4050 50  0000 L CNN
+F 0 "RN7903" V 1950 4050 50  0000 L CNN
 F 1 "10MΩ" H 2100 3700 50  0001 L CNN
 F 2 "Resistor_THT:R_Array_SIP9" V 2925 4100 50  0001 C CNN
@@
 AR Path="/D1BB8DB4/5F317CB5/62F1D24C" Ref="RN7904"  Part="1"
 AR Path="/D1BB8DB4/5F746103/62F1D24C" Ref="RN5204"  Part="1"
-F 0 "RN5204" V 1950 5000 50  0000 C CNN
+F 0 "RN7904" V 1950 5000 50  0000 C CNN
 F 1 "100KΩ" V 2250 4700 50  0001 C CNN
 F 2 "Resistor_THT:R_Array_SIP9" H 3200 5100 50  0001 L CNN
@@
 AR Path="/D1BB8DB4/5F317CB5/62F2A731" Ref="RN7901"  Part="1"
 AR Path="/D1BB8DB4/5F746103/62F2A731" Ref="RN5201"  Part="1"
-F 0 "RN5201" V 1950 3200 50  0000 C CNN
+F 0 "RN7901" V 1950 3200 50  0000 C CNN
 F 1 "100KΩ" V 2250 2900 50  0001 C CNN
 F 2 "Resistor_THT:R_Array_SIP9" H 3200 3300 50  0001 L CNN
@@
 AR Path="/D1BB8DB4/5F317CB5/624D8B2F" Ref="C7909"  Part="1"
 AR Path="/D1BB8DB4/5F746103/624D8B2F" Ref="C5209"  Part="1"
-F 0 "C5209" H 6100 2950 50  0000 L CNN
+F 0 "C7909" H 6100 2950 50  0000 L CNN
 F 1 "10uF" H 6291 3105 50  0001 L CNN
 F 2 "Capacitor_THT:C_Disc_D7.5mm_W5.0mm_P5.00mm" H 6200 3150 50  0001 C CNN
@@
 AR Path="/D1BB8DB4/5F317CB5/624D8B37" Ref="C7910"  Part="1"
 AR Path="/D1BB8DB4/5F746103/624D8B37" Ref="C5210"  Part="1"
-F 0 "C5210" H 6350 2950 50  0000 L CNN
+F 0 "C7910" H 6350 2950 50  0000 L CNN
 F 1 "0.1uF" H 6541 3105 50  0001 L CNN
 F 2 "Capacitor_THT:C_Disc_D7.5mm_W5.0mm_P5.00mm" H 6450 3150 50  0001 C CNN
@@
 AR Path="/D1BB8DB4/5F317CB5/624D8B3E" Ref="#PWR0204"  Part="1"
 AR Path="/D1BB8DB4/5F746103/624D8B3E" Ref="#PWR0198"  Part="1"
-F 0 "#PWR0198" H 6450 2800 50  0001 C CNN
+F 0 "#PWR0204" H 6450 2800 50  0001 C CNN
 F 1 "GND" V 6455 2922 50  0000 R CNN
 F 2 "" H 6450 3050 50  0001 C CNN

Commit message: More cleanup
Other:
- moved on the sheet: RN7902

Commit message: More cleanup
Connections:
- net +5V: no longer RN7901.1 (common), RN7904.1 (common)
- net GND: now also RN7901.1 (common), RN7904.1 (common)
Changed lines of the file:
@@
 Wire Wire Line
 	5700 4050 5900 4050
-$Comp
-L power:+5V #PWR?
-U 1 1 60365B8C
-P 2250 5300
-AR Path="/D16552B4/5FA17F38/60365B8C" Ref="#PWR?"  Part="1"
-AR Path="/D16552B4/5FA17F52/60365B8C" Ref="#PWR?"  Part="1"
-AR Path="/D16552B4/5FA17F6C/60365B8C" Ref="#PWR?"  Part="1"
-AR Path="/D16552B4/5FA17F86/60365B8C" Ref="#PWR?"  Part="1"
-AR Path="/D1BB8DB4/5F317CB5/60365B8C" Ref="#PWR07903"  Part="1"
-AR Path="/D1BB8DB4/5F746103/60365B8C" Ref="#PWR05203"  Part="1"
-F 0 "#PWR07903" H 2250 5150 50  0001 C CNN
-F 1 "+5V" H 2265 5473 50  0000 C CNN
-F 2 "" H 2250 5300 50  0001 C CNN
-F 3 "" H 2250 5300 50  0001 C CNN
-	1    2250 5300
-	-1   0    0    1
-$EndComp
 Wire Wire Line
 	6700 3850 6950 3850
@@
 	0    -1   1    0
 $EndComp
-Connection ~ 2250 3700
-Wire Wire Line
-	2250 3700 2250 4600
 $Comp
 L Device:R_Network08 RN?
@@
 	0    -1   1    0
 $EndComp
-Wire Wire Line
-	2250 2800 2250 3700
 $Comp
 L Device:R_Network08 RN?
@@
 	0    -1   1    0
 $EndComp
-Connection ~ 2250 4600
-Wire Wire Line
-	2250 4600 2250 5300
 Wire Wire Line
 	9350 2400 10350 2400
@@
 Wire Wire Line
 	7000 3250 7000 3950
+$Comp
+L power:+5V #PWR?
+U 1 1 6027D066
+P 2250 3700
+AR Path="/D16552B4/5FA17F38/6027D066" Ref="#PWR?"  Part="1"
+AR Path="/D16552B4/5FA17F52/6027D066" Ref="#PWR?"  Part="1"
+AR Path="/D16552B4/5FA17F6C/6027D066" Ref="#PWR?"  Part="1"
+AR Path="/D16552B4/5FA17F86/6027D066" Ref="#PWR?"  Part="1"
+F 0 "#PWR?" H 2250 3550 50  0001 C CNN
+F 1 "+5V" H 2400 3750 50  0000 C CNN
+F 2 "" H 2250 3700 50  0001 C CNN
+F 3 "" H 2250 3700 50  0001 C CNN
+	1    2250 3700
+	-1   0    0    1
+$EndComp
+$Comp
+L power:GND #PWR?
+U 1 1 6027D06C
+P 2250 2800
+F 0 "#PWR?" H 2250 2550 50  0001 C CNN
+F 1 "GND" H 2100 2750 50  0000 C CNN
+F 2 "" H 2250 2800 50  0001 C CNN
+F 3 "" H 2250 2800 50  0001 C CNN
+	1    2250 2800
+	1    0    0    -1
+$EndComp
+$Comp
+L power:GND #PWR?
+U 1 1 6027D072
+P 2250 4600
+F 0 "#PWR?" H 2250 4350 50  0001 C CNN
+F 1 "GND" H 2100 4550 50  0000 C CNN
+F 2 "" H 2250 4600 50  0001 C CNN
+F 3 "" H 2250 4600 50  0001 C CNN
+	1    2250 4600
+	1    0    0    -1
+$EndComp
 $EndSCHEMATC
