File: boatcontrol/6AmpCircuit.sch (KiCad schematic (older format))
At the start: 5 parts, among them K8701 G5RL-K1A-E-DC12, Q8701 T9-818 6A, SW8701 ESB30, SW8702 ESB30

Commit message: More cleanup
Parts:
- D8701: value 20mA R/G -> 20mA R/G CA
Changed lines of the file:
@@
 $Descr A4 11693 8268
 encoding utf-8
-Sheet 85 97
+Sheet 96 97
 Title "Boat Control Hat"
 Date "2020-07-09"
@@
 AR Path="/D1BB8DB4/5F746103/60365C49/D2F4D9A7" Ref="D5901"  Part="1"
 AR Path="/D1BB8DB4/5F746103/60365C53/D2F4D9A7" Ref="D6001"  Part="1"
-F 0 "D8601" H 5400 4100 50  0000 C CNN
-F 1 "20mA R/G" H 5550 4000 50  0000 C CNN
+F 0 "D8401" H 5400 4100 50  0000 C CNN
+F 1 "20mA R/G CA" H 5550 4000 50  0000 C CNN
 F 2 "LED_THT:LED_D5.0mm-3" H 5600 4250 50  0001 C CNN
 F 3 "http://www.kingbrightusa.com/images/catalog/SPEC/WP59EGW-CA.pdf" H 5600 4250 50  0001 C CNN
@@
 AR Path="/D1BB8DB4/5F746103/60365C49/D2F4DB56" Ref="K5901"  Part="1"
 AR Path="/D1BB8DB4/5F746103/60365C53/D2F4DB56" Ref="K6001"  Part="1"
-F 0 "K8601" H 6750 4250 50  0000 L CNN
+F 0 "K8401" H 6750 4250 50  0000 L CNN
 F 1 "G5RL-K1A-E-DC12" H 7100 4250 50  0000 L CNN
 F 2 "RELAY_G5RL-K1A-E-DC12" H 7100 4400 50  0001 L BNN
@@
 AR Path="/D1BB8DB4/5F746103/60365C49/D2F4D9AA" Ref="Q5901"  Part="1"
 AR Path="/D1BB8DB4/5F746103/60365C53/D2F4D9AA" Ref="Q6001"  Part="1"
-F 0 "Q8601" V 6650 3200 50  0000 R CNN
+F 0 "Q8401" V 6650 3200 50  0000 R CNN
 F 1 "T9-818 6A" V 6650 2950 50  0000 R CNN
 F 2 "BoatControl:Schurter_Circuit_Breaker" H 6650 3550 50  0001 C CNN
@@
 AR Path="/D1BB8DB4/5F746103/60365C49/D2F4D9AB" Ref="SW5901"  Part="1"
 AR Path="/D1BB8DB4/5F746103/60365C53/D2F4D9AB" Ref="SW6001"  Part="1"
-F 0 "SW8601" H 4250 4750 50  0000 C CNN
+F 0 "SW8401" H 4250 4750 50  0000 C CNN
 F 1 " ESB30" H 4250 3800 50  0000 C CNN
 F 2 "BoatControl:SW_PUSH_ESB30_DPDT" H 4500 3950 50  0001 C CNN
@@
 AR Path="/D1BB8DB4/5F746103/60365C49/D2F4D9A9" Ref="SW5902"  Part="1"
 AR Path="/D1BB8DB4/5F746103/60365C53/D2F4D9A9" Ref="SW6002"  Part="1"
-F 0 "SW8602" H 4200 5900 50  0000 C CNN
+F 0 "SW8402" H 4200 5900 50  0000 C CNN
 F 1 " ESB30" H 4300 4750 50  0000 C CNN
 F 2 "BoatControl:SW_PUSH_ESB30_DPDT" H 4500 5000 50  0001 C CNN
@@
 AR Path="/D1BB8DB4/5F75E923/60474907/60D74A5A" Ref="#PWR?"  Part="1"
 AR Path="/D1BB8DB4/5F75E923/60474911/60D74A5A" Ref="#PWR?"  Part="1"
-F 0 "#PWR0151" H 6150 4100 50  0001 C CNN
+F 0 "#PWR0147" H 6150 4100 50  0001 C CNN
 F 1 "+12P" H 6165 4423 50  0000 C CNN
 F 2 "" H 6150 4250 50  0001 C CNN
@@
 AR Path="/D1BB8DB4/5F75E923/60474907/60D74A7B" Ref="#PWR?"  Part="1"
 AR Path="/D1BB8DB4/5F75E923/60474911/60D74A7B" Ref="#PWR?"  Part="1"
-F 0 "#PWR0152" H 3950 4850 50  0001 C CNN
+F 0 "#PWR0148" H 3950 4850 50  0001 C CNN
 F 1 "GND" H 3955 4927 50  0000 C CNN
 F 2 "" H 3950 5100 50  0001 C CNN

Commit message: Add Node-RED flows
Changed lines of the file:
@@
 AR Path="/D1BB8DB4/5F746103/60365C49/D2F4D9A7" Ref="D5901"  Part="1"
 AR Path="/D1BB8DB4/5F746103/60365C53/D2F4D9A7" Ref="D6001"  Part="1"
-F 0 "D8401" H 5400 4100 50  0000 C CNN
+F 0 "D8601" H 5400 4100 50  0000 C CNN
 F 1 "20mA R/G CA" H 5550 4000 50  0000 C CNN
 F 2 "LED_THT:LED_D5.0mm-3" H 5600 4250 50  0001 C CNN
@@
 AR Path="/D1BB8DB4/5F746103/60365C49/D2F4DB56" Ref="K5901"  Part="1"
 AR Path="/D1BB8DB4/5F746103/60365C53/D2F4DB56" Ref="K6001"  Part="1"
-F 0 "K8401" H 6750 4250 50  0000 L CNN
+F 0 "K8601" H 6750 4250 50  0000 L CNN
 F 1 "G5RL-K1A-E-DC12" H 7100 4250 50  0000 L CNN
 F 2 "RELAY_G5RL-K1A-E-DC12" H 7100 4400 50  0001 L BNN
@@
 AR Path="/D1BB8DB4/5F746103/60365C49/D2F4D9AA" Ref="Q5901"  Part="1"
 AR Path="/D1BB8DB4/5F746103/60365C53/D2F4D9AA" Ref="Q6001"  Part="1"
-F 0 "Q8401" V 6650 3200 50  0000 R CNN
+F 0 "Q8601" V 6650 3200 50  0000 R CNN
 F 1 "T9-818 6A" V 6650 2950 50  0000 R CNN
 F 2 "BoatControl:Schurter_Circuit_Breaker" H 6650 3550 50  0001 C CNN
@@
 AR Path="/D1BB8DB4/5F746103/60365C49/D2F4D9AB" Ref="SW5901"  Part="1"
 AR Path="/D1BB8DB4/5F746103/60365C53/D2F4D9AB" Ref="SW6001"  Part="1"
-F 0 "SW8401" H 4250 4750 50  0000 C CNN
+F 0 "SW8601" H 4250 4750 50  0000 C CNN
 F 1 " ESB30" H 4250 3800 50  0000 C CNN
 F 2 "BoatControl:SW_PUSH_ESB30_DPDT" H 4500 3950 50  0001 C CNN
@@
 AR Path="/D1BB8DB4/5F746103/60365C49/D2F4D9A9" Ref="SW5902"  Part="1"
 AR Path="/D1BB8DB4/5F746103/60365C53/D2F4D9A9" Ref="SW6002"  Part="1"
-F 0 "SW8402" H 4200 5900 50  0000 C CNN
+F 0 "SW8602" H 4200 5900 50  0000 C CNN
 F 1 " ESB30" H 4300 4750 50  0000 C CNN
 F 2 "BoatControl:SW_PUSH_ESB30_DPDT" H 4500 5000 50  0001 C CNN

Commit message: Fix SB footprint and symbol
Parts:
- renumbered Q8701 to CB8701
Changed lines of the file:
@@
 $Descr A4 11693 8268
 encoding utf-8
-Sheet 96 97
+Sheet 83 97
 Title "Boat Control Hat"
 Date "2020-07-09"
@@
 AR Path="/D1BB8DB4/5F746103/60365C49/D2F4D9A7" Ref="D5901"  Part="1"
 AR Path="/D1BB8DB4/5F746103/60365C53/D2F4D9A7" Ref="D6001"  Part="1"
-F 0 "D8601" H 5400 4100 50  0000 C CNN
+F 0 "D8501" H 5400 4100 50  0000 C CNN
 F 1 "20mA R/G CA" H 5550 4000 50  0000 C CNN
 F 2 "LED_THT:LED_D5.0mm-3" H 5600 4250 50  0001 C CNN
@@
 AR Path="/D1BB8DB4/5F746103/60365C49/D2F4DB56" Ref="K5901"  Part="1"
 AR Path="/D1BB8DB4/5F746103/60365C53/D2F4DB56" Ref="K6001"  Part="1"
-F 0 "K8601" H 6750 4250 50  0000 L CNN
+F 0 "K8501" H 6750 4250 50  0000 L CNN
 F 1 "G5RL-K1A-E-DC12" H 7100 4250 50  0000 L CNN
 F 2 "RELAY_G5RL-K1A-E-DC12" H 7100 4400 50  0001 L BNN
@@
 AR Path="/D1BB8DB4/5F75E923/6067724E/D2F4D9AA" Ref="Q?"  Part="1"
 AR Path="/D1BB8DB4/5F75E923/60677477/D2F4D9AA" Ref="Q?"  Part="1"
-AR Path="/D1BB8DB4/5F317CB5/60365C53/D2F4D9AA" Ref="Q8701"  Part="1"
-AR Path="/D1BB8DB4/5F317CB5/60365C39/D2F4D9AA" Ref="Q8401"  Part="1"
-AR Path="/D1BB8DB4/5F317CB5/60365C41/D2F4D9AA" Ref="Q8501"  Part="1"
-AR Path="/D1BB8DB4/5F317CB5/60365C49/D2F4D9AA" Ref="Q8601"  Part="1"
-AR Path="/D1BB8DB4/5F746103/60365C39/D2F4D9AA" Ref="Q5701"  Part="1"
-AR Path="/D1BB8DB4/5F746103/60365C41/D2F4D9AA" Ref="Q5801"  Part="1"
-AR Path="/D1BB8DB4/5F746103/60365C49/D2F4D9AA" Ref="Q5901"  Part="1"
-AR Path="/D1BB8DB4/5F746103/60365C53/D2F4D9AA" Ref="Q6001"  Part="1"
-F 0 "Q8601" V 6650 3200 50  0000 R CNN
-F 1 "T9-818 6A" V 6650 2950 50  0000 R CNN
+AR Path="/D1BB8DB4/5F317CB5/60365C53/D2F4D9AA" Ref="CB8701"  Part="1"
+AR Path="/D1BB8DB4/5F317CB5/60365C39/D2F4D9AA" Ref="CB8401"  Part="1"
+AR Path="/D1BB8DB4/5F317CB5/60365C41/D2F4D9AA" Ref="CB8501"  Part="1"
+AR Path="/D1BB8DB4/5F317CB5/60365C49/D2F4D9AA" Ref="CB8601"  Part="1"
+AR Path="/D1BB8DB4/5F746103/60365C39/D2F4D9AA" Ref="CB5701"  Part="1"
+AR Path="/D1BB8DB4/5F746103/60365C41/D2F4D9AA" Ref="CB5801"  Part="1"
+AR Path="/D1BB8DB4/5F746103/60365C49/D2F4D9AA" Ref="CB5901"  Part="1"
+AR Path="/D1BB8DB4/5F746103/60365C53/D2F4D9AA" Ref="CB6001"  Part="1"
+F 0 "CB8501" V 6700 3000 50  0000 R CNN
+F 1 "T9-818 6A" V 6600 3000 50  0000 R CNN
 F 2 "BoatControl:Schurter_Circuit_Breaker" H 6650 3550 50  0001 C CNN
 F 3 "https://eu.mouser.com/datasheet/2/358/typ_T9-818-1276014.pdf" H 6650 3550 50  0001 C CNN
@@
 AR Path="/D1BB8DB4/5F746103/60365C49/D2F4D9AB" Ref="SW5901"  Part="1"
 AR Path="/D1BB8DB4/5F746103/60365C53/D2F4D9AB" Ref="SW6001"  Part="1"
-F 0 "SW8601" H 4250 4750 50  0000 C CNN
+F 0 "SW8501" H 4250 4750 50  0000 C CNN
 F 1 " ESB30" H 4250 3800 50  0000 C CNN
 F 2 "BoatControl:SW_PUSH_ESB30_DPDT" H 4500 3950 50  0001 C CNN
@@
 AR Path="/D1BB8DB4/5F746103/60365C49/D2F4D9A9" Ref="SW5902"  Part="1"
 AR Path="/D1BB8DB4/5F746103/60365C53/D2F4D9A9" Ref="SW6002"  Part="1"
-F 0 "SW8602" H 4200 5900 50  0000 C CNN
+F 0 "SW8502" H 4200 5900 50  0000 C CNN
 F 1 " ESB30" H 4300 4750 50  0000 C CNN
 F 2 "BoatControl:SW_PUSH_ESB30_DPDT" H 4500 5000 50  0001 C CNN
@@
 AR Path="/D1BB8DB4/5F75E923/60474907/60D74A5A" Ref="#PWR?"  Part="1"
 AR Path="/D1BB8DB4/5F75E923/60474911/60D74A5A" Ref="#PWR?"  Part="1"
-F 0 "#PWR0151" H 6150 4100 50  0001 C CNN
+F 0 "#PWR0149" H 6150 4100 50  0001 C CNN
 F 1 "+12P" H 6165 4423 50  0000 C CNN
 F 2 "" H 6150 4250 50  0001 C CNN
@@
 AR Path="/D1BB8DB4/5F75E923/60474907/60D74A7B" Ref="#PWR?"  Part="1"
 AR Path="/D1BB8DB4/5F75E923/60474911/60D74A7B" Ref="#PWR?"  Part="1"
-F 0 "#PWR0152" H 3950 4850 50  0001 C CNN
+F 0 "#PWR0150" H 3950 4850 50  0001 C CNN
 F 1 "GND" H 3955 4927 50  0000 C CNN
 F 2 "" H 3950 5100 50  0001 C CNN

Commit message: Cleanup
Parts:
- D8701: symbol Device:LED_Dual_ACA -> boatcontrol-rescue:LED_Dual_ACA-Device
Changed lines of the file:
@@
 $EndDescr
 $Comp
-L Device:LED_Dual_ACA D?
+L boatcontrol-rescue:LED_Dual_ACA-Device D?
 U 1 1 D2F4D9A7
 P 5600 4250
@@
 AR Path="/D1BB8DB4/5F746103/60365C49/D2F4D9A7" Ref="D5901"  Part="1"
 AR Path="/D1BB8DB4/5F746103/60365C53/D2F4D9A7" Ref="D6001"  Part="1"
-F 0 "D8501" H 5400 4100 50  0000 C CNN
+F 0 "D8601" H 5400 4100 50  0000 C CNN
 F 1 "20mA R/G CA" H 5550 4000 50  0000 C CNN
 F 2 "LED_THT:LED_D5.0mm-3" H 5600 4250 50  0001 C CNN
@@
 AR Path="/D1BB8DB4/5F746103/60365C49/D2F4DB56" Ref="K5901"  Part="1"
 AR Path="/D1BB8DB4/5F746103/60365C53/D2F4DB56" Ref="K6001"  Part="1"
-F 0 "K8501" H 6750 4250 50  0000 L CNN
+F 0 "K8601" H 6750 4250 50  0000 L CNN
 F 1 "G5RL-K1A-E-DC12" H 7100 4250 50  0000 L CNN
 F 2 "RELAY_G5RL-K1A-E-DC12" H 7100 4400 50  0001 L BNN
@@
 AR Path="/D1BB8DB4/5F746103/60365C49/D2F4D9AA" Ref="CB5901"  Part="1"
 AR Path="/D1BB8DB4/5F746103/60365C53/D2F4D9AA" Ref="CB6001"  Part="1"
-F 0 "CB8501" V 6700 3000 50  0000 R CNN
+F 0 "CB8601" V 6700 3000 50  0000 R CNN
 F 1 "T9-818 6A" V 6600 3000 50  0000 R CNN
 F 2 "BoatControl:Schurter_Circuit_Breaker" H 6650 3550 50  0001 C CNN
@@
 AR Path="/D1BB8DB4/5F746103/60365C49/D2F4D9AB" Ref="SW5901"  Part="1"
 AR Path="/D1BB8DB4/5F746103/60365C53/D2F4D9AB" Ref="SW6001"  Part="1"
-F 0 "SW8501" H 4250 4750 50  0000 C CNN
+F 0 "SW8601" H 4250 4750 50  0000 C CNN
 F 1 " ESB30" H 4250 3800 50  0000 C CNN
 F 2 "BoatControl:SW_PUSH_ESB30_DPDT" H 4500 3950 50  0001 C CNN
@@
 AR Path="/D1BB8DB4/5F746103/60365C49/D2F4D9A9" Ref="SW5902"  Part="1"
 AR Path="/D1BB8DB4/5F746103/60365C53/D2F4D9A9" Ref="SW6002"  Part="1"
-F 0 "SW8502" H 4200 5900 50  0000 C CNN
+F 0 "SW8602" H 4200 5900 50  0000 C CNN
 F 1 " ESB30" H 4300 4750 50  0000 C CNN
 F 2 "BoatControl:SW_PUSH_ESB30_DPDT" H 4500 5000 50  0001 C CNN
@@
 AR Path="/D1BB8DB4/5F75E923/60474907/60D74A5A" Ref="#PWR?"  Part="1"
 AR Path="/D1BB8DB4/5F75E923/60474911/60D74A5A" Ref="#PWR?"  Part="1"
-F 0 "#PWR0149" H 6150 4100 50  0001 C CNN
+F 0 "#PWR0151" H 6150 4100 50  0001 C CNN
 F 1 "+12P" H 6165 4423 50  0000 C CNN
 F 2 "" H 6150 4250 50  0001 C CNN
@@
 AR Path="/D1BB8DB4/5F75E923/60474907/60D74A7B" Ref="#PWR?"  Part="1"
 AR Path="/D1BB8DB4/5F75E923/60474911/60D74A7B" Ref="#PWR?"  Part="1"
-F 0 "#PWR0150" H 3950 4850 50  0001 C CNN
+F 0 "#PWR0152" H 3950 4850 50  0001 C CNN
 F 1 "GND" H 3955 4927 50  0000 C CNN
 F 2 "" H 3950 5100 50  0001 C CNN

Commit message: Fits
Changed lines of the file:
@@
 $Descr A4 11693 8268
 encoding utf-8
-Sheet 83 97
+Sheet 47 97
 Title "Boat Control Hat"
 Date "2020-07-09"
@@
 AR Path="/D1BB8DB4/5F746103/60365C49/D2F4D9A7" Ref="D5901"  Part="1"
 AR Path="/D1BB8DB4/5F746103/60365C53/D2F4D9A7" Ref="D6001"  Part="1"
-F 0 "D8601" H 5400 4100 50  0000 C CNN
+F 0 "D5701" H 5400 4100 50  0000 C CNN
 F 1 "20mA R/G CA" H 5550 4000 50  0000 C CNN
 F 2 "LED_THT:LED_D5.0mm-3" H 5600 4250 50  0001 C CNN
@@
 AR Path="/D1BB8DB4/5F746103/60365C49/D2F4DB56" Ref="K5901"  Part="1"
 AR Path="/D1BB8DB4/5F746103/60365C53/D2F4DB56" Ref="K6001"  Part="1"
-F 0 "K8601" H 6750 4250 50  0000 L CNN
+F 0 "K5701" H 6750 4250 50  0000 L CNN
 F 1 "G5RL-K1A-E-DC12" H 7100 4250 50  0000 L CNN
 F 2 "RELAY_G5RL-K1A-E-DC12" H 7100 4400 50  0001 L BNN
@@
 AR Path="/D1BB8DB4/5F746103/60365C49/D2F4D9AA" Ref="CB5901"  Part="1"
 AR Path="/D1BB8DB4/5F746103/60365C53/D2F4D9AA" Ref="CB6001"  Part="1"
-F 0 "CB8601" V 6700 3000 50  0000 R CNN
+F 0 "CB5701" V 6700 3000 50  0000 R CNN
 F 1 "T9-818 6A" V 6600 3000 50  0000 R CNN
 F 2 "BoatControl:Schurter_Circuit_Breaker" H 6650 3550 50  0001 C CNN
@@
 AR Path="/D1BB8DB4/5F746103/60365C49/D2F4D9AB" Ref="SW5901"  Part="1"
 AR Path="/D1BB8DB4/5F746103/60365C53/D2F4D9AB" Ref="SW6001"  Part="1"
-F 0 "SW8601" H 4250 4750 50  0000 C CNN
+F 0 "SW5701" H 4250 4750 50  0000 C CNN
 F 1 " ESB30" H 4250 3800 50  0000 C CNN
 F 2 "BoatControl:SW_PUSH_ESB30_DPDT" H 4500 3950 50  0001 C CNN
@@
 AR Path="/D1BB8DB4/5F746103/60365C49/D2F4D9A9" Ref="SW5902"  Part="1"
 AR Path="/D1BB8DB4/5F746103/60365C53/D2F4D9A9" Ref="SW6002"  Part="1"
-F 0 "SW8602" H 4200 5900 50  0000 C CNN
+F 0 "SW5702" H 4200 5900 50  0000 C CNN
 F 1 " ESB30" H 4300 4750 50  0000 C CNN
 F 2 "BoatControl:SW_PUSH_ESB30_DPDT" H 4500 5000 50  0001 C CNN

Commit message: Fix silkscreen logos and graphics
Changed lines of the file:
@@
 AR Path="/D1BB8DB4/5F746103/60365C49/D2F4D9A7" Ref="D5901"  Part="1"
 AR Path="/D1BB8DB4/5F746103/60365C53/D2F4D9A7" Ref="D6001"  Part="1"
-F 0 "D5701" H 5400 4100 50  0000 C CNN
+F 0 "D8601" H 5400 4100 50  0000 C CNN
 F 1 "20mA R/G CA" H 5550 4000 50  0000 C CNN
 F 2 "LED_THT:LED_D5.0mm-3" H 5600 4250 50  0001 C CNN
@@
 AR Path="/D1BB8DB4/5F746103/60365C49/D2F4DB56" Ref="K5901"  Part="1"
 AR Path="/D1BB8DB4/5F746103/60365C53/D2F4DB56" Ref="K6001"  Part="1"
-F 0 "K5701" H 6750 4250 50  0000 L CNN
+F 0 "K8601" H 6750 4250 50  0000 L CNN
 F 1 "G5RL-K1A-E-DC12" H 7100 4250 50  0000 L CNN
 F 2 "RELAY_G5RL-K1A-E-DC12" H 7100 4400 50  0001 L BNN
@@
 AR Path="/D1BB8DB4/5F746103/60365C49/D2F4D9AA" Ref="CB5901"  Part="1"
 AR Path="/D1BB8DB4/5F746103/60365C53/D2F4D9AA" Ref="CB6001"  Part="1"
-F 0 "CB5701" V 6700 3000 50  0000 R CNN
+F 0 "CB8601" V 6700 3000 50  0000 R CNN
 F 1 "T9-818 6A" V 6600 3000 50  0000 R CNN
 F 2 "BoatControl:Schurter_Circuit_Breaker" H 6650 3550 50  0001 C CNN
@@
 AR Path="/D1BB8DB4/5F746103/60365C49/D2F4D9AB" Ref="SW5901"  Part="1"
 AR Path="/D1BB8DB4/5F746103/60365C53/D2F4D9AB" Ref="SW6001"  Part="1"
-F 0 "SW5701" H 4250 4750 50  0000 C CNN
+F 0 "SW8601" H 4250 4750 50  0000 C CNN
 F 1 " ESB30" H 4250 3800 50  0000 C CNN
 F 2 "BoatControl:SW_PUSH_ESB30_DPDT" H 4500 3950 50  0001 C CNN
@@
 AR Path="/D1BB8DB4/5F746103/60365C49/D2F4D9A9" Ref="SW5902"  Part="1"
 AR Path="/D1BB8DB4/5F746103/60365C53/D2F4D9A9" Ref="SW6002"  Part="1"
-F 0 "SW5702" H 4200 5900 50  0000 C CNN
+F 0 "SW8602" H 4200 5900 50  0000 C CNN
 F 1 " ESB30" H 4300 4750 50  0000 C CNN
 F 2 "BoatControl:SW_PUSH_ESB30_DPDT" H 4500 5000 50  0001 C CNN

Commit message: shuffle
Changed lines of the file:
@@
 $Descr A4 11693 8268
 encoding utf-8
-Sheet 47 97
+Sheet 74 97
 Title "Boat Control Hat"
 Date "2020-07-09"
@@
 AR Path="/D1BB8DB4/5F746103/60365C49/D2F4D9A7" Ref="D5901"  Part="1"
 AR Path="/D1BB8DB4/5F746103/60365C53/D2F4D9A7" Ref="D6001"  Part="1"
-F 0 "D8601" H 5400 4100 50  0000 C CNN
+F 0 "D8401" H 5400 4100 50  0000 C CNN
 F 1 "20mA R/G CA" H 5550 4000 50  0000 C CNN
 F 2 "LED_THT:LED_D5.0mm-3" H 5600 4250 50  0001 C CNN
@@
 AR Path="/D1BB8DB4/5F746103/60365C49/D2F4DB56" Ref="K5901"  Part="1"
 AR Path="/D1BB8DB4/5F746103/60365C53/D2F4DB56" Ref="K6001"  Part="1"
-F 0 "K8601" H 6750 4250 50  0000 L CNN
+F 0 "K8401" H 6750 4250 50  0000 L CNN
 F 1 "G5RL-K1A-E-DC12" H 7100 4250 50  0000 L CNN
 F 2 "RELAY_G5RL-K1A-E-DC12" H 7100 4400 50  0001 L BNN
@@
 AR Path="/D1BB8DB4/5F746103/60365C49/D2F4D9AA" Ref="CB5901"  Part="1"
 AR Path="/D1BB8DB4/5F746103/60365C53/D2F4D9AA" Ref="CB6001"  Part="1"
-F 0 "CB8601" V 6700 3000 50  0000 R CNN
+F 0 "CB8401" V 6700 3000 50  0000 R CNN
 F 1 "T9-818 6A" V 6600 3000 50  0000 R CNN
 F 2 "BoatControl:Schurter_Circuit_Breaker" H 6650 3550 50  0001 C CNN
@@
 AR Path="/D1BB8DB4/5F746103/60365C49/D2F4D9AB" Ref="SW5901"  Part="1"
 AR Path="/D1BB8DB4/5F746103/60365C53/D2F4D9AB" Ref="SW6001"  Part="1"
-F 0 "SW8601" H 4250 4750 50  0000 C CNN
+F 0 "SW8401" H 4250 4750 50  0000 C CNN
 F 1 " ESB30" H 4250 3800 50  0000 C CNN
 F 2 "BoatControl:SW_PUSH_ESB30_DPDT" H 4500 3950 50  0001 C CNN
@@
 AR Path="/D1BB8DB4/5F746103/60365C49/D2F4D9A9" Ref="SW5902"  Part="1"
 AR Path="/D1BB8DB4/5F746103/60365C53/D2F4D9A9" Ref="SW6002"  Part="1"
-F 0 "SW8602" H 4200 5900 50  0000 C CNN
+F 0 "SW8402" H 4200 5900 50  0000 C CNN
 F 1 " ESB30" H 4300 4750 50  0000 C CNN
 F 2 "BoatControl:SW_PUSH_ESB30_DPDT" H 4500 5000 50  0001 C CNN
@@
 AR Path="/D1BB8DB4/5F75E923/60474907/60D74A5A" Ref="#PWR?"  Part="1"
 AR Path="/D1BB8DB4/5F75E923/60474911/60D74A5A" Ref="#PWR?"  Part="1"
-F 0 "#PWR0151" H 6150 4100 50  0001 C CNN
+F 0 "#PWR0147" H 6150 4100 50  0001 C CNN
 F 1 "+12P" H 6165 4423 50  0000 C CNN
 F 2 "" H 6150 4250 50  0001 C CNN
@@
 AR Path="/D1BB8DB4/5F75E923/60474907/60D74A7B" Ref="#PWR?"  Part="1"
 AR Path="/D1BB8DB4/5F75E923/60474911/60D74A7B" Ref="#PWR?"  Part="1"
-F 0 "#PWR0152" H 3950 4850 50  0001 C CNN
+F 0 "#PWR0148" H 3950 4850 50  0001 C CNN
 F 1 "GND" H 3955 4927 50  0000 C CNN
 F 2 "" H 3950 5100 50  0001 C CNN
