File: boatcontrol/CircuitControl.sch (KiCad schematic (older format))
At the start: 3 parts, among them SW4101 ESB30, SW4102 ESB30

Commit message: Fix SB footprint and symbol
Changed lines of the file:
@@
 $Descr A4 11693 8268
 encoding utf-8
-Sheet 7 97
+Sheet 4 97
 Title "Boat Control Hat"
 Date "2020-07-09"
@@
 AR Path="/601318CC/E15855D9/E150FD51/E13B21A8" Ref="SW9601"  Part="1"
 AR Path="/601318CC/E15855D9/E150AEB9/E13B21A8" Ref="SW9701"  Part="1"
-F 0 "SW9201" H 5500 3900 50  0000 C CNN
+F 0 "SW8901" H 5500 3900 50  0000 C CNN
 F 1 " ESB30" H 5550 4000 50  0000 C CNN
 F 2 "BoatControl:SW_PUSH_ESB30_DPDT" H 5750 4150 50  0001 C CNN
@@
 AR Path="/601318CC/E15855D9/E150FD51/E13B21B4" Ref="SW9602"  Part="1"
 AR Path="/601318CC/E15855D9/E150AEB9/E13B21B4" Ref="SW9702"  Part="1"
-F 0 "SW9202" H 5450 5050 50  0000 C CNN
+F 0 "SW8902" H 5450 5050 50  0000 C CNN
 F 1 " ESB30" H 5500 4950 50  0000 C CNN
 F 2 "BoatControl:SW_PUSH_ESB30_DPDT" H 5750 5200 50  0001 C CNN
@@
 AR Path="/601318CC/E15855D9/E150FD51/E13B21BC" Ref="D9601"  Part="1"
 AR Path="/601318CC/E15855D9/E150AEB9/E13B21BC" Ref="D9701"  Part="1"
-F 0 "D9201" H 6650 4250 50  0000 C CNN
+F 0 "D8901" H 6650 4250 50  0000 C CNN
 F 1 "20mA R/G CC" H 6800 4150 50  0000 C CNN
 F 2 "LED_THT:LED_D5.0mm-3" H 6850 4450 50  0001 C CNN

Commit message: Cleanup
Parts:
- D4101: symbol Device:LED_Dual_ACA -> boatcontrol-rescue:LED_Dual_ACA-Device
Changed lines of the file:
@@
 AR Path="/601318CC/E15855D9/E150FD51/E13B21A8" Ref="SW9601"  Part="1"
 AR Path="/601318CC/E15855D9/E150AEB9/E13B21A8" Ref="SW9701"  Part="1"
-F 0 "SW8901" H 5500 3900 50  0000 C CNN
+F 0 "SW4902" H 5500 3900 50  0000 C CNN
 F 1 " ESB30" H 5550 4000 50  0000 C CNN
 F 2 "BoatControl:SW_PUSH_ESB30_DPDT" H 5750 4150 50  0001 C CNN
@@
 AR Path="/601318CC/E15855D9/E150FD51/E13B21B4" Ref="SW9602"  Part="1"
 AR Path="/601318CC/E15855D9/E150AEB9/E13B21B4" Ref="SW9702"  Part="1"
-F 0 "SW8902" H 5450 5050 50  0000 C CNN
+F 0 "SW4901" H 5450 5050 50  0000 C CNN
 F 1 " ESB30" H 5500 4950 50  0000 C CNN
 F 2 "BoatControl:SW_PUSH_ESB30_DPDT" H 5750 5200 50  0001 C CNN
@@
 $EndComp
 $Comp
-L Device:LED_Dual_ACA D?
+L boatcontrol-rescue:LED_Dual_ACA-Device D?
 U 1 1 E13B21BC
 P 6850 4450
@@
 AR Path="/601318CC/E15855D9/E150FD51/E13B21BC" Ref="D9601"  Part="1"
 AR Path="/601318CC/E15855D9/E150AEB9/E13B21BC" Ref="D9701"  Part="1"
-F 0 "D8901" H 6650 4250 50  0000 C CNN
+F 0 "D4901" H 6650 4250 50  0000 C CNN
 F 1 "20mA R/G CC" H 6800 4150 50  0000 C CNN
 F 2 "LED_THT:LED_D5.0mm-3" H 6850 4450 50  0001 C CNN

Commit message: Newcluster
Changed lines of the file:
@@
 $Descr A4 11693 8268
 encoding utf-8
-Sheet 4 97
+Sheet 96 97
 Title "Boat Control Hat"
 Date "2020-07-09"
@@
 AR Path="/601318CC/E15855D9/E150FD51/E13B21A8" Ref="SW9601"  Part="1"
 AR Path="/601318CC/E15855D9/E150AEB9/E13B21A8" Ref="SW9701"  Part="1"
-F 0 "SW4902" H 5500 3900 50  0000 C CNN
+F 0 "SW4802" H 5500 3900 50  0000 C CNN
 F 1 " ESB30" H 5550 4000 50  0000 C CNN
 F 2 "BoatControl:SW_PUSH_ESB30_DPDT" H 5750 4150 50  0001 C CNN
@@
 AR Path="/601318CC/E15855D9/E150FD51/E13B21AE" Ref="#PWR0227"  Part="1"
 AR Path="/601318CC/E15855D9/E150AEB9/E13B21AE" Ref="#PWR0229"  Part="1"
-F 0 "#PWR04901" H 4300 4300 50  0001 C CNN
+F 0 "#PWR04801" H 4300 4300 50  0001 C CNN
 F 1 "+12P" V 4300 4700 50  0000 C CNN
 F 2 "" H 4300 4450 50  0001 C CNN
@@
 AR Path="/601318CC/E15855D9/E150FD51/E13B21B4" Ref="SW9602"  Part="1"
 AR Path="/601318CC/E15855D9/E150AEB9/E13B21B4" Ref="SW9702"  Part="1"
-F 0 "SW4901" H 5450 5050 50  0000 C CNN
+F 0 "SW4801" H 5450 5050 50  0000 C CNN
 F 1 " ESB30" H 5500 4950 50  0000 C CNN
 F 2 "BoatControl:SW_PUSH_ESB30_DPDT" H 5750 5200 50  0001 C CNN
@@
 AR Path="/601318CC/E15855D9/E150FD51/E13B21BC" Ref="D9601"  Part="1"
 AR Path="/601318CC/E15855D9/E150AEB9/E13B21BC" Ref="D9701"  Part="1"
-F 0 "D4901" H 6650 4250 50  0000 C CNN
+F 0 "D4801" H 6650 4250 50  0000 C CNN
 F 1 "20mA R/G CC" H 6800 4150 50  0000 C CNN
 F 2 "LED_THT:LED_D5.0mm-3" H 6850 4450 50  0001 C CNN
@@
 AR Path="/601318CC/E15855D9/E150FD51/5F521E18" Ref="#PWR0228"  Part="1"
 AR Path="/601318CC/E15855D9/E150AEB9/5F521E18" Ref="#PWR0230"  Part="1"
-F 0 "#PWR04902" H 7250 4200 50  0001 C CNN
+F 0 "#PWR04802" H 7250 4200 50  0001 C CNN
 F 1 "GND" V 7255 4322 50  0000 R CNN
 F 2 "" H 7250 4450 50  0001 C CNN

Commit message: organized
Changed lines of the file:
@@
 $Descr A4 11693 8268
 encoding utf-8
-Sheet 96 97
+Sheet 79 97
 Title "Boat Control Hat"
 Date "2020-07-09"
@@
 AR Path="/601318CC/E15855D9/E150FD51/E13B21A8" Ref="SW9601"  Part="1"
 AR Path="/601318CC/E15855D9/E150AEB9/E13B21A8" Ref="SW9701"  Part="1"
-F 0 "SW4802" H 5500 3900 50  0000 C CNN
+F 0 "SW9001" H 5500 3900 50  0000 C CNN
 F 1 " ESB30" H 5550 4000 50  0000 C CNN
 F 2 "BoatControl:SW_PUSH_ESB30_DPDT" H 5750 4150 50  0001 C CNN
@@
 AR Path="/601318CC/E15855D9/E150FD51/E13B21AE" Ref="#PWR0227"  Part="1"
 AR Path="/601318CC/E15855D9/E150AEB9/E13B21AE" Ref="#PWR0229"  Part="1"
-F 0 "#PWR04801" H 4300 4300 50  0001 C CNN
+F 0 "#PWR04901" H 4300 4300 50  0001 C CNN
 F 1 "+12P" V 4300 4700 50  0000 C CNN
 F 2 "" H 4300 4450 50  0001 C CNN
@@
 AR Path="/601318CC/E15855D9/E150FD51/E13B21B4" Ref="SW9602"  Part="1"
 AR Path="/601318CC/E15855D9/E150AEB9/E13B21B4" Ref="SW9702"  Part="1"
-F 0 "SW4801" H 5450 5050 50  0000 C CNN
+F 0 "SW9002" H 5450 5050 50  0000 C CNN
 F 1 " ESB30" H 5500 4950 50  0000 C CNN
 F 2 "BoatControl:SW_PUSH_ESB30_DPDT" H 5750 5200 50  0001 C CNN
@@
 AR Path="/601318CC/E15855D9/E150FD51/E13B21BC" Ref="D9601"  Part="1"
 AR Path="/601318CC/E15855D9/E150AEB9/E13B21BC" Ref="D9701"  Part="1"
-F 0 "D4801" H 6650 4250 50  0000 C CNN
+F 0 "D9001" H 6650 4250 50  0000 C CNN
 F 1 "20mA R/G CC" H 6800 4150 50  0000 C CNN
 F 2 "LED_THT:LED_D5.0mm-3" H 6850 4450 50  0001 C CNN
@@
 AR Path="/601318CC/E15855D9/E150FD51/5F521E18" Ref="#PWR0228"  Part="1"
 AR Path="/601318CC/E15855D9/E150AEB9/5F521E18" Ref="#PWR0230"  Part="1"
-F 0 "#PWR04802" H 7250 4200 50  0001 C CNN
+F 0 "#PWR04902" H 7250 4200 50  0001 C CNN
 F 1 "GND" V 7255 4322 50  0000 R CNN
 F 2 "" H 7250 4450 50  0001 C CNN

Commit message: better
Changed lines of the file:
@@
 $Descr A4 11693 8268
 encoding utf-8
-Sheet 79 97
+Sheet 85 97
 Title "Boat Control Hat"
 Date "2020-07-09"
@@
 AR Path="/601318CC/E15855D9/E150FD51/E13B21A8" Ref="SW9601"  Part="1"
 AR Path="/601318CC/E15855D9/E150AEB9/E13B21A8" Ref="SW9701"  Part="1"
-F 0 "SW9001" H 5500 3900 50  0000 C CNN
+F 0 "SW9601" H 5500 3900 50  0000 C CNN
 F 1 " ESB30" H 5550 4000 50  0000 C CNN
 F 2 "BoatControl:SW_PUSH_ESB30_DPDT" H 5750 4150 50  0001 C CNN
@@
 AR Path="/601318CC/E15855D9/E150FD51/E13B21B4" Ref="SW9602"  Part="1"
 AR Path="/601318CC/E15855D9/E150AEB9/E13B21B4" Ref="SW9702"  Part="1"
-F 0 "SW9002" H 5450 5050 50  0000 C CNN
+F 0 "SW9602" H 5450 5050 50  0000 C CNN
 F 1 " ESB30" H 5500 4950 50  0000 C CNN
 F 2 "BoatControl:SW_PUSH_ESB30_DPDT" H 5750 5200 50  0001 C CNN
@@
 AR Path="/601318CC/E15855D9/E150FD51/E13B21BC" Ref="D9601"  Part="1"
 AR Path="/601318CC/E15855D9/E150AEB9/E13B21BC" Ref="D9701"  Part="1"
-F 0 "D9001" H 6650 4250 50  0000 C CNN
+F 0 "D9601" H 6650 4250 50  0000 C CNN
 F 1 "20mA R/G CC" H 6800 4150 50  0000 C CNN
 F 2 "LED_THT:LED_D5.0mm-3" H 6850 4450 50  0001 C CNN

Commit message: Fix rescued symbols
Parts:
- D4101: symbol boatcontrol-rescue:LED_Dual_ACA-Device -> Device:LED_Dual_AKA
Changed lines of the file:
@@
 $EndComp
 $Comp
-L boatcontrol-rescue:LED_Dual_ACA-Device D?
+L Device:LED_Dual_AKA D?
 U 1 1 E13B21BC
 P 6850 4450

Commit message: More cleanup
Changed lines of the file:
@@
 AR Path="/601318CC/E15855D9/E150FD51/E13B21A8" Ref="SW9601"  Part="1"
 AR Path="/601318CC/E15855D9/E150AEB9/E13B21A8" Ref="SW9701"  Part="1"
-F 0 "SW9601" H 5500 3900 50  0000 C CNN
+AR Path="/626FCFE3/E142CD30/E14BA326/E13B21A8" Ref="SW?"  Part="1"
+AR Path="/626FCFE3/E142CD30/E150D6D7/E13B21A8" Ref="SW?"  Part="1"
+AR Path="/626FCFE3/E142CD30/E150FD51/E13B21A8" Ref="SW?"  Part="1"
+AR Path="/626FCFE3/E142CD30/E150AEB9/E13B21A8" Ref="SW?"  Part="1"
+AR Path="/626FCFE3/E15855D9/E14BA326/E13B21A8" Ref="SW?"  Part="1"
+AR Path="/626FCFE3/E15855D9/E150D6D7/E13B21A8" Ref="SW?"  Part="1"
+AR Path="/626FCFE3/E15855D9/E150FD51/E13B21A8" Ref="SW?"  Part="1"
+AR Path="/626FCFE3/E15855D9/E150AEB9/E13B21A8" Ref="SW?"  Part="1"
+AR Path="/626FD005/E142CD30/E14BA326/E13B21A8" Ref="SW?"  Part="1"
+AR Path="/626FD005/E142CD30/E150D6D7/E13B21A8" Ref="SW?"  Part="1"
+AR Path="/626FD005/E142CD30/E150FD51/E13B21A8" Ref="SW?"  Part="1"
+AR Path="/626FD005/E142CD30/E150AEB9/E13B21A8" Ref="SW?"  Part="1"
+AR Path="/626FD005/E15855D9/E14BA326/E13B21A8" Ref="SW?"  Part="1"
+AR Path="/626FD005/E15855D9/E150D6D7/E13B21A8" Ref="SW?"  Part="1"
+AR Path="/626FD005/E15855D9/E150FD51/E13B21A8" Ref="SW?"  Part="1"
+AR Path="/626FD005/E15855D9/E150AEB9/E13B21A8" Ref="SW?"  Part="1"
+F 0 "SW?" H 5500 3900 50  0000 C CNN
 F 1 " ESB30" H 5550 4000 50  0000 C CNN
 F 2 "BoatControl:SW_PUSH_ESB30_DPDT" H 5750 4150 50  0001 C CNN
@@
 AR Path="/601318CC/E15855D9/E150FD51/E13B21AE" Ref="#PWR0227"  Part="1"
 AR Path="/601318CC/E15855D9/E150AEB9/E13B21AE" Ref="#PWR0229"  Part="1"
-F 0 "#PWR04901" H 4300 4300 50  0001 C CNN
+AR Path="/626FCFE3/E142CD30/E14BA326/E13B21AE" Ref="#PWR?"  Part="1"
+AR Path="/626FCFE3/E142CD30/E150D6D7/E13B21AE" Ref="#PWR?"  Part="1"
+AR Path="/626FCFE3/E142CD30/E150FD51/E13B21AE" Ref="#PWR?"  Part="1"
+AR Path="/626FCFE3/E142CD30/E150AEB9/E13B21AE" Ref="#PWR?"  Part="1"
+AR Path="/626FCFE3/E15855D9/E14BA326/E13B21AE" Ref="#PWR?"  Part="1"
+AR Path="/626FCFE3/E15855D9/E150D6D7/E13B21AE" Ref="#PWR?"  Part="1"
+AR Path="/626FCFE3/E15855D9/E150FD51/E13B21AE" Ref="#PWR?"  Part="1"
+AR Path="/626FCFE3/E15855D9/E150AEB9/E13B21AE" Ref="#PWR?"  Part="1"
+AR Path="/626FD005/E142CD30/E14BA326/E13B21AE" Ref="#PWR?"  Part="1"
+AR Path="/626FD005/E142CD30/E150D6D7/E13B21AE" Ref="#PWR?"  Part="1"
+AR Path="/626FD005/E142CD30/E150FD51/E13B21AE" Ref="#PWR?"  Part="1"
+AR Path="/626FD005/E142CD30/E150AEB9/E13B21AE" Ref="#PWR?"  Part="1"
+AR Path="/626FD005/E15855D9/E14BA326/E13B21AE" Ref="#PWR?"  Part="1"
+AR Path="/626FD005/E15855D9/E150D6D7/E13B21AE" Ref="#PWR?"  Part="1"
+AR Path="/626FD005/E15855D9/E150FD51/E13B21AE" Ref="#PWR?"  Part="1"
+AR Path="/626FD005/E15855D9/E150AEB9/E13B21AE" Ref="#PWR?"  Part="1"
+F 0 "#PWR?" H 4300 4300 50  0001 C CNN
 F 1 "+12P" V 4300 4700 50  0000 C CNN
 F 2 "" H 4300 4450 50  0001 C CNN
@@
 AR Path="/601318CC/E15855D9/E150FD51/E13B21B4" Ref="SW9602"  Part="1"
 AR Path="/601318CC/E15855D9/E150AEB9/E13B21B4" Ref="SW9702"  Part="1"
-F 0 "SW9602" H 5450 5050 50  0000 C CNN
+AR Path="/626FCFE3/E142CD30/E14BA326/E13B21B4" Ref="SW?"  Part="1"
+AR Path="/626FCFE3/E142CD30/E150D6D7/E13B21B4" Ref="SW?"  Part="1"
+AR Path="/626FCFE3/E142CD30/E150FD51/E13B21B4" Ref="SW?"  Part="1"
+AR Path="/626FCFE3/E142CD30/E150AEB9/E13B21B4" Ref="SW?"  Part="1"
+AR Path="/626FCFE3/E15855D9/E14BA326/E13B21B4" Ref="SW?"  Part="1"
+AR Path="/626FCFE3/E15855D9/E150D6D7/E13B21B4" Ref="SW?"  Part="1"
+AR Path="/626FCFE3/E15855D9/E150FD51/E13B21B4" Ref="SW?"  Part="1"
+AR Path="/626FCFE3/E15855D9/E150AEB9/E13B21B4" Ref="SW?"  Part="1"
+AR Path="/626FD005/E142CD30/E14BA326/E13B21B4" Ref="SW?"  Part="1"
+AR Path="/626FD005/E142CD30/E150D6D7/E13B21B4" Ref="SW?"  Part="1"
+AR Path="/626FD005/E142CD30/E150FD51/E13B21B4" Ref="SW?"  Part="1"
+AR Path="/626FD005/E142CD30/E150AEB9/E13B21B4" Ref="SW?"  Part="1"
+AR Path="/626FD005/E15855D9/E14BA326/E13B21B4" Ref="SW?"  Part="1"
+AR Path="/626FD005/E15855D9/E150D6D7/E13B21B4" Ref="SW?"  Part="1"
+AR Path="/626FD005/E15855D9/E150FD51/E13B21B4" Ref="SW?"  Part="1"
+AR Path="/626FD005/E15855D9/E150AEB9/E13B21B4" Ref="SW?"  Part="1"
+F 0 "SW?" H 5450 5050 50  0000 C CNN
 F 1 " ESB30" H 5500 4950 50  0000 C CNN
 F 2 "BoatControl:SW_PUSH_ESB30_DPDT" H 5750 5200 50  0001 C CNN
@@
 AR Path="/601318CC/E15855D9/E150FD51/E13B21BC" Ref="D9601"  Part="1"
 AR Path="/601318CC/E15855D9/E150AEB9/E13B21BC" Ref="D9701"  Part="1"
-F 0 "D9601" H 6650 4250 50  0000 C CNN
+AR Path="/626FCFE3/E142CD30/E14BA326/E13B21BC" Ref="D?"  Part="1"
+AR Path="/626FCFE3/E142CD30/E150D6D7/E13B21BC" Ref="D?"  Part="1"
+AR Path="/626FCFE3/E142CD30/E150FD51/E13B21BC" Ref="D?"  Part="1"
+AR Path="/626FCFE3/E142CD30/E150AEB9/E13B21BC" Ref="D?"  Part="1"
+AR Path="/626FCFE3/E15855D9/E14BA326/E13B21BC" Ref="D?"  Part="1"
+AR Path="/626FCFE3/E15855D9/E150D6D7/E13B21BC" Ref="D?"  Part="1"
+AR Path="/626FCFE3/E15855D9/E150FD51/E13B21BC" Ref="D?"  Part="1"
+AR Path="/626FCFE3/E15855D9/E150AEB9/E13B21BC" Ref="D?"  Part="1"
+AR Path="/626FD005/E142CD30/E14BA326/E13B21BC" Ref="D?"  Part="1"
+AR Path="/626FD005/E142CD30/E150D6D7/E13B21BC" Ref="D?"  Part="1"
+AR Path="/626FD005/E142CD30/E150FD51/E13B21BC" Ref="D?"  Part="1"
+AR Path="/626FD005/E142CD30/E150AEB9/E13B21BC" Ref="D?"  Part="1"
+AR Path="/626FD005/E15855D9/E14BA326/E13B21BC" Ref="D?"  Part="1"
+AR Path="/626FD005/E15855D9/E150D6D7/E13B21BC" Ref="D?"  Part="1"
+AR Path="/626FD005/E15855D9/E150FD51/E13B21BC" Ref="D?"  Part="1"
+AR Path="/626FD005/E15855D9/E150AEB9/E13B21BC" Ref="D?"  Part="1"
+F 0 "D?" H 6650 4250 50  0000 C CNN
 F 1 "20mA R/G CC" H 6800 4150 50  0000 C CNN
 F 2 "LED_THT:LED_D5.0mm-3" H 6850 4450 50  0001 C CNN
@@
 AR Path="/601318CC/E15855D9/E150FD51/5F521E18" Ref="#PWR0228"  Part="1"
 AR Path="/601318CC/E15855D9/E150AEB9/5F521E18" Ref="#PWR0230"  Part="1"
-F 0 "#PWR04902" H 7250 4200 50  0001 C CNN
+AR Path="/626FCFE3/E142CD30/E14BA326/5F521E18" Ref="#PWR?"  Part="1"
+AR Path="/626FCFE3/E142CD30/E150D6D7/5F521E18" Ref="#PWR?"  Part="1"
+AR Path="/626FCFE3/E142CD30/E150FD51/5F521E18" Ref="#PWR?"  Part="1"
+AR Path="/626FCFE3/E142CD30/E150AEB9/5F521E18" Ref="#PWR?"  Part="1"
+AR Path="/626FCFE3/E15855D9/E14BA326/5F521E18" Ref="#PWR?"  Part="1"
+AR Path="/626FCFE3/E15855D9/E150D6D7/5F521E18" Ref="#PWR?"  Part="1"
+AR Path="/626FCFE3/E15855D9/E150FD51/5F521E18" Ref="#PWR?"  Part="1"
+AR Path="/626FCFE3/E15855D9/E150AEB9/5F521E18" Ref="#PWR?"  Part="1"
+AR Path="/626FD005/E142CD30/E14BA326/5F521E18" Ref="#PWR?"  Part="1"
+AR Path="/626FD005/E142CD30/E150D6D7/5F521E18" Ref="#PWR?"  Part="1"
+AR Path="/626FD005/E142CD30/E150FD51/5F521E18" Ref="#PWR?"  Part="1"
+AR Path="/626FD005/E142CD30/E150AEB9/5F521E18" Ref="#PWR?"  Part="1"
+AR Path="/626FD005/E15855D9/E14BA326/5F521E18" Ref="#PWR?"  Part="1"
+AR Path="/626FD005/E15855D9/E150D6D7/5F521E18" Ref="#PWR?"  Part="1"
+AR Path="/626FD005/E15855D9/E150FD51/5F521E18" Ref="#PWR?"  Part="1"
+AR Path="/626FD005/E15855D9/E150AEB9/5F521E18" Ref="#PWR?"  Part="1"
+F 0 "#PWR?" H 7250 4200 50  0001 C CNN
 F 1 "GND" V 7255 4322 50  0000 R CNN
 F 2 "" H 7250 4450 50  0001 C CNN

Commit message: Add xors on input
Changed lines of the file:
@@
 $Descr A4 11693 8268
 encoding utf-8
-Sheet 85 97
+Sheet 89 97
 Title "Boat Control Hat"
 Date "2020-07-09"
@@
 AR Path="/626FD005/E15855D9/E150FD51/E13B21A8" Ref="SW?"  Part="1"
 AR Path="/626FD005/E15855D9/E150AEB9/E13B21A8" Ref="SW?"  Part="1"
-F 0 "SW?" H 5500 3900 50  0000 C CNN
+F 0 "SW4102" H 5500 3900 50  0000 C CNN
 F 1 " ESB30" H 5550 4000 50  0000 C CNN
 F 2 "BoatControl:SW_PUSH_ESB30_DPDT" H 5750 4150 50  0001 C CNN
@@
 AR Path="/626FD005/E15855D9/E150FD51/E13B21AE" Ref="#PWR?"  Part="1"
 AR Path="/626FD005/E15855D9/E150AEB9/E13B21AE" Ref="#PWR?"  Part="1"
-F 0 "#PWR?" H 4300 4300 50  0001 C CNN
+F 0 "#PWR04101" H 4300 4300 50  0001 C CNN
 F 1 "+12P" V 4300 4700 50  0000 C CNN
 F 2 "" H 4300 4450 50  0001 C CNN
@@
 AR Path="/626FD005/E15855D9/E150FD51/E13B21B4" Ref="SW?"  Part="1"
 AR Path="/626FD005/E15855D9/E150AEB9/E13B21B4" Ref="SW?"  Part="1"
-F 0 "SW?" H 5450 5050 50  0000 C CNN
+F 0 "SW4101" H 5450 5050 50  0000 C CNN
 F 1 " ESB30" H 5500 4950 50  0000 C CNN
 F 2 "BoatControl:SW_PUSH_ESB30_DPDT" H 5750 5200 50  0001 C CNN
@@
 AR Path="/626FD005/E15855D9/E150FD51/E13B21BC" Ref="D?"  Part="1"
 AR Path="/626FD005/E15855D9/E150AEB9/E13B21BC" Ref="D?"  Part="1"
-F 0 "D?" H 6650 4250 50  0000 C CNN
+F 0 "D4101" H 6650 4250 50  0000 C CNN
 F 1 "20mA R/G CC" H 6800 4150 50  0000 C CNN
 F 2 "LED_THT:LED_D5.0mm-3" H 6850 4450 50  0001 C CNN
@@
 AR Path="/626FD005/E15855D9/E150FD51/5F521E18" Ref="#PWR?"  Part="1"
 AR Path="/626FD005/E15855D9/E150AEB9/5F521E18" Ref="#PWR?"  Part="1"
-F 0 "#PWR?" H 7250 4200 50  0001 C CNN
+F 0 "#PWR04102" H 7250 4200 50  0001 C CNN
 F 1 "GND" V 7255 4322 50  0000 R CNN
 F 2 "" H 7250 4450 50  0001 C CNN
@@
 	1    0    0    -1
 $EndComp
-Text Notes 2700 3100 0    50   ~ 0
-Buttons offer manual overide of relays using direct 12V.\n\nThere is no timing/pulse  circuit when operating  the switches so care should be taken not to energise relay coils for more than a few seconds.\n\nSetting each coil to "on" will disable the opposing coil to prevent both coils from being energnized at the same time.\n\nMomentary switches are easy to use and recommended.\n\nNon-momentary (latching) switches can be used by "double-clicking" and the advantage of these is that the relay can be disabled completely by setting both swtiches to the "on" position.\n\n
 Text HLabel 6550 4350 0    50   Input ~ 0
 ON_LED
@@
 Wire Wire Line
 	5200 4700 5550 4700
+Text Notes 2700 3100 0    50   ~ 0
+Buttons offer manual overide of relays using direct 12V.\n\nThere is no timing/pulse  circuit when operating  the switches so care should be taken not to energise relay coils for more than a few seconds.\n\nSetting each coil to "on" will disable the opposing coil to prevent both coils from being energnized at the same time.\n\nMomentary switches are easy to use and recommended.\n\nNon-momentary (latching) switches can be used by "double-clicking" and the advantage of these is that the relay can be disabled completely by setting both swtiches to the "on" position.\n\n
 $EndSCHEMATC
