File: boatcontrol/MultiVibratorB.sch (KiCad schematic (older format))
At the start: 5 parts, among them IC401 CD74HCT221E, U302 74HC86

Commit message: Cleaner
Changed lines of the file:
@@
 $Descr A4 11693 8268
 encoding utf-8
-Sheet 35 97
+Sheet 69 97
 Title "Boat Control Hat"
 Date ""
@@
 AR Path="/D1BB8DB4/5F75E923/604747F3/5FD2B9DE" Ref="IC7301"  Part="1"
 AR Path="/D1BB8DB4/5F75E923/604747FF/5FD2B9DE" Ref="IC7401"  Part="1"
-F 0 "IC3401" H 5450 4215 50  0000 C CNN
+F 0 "IC8101" H 5450 4215 50  0000 C CNN
 F 1 "CD74HCT221E" H 5450 4124 50  0000 C CNN
 F 2 "DIP794W53P254L1930H508Q16N" H 5900 4050 50  0001 L CNN
@@
 AR Path="/D1BB8DB4/5F75E923/604747F3/60314A0F" Ref="#PWR07302"  Part="1"
 AR Path="/D1BB8DB4/5F75E923/604747FF/60314A0F" Ref="#PWR07402"  Part="1"
-F 0 "#PWR03402" H 4850 4400 50  0001 C CNN
+F 0 "#PWR08102" H 4850 4400 50  0001 C CNN
 F 1 "GND" H 4700 4600 50  0000 C CNN
 F 2 "" H 4850 4650 50  0001 C CNN
@@
 AR Path="/D1BB8DB4/5F75E923/604747F3/5FD9FC74" Ref="#PWR07301"  Part="1"
 AR Path="/D1BB8DB4/5F75E923/604747FF/5FD9FC74" Ref="#PWR07401"  Part="1"
-F 0 "#PWR03401" H 6050 3800 50  0001 C CNN
+F 0 "#PWR08101" H 6050 3800 50  0001 C CNN
 F 1 "+5V" V 6000 4050 50  0000 L CNN
 F 2 "" H 6050 3950 50  0001 C CNN
@@
 AR Path="/D1BB8DB4/5F317CB5/60365B0F/61CAF5C8" Ref="#PWR0183"  Part="1"
 AR Path="/D1BB8DB4/5F317CB5/60365B35/61CAF5C8" Ref="#PWR0185"  Part="1"
-F 0 "#PWR0170" H 6050 3500 50  0001 C CNN
+F 0 "#PWR0184" H 6050 3500 50  0001 C CNN
 F 1 "GND" V 6055 3622 50  0000 R CNN
 F 2 "" H 6050 3750 50  0001 C CNN
@@
 AR Path="/D1BB8DB4/5F317CB5/60365B0F/61CAE2AB" Ref="C8001"  Part="1"
 AR Path="/D1BB8DB4/5F317CB5/60365B35/61CAE2AB" Ref="C8201"  Part="1"
-F 0 "C3401" H 5900 3650 50  0000 L CNN
+F 0 "C8101" H 5900 3650 50  0000 L CNN
 F 1 "0.1μF" H 6141 3805 50  0001 L CNN
 F 2 "Capacitor_THT:C_Disc_D7.5mm_W5.0mm_P5.00mm" H 6050 3850 50  0001 C CNN
@@
 AR Path="/D1BB8DB4/5F317CB5/60365B29/602120C6" Ref="C8103"  Part="1"
 AR Path="/D1BB8DB4/5F317CB5/60365B41/602120C6" Ref="C8303"  Part="1"
-F 0 "C3403" H 6950 4800 50  0000 L CNN
+F 0 "C8103" H 6950 4800 50  0000 L CNN
 F 1 "1µF" H 6000 4650 50  0001 L CNN
 F 2 "Capacitor_THT:C_Disc_D7.5mm_W5.0mm_P5.00mm" H 6850 4750 50  0001 C CNN
@@
 AR Path="/D1BB8DB4/5F317CB5/60365B29/60314A11" Ref="#PWR0350"  Part="1"
 AR Path="/D1BB8DB4/5F317CB5/60365B41/60314A11" Ref="#PWR0354"  Part="1"
-F 0 "#PWR0293" H 6850 4600 50  0001 C CNN
+F 0 "#PWR0350" H 6850 4600 50  0001 C CNN
 F 1 "GND" H 6855 4677 50  0000 C CNN
 F 2 "" H 6850 4850 50  0001 C CNN
@@
 AR Path="/D1BB8DB4/5F317CB5/60365B29/60216860" Ref="#PWR0351"  Part="1"
 AR Path="/D1BB8DB4/5F317CB5/60365B41/60216860" Ref="#PWR0355"  Part="1"
-F 0 "#PWR0294" H 3650 4100 50  0001 C CNN
+F 0 "#PWR0351" H 3650 4100 50  0001 C CNN
 F 1 "GND" H 3655 4177 50  0000 C CNN
 F 2 "" H 3650 4350 50  0001 C CNN
@@
 AR Path="/D1BB8DB4/5F317CB5/60365B29/6021685A" Ref="C8102"  Part="1"
 AR Path="/D1BB8DB4/5F317CB5/60365B41/6021685A" Ref="C8302"  Part="1"
-F 0 "C3402" H 3300 4300 50  0000 L CNN
+F 0 "C8102" H 3300 4300 50  0000 L CNN
 F 1 "1µF" H 2800 4150 50  0001 L CNN
 F 2 "Capacitor_THT:C_Disc_D7.5mm_W5.0mm_P5.00mm" H 3650 4250 50  0001 C CNN
@@
 AR Path="/D1BB8DB4/5F317CB5/60365B29/604BDC57" Ref="U7902"  Part="3"
 AR Path="/D1BB8DB4/5F317CB5/60365B41/604BDC57" Ref="U7903"  Part="3"
-F 0 "U3003" H 3950 4375 50  0000 C CNN
+F 0 "U7902" H 3950 4375 50  0000 C CNN
 F 1 "74HC86" H 3950 4284 50  0000 C CNN
 F 2 "" H 3950 4050 50  0001 C CNN
@@
 AR Path="/D1BB8DB4/5F317CB5/60365B29/604BF9DE" Ref="U7902"  Part="4"
 AR Path="/D1BB8DB4/5F317CB5/60365B41/604BF9DE" Ref="U7903"  Part="4"
-F 0 "U3003" H 6450 4900 50  0000 C CNN
+F 0 "U7902" H 6450 4900 50  0000 C CNN
 F 1 "74HC86" H 6450 4800 50  0000 C CNN
 F 2 "" H 6550 4550 50  0001 C CNN

Commit message: I give up, SMD resistors for RJ45
Changed lines of the file:
@@
 $Descr A4 11693 8268
 encoding utf-8
-Sheet 69 97
+Sheet 44 97
 Title "Boat Control Hat"
 Date ""
@@
 AR Path="/D1BB8DB4/5F75E923/604747F3/5FD2B9DE" Ref="IC7301"  Part="1"
 AR Path="/D1BB8DB4/5F75E923/604747FF/5FD2B9DE" Ref="IC7401"  Part="1"
-F 0 "IC8101" H 5450 4215 50  0000 C CNN
+F 0 "IC8301" H 5450 4215 50  0000 C CNN
 F 1 "CD74HCT221E" H 5450 4124 50  0000 C CNN
 F 2 "DIP794W53P254L1930H508Q16N" H 5900 4050 50  0001 L CNN
@@
 AR Path="/D1BB8DB4/5F317CB5/60365B0F/61CAE2AB" Ref="C8001"  Part="1"
 AR Path="/D1BB8DB4/5F317CB5/60365B35/61CAE2AB" Ref="C8201"  Part="1"
-F 0 "C8101" H 5900 3650 50  0000 L CNN
+F 0 "C8301" H 5900 3650 50  0000 L CNN
 F 1 "0.1μF" H 6141 3805 50  0001 L CNN
 F 2 "Capacitor_THT:C_Disc_D7.5mm_W5.0mm_P5.00mm" H 6050 3850 50  0001 C CNN
@@
 AR Path="/D1BB8DB4/5F317CB5/60365B29/602120C6" Ref="C8103"  Part="1"
 AR Path="/D1BB8DB4/5F317CB5/60365B41/602120C6" Ref="C8303"  Part="1"
-F 0 "C8103" H 6950 4800 50  0000 L CNN
+F 0 "C8303" H 6950 4800 50  0000 L CNN
 F 1 "1µF" H 6000 4650 50  0001 L CNN
 F 2 "Capacitor_THT:C_Disc_D7.5mm_W5.0mm_P5.00mm" H 6850 4750 50  0001 C CNN
@@
 AR Path="/D1BB8DB4/5F317CB5/60365B29/6021685A" Ref="C8102"  Part="1"
 AR Path="/D1BB8DB4/5F317CB5/60365B41/6021685A" Ref="C8302"  Part="1"
-F 0 "C8102" H 3300 4300 50  0000 L CNN
+F 0 "C8302" H 3300 4300 50  0000 L CNN
 F 1 "1µF" H 2800 4150 50  0001 L CNN
 F 2 "Capacitor_THT:C_Disc_D7.5mm_W5.0mm_P5.00mm" H 3650 4250 50  0001 C CNN
@@
 AR Path="/D1BB8DB4/5F317CB5/60365B29/604BDC57" Ref="U7902"  Part="3"
 AR Path="/D1BB8DB4/5F317CB5/60365B41/604BDC57" Ref="U7903"  Part="3"
-F 0 "U7902" H 3950 4375 50  0000 C CNN
+F 0 "U7903" H 3950 4375 50  0000 C CNN
 F 1 "74HC86" H 3950 4284 50  0000 C CNN
 F 2 "" H 3950 4050 50  0001 C CNN
@@
 AR Path="/D1BB8DB4/5F317CB5/60365B29/604BF9DE" Ref="U7902"  Part="4"
 AR Path="/D1BB8DB4/5F317CB5/60365B41/604BF9DE" Ref="U7903"  Part="4"
-F 0 "U7902" H 6450 4900 50  0000 C CNN
+F 0 "U7903" H 6450 4900 50  0000 C CNN
 F 1 "74HC86" H 6450 4800 50  0000 C CNN
 F 2 "" H 6550 4550 50  0001 C CNN

Commit message: NewPattern before split
Changed lines of the file:
@@
 $Descr A4 11693 8268
 encoding utf-8
-Sheet 44 97
+Sheet 60 97
 Title "Boat Control Hat"
 Date ""
@@
 AR Path="/D1BB8DB4/5F75E923/604747F3/5FD2B9DE" Ref="IC7301"  Part="1"
 AR Path="/D1BB8DB4/5F75E923/604747FF/5FD2B9DE" Ref="IC7401"  Part="1"
-F 0 "IC8301" H 5450 4215 50  0000 C CNN
+F 0 "IC7201" H 5450 4215 50  0000 C CNN
 F 1 "CD74HCT221E" H 5450 4124 50  0000 C CNN
 F 2 "DIP794W53P254L1930H508Q16N" H 5900 4050 50  0001 L CNN
@@
 AR Path="/D1BB8DB4/5F317CB5/60365B0F/61CAE2AB" Ref="C8001"  Part="1"
 AR Path="/D1BB8DB4/5F317CB5/60365B35/61CAE2AB" Ref="C8201"  Part="1"
-F 0 "C8301" H 5900 3650 50  0000 L CNN
+F 0 "C7201" H 5900 3650 50  0000 L CNN
 F 1 "0.1μF" H 6141 3805 50  0001 L CNN
 F 2 "Capacitor_THT:C_Disc_D7.5mm_W5.0mm_P5.00mm" H 6050 3850 50  0001 C CNN
@@
 AR Path="/D1BB8DB4/5F317CB5/60365B29/602120C6" Ref="C8103"  Part="1"
 AR Path="/D1BB8DB4/5F317CB5/60365B41/602120C6" Ref="C8303"  Part="1"
-F 0 "C8303" H 6950 4800 50  0000 L CNN
+F 0 "C7203" H 6950 4800 50  0000 L CNN
 F 1 "1µF" H 6000 4650 50  0001 L CNN
 F 2 "Capacitor_THT:C_Disc_D7.5mm_W5.0mm_P5.00mm" H 6850 4750 50  0001 C CNN
@@
 AR Path="/D1BB8DB4/5F317CB5/60365B29/6021685A" Ref="C8102"  Part="1"
 AR Path="/D1BB8DB4/5F317CB5/60365B41/6021685A" Ref="C8302"  Part="1"
-F 0 "C8302" H 3300 4300 50  0000 L CNN
+F 0 "C7202" H 3300 4300 50  0000 L CNN
 F 1 "1µF" H 2800 4150 50  0001 L CNN
 F 2 "Capacitor_THT:C_Disc_D7.5mm_W5.0mm_P5.00mm" H 3650 4250 50  0001 C CNN
@@
 AR Path="/D1BB8DB4/5F317CB5/60365B29/604BDC57" Ref="U7902"  Part="3"
 AR Path="/D1BB8DB4/5F317CB5/60365B41/604BDC57" Ref="U7903"  Part="3"
-F 0 "U7903" H 3950 4375 50  0000 C CNN
+F 0 "U7002" H 3950 4375 50  0000 C CNN
 F 1 "74HC86" H 3950 4284 50  0000 C CNN
 F 2 "" H 3950 4050 50  0001 C CNN
@@
 AR Path="/D1BB8DB4/5F317CB5/60365B29/604BF9DE" Ref="U7902"  Part="4"
 AR Path="/D1BB8DB4/5F317CB5/60365B41/604BF9DE" Ref="U7903"  Part="4"
-F 0 "U7903" H 6450 4900 50  0000 C CNN
+F 0 "U7002" H 6450 4900 50  0000 C CNN
 F 1 "74HC86" H 6450 4800 50  0000 C CNN
 F 2 "" H 6550 4550 50  0001 C CNN

Commit message: Let's fix this
Changed lines of the file:
@@
 $Descr A4 11693 8268
 encoding utf-8
-Sheet 60 97
+Sheet 66 97
 Title "Boat Control Hat"
 Date ""
@@
 AR Path="/D1BB8DB4/5F75E923/604747F3/5FD2B9DE" Ref="IC7301"  Part="1"
 AR Path="/D1BB8DB4/5F75E923/604747FF/5FD2B9DE" Ref="IC7401"  Part="1"
-F 0 "IC7201" H 5450 4215 50  0000 C CNN
+F 0 "IC7401" H 5450 4215 50  0000 C CNN
 F 1 "CD74HCT221E" H 5450 4124 50  0000 C CNN
 F 2 "DIP794W53P254L1930H508Q16N" H 5900 4050 50  0001 L CNN
@@
 AR Path="/D1BB8DB4/5F317CB5/60365B0F/61CAE2AB" Ref="C8001"  Part="1"
 AR Path="/D1BB8DB4/5F317CB5/60365B35/61CAE2AB" Ref="C8201"  Part="1"
-F 0 "C7201" H 5900 3650 50  0000 L CNN
+F 0 "C7401" H 5900 3650 50  0000 L CNN
 F 1 "0.1μF" H 6141 3805 50  0001 L CNN
 F 2 "Capacitor_THT:C_Disc_D7.5mm_W5.0mm_P5.00mm" H 6050 3850 50  0001 C CNN
@@
 AR Path="/D1BB8DB4/5F317CB5/60365B29/602120C6" Ref="C8103"  Part="1"
 AR Path="/D1BB8DB4/5F317CB5/60365B41/602120C6" Ref="C8303"  Part="1"
-F 0 "C7203" H 6950 4800 50  0000 L CNN
+F 0 "C7403" H 6950 4800 50  0000 L CNN
 F 1 "1µF" H 6000 4650 50  0001 L CNN
 F 2 "Capacitor_THT:C_Disc_D7.5mm_W5.0mm_P5.00mm" H 6850 4750 50  0001 C CNN
@@
 AR Path="/D1BB8DB4/5F317CB5/60365B29/6021685A" Ref="C8102"  Part="1"
 AR Path="/D1BB8DB4/5F317CB5/60365B41/6021685A" Ref="C8302"  Part="1"
-F 0 "C7202" H 3300 4300 50  0000 L CNN
+F 0 "C7402" H 3300 4300 50  0000 L CNN
 F 1 "1µF" H 2800 4150 50  0001 L CNN
 F 2 "Capacitor_THT:C_Disc_D7.5mm_W5.0mm_P5.00mm" H 3650 4250 50  0001 C CNN
@@
 AR Path="/D1BB8DB4/5F317CB5/60365B29/604BDC57" Ref="U7902"  Part="3"
 AR Path="/D1BB8DB4/5F317CB5/60365B41/604BDC57" Ref="U7903"  Part="3"
-F 0 "U7002" H 3950 4375 50  0000 C CNN
+F 0 "U7003" H 3950 4375 50  0000 C CNN
 F 1 "74HC86" H 3950 4284 50  0000 C CNN
 F 2 "" H 3950 4050 50  0001 C CNN
@@
 AR Path="/D1BB8DB4/5F317CB5/60365B29/604BF9DE" Ref="U7902"  Part="4"
 AR Path="/D1BB8DB4/5F317CB5/60365B41/604BF9DE" Ref="U7903"  Part="4"
-F 0 "U7002" H 6450 4900 50  0000 C CNN
+F 0 "U7003" H 6450 4900 50  0000 C CNN
 F 1 "74HC86" H 6450 4800 50  0000 C CNN
 F 2 "" H 6550 4550 50  0001 C CNN

Commit message: Stepping stone
Changed lines of the file:
@@
 $Descr A4 11693 8268
 encoding utf-8
-Sheet 66 97
+Sheet 51 97
 Title "Boat Control Hat"
 Date ""
@@
 AR Path="/D1BB8DB4/5F75E923/604747F3/5FD2B9DE" Ref="IC7301"  Part="1"
 AR Path="/D1BB8DB4/5F75E923/604747FF/5FD2B9DE" Ref="IC7401"  Part="1"
-F 0 "IC7401" H 5450 4215 50  0000 C CNN
+F 0 "IC6301" H 5450 4215 50  0000 C CNN
 F 1 "CD74HCT221E" H 5450 4124 50  0000 C CNN
 F 2 "DIP794W53P254L1930H508Q16N" H 5900 4050 50  0001 L CNN
@@
 AR Path="/D1BB8DB4/5F317CB5/60365B0F/61CAE2AB" Ref="C8001"  Part="1"
 AR Path="/D1BB8DB4/5F317CB5/60365B35/61CAE2AB" Ref="C8201"  Part="1"
-F 0 "C7401" H 5900 3650 50  0000 L CNN
+F 0 "C6301" H 5900 3650 50  0000 L CNN
 F 1 "0.1μF" H 6141 3805 50  0001 L CNN
 F 2 "Capacitor_THT:C_Disc_D7.5mm_W5.0mm_P5.00mm" H 6050 3850 50  0001 C CNN
@@
 AR Path="/D1BB8DB4/5F317CB5/60365B29/602120C6" Ref="C8103"  Part="1"
 AR Path="/D1BB8DB4/5F317CB5/60365B41/602120C6" Ref="C8303"  Part="1"
-F 0 "C7403" H 6950 4800 50  0000 L CNN
+F 0 "C6303" H 6950 4800 50  0000 L CNN
 F 1 "1µF" H 6000 4650 50  0001 L CNN
 F 2 "Capacitor_THT:C_Disc_D7.5mm_W5.0mm_P5.00mm" H 6850 4750 50  0001 C CNN
@@
 AR Path="/D1BB8DB4/5F317CB5/60365B29/6021685A" Ref="C8102"  Part="1"
 AR Path="/D1BB8DB4/5F317CB5/60365B41/6021685A" Ref="C8302"  Part="1"
-F 0 "C7402" H 3300 4300 50  0000 L CNN
+F 0 "C6302" H 3300 4300 50  0000 L CNN
 F 1 "1µF" H 2800 4150 50  0001 L CNN
 F 2 "Capacitor_THT:C_Disc_D7.5mm_W5.0mm_P5.00mm" H 3650 4250 50  0001 C CNN
@@
 AR Path="/D1BB8DB4/5F317CB5/60365B29/604BDC57" Ref="U7902"  Part="3"
 AR Path="/D1BB8DB4/5F317CB5/60365B41/604BDC57" Ref="U7903"  Part="3"
-F 0 "U7003" H 3950 4375 50  0000 C CNN
+F 0 "U6102" H 3950 4375 50  0000 C CNN
 F 1 "74HC86" H 3950 4284 50  0000 C CNN
 F 2 "" H 3950 4050 50  0001 C CNN
@@
 AR Path="/D1BB8DB4/5F317CB5/60365B29/604BF9DE" Ref="U7902"  Part="4"
 AR Path="/D1BB8DB4/5F317CB5/60365B41/604BF9DE" Ref="U7903"  Part="4"
-F 0 "U7003" H 6450 4900 50  0000 C CNN
+F 0 "U6102" H 6450 4900 50  0000 C CNN
 F 1 "74HC86" H 6450 4800 50  0000 C CNN
 F 2 "" H 6550 4550 50  0001 C CNN

Commit message: Let's do this
Changed lines of the file:
@@
 $Descr A4 11693 8268
 encoding utf-8
-Sheet 51 97
+Sheet 8 97
 Title "Boat Control Hat"
 Date ""
@@
 AR Path="/D1BB8DB4/5F75E923/604747F3/5FD2B9DE" Ref="IC7301"  Part="1"
 AR Path="/D1BB8DB4/5F75E923/604747FF/5FD2B9DE" Ref="IC7401"  Part="1"
-F 0 "IC6301" H 5450 4215 50  0000 C CNN
+F 0 "IC701" H 5450 4215 50  0000 C CNN
 F 1 "CD74HCT221E" H 5450 4124 50  0000 C CNN
 F 2 "DIP794W53P254L1930H508Q16N" H 5900 4050 50  0001 L CNN
@@
 AR Path="/D1BB8DB4/5F75E923/604747F3/60314A0F" Ref="#PWR07302"  Part="1"
 AR Path="/D1BB8DB4/5F75E923/604747FF/60314A0F" Ref="#PWR07402"  Part="1"
-F 0 "#PWR08302" H 4850 4400 50  0001 C CNN
+F 0 "#PWR0702" H 4850 4400 50  0001 C CNN
 F 1 "GND" H 4700 4600 50  0000 C CNN
 F 2 "" H 4850 4650 50  0001 C CNN
@@
 AR Path="/D1BB8DB4/5F75E923/604747F3/5FD9FC74" Ref="#PWR07301"  Part="1"
 AR Path="/D1BB8DB4/5F75E923/604747FF/5FD9FC74" Ref="#PWR07401"  Part="1"
-F 0 "#PWR08301" H 6050 3800 50  0001 C CNN
+F 0 "#PWR0701" H 6050 3800 50  0001 C CNN
 F 1 "+5V" V 6000 4050 50  0000 L CNN
 F 2 "" H 6050 3950 50  0001 C CNN
@@
 AR Path="/D1BB8DB4/5F317CB5/60365B0F/61CAF5C8" Ref="#PWR0183"  Part="1"
 AR Path="/D1BB8DB4/5F317CB5/60365B35/61CAF5C8" Ref="#PWR0185"  Part="1"
-F 0 "#PWR0186" H 6050 3500 50  0001 C CNN
+F 0 "#PWR0158" H 6050 3500 50  0001 C CNN
 F 1 "GND" V 6055 3622 50  0000 R CNN
 F 2 "" H 6050 3750 50  0001 C CNN
@@
 AR Path="/D1BB8DB4/5F317CB5/60365B0F/61CAE2AB" Ref="C8001"  Part="1"
 AR Path="/D1BB8DB4/5F317CB5/60365B35/61CAE2AB" Ref="C8201"  Part="1"
-F 0 "C6301" H 5900 3650 50  0000 L CNN
+F 0 "C701" H 5900 3650 50  0000 L CNN
 F 1 "0.1μF" H 6141 3805 50  0001 L CNN
 F 2 "Capacitor_THT:C_Disc_D7.5mm_W5.0mm_P5.00mm" H 6050 3850 50  0001 C CNN
@@
 AR Path="/D1BB8DB4/5F317CB5/60365B29/602120C6" Ref="C8103"  Part="1"
 AR Path="/D1BB8DB4/5F317CB5/60365B41/602120C6" Ref="C8303"  Part="1"
-F 0 "C6303" H 6950 4800 50  0000 L CNN
+F 0 "C703" H 6950 4800 50  0000 L CNN
 F 1 "1µF" H 6000 4650 50  0001 L CNN
 F 2 "Capacitor_THT:C_Disc_D7.5mm_W5.0mm_P5.00mm" H 6850 4750 50  0001 C CNN
@@
 AR Path="/D1BB8DB4/5F317CB5/60365B29/60314A11" Ref="#PWR0350"  Part="1"
 AR Path="/D1BB8DB4/5F317CB5/60365B41/60314A11" Ref="#PWR0354"  Part="1"
-F 0 "#PWR0354" H 6850 4600 50  0001 C CNN
+F 0 "#PWR0251" H 6850 4600 50  0001 C CNN
 F 1 "GND" H 6855 4677 50  0000 C CNN
 F 2 "" H 6850 4850 50  0001 C CNN
@@
 AR Path="/D1BB8DB4/5F317CB5/60365B29/60216860" Ref="#PWR0351"  Part="1"
 AR Path="/D1BB8DB4/5F317CB5/60365B41/60216860" Ref="#PWR0355"  Part="1"
-F 0 "#PWR0355" H 3650 4100 50  0001 C CNN
+F 0 "#PWR0252" H 3650 4100 50  0001 C CNN
 F 1 "GND" H 3655 4177 50  0000 C CNN
 F 2 "" H 3650 4350 50  0001 C CNN
@@
 AR Path="/D1BB8DB4/5F317CB5/60365B29/6021685A" Ref="C8102"  Part="1"
 AR Path="/D1BB8DB4/5F317CB5/60365B41/6021685A" Ref="C8302"  Part="1"
-F 0 "C6302" H 3300 4300 50  0000 L CNN
+F 0 "C702" H 3300 4300 50  0000 L CNN
 F 1 "1µF" H 2800 4150 50  0001 L CNN
 F 2 "Capacitor_THT:C_Disc_D7.5mm_W5.0mm_P5.00mm" H 3650 4250 50  0001 C CNN
@@
 AR Path="/D1BB8DB4/5F317CB5/60365B29/604BDC57" Ref="U7902"  Part="3"
 AR Path="/D1BB8DB4/5F317CB5/60365B41/604BDC57" Ref="U7903"  Part="3"
-F 0 "U6102" H 3950 4375 50  0000 C CNN
+F 0 "U303" H 3950 4375 50  0000 C CNN
 F 1 "74HC86" H 3950 4284 50  0000 C CNN
 F 2 "" H 3950 4050 50  0001 C CNN
@@
 AR Path="/D1BB8DB4/5F317CB5/60365B29/604BF9DE" Ref="U7902"  Part="4"
 AR Path="/D1BB8DB4/5F317CB5/60365B41/604BF9DE" Ref="U7903"  Part="4"
-F 0 "U6102" H 6450 4900 50  0000 C CNN
+F 0 "U303" H 6450 4900 50  0000 C CNN
 F 1 "74HC86" H 6450 4800 50  0000 C CNN
 F 2 "" H 6550 4550 50  0001 C CNN
