File: boatcontrol/MultiVibratorB.sch (KiCad schematic (older format))
At the start: 5 parts, among them IC401 CD74HCT221E, U302 74HC86

Commit message: Power
Changed lines of the file:
@@
 $Descr A4 11693 8268
 encoding utf-8
-Sheet 66 97
+Sheet 8 97
 Title "Boat Control Hat"
 Date ""
@@
 AR Path="/D1BB8DB4/5F75E923/604747F3/5FD2B9DE" Ref="IC7301"  Part="1"
 AR Path="/D1BB8DB4/5F75E923/604747FF/5FD2B9DE" Ref="IC7401"  Part="1"
-F 0 "IC7401" H 5450 4215 50  0000 C CNN
+F 0 "IC701" H 5450 4215 50  0000 C CNN
 F 1 "CD74HCT221E" H 5450 4124 50  0000 C CNN
 F 2 "DIP794W53P254L1930H508Q16N" H 5900 4050 50  0001 L CNN
@@
 AR Path="/D1BB8DB4/5F317CB5/60365B0F/61CAE2AB" Ref="C8001"  Part="1"
 AR Path="/D1BB8DB4/5F317CB5/60365B35/61CAE2AB" Ref="C8201"  Part="1"
-F 0 "C7401" H 5900 3650 50  0000 L CNN
+F 0 "C701" H 5900 3650 50  0000 L CNN
 F 1 "0.1μF" H 6141 3805 50  0001 L CNN
 F 2 "Capacitor_THT:C_Disc_D7.5mm_W5.0mm_P5.00mm" H 6050 3850 50  0001 C CNN
@@
 AR Path="/D1BB8DB4/5F317CB5/60365B29/602120C6" Ref="C8103"  Part="1"
 AR Path="/D1BB8DB4/5F317CB5/60365B41/602120C6" Ref="C8303"  Part="1"
-F 0 "C7403" H 6950 4800 50  0000 L CNN
+F 0 "C703" H 6950 4800 50  0000 L CNN
 F 1 "1µF" H 6000 4650 50  0001 L CNN
 F 2 "Capacitor_THT:C_Disc_D7.5mm_W5.0mm_P5.00mm" H 6850 4750 50  0001 C CNN
@@
 AR Path="/D1BB8DB4/5F317CB5/60365B29/6021685A" Ref="C8102"  Part="1"
 AR Path="/D1BB8DB4/5F317CB5/60365B41/6021685A" Ref="C8302"  Part="1"
-F 0 "C7402" H 3300 4300 50  0000 L CNN
+F 0 "C702" H 3300 4300 50  0000 L CNN
 F 1 "1µF" H 2800 4150 50  0001 L CNN
 F 2 "Capacitor_THT:C_Disc_D7.5mm_W5.0mm_P5.00mm" H 3650 4250 50  0001 C CNN
@@
 AR Path="/D1BB8DB4/5F317CB5/60365B29/604BDC57" Ref="U7902"  Part="3"
 AR Path="/D1BB8DB4/5F317CB5/60365B41/604BDC57" Ref="U7903"  Part="3"
-F 0 "U7003" H 3950 4375 50  0000 C CNN
+F 0 "U303" H 3950 4375 50  0000 C CNN
 F 1 "74HC86" H 3950 4284 50  0000 C CNN
 F 2 "" H 3950 4050 50  0001 C CNN
@@
 AR Path="/D1BB8DB4/5F317CB5/60365B29/604BF9DE" Ref="U7902"  Part="4"
 AR Path="/D1BB8DB4/5F317CB5/60365B41/604BF9DE" Ref="U7903"  Part="4"
-F 0 "U7003" H 6450 4900 50  0000 C CNN
+F 0 "U303" H 6450 4900 50  0000 C CNN
 F 1 "74HC86" H 6450 4800 50  0000 C CNN
 F 2 "" H 6550 4550 50  0001 C CNN

Commit message: Start over
Changed lines of the file:
@@
 $Descr A4 11693 8268
 encoding utf-8
-Sheet 8 97
+Sheet 71 97
 Title "Boat Control Hat"
 Date ""
@@
 AR Path="/D1BB8DB4/5F75E923/604747F3/5FD2B9DE" Ref="IC7301"  Part="1"
 AR Path="/D1BB8DB4/5F75E923/604747FF/5FD2B9DE" Ref="IC7401"  Part="1"
-F 0 "IC701" H 5450 4215 50  0000 C CNN
+F 0 "IC8301" H 5450 4215 50  0000 C CNN
 F 1 "CD74HCT221E" H 5450 4124 50  0000 C CNN
 F 2 "DIP794W53P254L1930H508Q16N" H 5900 4050 50  0001 L CNN
@@
 	1    0    0    -1
 $EndComp
-Text HLabel 3650 4150 0    50   Input ~ 0
-AN_ON
 $Comp
 L power:GND #PWR?
@@
 Text HLabel 6050 4250 2    50   Output ~ 0
 MUX_ON
-Text HLabel 6900 4650 2    50   Input ~ 0
+Text HLabel 6850 4650 2    50   Input ~ 0
 AN_OFF
 Text HLabel 6850 4450 2    50   Input ~ 0
@@
 AR Path="/D1BB8DB4/5F317CB5/60365B0F/61CAE2AB" Ref="C8001"  Part="1"
 AR Path="/D1BB8DB4/5F317CB5/60365B35/61CAE2AB" Ref="C8201"  Part="1"
-F 0 "C701" H 5900 3650 50  0000 L CNN
+F 0 "C8301" H 5900 3650 50  0000 L CNN
 F 1 "0.1μF" H 6141 3805 50  0001 L CNN
 F 2 "Capacitor_THT:C_Disc_D7.5mm_W5.0mm_P5.00mm" H 6050 3850 50  0001 C CNN
@@
 AR Path="/D1BB8DB4/5F317CB5/60365B29/602120C6" Ref="C8103"  Part="1"
 AR Path="/D1BB8DB4/5F317CB5/60365B41/602120C6" Ref="C8303"  Part="1"
-F 0 "C703" H 6950 4800 50  0000 L CNN
+F 0 "C8303" H 6950 4800 50  0000 L CNN
 F 1 "1µF" H 6000 4650 50  0001 L CNN
 F 2 "Capacitor_THT:C_Disc_D7.5mm_W5.0mm_P5.00mm" H 6850 4750 50  0001 C CNN
@@
 AR Path="/D1BB8DB4/5F317CB5/60365B29/6021685A" Ref="C8102"  Part="1"
 AR Path="/D1BB8DB4/5F317CB5/60365B41/6021685A" Ref="C8302"  Part="1"
-F 0 "C702" H 3300 4300 50  0000 L CNN
+F 0 "C8302" H 3300 4300 50  0000 L CNN
 F 1 "1µF" H 2800 4150 50  0001 L CNN
 F 2 "Capacitor_THT:C_Disc_D7.5mm_W5.0mm_P5.00mm" H 3650 4250 50  0001 C CNN
@@
 Wire Wire Line
 	6050 4550 6250 4550
-Wire Wire Line
-	6900 4650 6850 4650
 Wire Wire Line
 	6250 4650 6250 4850
@@
 AR Path="/D1BB8DB4/5F317CB5/60365B29/604BDC57" Ref="U7902"  Part="3"
 AR Path="/D1BB8DB4/5F317CB5/60365B41/604BDC57" Ref="U7903"  Part="3"
-F 0 "U303" H 3950 4375 50  0000 C CNN
+F 0 "U7903" H 3950 4375 50  0000 C CNN
 F 1 "74HC86" H 3950 4284 50  0000 C CNN
 F 2 "" H 3950 4050 50  0001 C CNN
@@
 	1    0    0    -1
 $EndComp
-Connection ~ 6850 4650
 Text Notes 5750 5050 0    50   ~ 0
 OFF side
@@
 AR Path="/D1BB8DB4/5F317CB5/60365B29/604BF9DE" Ref="U7902"  Part="4"
 AR Path="/D1BB8DB4/5F317CB5/60365B41/604BF9DE" Ref="U7903"  Part="4"
-F 0 "U303" H 6450 4900 50  0000 C CNN
+F 0 "U7903" H 6450 4900 50  0000 C CNN
 F 1 "74HC86" H 6450 4800 50  0000 C CNN
 F 2 "" H 6550 4550 50  0001 C CNN
@@
 	-1   0    0    -1
 $EndComp
+Text HLabel 3650 4150 0    50   Input ~ 0
+AN_ON
 $EndSCHEMATC

Commit message: Going
Changed lines of the file:
@@
 $Descr A4 11693 8268
 encoding utf-8
-Sheet 71 97
+Sheet 8 97
 Title "Boat Control Hat"
 Date ""
@@
 AR Path="/D1BB8DB4/5F75E923/604747F3/5FD2B9DE" Ref="IC7301"  Part="1"
 AR Path="/D1BB8DB4/5F75E923/604747FF/5FD2B9DE" Ref="IC7401"  Part="1"
-F 0 "IC8301" H 5450 4215 50  0000 C CNN
+F 0 "IC701" H 5450 4215 50  0000 C CNN
 F 1 "CD74HCT221E" H 5450 4124 50  0000 C CNN
 F 2 "DIP794W53P254L1930H508Q16N" H 5900 4050 50  0001 L CNN
@@
 AR Path="/D1BB8DB4/5F317CB5/60365B0F/61CAE2AB" Ref="C8001"  Part="1"
 AR Path="/D1BB8DB4/5F317CB5/60365B35/61CAE2AB" Ref="C8201"  Part="1"
-F 0 "C8301" H 5900 3650 50  0000 L CNN
+F 0 "C701" H 5900 3650 50  0000 L CNN
 F 1 "0.1μF" H 6141 3805 50  0001 L CNN
 F 2 "Capacitor_THT:C_Disc_D7.5mm_W5.0mm_P5.00mm" H 6050 3850 50  0001 C CNN
@@
 AR Path="/D1BB8DB4/5F317CB5/60365B29/602120C6" Ref="C8103"  Part="1"
 AR Path="/D1BB8DB4/5F317CB5/60365B41/602120C6" Ref="C8303"  Part="1"
-F 0 "C8303" H 6950 4800 50  0000 L CNN
+F 0 "C703" H 6950 4800 50  0000 L CNN
 F 1 "1µF" H 6000 4650 50  0001 L CNN
 F 2 "Capacitor_THT:C_Disc_D7.5mm_W5.0mm_P5.00mm" H 6850 4750 50  0001 C CNN
@@
 AR Path="/D1BB8DB4/5F317CB5/60365B29/6021685A" Ref="C8102"  Part="1"
 AR Path="/D1BB8DB4/5F317CB5/60365B41/6021685A" Ref="C8302"  Part="1"
-F 0 "C8302" H 3300 4300 50  0000 L CNN
+F 0 "C702" H 3300 4300 50  0000 L CNN
 F 1 "1µF" H 2800 4150 50  0001 L CNN
 F 2 "Capacitor_THT:C_Disc_D7.5mm_W5.0mm_P5.00mm" H 3650 4250 50  0001 C CNN
@@
 AR Path="/D1BB8DB4/5F317CB5/60365B29/604BDC57" Ref="U7902"  Part="3"
 AR Path="/D1BB8DB4/5F317CB5/60365B41/604BDC57" Ref="U7903"  Part="3"
-F 0 "U7903" H 3950 4375 50  0000 C CNN
+F 0 "U303" H 3950 4375 50  0000 C CNN
 F 1 "74HC86" H 3950 4284 50  0000 C CNN
 F 2 "" H 3950 4050 50  0001 C CNN
@@
 AR Path="/D1BB8DB4/5F317CB5/60365B29/604BF9DE" Ref="U7902"  Part="4"
 AR Path="/D1BB8DB4/5F317CB5/60365B41/604BF9DE" Ref="U7903"  Part="4"
-F 0 "U7903" H 6450 4900 50  0000 C CNN
+F 0 "U303" H 6450 4900 50  0000 C CNN
 F 1 "74HC86" H 6450 4800 50  0000 C CNN
 F 2 "" H 6550 4550 50  0001 C CNN
