File: boatcontrol/MultiVibratorA.sch (KiCad schematic (older format))
At the start: 5 parts, among them IC401 CD74HCT221E, U2103 74HC86

Commit message: Stepping stone
Changed lines of the file:
@@
 $Descr A4 11693 8268
 encoding utf-8
-Sheet 41 97
+Sheet 68 97
 Title "Boat Control Hat"
 Date ""
@@
 AR Path="/D1BB8DB4/5F75E923/604747F3/603A29DF" Ref="IC7301"  Part="1"
 AR Path="/D1BB8DB4/5F75E923/604747FF/603A29DF" Ref="IC7401"  Part="1"
-F 0 "IC5301" H 5450 4215 50  0000 C CNN
+F 0 "IC8001" H 5450 4215 50  0000 C CNN
 F 1 "CD74HCT221E" H 5450 4124 50  0000 C CNN
 F 2 "DIP794W53P254L1930H508Q16N" H 5900 4050 50  0001 L CNN
@@
 AR Path="/D1BB8DB4/5F317CB5/60365B0F/603A29E8" Ref="C8001"  Part="1"
 AR Path="/D1BB8DB4/5F317CB5/60365B35/603A29E8" Ref="C8201"  Part="1"
-F 0 "C5301" H 5900 3650 50  0000 L CNN
+F 0 "C8001" H 5900 3650 50  0000 L CNN
 F 1 "0.1μF" H 6141 3805 50  0001 L CNN
 F 2 "Capacitor_THT:C_Disc_D7.5mm_W5.0mm_P5.00mm" H 6050 3850 50  0001 C CNN
@@
 AR Path="/D1BB8DB4/5F75E923/604747F3/60314A10" Ref="C7303"  Part="1"
 AR Path="/D1BB8DB4/5F317CB5/60365B35/60314A10" Ref="C8203"  Part="1"
-F 0 "C5303" H 6950 4800 50  0000 L CNN
+F 0 "C8003" H 6950 4800 50  0000 L CNN
 F 1 "1µF" H 6000 4650 50  0001 L CNN
 F 2 "Capacitor_THT:C_Disc_D7.5mm_W5.0mm_P5.00mm" H 6850 4750 50  0001 C CNN
@@
 AR Path="/D1BB8DB4/5F75E923/604747F3/60416EE6" Ref="U7003"  Part="1"
 AR Path="/D1BB8DB4/5F317CB5/60365B35/60416EE6" Ref="U7903"  Part="1"
-F 0 "U4002" H 3950 4350 50  0000 C CNN
+F 0 "U7902" H 3950 4350 50  0000 C CNN
 F 1 "74HC86" H 3950 4250 50  0000 C CNN
 F 2 "" H 3950 4050 50  0001 C CNN
@@
 AR Path="/D1BB8DB4/5F75E923/604747F3/60314A12" Ref="C7302"  Part="1"
 AR Path="/D1BB8DB4/5F317CB5/60365B35/60314A12" Ref="C8202"  Part="1"
-F 0 "C5302" H 3300 4300 50  0000 L CNN
+F 0 "C8002" H 3300 4300 50  0000 L CNN
 F 1 "1µF" H 2800 4150 50  0001 L CNN
 F 2 "Capacitor_THT:C_Disc_D7.5mm_W5.0mm_P5.00mm" H 3650 4250 50  0001 C CNN
@@
 AR Path="/D1BB8DB4/5F75E923/604747F3/60491845" Ref="U7003"  Part="2"
 AR Path="/D1BB8DB4/5F317CB5/60365B35/60491845" Ref="U7903"  Part="2"
-F 0 "U4002" H 6500 4750 50  0000 C CNN
+F 0 "U7902" H 6500 4750 50  0000 C CNN
 F 1 "74HC86" H 6500 4850 50  0000 C CNN
 F 2 "" H 6550 4550 50  0001 C CNN

Commit message: Let's do this
Changed lines of the file:
@@
 $Descr A4 11693 8268
 encoding utf-8
-Sheet 68 97
+Sheet 9 97
 Title "Boat Control Hat"
 Date ""
@@
 AR Path="/D1BB8DB4/5F75E923/604747F3/603A29DF" Ref="IC7301"  Part="1"
 AR Path="/D1BB8DB4/5F75E923/604747FF/603A29DF" Ref="IC7401"  Part="1"
-F 0 "IC8001" H 5450 4215 50  0000 C CNN
+F 0 "IC601" H 5450 4215 50  0000 C CNN
 F 1 "CD74HCT221E" H 5450 4124 50  0000 C CNN
 F 2 "DIP794W53P254L1930H508Q16N" H 5900 4050 50  0001 L CNN
@@
 AR Path="/D1BB8DB4/5F75E923/604747F3/5FDA22CD" Ref="#PWR07302"  Part="1"
 AR Path="/D1BB8DB4/5F75E923/604747FF/5FDA22CD" Ref="#PWR07402"  Part="1"
-F 0 "#PWR08202" H 4850 4400 50  0001 C CNN
+F 0 "#PWR0602" H 4850 4400 50  0001 C CNN
 F 1 "GND" H 4700 4600 50  0000 C CNN
 F 2 "" H 4850 4650 50  0001 C CNN
@@
 AR Path="/D1BB8DB4/5F75E923/604747F3/603A29E0" Ref="#PWR07301"  Part="1"
 AR Path="/D1BB8DB4/5F75E923/604747FF/603A29E0" Ref="#PWR07401"  Part="1"
-F 0 "#PWR08201" H 6050 3800 50  0001 C CNN
+F 0 "#PWR0601" H 6050 3800 50  0001 C CNN
 F 1 "+5V" V 6000 4050 50  0000 L CNN
 F 2 "" H 6050 3950 50  0001 C CNN
@@
 AR Path="/D1BB8DB4/5F317CB5/60365B0F/603A29E9" Ref="#PWR0183"  Part="1"
 AR Path="/D1BB8DB4/5F317CB5/60365B35/603A29E9" Ref="#PWR0185"  Part="1"
-F 0 "#PWR0185" H 6050 3500 50  0001 C CNN
+F 0 "#PWR0157" H 6050 3500 50  0001 C CNN
 F 1 "GND" V 6055 3622 50  0000 R CNN
 F 2 "" H 6050 3750 50  0001 C CNN
@@
 AR Path="/D1BB8DB4/5F317CB5/60365B0F/603A29E8" Ref="C8001"  Part="1"
 AR Path="/D1BB8DB4/5F317CB5/60365B35/603A29E8" Ref="C8201"  Part="1"
-F 0 "C8001" H 5900 3650 50  0000 L CNN
+F 0 "C601" H 5900 3650 50  0000 L CNN
 F 1 "0.1μF" H 6141 3805 50  0001 L CNN
 F 2 "Capacitor_THT:C_Disc_D7.5mm_W5.0mm_P5.00mm" H 6050 3850 50  0001 C CNN
@@
 AR Path="/D1BB8DB4/5F75E923/604747F3/60314A10" Ref="C7303"  Part="1"
 AR Path="/D1BB8DB4/5F317CB5/60365B35/60314A10" Ref="C8203"  Part="1"
-F 0 "C8003" H 6950 4800 50  0000 L CNN
+F 0 "C603" H 6950 4800 50  0000 L CNN
 F 1 "1µF" H 6000 4650 50  0001 L CNN
 F 2 "Capacitor_THT:C_Disc_D7.5mm_W5.0mm_P5.00mm" H 6850 4750 50  0001 C CNN
@@
 AR Path="/D1BB8DB4/5F75E923/604747F3/602124D8" Ref="#PWR0337"  Part="1"
 AR Path="/D1BB8DB4/5F317CB5/60365B35/602124D8" Ref="#PWR0352"  Part="1"
-F 0 "#PWR0352" H 6850 4600 50  0001 C CNN
+F 0 "#PWR0253" H 6850 4600 50  0001 C CNN
 F 1 "GND" H 6855 4677 50  0000 C CNN
 F 2 "" H 6850 4850 50  0001 C CNN
@@
 AR Path="/D1BB8DB4/5F75E923/604747F3/60416EE6" Ref="U7003"  Part="1"
 AR Path="/D1BB8DB4/5F317CB5/60365B35/60416EE6" Ref="U7903"  Part="1"
-F 0 "U7902" H 3950 4350 50  0000 C CNN
+F 0 "U303" H 3950 4350 50  0000 C CNN
 F 1 "74HC86" H 3950 4250 50  0000 C CNN
 F 2 "" H 3950 4050 50  0001 C CNN
@@
 AR Path="/D1BB8DB4/5F75E923/604747F3/603A29E5" Ref="#PWR0338"  Part="1"
 AR Path="/D1BB8DB4/5F317CB5/60365B35/603A29E5" Ref="#PWR0353"  Part="1"
-F 0 "#PWR0353" H 3650 4100 50  0001 C CNN
+F 0 "#PWR0254" H 3650 4100 50  0001 C CNN
 F 1 "GND" H 3655 4177 50  0000 C CNN
 F 2 "" H 3650 4350 50  0001 C CNN
@@
 AR Path="/D1BB8DB4/5F75E923/604747F3/60314A12" Ref="C7302"  Part="1"
 AR Path="/D1BB8DB4/5F317CB5/60365B35/60314A12" Ref="C8202"  Part="1"
-F 0 "C8002" H 3300 4300 50  0000 L CNN
+F 0 "C602" H 3300 4300 50  0000 L CNN
 F 1 "1µF" H 2800 4150 50  0001 L CNN
 F 2 "Capacitor_THT:C_Disc_D7.5mm_W5.0mm_P5.00mm" H 3650 4250 50  0001 C CNN
@@
 AR Path="/D1BB8DB4/5F75E923/604747F3/60491845" Ref="U7003"  Part="2"
 AR Path="/D1BB8DB4/5F317CB5/60365B35/60491845" Ref="U7903"  Part="2"
-F 0 "U7902" H 6500 4750 50  0000 C CNN
+F 0 "U303" H 6500 4750 50  0000 C CNN
 F 1 "74HC86" H 6500 4850 50  0000 C CNN
 F 2 "" H 6550 4550 50  0001 C CNN

Commit message: Probably OK
Changed lines of the file:
@@
 $Descr A4 11693 8268
 encoding utf-8
-Sheet 9 97
+Sheet 18 97
 Title "Boat Control Hat"
 Date ""
@@
 AR Path="/D1BB8DB4/5F75E923/604747F3/603A29DF" Ref="IC7301"  Part="1"
 AR Path="/D1BB8DB4/5F75E923/604747FF/603A29DF" Ref="IC7401"  Part="1"
-F 0 "IC601" H 5450 4215 50  0000 C CNN
+F 0 "IC1501" H 5450 4215 50  0000 C CNN
 F 1 "CD74HCT221E" H 5450 4124 50  0000 C CNN
 F 2 "DIP794W53P254L1930H508Q16N" H 5900 4050 50  0001 L CNN
@@
 AR Path="/D1BB8DB4/5F317CB5/60365B0F/603A29E8" Ref="C8001"  Part="1"
 AR Path="/D1BB8DB4/5F317CB5/60365B35/603A29E8" Ref="C8201"  Part="1"
-F 0 "C601" H 5900 3650 50  0000 L CNN
+F 0 "C1501" H 5900 3650 50  0000 L CNN
 F 1 "0.1μF" H 6141 3805 50  0001 L CNN
 F 2 "Capacitor_THT:C_Disc_D7.5mm_W5.0mm_P5.00mm" H 6050 3850 50  0001 C CNN
@@
 AR Path="/D1BB8DB4/5F75E923/604747F3/60314A10" Ref="C7303"  Part="1"
 AR Path="/D1BB8DB4/5F317CB5/60365B35/60314A10" Ref="C8203"  Part="1"
-F 0 "C603" H 6950 4800 50  0000 L CNN
+F 0 "C1503" H 6950 4800 50  0000 L CNN
 F 1 "1µF" H 6000 4650 50  0001 L CNN
 F 2 "Capacitor_THT:C_Disc_D7.5mm_W5.0mm_P5.00mm" H 6850 4750 50  0001 C CNN
@@
 AR Path="/D1BB8DB4/5F75E923/604747F3/60416EE6" Ref="U7003"  Part="1"
 AR Path="/D1BB8DB4/5F317CB5/60365B35/60416EE6" Ref="U7903"  Part="1"
-F 0 "U303" H 3950 4350 50  0000 C CNN
+F 0 "U1203" H 3950 4350 50  0000 C CNN
 F 1 "74HC86" H 3950 4250 50  0000 C CNN
 F 2 "" H 3950 4050 50  0001 C CNN
@@
 AR Path="/D1BB8DB4/5F75E923/604747F3/60314A12" Ref="C7302"  Part="1"
 AR Path="/D1BB8DB4/5F317CB5/60365B35/60314A12" Ref="C8202"  Part="1"
-F 0 "C602" H 3300 4300 50  0000 L CNN
+F 0 "C1502" H 3300 4300 50  0000 L CNN
 F 1 "1µF" H 2800 4150 50  0001 L CNN
 F 2 "Capacitor_THT:C_Disc_D7.5mm_W5.0mm_P5.00mm" H 3650 4250 50  0001 C CNN
@@
 AR Path="/D1BB8DB4/5F75E923/604747F3/60491845" Ref="U7003"  Part="2"
 AR Path="/D1BB8DB4/5F317CB5/60365B35/60491845" Ref="U7903"  Part="2"
-F 0 "U303" H 6500 4750 50  0000 C CNN
+F 0 "U1203" H 6500 4750 50  0000 C CNN
 F 1 "74HC86" H 6500 4850 50  0000 C CNN
 F 2 "" H 6550 4550 50  0001 C CNN

Commit message: Start over
Changed lines of the file:
@@
 Text HLabel 6050 4250 2    50   Output ~ 0
 MUX_ON
-Text HLabel 6900 4650 2    50   Input ~ 0
+Text HLabel 6850 4650 2    50   Input ~ 0
 AN_OFF
 Text HLabel 6850 4450 2    50   Input ~ 0
@@
 	6050 4550 6250 4550
 Wire Wire Line
-	6900 4650 6850 4650
-Connection ~ 6850 4650
-Wire Wire Line
 	6250 4650 6250 4850

Commit message: Going
Changed lines of the file:
@@
 $Descr A4 11693 8268
 encoding utf-8
-Sheet 18 97
+Sheet 37 97
 Title "Boat Control Hat"
 Date ""
@@
 AR Path="/D1BB8DB4/5F75E923/604747F3/603A29DF" Ref="IC7301"  Part="1"
 AR Path="/D1BB8DB4/5F75E923/604747FF/603A29DF" Ref="IC7401"  Part="1"
-F 0 "IC1501" H 5450 4215 50  0000 C CNN
+F 0 "IC401" H 5450 4215 50  0000 C CNN
 F 1 "CD74HCT221E" H 5450 4124 50  0000 C CNN
 F 2 "DIP794W53P254L1930H508Q16N" H 5900 4050 50  0001 L CNN
@@
 AR Path="/D1BB8DB4/5F317CB5/60365B0F/603A29E8" Ref="C8001"  Part="1"
 AR Path="/D1BB8DB4/5F317CB5/60365B35/603A29E8" Ref="C8201"  Part="1"
-F 0 "C1501" H 5900 3650 50  0000 L CNN
+F 0 "C401" H 5900 3650 50  0000 L CNN
 F 1 "0.1μF" H 6141 3805 50  0001 L CNN
 F 2 "Capacitor_THT:C_Disc_D7.5mm_W5.0mm_P5.00mm" H 6050 3850 50  0001 C CNN
@@
 AR Path="/D1BB8DB4/5F75E923/604747F3/60314A10" Ref="C7303"  Part="1"
 AR Path="/D1BB8DB4/5F317CB5/60365B35/60314A10" Ref="C8203"  Part="1"
-F 0 "C1503" H 6950 4800 50  0000 L CNN
+F 0 "C403" H 6950 4800 50  0000 L CNN
 F 1 "1µF" H 6000 4650 50  0001 L CNN
 F 2 "Capacitor_THT:C_Disc_D7.5mm_W5.0mm_P5.00mm" H 6850 4750 50  0001 C CNN
@@
 AR Path="/D1BB8DB4/5F75E923/604747F3/60416EE6" Ref="U7003"  Part="1"
 AR Path="/D1BB8DB4/5F317CB5/60365B35/60416EE6" Ref="U7903"  Part="1"
-F 0 "U1203" H 3950 4350 50  0000 C CNN
+F 0 "U302" H 3950 4350 50  0000 C CNN
 F 1 "74HC86" H 3950 4250 50  0000 C CNN
 F 2 "" H 3950 4050 50  0001 C CNN
@@
 AR Path="/D1BB8DB4/5F75E923/604747F3/60314A12" Ref="C7302"  Part="1"
 AR Path="/D1BB8DB4/5F317CB5/60365B35/60314A12" Ref="C8202"  Part="1"
-F 0 "C1502" H 3300 4300 50  0000 L CNN
+F 0 "C402" H 3300 4300 50  0000 L CNN
 F 1 "1µF" H 2800 4150 50  0001 L CNN
 F 2 "Capacitor_THT:C_Disc_D7.5mm_W5.0mm_P5.00mm" H 3650 4250 50  0001 C CNN
@@
 AR Path="/D1BB8DB4/5F75E923/604747F3/60491845" Ref="U7003"  Part="2"
 AR Path="/D1BB8DB4/5F317CB5/60365B35/60491845" Ref="U7903"  Part="2"
-F 0 "U1203" H 6500 4750 50  0000 C CNN
+F 0 "U302" H 6500 4750 50  0000 C CNN
 F 1 "74HC86" H 6500 4850 50  0000 C CNN
 F 2 "" H 6550 4550 50  0001 C CNN

Commit message: Wired
Changed lines of the file:
@@
 $Descr A4 11693 8268
 encoding utf-8
-Sheet 37 97
+Sheet 41 97
 Title "Boat Control Hat"
 Date ""
@@
 AR Path="/D1BB8DB4/5F75E923/604747F3/603A29DF" Ref="IC7301"  Part="1"
 AR Path="/D1BB8DB4/5F75E923/604747FF/603A29DF" Ref="IC7401"  Part="1"
-F 0 "IC401" H 5450 4215 50  0000 C CNN
+F 0 "IC5301" H 5450 4215 50  0000 C CNN
 F 1 "CD74HCT221E" H 5450 4124 50  0000 C CNN
 F 2 "DIP794W53P254L1930H508Q16N" H 5900 4050 50  0001 L CNN
@@
 AR Path="/D1BB8DB4/5F317CB5/60365B0F/603A29E8" Ref="C8001"  Part="1"
 AR Path="/D1BB8DB4/5F317CB5/60365B35/603A29E8" Ref="C8201"  Part="1"
-F 0 "C401" H 5900 3650 50  0000 L CNN
+F 0 "C5301" H 5900 3650 50  0000 L CNN
 F 1 "0.1μF" H 6141 3805 50  0001 L CNN
 F 2 "Capacitor_THT:C_Disc_D7.5mm_W5.0mm_P5.00mm" H 6050 3850 50  0001 C CNN
@@
 AR Path="/D1BB8DB4/5F75E923/604747F3/60314A10" Ref="C7303"  Part="1"
 AR Path="/D1BB8DB4/5F317CB5/60365B35/60314A10" Ref="C8203"  Part="1"
-F 0 "C403" H 6950 4800 50  0000 L CNN
+F 0 "C5303" H 6950 4800 50  0000 L CNN
 F 1 "1µF" H 6000 4650 50  0001 L CNN
 F 2 "Capacitor_THT:C_Disc_D7.5mm_W5.0mm_P5.00mm" H 6850 4750 50  0001 C CNN
@@
 AR Path="/D1BB8DB4/5F75E923/604747F3/60416EE6" Ref="U7003"  Part="1"
 AR Path="/D1BB8DB4/5F317CB5/60365B35/60416EE6" Ref="U7903"  Part="1"
-F 0 "U302" H 3950 4350 50  0000 C CNN
+F 0 "U4002" H 3950 4350 50  0000 C CNN
 F 1 "74HC86" H 3950 4250 50  0000 C CNN
 F 2 "" H 3950 4050 50  0001 C CNN
@@
 AR Path="/D1BB8DB4/5F75E923/604747F3/60314A12" Ref="C7302"  Part="1"
 AR Path="/D1BB8DB4/5F317CB5/60365B35/60314A12" Ref="C8202"  Part="1"
-F 0 "C402" H 3300 4300 50  0000 L CNN
+F 0 "C5302" H 3300 4300 50  0000 L CNN
 F 1 "1µF" H 2800 4150 50  0001 L CNN
 F 2 "Capacitor_THT:C_Disc_D7.5mm_W5.0mm_P5.00mm" H 3650 4250 50  0001 C CNN
@@
 AR Path="/D1BB8DB4/5F75E923/604747F3/60491845" Ref="U7003"  Part="2"
 AR Path="/D1BB8DB4/5F317CB5/60365B35/60491845" Ref="U7903"  Part="2"
-F 0 "U302" H 6500 4750 50  0000 C CNN
+F 0 "U4002" H 6500 4750 50  0000 C CNN
 F 1 "74HC86" H 6500 4850 50  0000 C CNN
 F 2 "" H 6550 4550 50  0001 C CNN

Commit message: Deleting second heatsink
Changed lines of the file:
@@
 $Descr A4 11693 8268
 encoding utf-8
-Sheet 41 97
+Sheet 18 97
 Title "Boat Control Hat"
 Date ""
@@
 AR Path="/D1BB8DB4/5F75E923/604747F3/603A29DF" Ref="IC7301"  Part="1"
 AR Path="/D1BB8DB4/5F75E923/604747FF/603A29DF" Ref="IC7401"  Part="1"
-F 0 "IC5301" H 5450 4215 50  0000 C CNN
+F 0 "IC2401" H 5450 4215 50  0000 C CNN
 F 1 "CD74HCT221E" H 5450 4124 50  0000 C CNN
 F 2 "DIP794W53P254L1930H508Q16N" H 5900 4050 50  0001 L CNN
@@
 AR Path="/D1BB8DB4/5F75E923/604747F3/5FDA22CD" Ref="#PWR07302"  Part="1"
 AR Path="/D1BB8DB4/5F75E923/604747FF/5FDA22CD" Ref="#PWR07402"  Part="1"
-F 0 "#PWR08202" H 4850 4400 50  0001 C CNN
+F 0 "#PWR02402" H 4850 4400 50  0001 C CNN
 F 1 "GND" H 4700 4600 50  0000 C CNN
 F 2 "" H 4850 4650 50  0001 C CNN
@@
 AR Path="/D1BB8DB4/5F75E923/604747F3/603A29E0" Ref="#PWR07301"  Part="1"
 AR Path="/D1BB8DB4/5F75E923/604747FF/603A29E0" Ref="#PWR07401"  Part="1"
-F 0 "#PWR08201" H 6050 3800 50  0001 C CNN
+F 0 "#PWR02401" H 6050 3800 50  0001 C CNN
 F 1 "+5V" V 6000 4050 50  0000 L CNN
 F 2 "" H 6050 3950 50  0001 C CNN
@@
 AR Path="/D1BB8DB4/5F317CB5/60365B0F/603A29E9" Ref="#PWR0183"  Part="1"
 AR Path="/D1BB8DB4/5F317CB5/60365B35/603A29E9" Ref="#PWR0185"  Part="1"
-F 0 "#PWR0185" H 6050 3500 50  0001 C CNN
+F 0 "#PWR0165" H 6050 3500 50  0001 C CNN
 F 1 "GND" V 6055 3622 50  0000 R CNN
 F 2 "" H 6050 3750 50  0001 C CNN
@@
 AR Path="/D1BB8DB4/5F317CB5/60365B0F/603A29E8" Ref="C8001"  Part="1"
 AR Path="/D1BB8DB4/5F317CB5/60365B35/603A29E8" Ref="C8201"  Part="1"
-F 0 "C5301" H 5900 3650 50  0000 L CNN
+F 0 "C2401" H 5900 3650 50  0000 L CNN
 F 1 "0.1μF" H 6141 3805 50  0001 L CNN
 F 2 "Capacitor_THT:C_Disc_D7.5mm_W5.0mm_P5.00mm" H 6050 3850 50  0001 C CNN
@@
 AR Path="/D1BB8DB4/5F75E923/604747F3/60314A10" Ref="C7303"  Part="1"
 AR Path="/D1BB8DB4/5F317CB5/60365B35/60314A10" Ref="C8203"  Part="1"
-F 0 "C5303" H 6950 4800 50  0000 L CNN
+F 0 "C2403" H 6950 4800 50  0000 L CNN
 F 1 "1µF" H 6000 4650 50  0001 L CNN
 F 2 "Capacitor_THT:C_Disc_D7.5mm_W5.0mm_P5.00mm" H 6850 4750 50  0001 C CNN
@@
 AR Path="/D1BB8DB4/5F75E923/604747F3/602124D8" Ref="#PWR0337"  Part="1"
 AR Path="/D1BB8DB4/5F317CB5/60365B35/602124D8" Ref="#PWR0352"  Part="1"
-F 0 "#PWR0352" H 6850 4600 50  0001 C CNN
+F 0 "#PWR0281" H 6850 4600 50  0001 C CNN
 F 1 "GND" H 6855 4677 50  0000 C CNN
 F 2 "" H 6850 4850 50  0001 C CNN
@@
 AR Path="/D1BB8DB4/5F75E923/604747F3/60416EE6" Ref="U7003"  Part="1"
 AR Path="/D1BB8DB4/5F317CB5/60365B35/60416EE6" Ref="U7903"  Part="1"
-F 0 "U4002" H 3950 4350 50  0000 C CNN
+F 0 "U2103" H 3950 4350 50  0000 C CNN
 F 1 "74HC86" H 3950 4250 50  0000 C CNN
 F 2 "" H 3950 4050 50  0001 C CNN
@@
 AR Path="/D1BB8DB4/5F75E923/604747F3/603A29E5" Ref="#PWR0338"  Part="1"
 AR Path="/D1BB8DB4/5F317CB5/60365B35/603A29E5" Ref="#PWR0353"  Part="1"
-F 0 "#PWR0353" H 3650 4100 50  0001 C CNN
+F 0 "#PWR0282" H 3650 4100 50  0001 C CNN
 F 1 "GND" H 3655 4177 50  0000 C CNN
 F 2 "" H 3650 4350 50  0001 C CNN
@@
 AR Path="/D1BB8DB4/5F75E923/604747F3/60314A12" Ref="C7302"  Part="1"
 AR Path="/D1BB8DB4/5F317CB5/60365B35/60314A12" Ref="C8202"  Part="1"
-F 0 "C5302" H 3300 4300 50  0000 L CNN
+F 0 "C2402" H 3300 4300 50  0000 L CNN
 F 1 "1µF" H 2800 4150 50  0001 L CNN
 F 2 "Capacitor_THT:C_Disc_D7.5mm_W5.0mm_P5.00mm" H 3650 4250 50  0001 C CNN
@@
 AR Path="/D1BB8DB4/5F75E923/604747F3/60491845" Ref="U7003"  Part="2"
 AR Path="/D1BB8DB4/5F317CB5/60365B35/60491845" Ref="U7903"  Part="2"
-F 0 "U4002" H 6500 4750 50  0000 C CNN
+F 0 "U2103" H 6500 4750 50  0000 C CNN
 F 1 "74HC86" H 6500 4850 50  0000 C CNN
 F 2 "" H 6550 4550 50  0001 C CNN
