File: addon/NonLatchingNO30A/NonLatchingNO30A.kicad_pcb (KiCad board)
At the start: 4 copper layers, 153 x 114 mm, 27 parts, among them J101 Conn_02x20_Odd_Even Header, J102 TBP01R2W-508-16BE, J103 TBP01R2W-508-16BE, K101 ALFG2PF121, K102 ALFG2PF121, K103 ALFG2PF121, K104 ALFG2PF121, K105 ALFG2PF121, K106 ALFG2PF121, K107 ALFG2PF121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

Commit message: Headless ants
Parts:
- G102: moved to B.Cu
- moved G102 7.50 mm to (74.8, 121.0)
