File: addon/SwitchBreakout/SwitchBreakout.kicad_pcb (KiCad board)
At the start: 2 copper layers, 127.8 x 194.6 mm, 209 parts, among them IC1 SN74HCS72QPWRQ1, IC10 SN74HCS72QPWRQ1, IC11 SN74HCS72QPWRQ1, IC12 SN74HCS72QPWRQ1, IC13 SN74HCS72QPWRQ1, IC14 SN74HCS72QPWRQ1, IC15 SN74HCS72QPWRQ1, IC16 SN74HCS72QPWRQ1, IC2 SN74HCS72QPWRQ1, IC3 SN74HCS72QPWRQ1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

Commit message: Topper
Routing:
- net Net-(F72-Pad1): track 0.00 -> 95.1 mm
- net Net-(F70-Pad1): track 0.00 -> 86.5 mm
- net Net-(F76-Pad1): track 0.00 -> 86.0 mm
- net Net-(F80-Pad1): track 0.00 -> 77.5 mm
- net Net-(F74-Pad1): track 0.00 -> 76.0 mm
- net Net-(F55-Pad1): track 72.6 -> 0.00 mm
- net Net-(F84-Pad1): track 0.00 -> 69.5 mm
- net Net-(F94-Pad1): track 0.00 -> 66.0 mm
- net Net-(F71-Pad1): track 0.00 -> 65.9 mm
- net Net-(F90-Pad1): track 0.00 -> 65.5 mm
- net Net-(F78-Pad1): track 0.00 -> 64.5 mm
- net Net-(F86-Pad1): track 0.00 -> 62.4 mm
- net Net-(F82-Pad1): track 0.00 -> 60.8 mm
- net Net-(F75-Pad1): track 0.00 -> 58.8 mm
- net Net-(F69-Pad1): track 0.00 -> 55.1 mm
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
Commit message: Bugfixing
Parts:
- moved F93 4.95 mm to (178.7, 103.8), turned to 180 degrees
Routing:
- net Net-(F62-Pad1): track 0.00 -> 108.6 mm
- net Net-(F55-Pad1): track 0.00 -> 67.8 mm
- net Net-(F79-Pad1): track 0.00 -> 46.1 mm
- net Net-(F28-Pad2): track 0.00 -> 16.3 mm
- net Net-(F8-Pad2): track 0.00 -> 16.3 mm
- net Net-(F16-Pad2): track 0.00 -> 15.0 mm
- net Net-(F20-Pad2): track 0.00 -> 15.0 mm
- net Net-(F24-Pad2): track 0.00 -> 15.0 mm
- net Net-(F65-Pad1): track 72.9 -> 86.2 mm
- net Net-(F93-Pad2): track 0.00 -> 10.9 mm
- net Net-(F90-Pad2): track 0.00 -> 10.9 mm
- net Net-(F89-Pad2): track 0.00 -> 10.9 mm
- net Net-(F86-Pad2): track 0.00 -> 10.9 mm
- net Net-(F85-Pad2): track 0.00 -> 10.9 mm
- net Net-(F82-Pad2): track 0.00 -> 10.9 mm
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
Commit message: Right side
Connections:
- RN1 pad 2: /D-Latch 1-8/D-Latch 0/CLK1 -> /D-Latch 1-8/D-Latch 0/CLK2
- RN1 pad 3: /D-Latch 1-8/D-Latch 0/CLK2 -> /D-Latch 1-8/D-Latch 0/CLK1
- RN1 pad 4: /D-Latch 1-8/D-Latch 1/CLK1 -> /D-Latch 1-8/D-Latch 1/CLK2
- RN1 pad 5: /D-Latch 1-8/D-Latch 1/CLK2 -> /D-Latch 1-8/D-Latch 1/CLK1
- RN1 pad 6: /D-Latch 1-8/D-Latch 2/CLK1 -> /D-Latch 1-8/D-Latch 2/CLK2
- RN1 pad 7: /D-Latch 1-8/D-Latch 2/CLK2 -> /D-Latch 1-8/D-Latch 2/CLK1
- RN1 pad 8: /D-Latch 1-8/D-Latch 4/CLK1 -> /D-Latch 1-8/D-Latch 4/CLK2
- RN1 pad 9: /D-Latch 1-8/D-Latch 4/CLK2 -> /D-Latch 1-8/D-Latch 4/CLK1
- RN3 pad 2: /D-Lach 9-16/D-Latch 0/CLK1 -> /D-Lach 9-16/D-Latch 0/CLK2
- RN3 pad 3: /D-Lach 9-16/D-Latch 0/CLK2 -> /D-Lach 9-16/D-Latch 0/CLK1
- RN3 pad 4: /D-Lach 9-16/D-Latch 1/CLK1 -> /D-Lach 9-16/D-Latch 1/CLK2
- RN3 pad 5: /D-Lach 9-16/D-Latch 1/CLK2 -> /D-Lach 9-16/D-Latch 1/CLK1
- RN3 pad 6: /D-Lach 9-16/D-Latch 2/CLK1 -> /D-Lach 9-16/D-Latch 2/CLK2
- RN3 pad 7: /D-Lach 9-16/D-Latch 2/CLK2 -> /D-Lach 9-16/D-Latch 2/CLK1
- RN3 pad 8: /D-Lach 9-16/D-Latch 4/CLK1 -> /D-Lach 9-16/D-Latch 4/CLK2
- RN3 pad 9: /D-Lach 9-16/D-Latch 4/CLK2 -> /D-Lach 9-16/D-Latch 4/CLK1
- RN5 pad 2: /D-Latch 17-24/D-Latch 0/CLK1 -> /D-Latch 17-24/D-Latch 0/CLK2
- RN5 pad 3: /D-Latch 17-24/D-Latch 0/CLK2 -> /D-Latch 17-24/D-Latch 0/CLK1
- RN5 pad 4: /D-Latch 17-24/D-Latch 1/CLK1 -> /D-Latch 17-24/D-Latch 1/CLK2
- RN5 pad 5: /D-Latch 17-24/D-Latch 1/CLK2 -> /D-Latch 17-24/D-Latch 1/CLK1
- RN5 pad 6: /D-Latch 17-24/D-Latch 2/CLK1 -> /D-Latch 17-24/D-Latch 2/CLK2
- RN5 pad 7: /D-Latch 17-24/D-Latch 2/CLK2 -> /D-Latch 17-24/D-Latch 2/CLK1
- RN5 pad 8: /D-Latch 17-24/D-Latch 4/CLK1 -> /D-Latch 17-24/D-Latch 4/CLK2
- RN5 pad 9: /D-Latch 17-24/D-Latch 4/CLK2 -> /D-Latch 17-24/D-Latch 4/CLK1
- RN7 pad 2: /D-Latch 25-32/D-Latch 0/CLK1 -> /D-Latch 25-32/D-Latch 0/CLK2
- RN7 pad 3: /D-Latch 25-32/D-Latch 0/CLK2 -> /D-Latch 25-32/D-Latch 0/CLK1
- RN7 pad 4: /D-Latch 25-32/D-Latch 1/CLK1 -> /D-Latch 25-32/D-Latch 1/CLK2
- RN7 pad 5: /D-Latch 25-32/D-Latch 1/CLK2 -> /D-Latch 25-32/D-Latch 1/CLK1
- RN7 pad 6: /D-Latch 25-32/D-Latch 2/CLK1 -> /D-Latch 25-32/D-Latch 2/CLK2
- RN7 pad 7: /D-Latch 25-32/D-Latch 2/CLK2 -> /D-Latch 25-32/D-Latch 2/CLK1
- RN7 pad 8: /D-Latch 25-32/D-Latch 4/CLK1 -> /D-Latch 25-32/D-Latch 4/CLK2
- RN7 pad 9: /D-Latch 25-32/D-Latch 4/CLK2 -> /D-Latch 25-32/D-Latch 4/CLK1
Routing:
- net /D-Lach 9-16/D-Latch 2/CLK2: track 0.00 -> 76.2 mm
- net /D-Lach 9-16/D-Latch 4/CLK2: track 0.00 -> 67.2 mm
- net /D-Lach 9-16/D-Latch 2/CLK1: track 0.00 -> 62.8 mm
- net /D-Lach 9-16/D-Latch 0/CLK2: track 41.9 -> 102.8 mm
- net /D-Latch 25-32/D-Latch 4/CLK1: track 0.00 -> 60.3 mm
- net /D-Lach 9-16/D-Latch 0/CLK1: track 32.0 -> 87.6 mm
- net /D-Latch 25-32/D-Latch 4/CLK2: track 0.00 -> 53.7 mm
- net /D-Latch 25-32/D-Latch 2/CLK1: track 0.00 -> 50.1 mm
- net /D-Lach 9-16/D-Latch 4/CLK1: track 0.00 -> 49.2 mm
- net /D-Lach 9-16/D-Latch 1/CLK2: track 43.0 -> 91.9 mm
- net /D-Lach 9-16/D-Latch 2/BTN2: track 0.00 -> 48.8 mm
- net /D-Lach 9-16/D-Latch 4/BTN2: track 0.00 -> 48.8 mm
- net /D-Latch 25-32/D-Latch 2/CLK2: track 0.00 -> 41.8 mm
- net /D-Lach 9-16/D-Latch 1/CLK1: track 33.1 -> 74.5 mm
- net /D-Lach 9-16/D-Latch 4/BTN1: track 0.00 -> 41.0 mm
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
Commit message: Swirls
Routing:
- net /D-Lach 9-16/D-Latch 0/CLK2: track 102.8 -> 41.9 mm
- net /D-Lach 9-16/D-Latch 0/CLK1: track 87.6 -> 32.0 mm
- net /D-Lach 9-16/D-Latch 1/CLK2: track 91.9 -> 43.0 mm
- net /D-Latch 25-32/D-Latch 4/BTN2: track 0.00 -> 48.7 mm
- net /D-Latch 25-32/D-Latch 1/BTN2: track 0.00 -> 48.7 mm
- net /D-Latch 25-32/D-Latch 2/BTN2: track 0.00 -> 48.7 mm
- net /D-Lach 9-16/D-Latch 1/CLK1: track 74.5 -> 33.1 mm
- net /D-Latch 25-32/D-Latch 1/BTN1: track 0.00 -> 41.2 mm
- net /D-Latch 25-32/D-Latch 0/BTN1: track 0.00 -> 40.8 mm
- net /D-Latch 25-32/D-Latch 4/BTN1: track 0.00 -> 40.5 mm
- net /D-Latch 25-32/D-Latch 2/BTN1: track 0.00 -> 39.5 mm
- net /D-Lach 9-16/D-Latch 2/CLK2: track 76.2 -> 42.0 mm
- net /D-Lach 9-16/D-Latch 2/CLK1: track 62.8 -> 32.4 mm
- net /A6: track 0.00 -> 30.3 mm
- net /D-Latch 25-32/D-Latch 4/CLK1: track 60.3 -> 33.1 mm
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
Commit message: Red
Routing:
- net /D-Latch 1-8/D-Latch 2/BTN2: track 0.00 -> 32.1 mm
- net /D-Latch 17-24/D-Latch 4/BTN2: track 0.00 -> 32.1 mm
- net /D-Latch 17-24/D-Latch 2/BTN2: track 0.00 -> 32.1 mm
- net /D-Latch 17-24/D-Latch 1/BTN2: track 0.00 -> 32.1 mm
- net /D-Latch 17-24/D-Latch 0/BTN2: track 0.00 -> 32.1 mm
- net /D-Latch 1-8/D-Latch 4/BTN2: track 0.00 -> 32.0 mm
- net /D-Latch 17-24/D-Latch 4/CLK2: track 0.00 -> 24.5 mm
- net /D-Latch 17-24/D-Latch 2/CLK2: track 0.00 -> 24.5 mm
- net /D-Latch 1-8/D-Latch 2/CLK2: track 0.00 -> 24.5 mm
- net /D-Latch 17-24/D-Latch 1/CLK2: track 0.00 -> 24.5 mm
- net /D-Latch 17-24/D-Latch 0/CLK2: track 0.00 -> 24.5 mm
- net /D-Latch 1-8/D-Latch 4/CLK2: track 0.00 -> 24.4 mm
- net /E4: track 0.00 -> 19.0 mm
- net /H4: track 0.00 -> 19.0 mm
- net /M4: track 0.00 -> 18.9 mm
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
Commit message: UP
Routing:
- added copper zone on F.Cu, net GND
- added copper zone on B.Cu, net VCC
Changed lines of the file:
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@@
     (thickness 1.6)
     (drawings 8)
-    (tracks 1933)
+    (tracks 1932)
     (zones 0)
     (modules 209)
@@
   (segment (start 200.682511 194.200009) (end 200.682511 198.169991) (width 0.25) (layer B.Cu) (net 40))
   (segment (start 195.834 187.325) (end 195.834 190.169722) (width 0.25) (layer B.Cu) (net 40))
-  (segment (start 193.294 198.135) (end 196.349678 198.135) (width 0.25) (layer B.Cu) (net 41))
   (segment (start 201.652999 188.063999) (end 200.914 187.325) (width 0.25) (layer B.Cu) (net 41))
-  (segment (start 200.540303 199.585019) (end 201.652999 198.472323) (width 0.25) (layer B.Cu) (net 41))
   (segment (start 201.652999 198.472323) (end 201.652999 188.063999) (width 0.25) (layer B.Cu) (net 41))
-  (segment (start 197.799698 199.58502) (end 200.540303 199.585019) (width 0.25) (layer B.Cu) (net 41))
-  (segment (start 196.349678 198.135) (end 197.799698 199.58502) (width 0.25) (layer B.Cu) (net 41))
+  (segment (start 193.294 198.61) (end 193.294 198.135) (width 0.25) (layer B.Cu) (net 41))
+  (segment (start 194.269019 199.585019) (end 193.294 198.61) (width 0.25) (layer B.Cu) (net 41))
+  (segment (start 200.540303 199.585019) (end 194.269019 199.585019) (width 0.25) (layer B.Cu) (net 41))
+  (segment (start 201.652999 198.472323) (end 200.540303 199.585019) (width 0.25) (layer B.Cu) (net 41))
   (segment (start 194.2815 195.535) (end 193.294 195.535) (width 0.25) (layer B.Cu) (net 42))
   (segment (start 194.356501 195.610001) (end 194.2815 195.535) (width 0.25) (layer B.Cu) (net 42))
@@
   (segment (start 194.191502 197.485) (end 194.356501 197.320001) (width 0.25) (layer B.Cu) (net 42))
   (segment (start 193.294 197.485) (end 194.191502 197.485) (width 0.25) (layer B.Cu) (net 42))
-  (segment (start 198.374 188.370103) (end 198.374 187.325) (width 0.25) (layer B.Cu) (net 42))
-  (segment (start 198.374 190.5) (end 198.374 188.370103) (width 0.25) (layer B.Cu) (net 42))
-  (segment (start 201.132521 198.356391) (end 201.132521 193.258521) (width 0.25) (layer B.Cu) (net 42))
-  (segment (start 200.353902 199.13501) (end 201.132521 198.356391) (width 0.25) (layer B.Cu) (net 42))
-  (segment (start 197.986098 199.13501) (end 200.353902 199.13501) (width 0.25) (layer B.Cu) (net 42))
-  (segment (start 196.336088 197.485) (end 197.986098 199.13501) (width 0.25) (layer B.Cu) (net 42))
-  (segment (start 201.132521 193.258521) (end 198.374 190.5) (width 0.25) (layer B.Cu) (net 42))
-  (segment (start 193.294 197.485) (end 196.336088 197.485) (width 0.25) (layer B.Cu) (net 42))
+  (segment (start 194.2815 197.485) (end 193.294 197.485) (width 0.25) (layer B.Cu) (net 42))
+  (segment (start 195.931511 199.135011) (end 194.2815 197.485) (width 0.25) (layer B.Cu) (net 42))
+  (segment (start 200.353901 199.135011) (end 195.931511 199.135011) (width 0.25) (layer B.Cu) (net 42))
+  (segment (start 201.132521 198.356391) (end 200.353901 199.135011) (width 0.25) (layer B.Cu) (net 42))
+  (segment (start 201.132521 193.258521) (end 201.132521 198.356391) (width 0.25) (layer B.Cu) (net 42))
+  (segment (start 198.374 190.5) (end 201.132521 193.258521) (width 0.25) (layer B.Cu) (net 42))
+  (segment (start 198.374 187.325) (end 198.374 190.5) (width 0.25) (layer B.Cu) (net 42))
   (segment (start 179.314 188.370103) (end 179.314 187.325) (width 0.25) (layer B.Cu) (net 43))
   (segment (start 179.314 190.4145) (end 179.314 188.370103) (width 0.25) (layer B.Cu) (net 43))
@@
   (segment (start 118.634531 188.865531) (end 118.63453 198.572792) (width 0.25) (layer B.Cu) (net 69))
   (segment (start 117.094 187.325) (end 118.634531 188.865531) (width 0.25) (layer B.Cu) (net 69))
-  (segment (start 111.3335 197.515) (end 110.346 197.515) (width 0.25) (layer B.Cu) (net 70))
-  (segment (start 111.408501 197.439999) (end 111.3335 197.515) (width 0.25) (layer B.Cu) (net 70))
-  (segment (start 111.408501 195.640001) (end 111.408501 197.439999) (width 0.25) (layer B.Cu) (net 70))
+  (segment (start 118.184521 190.650799) (end 115.597721 188.063999) (width 0.25) (layer B.Cu) (net 70))
+  (segment (start 113.388088 197.515) (end 115.038099 199.165011) (width 0.25) (layer B.Cu) (net 70))
   (segment (start 111.3335 195.565) (end 111.408501 195.640001) (width 0.25) (layer B.Cu) (net 70))
-  (segment (start 110.346 195.565) (end 111.3335 195.565) (width 0.25) (layer B.Cu) (net 70))
-  (segment (start 118.184521 198.386391) (end 118.184521 190.650799) (width 0.25) (layer B.Cu) (net 70))
-  (segment (start 117.405902 199.16501) (end 118.184521 198.386391) (width 0.25) (layer B.Cu) (net 70))
   (segment (start 115.038099 199.165011) (end 117.405902 199.16501) (width 0.25) (layer B.Cu) (net 70))
+  (segment (start 111.408501 195.640001) (end 111.408501 197.439999) (width 0.25) (layer B.Cu) (net 70))
   (segment (start 115.292999 188.063999) (end 114.554 187.325) (width 0.25) (layer B.Cu) (net 70))
-  (segment (start 118.184521 190.650799) (end 115.597721 188.063999) (width 0.25) (layer B.Cu) (net 70))
-  (segment (start 113.388088 197.515) (end 115.038099 199.165011) (width 0.25) (layer B.Cu) (net 70))
-  (segment (start 115.597721 188.063999) (end 115.292999 188.063999) (width 0.25) (layer B.Cu) (net 70))
+  (segment (start 117.405902 199.16501) (end 118.184521 198.386391) (width 0.25) (layer B.Cu) (net 70))
+  (segment (start 110.346 195.565) (end 111.3335 195.565) (width 0.25) (layer B.Cu) (net 70))
+  (segment (start 111.408501 197.439999) (end 111.3335 197.515) (width 0.25) (layer B.Cu) (net 70))
+  (segment (start 118.184521 198.386391) (end 118.184521 190.650799) (width 0.25) (layer B.Cu) (net 70))
   (segment (start 110.346 197.515) (end 113.388088 197.515) (width 0.25) (layer B.Cu) (net 70))
+  (segment (start 115.597721 188.063999) (end 115.292999 188.063999) (width 0.25) (layer B.Cu) (net 70))
+  (segment (start 111.3335 197.515) (end 110.346 197.515) (width 0.25) (layer B.Cu) (net 70))
   (segment (start 127.605 194.915) (end 127.9345 194.915) (width 0.25) (layer B.Cu) (net 71))
   (segment (start 126.189999 193.499999) (end 127.605 194.915) (width 0.25) (layer B.Cu) (net 71))
@@
   (segment (start 194.552001 117.544999) (end 198.167001 121.159999) (width 0.4) (layer F.Cu) (net 386))
   (segment (start 170.874018 107.88002) (end 183.955018 107.88002) (width 0.4) (layer F.Cu) (net 386))
+  (zone (net 1) (net_name GND) (layer F.Cu) (hatch edge 0.508)
+    (connect_pads (clearance 0.508))
+    (min_thickness 0.254)
+    (fill (arc_segments 32) (thermal_gap 0.508) (thermal_bridge_width 0.508))
+    (polygon
+      (pts
+        (xy 226 208.5) (xy 97 208.5) (xy 97 12) (xy 226 12)
+      )
+    )
+  )
+  (zone (net 2) (net_name VCC) (layer B.Cu) (hatch edge 0.508)
+    (connect_pads (clearance 0.508))
+    (min_thickness 0.254)
+    (fill (arc_segments 32) (thermal_gap 0.508) (thermal_bridge_width 0.508))
+    (polygon
+      (pts
+        (xy 226 208.5) (xy 97 208.5) (xy 97 12) (xy 226 12)
+      )
+    )
+  )
 )

Commit message: Steps
Parts:
- removed H3, H4: MountingHole, MountingHole:MountingHole_3.2mm_M3
Routing:
- net /I1: track 0.00 -> 218.2 mm
- net /J1: track 0.00 -> 204.3 mm
- net /I5: track 0.00 -> 199.1 mm
- net /I2: track 15.8 -> 211.2 mm
- net /J5: track 0.00 -> 193.0 mm, vias 0 -> 1
- net /I4: track 19.0 -> 209.9 mm
- net /I6: track 25.6 -> 209.2 mm
- net /J2: track 15.4 -> 197.8 mm
- net /K1: track 0.00 -> 181.9 mm
- net /I8: track 21.5 -> 199.9 mm
- net /J4: track 18.5 -> 196.1 mm
- net /J6: track 24.1 -> 193.2 mm
- net /K5: track 0.00 -> 167.0 mm, vias 0 -> 1
- net /K2: track 15.2 -> 175.8 mm
- net /J8: track 21.0 -> 179.5 mm
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
Commit message: Patcha patcha
Routing:
- net /D4: track 18.6 -> 233.5 mm
- net /D5: track 0.00 -> 198.7 mm
- net /D6: track 24.8 -> 219.6 mm
- net /D8: track 21.3 -> 209.1 mm
- net /D1: track 0.00 -> 181.5 mm, vias 0 -> 1
- net /D2: track 15.1 -> 186.3 mm, vias 0 -> 1
- net /L1: track 0.00 -> 160.3 mm
- net /L2: track 15.2 -> 153.9 mm
- net /L4: track 18.5 -> 150.7 mm
- net /D-Latch 1-8/BTN1: track 0.00 -> 107.0 mm
- net /D-Latch 1-8/BTN2: track 0.00 -> 95.7 mm
- net /L5: track 0.00 -> 94.7 mm, vias 0 -> 1
- net /L8: track 21.3 -> 115.4 mm
- net /L6: track 24.0 -> 116.9 mm
- net /D-Latch 1-8/BTN3: track 0.00 -> 84.9 mm
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